Commit message: adding proper package depends, first attempt with phoebe modifications to standard ridgeback

File: phoebe_description/urdf/jaco01_customization.urdf.xacro (robot description, xacro)
@@ -1,4 +1,6 @@
 <?xml version="1.0"?>
 <robot xmlns:xacro="http://wiki.ros.org/xacro">
+  <!-- Macro for phoebe customization -->
+  <xacro:macro name="jaco01_customization">
   <material name="grey">
     <color rgba="0.5 0.5 0.5 1"/>
@@ -8,12 +10,12 @@
     <visual>
       <geometry>
-        <mesh filename="package://jaco01_ridgeback_description/meshes/lift_rails.STL"/>
-      </geometry>
-      <material name="black" />
+        <mesh filename="package://phoebe_description/meshes/visual/jaco01_meshes/lift_rails.STL"/>
+      </geometry>
+      <material name="clearpath_black" />
     </visual>
     <collision>
       <origin xyz="0.000 -0.000 0.020"/>
       <geometry>
-        <!--<mesh filename="package://jaco01_ridgeback_description/meshes/lift_rails.STL"/>-->
+        <!--<mesh filename="package://phoebe_description/meshes/visual/jaco01_meshes/lift_rails.STL"/>-->
         <box size="0.220 0.730 0.040"/>
       </geometry>
@@ -21,5 +23,5 @@
   </link>
   <joint name="lift_rails_joint" type="fixed">
-    <parent link="mid_mount" />
+    <parent link="default_mount" />
     <child link="lift_rails" />
     <origin xyz="0 0 0" rpy="0 0 0" />
@@ -29,12 +31,12 @@
     <visual>
       <geometry>
-        <mesh filename="package://jaco01_ridgeback_description/meshes/shelf.STL"/>
-      </geometry>
-      <material name="black" />
+        <mesh filename="package://phoebe_description/meshes/visual/jaco01_meshes/shelf.STL"/>
+      </geometry>
+      <material name="clearpath_black" />
     </visual>
     <collision>
       <origin xyz="-0.289 0.000 0.113"/>
       <geometry>
-        <!--<mesh filename="package://jaco01_ridgeback_description/meshes/shelf.STL"/>-->
+        <!--<mesh filename="package://phoebe_description/meshes/visual/jaco01_meshes/shelf.STL"/>-->
         <box size="0.379 0.790 0.226"/>
       </geometry>
@@ -42,5 +44,5 @@
   </link>
   <joint name="rear_shelf_joint" type="fixed">
-    <parent link="mid_mount" />
+    <parent link="default_mount" />
     <child link="rear_shelf" />
     <origin xyz="0 0 0" rpy="0 0 0" />
@@ -50,12 +52,12 @@
     <visual>
       <geometry>
-        <mesh filename="package://jaco01_ridgeback_description/meshes/shelf.STL"/>
-      </geometry>
-      <material name="black" />
+        <mesh filename="package://phoebe_description/meshes/visual/jaco01_meshes/shelf.STL"/>
+      </geometry>
+      <material name="clearpath_black" />
     </visual>
     <collision>
       <origin xyz="-0.289 0.000 0.113"/>
       <geometry>
-        <!--<mesh filename="package://jaco01_ridgeback_description/meshes/shelf.STL"/>-->
+        <!--<mesh filename="package://phoebe_description/meshes/visual/jaco01_meshes/shelf.STL"/>-->
         <box size="0.379 0.790 0.226"/>
       </geometry>
@@ -63,5 +65,5 @@
   </link>
   <joint name="front_shelf_joint" type="fixed">
-    <parent link="mid_mount" />
+    <parent link="default_mount" />
     <child link="front_shelf" />
     <origin xyz="0 0 0" rpy="0 0 ${pi}" />
@@ -71,7 +73,7 @@
     <visual>
       <geometry>
-        <mesh filename="package://jaco01_ridgeback_description/meshes/monitor_hinge_base.STL"/>
-      </geometry>
-      <material name="black" />
+        <mesh filename="package://phoebe_description/meshes/visual/jaco01_meshes/monitor_hinge_base.STL"/>
+      </geometry>
+      <material name="clearpath_black" />
     </visual>
     <collision>
@@ -79,10 +81,10 @@
       <geometry>
         <box size="0.040 0.450 0.036"/>
-        <!--<mesh filename="package://jaco01_ridgeback_description/meshes/monitor_hinge_base.STL"/>-->
+        <!--<mesh filename="package://phoebe_description/meshes/visual/jaco01_meshes/monitor_hinge_base.STL"/>-->
       </geometry>
     </collision>
   </link>
   <joint name="monitor_hinge_base_joint" type="fixed">
-    <parent link="mid_mount" />
+    <parent link="default_mount" />
     <child link="monitor_hinge_base" />
     <origin xyz="-0.4 0 0.24635" rpy="0 0 0" />
@@ -92,12 +94,12 @@
     <visual>
       <geometry>
-        <mesh filename="package://jaco01_ridgeback_description/meshes/monitor_hinge_top.STL"/>
-      </geometry>
-      <material name="black" />
+        <mesh filename="package://phoebe_description/meshes/visual/jaco01_meshes/monitor_hinge_top.STL"/>
+      </geometry>
+      <material name="clearpath_black" />
     </visual>
     <collision>
       <origin xyz="-0.013 0.000 0.000"/>
       <geometry>
-        <!--<mesh filename="package://jaco01_ridgeback_description/meshes/monitor_hinge_top.STL"/>-->
+        <!--<mesh filename="package://phoebe_description/meshes/visual/jaco01_meshes/monitor_hinge_top.STL"/>-->
         <box size="0.055 0.450 0.040"/>
       </geometry>
@@ -113,12 +115,12 @@
     <visual>
       <geometry>
-        <mesh filename="package://jaco01_ridgeback_description/meshes/monitor.STL"/>
-      </geometry>
-      <material name="black" />
+        <mesh filename="package://phoebe_description/meshes/visual/jaco01_meshes/monitor.STL"/>
+      </geometry>
+      <material name="clearpath_black" />
     </visual>
     <collision>
       <origin xyz="-0.015 0.000 -0.008"/>
       <geometry>
-        <!-- <mesh filename="package://jaco01_ridgeback_description/meshes/monitor.STL"/> -->
+        <!-- <mesh filename="package://phoebe_description/meshes/visual/jaco01_meshes/monitor.STL"/> -->
         <box size="0.071 0.260 0.176"/>
       </geometry>
@@ -134,12 +136,12 @@
     <visual>
       <geometry>
-        <mesh filename="package://jaco01_ridgeback_description/meshes/monitor.STL"/>
-      </geometry>
-      <material name="black" />
+        <mesh filename="package://phoebe_description/meshes/visual/jaco01_meshes/monitor.STL"/>
+      </geometry>
+      <material name="clearpath_black" />
     </visual>
     <collision>
       <origin xyz="-0.015 0.000 -0.008"/>
       <geometry>
-        <!-- <mesh filename="package://jaco01_ridgeback_description/meshes/monitor.STL"/> -->
+        <!-- <mesh filename="package://phoebe_description/meshes/visual/jaco01_meshes/monitor.STL"/> -->
         <box size="0.071 0.260 0.176"/>
       </geometry>
@@ -155,5 +157,5 @@
     <visual>
       <geometry>
-        <mesh filename="package://jaco01_ridgeback_description/meshes/ur_control_box.STL"/>
+        <mesh filename="package://phoebe_description/meshes/visual/jaco01_meshes/ur_control_box.STL"/>
       </geometry>
       <material name="grey" />
@@ -163,10 +165,10 @@
       <geometry>
         <box size="0.199 0.502 0.195"/>
-        <!-- <mesh filename="package://jaco01_ridgeback_description/meshes/ur_control_box.STL"/> -->
+        <!-- <mesh filename="package://phoebe_description/meshes/visual/jaco01_meshes/ur_control_box.STL"/> -->
       </geometry>
     </collision>
   </link>
   <joint name="rear_ur_control_box_joint" type="fixed">
-    <parent link="mid_mount" />
+    <parent link="default_mount" />
     <child link="rear_ur_control_box" />
     <origin xyz="-0.44274 0.13 0" rpy="0 0 0" />
@@ -176,5 +178,5 @@
     <visual>
       <geometry>
-        <mesh filename="package://jaco01_ridgeback_description/meshes/ur_control_box.STL"/>
+        <mesh filename="package://phoebe_description/meshes/visual/jaco01_meshes/ur_control_box.STL"/>
       </geometry>
       <material name="grey" />
@@ -184,10 +186,10 @@
       <geometry>
         <box size="0.199 0.502 0.195"/>
-        <!-- <mesh filename="package://jaco01_ridgeback_description/meshes/ur_control_box.STL"/> -->
+        <!-- <mesh filename="package://phoebe_description/meshes/visual/jaco01_meshes/ur_control_box.STL"/> -->
       </geometry>
     </collision>
   </link>
   <joint name="front_ur_control_box_joint" type="fixed">
-    <parent link="mid_mount" />
+    <parent link="default_mount" />
     <child link="front_ur_control_box" />
     <origin xyz="0.44274 -0.13 0" rpy="0 0 ${pi}" />
@@ -197,5 +199,5 @@
     <visual>
       <geometry>
-        <mesh filename="package://jaco01_ridgeback_description/meshes/scu.STL"/>
+        <mesh filename="package://phoebe_description/meshes/visual/jaco01_meshes/scu.STL"/>
       </geometry>
       <material name="grey" />
@@ -204,5 +206,5 @@
       <origin xyz="0.000 0.002 0.043"/>
       <geometry>
-        <!-- <mesh filename="package://jaco01_ridgeback_description/meshes/scu.STL"/> -->
+        <!-- <mesh filename="package://phoebe_description/meshes/visual/jaco01_meshes/scu.STL"/> -->
         <box size="0.140 0.365 0.087"/>
       </geometry>
@@ -210,5 +212,5 @@
   </link>
   <joint name="rear_scu_joint" type="fixed">
-    <parent link="mid_mount" />
+    <parent link="default_mount" />
     <child link="rear_scu" />
     <origin xyz="-0.18187 0 0" rpy="0 0 0" />
@@ -218,5 +220,5 @@
     <visual>
       <geometry>
-        <mesh filename="package://jaco01_ridgeback_description/meshes/scu.STL"/>
+        <mesh filename="package://phoebe_description/meshes/visual/jaco01_meshes/scu.STL"/>
       </geometry>
       <material name="grey" />
@@ -225,5 +227,5 @@
       <origin xyz="0.000 0.002 0.043"/>
       <geometry>
-        <!-- <mesh filename="package://jaco01_ridgeback_description/meshes/scu.STL"/> -->
+        <!-- <mesh filename="package://phoebe_description/meshes/visual/jaco01_meshes/scu.STL"/> -->
         <box size="0.140 0.365 0.087"/>
       </geometry>
@@ -231,5 +233,5 @@
   </link>
   <joint name="front_scu_joint" type="fixed">
-    <parent link="mid_mount" />
+    <parent link="default_mount" />
     <child link="front_scu" />
     <origin xyz="0.18187 0 0" rpy="0 0 ${pi}" />
@@ -239,12 +241,12 @@
     <visual>
       <geometry>
-        <mesh filename="package://jaco01_ridgeback_description/meshes/autec_receiver.STL"/>
-      </geometry>
-      <material name="yellow" />
+        <mesh filename="package://phoebe_description/meshes/visual/jaco01_meshes/autec_receiver.STL"/>
+      </geometry>
+      <material name="clearpath_yellow" />
     </visual>
     <collision>
       <origin xyz="0.008 0.000 0.031"/>
       <geometry>
-        <!-- <mesh filename="package://jaco01_ridgeback_description/meshes/autec_receiver.STL"/> -->
+        <!-- <mesh filename="package://phoebe_description/meshes/visual/jaco01_meshes/autec_receiver.STL"/> -->
         <box size="0.255 0.142 0.062"/>
       </geometry>
@@ -252,5 +254,5 @@
   </link>
   <joint name="autec_receiver_joint" type="fixed">
-    <parent link="mid_mount" />
+    <parent link="default_mount" />
     <child link="autec_receiver" />
     <origin xyz="-0.26 -0.29909 0" rpy="0 0 0" />
@@ -260,12 +262,12 @@
     <visual>
       <geometry>
-        <mesh filename="package://jaco01_ridgeback_description/meshes/wifi_antenna.STL"/>
-      </geometry>
-      <material name="black" />
+        <mesh filename="package://phoebe_description/meshes/visual/jaco01_meshes/wifi_antenna.STL"/>
+      </geometry>
+      <material name="clearpath_black" />
     </visual>
     <collision>
       <origin xyz="-0.003 0.000 0.089"/>
       <geometry>
-        <!-- <mesh filename="package://jaco01_ridgeback_description/meshes/wifi_antenna.STL"/> -->
+        <!-- <mesh filename="package://phoebe_description/meshes/visual/jaco01_meshes/wifi_antenna.STL"/> -->
         <cylinder radius="0.033" length="0.229"/>
       </geometry>
@@ -273,5 +275,5 @@
   </link>
   <joint name="right_wifi_antenna_joint" type="fixed">
-    <parent link="mid_mount" />
+    <parent link="default_mount" />
     <child link="right_wifi_antenna" />
     <origin xyz="-0.086 -0.384 0.22" rpy="0 0 0" />
@@ -281,12 +283,12 @@
     <visual>
       <geometry>
-        <mesh filename="package://jaco01_ridgeback_description/meshes/wifi_antenna.STL"/>
-      </geometry>
-      <material name="black" />
+        <mesh filename="package://phoebe_description/meshes/visual/jaco01_meshes/wifi_antenna.STL"/>
+      </geometry>
+      <material name="clearpath_black" />
     </visual>
     <collision>
       <origin xyz="-0.003 0.000 0.089"/>
       <geometry>
-        <!-- <mesh filename="package://jaco01_ridgeback_description/meshes/wifi_antenna.STL"/> -->
+        <!-- <mesh filename="package://phoebe_description/meshes/visual/jaco01_meshes/wifi_antenna.STL"/> -->
         <cylinder radius="0.033" length="0.229"/>
       </geometry>
@@ -294,5 +296,5 @@
   </link>
   <joint name="left_wifi_antenna_joint" type="fixed">
-    <parent link="mid_mount" />
+    <parent link="default_mount" />
     <child link="left_wifi_antenna" />
     <origin xyz="-0.086 0.384 0.22" rpy="0 0 0" />
@@ -302,12 +304,12 @@
     <visual>
       <geometry>
-        <mesh filename="package://jaco01_ridgeback_description/meshes/autec_antenna.STL"/>
-      </geometry>
-      <material name="black" />
+        <mesh filename="package://phoebe_description/meshes/visual/jaco01_meshes/autec_antenna.STL"/>
+      </geometry>
+      <material name="clearpath_black" />
     </visual>
     <collision>
       <origin xyz="0.002 0.000 0.049"/>
       <geometry>
-        <!-- <mesh filename="package://jaco01_ridgeback_description/meshes/autec_antenna.STL"/> -->
+        <!-- <mesh filename="package://phoebe_description/meshes/visual/jaco01_meshes/autec_antenna.STL"/> -->
         <cylinder radius="0.037" length="0.147"/>
       </geometry>
@@ -315,5 +317,5 @@
   </link>
   <joint name="autec_antenna_joint" type="fixed">
-    <parent link="mid_mount" />
+    <parent link="default_mount" />
     <child link="autec_antenna" />
     <origin xyz="0.0845 -0.384 0.22" rpy="0 0 0" />
@@ -336,5 +338,5 @@
   </link>
   <joint name="left_ewellix_mount_flange_joint" type="fixed">
-    <parent link="mid_mount"/>
+    <parent link="default_mount"/>
     <child link="left_ewellix_mount_flange_link"/>
     <origin xyz="0 $(optenv LEFT_LIFT_Y 0.2) 0.04" rpy="0 0 0" />
@@ -357,10 +359,11 @@
   </link>
   <joint name="right_ewellix_mount_flange_joint" type="fixed">
-    <parent link="mid_mount"/>
+    <parent link="default_mount"/>
     <child link="right_ewellix_mount_flange_link"/>
     <origin xyz="0 -$(optenv RIGHT_LIFT_Y 0.2) 0.04" rpy="0 0 0" />
   </joint>
 <!-- Ewellix lift column xacro -->
-  <xacro:include filename="$(find ewellix_tlt)/urdf/ewellix_lift_500mm.urdf.xacro" />
+  <!-- OLD VERSION -->
+  <!-- <xacro:include filename="$(find ewellix_lift)/urdf/ewellix_lift_500mm.urdf.xacro" />
   <xacro:ewellix_lift_500mm prefix="left_" parent="left_ewellix_mount_flange_link" cut_model="1">
     <origin xyz="0.0 0.0 0.015" rpy="0 0 0" />
@@ -368,21 +371,64 @@
   <xacro:ewellix_lift_500mm prefix="right_" parent="right_ewellix_mount_flange_link" cut_model="1">
     <origin xyz="0.0 0.0 0.015" rpy="0 0 0" />
-  </xacro:ewellix_lift_500mm>
+  </xacro:ewellix_lift_500mm> -->
+  <!-- end OLD VERSION -->
+  <!-- clearpath ewellix -->
+  <xacro:include filename="$(find clearpath_manipulators_description)/urdf/lift/ewellix.urdf.xacro"/>
+  <xacro:ewellix name="left" parent_link="left_ewellix_mount_flange_link">
+    <origin xyz="0.0 0.0 0.015" rpy="0 0 0"/>
+  </xacro:ewellix>
+  <xacro:ewellix name="right" parent_link="right_ewellix_mount_flange_link">
+    <origin xyz="0.0 0.0 0.015" rpy="0 0 0"/>
+  </xacro:ewellix>
+  <!-- end clearpath ewellix -->
+  <!-- our_ewellix -->
+    <xacro:include filename="$(find ewellix_liftkit_description)/urdf/ewellix_lift.xacro"/>
+    <xacro:include filename="$(find ewellix_liftkit_description)/urdf/properties.xacro"/>
+    <!-- use_fake_hardware="$(arg use_fake_hardware)"
+    com_port="$(arg com_port)" -->
+    <!-- base is 0.015 from clearpath description. 0.295 is from ewellix_lift.xacro -->
+    <!-- <xacro:ewellix_lift
+    name="left_ewellix"
+    is_700="false"
+    is_500="true"
+    tf_prefix="left_"
+    parent="left_ewellix_mount_flange_link"
+    height_limit="0.5"
+    omit_plates="true"
+  >
+    <origin xyz="0 0 ${0.015+0.295}" rpy="0 0 0"/>
+  </xacro:ewellix_lift> -->
+    <!-- use_fake_hardware="$(arg use_fake_hardware)"
+    com_port="$(arg com_port)" -->
+    <!-- base is 0.015 from clearpath description. 0.295 is from ewellix_lift.xacro -->
+    <!-- <xacro:ewellix_lift
+    name="right_ewellix"
+    is_700="false"
+    is_500="true"
+    tf_prefix="right_"
+    parent="right_ewellix_mount_flange_link"
+    height_limit="0.5"
+    omit_plates="true"
+  >
+    <origin xyz="0 0 ${0.015+0.295}" rpy="0 0 0"/>
+  </xacro:ewellix_lift> -->
+  <!-- end our_ewellix -->
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
File: phoebe_description/urdf/phoebe.urdf.xacro (robot description, xacro)
@@ -13,3 +13,5 @@
         ns="$(arg ns)"
     />
+    <xacro:include filename="$(find phoebe_description)/urdf/jaco01_customization.urdf.xacro" />
+    <xacro:jaco01_customization/>
 </robot>

Commit message: integrating in handes

File: phoebe_description/urdf/jaco01_customization.urdf.xacro (robot description, xacro)
@@ -375,18 +375,18 @@
   <!-- clearpath ewellix -->
   <xacro:include filename="$(find clearpath_manipulators_description)/urdf/lift/ewellix.urdf.xacro"/>
-  <xacro:ewellix name="left" parent_link="left_ewellix_mount_flange_link">
+  <xacro:ewellix name="left" parent_link="left_ewellix_mount_flange_link" add_plate="false">
     <origin xyz="0.0 0.0 0.015" rpy="0 0 0"/>
   </xacro:ewellix>
-  <xacro:ewellix name="right" parent_link="right_ewellix_mount_flange_link">
+  <xacro:ewellix name="right" parent_link="right_ewellix_mount_flange_link" add_plate="false">
     <origin xyz="0.0 0.0 0.015" rpy="0 0 0"/>
   </xacro:ewellix>
   <!-- end clearpath ewellix -->
   <!-- our_ewellix -->
-    <xacro:include filename="$(find ewellix_liftkit_description)/urdf/ewellix_lift.xacro"/>
-    <xacro:include filename="$(find ewellix_liftkit_description)/urdf/properties.xacro"/>
-    <!-- use_fake_hardware="$(arg use_fake_hardware)"
-    com_port="$(arg com_port)" -->
-    <!-- base is 0.015 from clearpath description. 0.295 is from ewellix_lift.xacro -->
-    <!-- <xacro:ewellix_lift
+  <!-- use_fake_hardware="$(arg use_fake_hardware)"
+  com_port="$(arg com_port)" -->
+  <!-- base is 0.015 from clearpath description. 0.2457 is from ewellix_lift.xacro -->
+  <!-- <xacro:include filename="$(find ewellix_liftkit_description)/urdf/ewellix_lift.xacro"/>
+  <xacro:include filename="$(find ewellix_liftkit_description)/urdf/properties.xacro"/>
+  <xacro:ewellix_lift
     name="left_ewellix"
     is_700="false"
@@ -397,10 +397,7 @@
     omit_plates="true"
   >
-    <origin xyz="0 0 ${0.015+0.295}" rpy="0 0 0"/>
-  </xacro:ewellix_lift> -->
-    <!-- use_fake_hardware="$(arg use_fake_hardware)"
-    com_port="$(arg com_port)" -->
-    <!-- base is 0.015 from clearpath description. 0.295 is from ewellix_lift.xacro -->
-    <!-- <xacro:ewellix_lift
+    <origin xyz="0 0 ${0.0075+0.2457}" rpy="0 0 0"/>
+  </xacro:ewellix_lift>
+  <xacro:ewellix_lift
     name="right_ewellix"
     is_700="false"
@@ -411,5 +408,5 @@
     omit_plates="true"
   >
-    <origin xyz="0 0 ${0.015+0.295}" rpy="0 0 0"/>
+    <origin xyz="0 0 ${0.0075+0.2457}" rpy="0 0 0"/>
   </xacro:ewellix_lift> -->
   <!-- end our_ewellix -->
@@ -532,11 +529,21 @@
     </xacro:ur_robot>
 <!-- Hand-E Grippers -->
-  <!-- <xacro:include filename="$(find robotiq_hande_gripper_visualization)/urdf/robotiq_ur_hande.urdf.xacro"/>
-  <xacro:robotiq_ur_hande parent="left_ur_arm_tool0" prefix="left_gripper_">
-    <origin xyz="0 0 0" rpy="0 0 0"/>
-  </xacro:robotiq_ur_hande>
-  <xacro:robotiq_ur_hande parent="right_ur_arm_tool0" prefix="right_gripper_">
-    <origin xyz="0 0 0" rpy="0 0 0"/>
-  </xacro:robotiq_ur_hande> -->
+    <!-- com_port="${com_port_hande}"
+    use_fake_hardware="${use_fake_hardware}" -->
+    <xacro:include filename="$(find dextivr_hande_description)/urdf/dextivr_hande.xacro"/>
+    <xacro:dextivr_hande
+      name="right_dextivr_hande"
+      tf_prefix="right_"
+      parent="right_ur_arm_tool0"
+      finger_xacro="fngr_original">
+      <origin xyz="0 0 0" rpy="0 0 ${radians(-90)}"/>
+    </xacro:dextivr_hande>
+    <xacro:dextivr_hande
+      name="left_dextivr_hande"
+      tf_prefix="left_"
+      parent="left_ur_arm_tool0"
+      finger_xacro="fngr_original">
+      <origin xyz="0 0 0" rpy="0 0 ${radians(-90)}"/>
+    </xacro:dextivr_hande>
   </xacro:macro>
 </robot>
