Commit message: adding more parameters and implementing tf_prefix for whole phoebe stack

File: phoebe_description/urdf/jaco01_customization.urdf.xacro (robot description, xacro)
@@ -2,10 +2,25 @@
 <robot xmlns:xacro="http://wiki.ros.org/xacro">
   <!-- Macro for phoebe customization -->
-  <xacro:macro name="jaco01_customization">
+  <xacro:macro
+    name="jaco01_customization"
+    params="
+      use_fake_hardware:='false'
+      sim_ignition:='false'
+      tf_prefix:=''
+      left_ewellix_com_port:='/dev/ttyUSB0'
+      right_ewellix_com_port:='/dev/ttyUSB1'
+      left_hande_com_port:='/dev/ttyUSB2'
+      right_hande_com_port:='/dev/ttyUSB3'
+      left_ur_ip_addr:='192.168.131.40'
+      right_ur_ip_addr:='192.168.131.41'
+      left_ur_kinematics_file:='$(find ur_description)/config/ur5e/default_kinematics.yaml'
+      right_ur_kinematics_file:='(find ur_description)/config/ur5e/default_kinematics.yaml'
+    "
+  >
   <material name="grey">
     <color rgba="0.5 0.5 0.5 1"/>
   </material>
-<!-- Mounting rails for lifts -->
-  <link name="lift_rails">
+  <!-- Mounting rails for lifts -->
+  <link name="${tf_prefix}lift_rails">
     <visual>
       <geometry>
@@ -22,11 +37,11 @@
     </collision>
   </link>
-  <joint name="lift_rails_joint" type="fixed">
-    <parent link="default_mount" />
-    <child link="lift_rails" />
+  <joint name="${tf_prefix}lift_rails_joint" type="fixed">
+    <parent link="${tf_prefix}default_mount" />
+    <child link="${tf_prefix}lift_rails" />
     <origin xyz="0 0 0" rpy="0 0 0" />
   </joint>
-<!-- Rear shelf -->
-  <link name="rear_shelf">
+  <!-- Rear shelf -->
+  <link name="${tf_prefix}rear_shelf">
     <visual>
       <geometry>
@@ -43,11 +58,11 @@
     </collision>
   </link>
-  <joint name="rear_shelf_joint" type="fixed">
-    <parent link="default_mount" />
-    <child link="rear_shelf" />
+  <joint name="${tf_prefix}rear_shelf_joint" type="fixed">
+    <parent link="${tf_prefix}default_mount" />
+    <child link="${tf_prefix}rear_shelf" />
     <origin xyz="0 0 0" rpy="0 0 0" />
   </joint>
-<!-- Front shelf -->
-  <link name="front_shelf">
+  <!-- Front shelf -->
+  <link name="${tf_prefix}front_shelf">
     <visual>
       <geometry>
@@ -64,11 +79,11 @@
     </collision>
   </link>
-  <joint name="front_shelf_joint" type="fixed">
-    <parent link="default_mount" />
-    <child link="front_shelf" />
+  <joint name="${tf_prefix}front_shelf_joint" type="fixed">
+    <parent link="${tf_prefix}default_mount" />
+    <child link="${tf_prefix}front_shelf" />
     <origin xyz="0 0 0" rpy="0 0 ${pi}" />
   </joint>
-<!-- Monitor hinge base -->
-  <link name="monitor_hinge_base">
+  <!-- Monitor hinge base -->
+  <link name="${tf_prefix}monitor_hinge_base">
     <visual>
       <geometry>
@@ -85,11 +100,11 @@
     </collision>
   </link>
-  <joint name="monitor_hinge_base_joint" type="fixed">
-    <parent link="default_mount" />
-    <child link="monitor_hinge_base" />
+  <joint name="${tf_prefix}monitor_hinge_base_joint" type="fixed">
+    <parent link="${tf_prefix}default_mount" />
+    <child link="${tf_prefix}monitor_hinge_base" />
     <origin xyz="-0.4 0 0.24635" rpy="0 0 0" />
   </joint>
-<!-- Monitor hinge top -->
-  <link name="monitor_hinge_top">
+  <!-- Monitor hinge top -->
+  <link name="${tf_prefix}monitor_hinge_top">
     <visual>
       <geometry>
@@ -106,11 +121,11 @@
     </collision>
   </link>
-  <joint name="monitor_hinge_top_joint" type="fixed">
-    <parent link="monitor_hinge_base" />
-    <child link="monitor_hinge_top" />
+  <joint name="${tf_prefix}monitor_hinge_top_joint" type="fixed">
+    <parent link="${tf_prefix}monitor_hinge_base" />
+    <child link="${tf_prefix}monitor_hinge_top" />
     <origin xyz="0 0 0" rpy="0 0.74 0" />
   </joint>
-<!-- Left monitor -->
-  <link name="left_monitor">
+  <!-- Left monitor -->
+  <link name="${tf_prefix}left_monitor">
     <visual>
       <geometry>
@@ -127,11 +142,11 @@
     </collision>
   </link>
-  <joint name="left_monitor_joint" type="fixed">
-    <parent link="monitor_hinge_top" />
-    <child link="left_monitor" />
+  <joint name="${tf_prefix}left_monitor_joint" type="fixed">
+    <parent link="${tf_prefix}monitor_hinge_top" />
+    <child link="${tf_prefix}left_monitor" />
     <origin xyz="-0.04 0.18 0.01" rpy="0 0 0" />
   </joint>
-<!-- Right monitor -->
-  <link name="right_monitor">
+  <!-- Right monitor -->
+  <link name="${tf_prefix}right_monitor">
     <visual>
       <geometry>
@@ -148,11 +163,11 @@
     </collision>
   </link>
-  <joint name="right_monitor_joint" type="fixed">
-    <parent link="monitor_hinge_top" />
-    <child link="right_monitor" />
+  <joint name="${tf_prefix}right_monitor_joint" type="fixed">
+    <parent link="${tf_prefix}monitor_hinge_top" />
+    <child link="${tf_prefix}right_monitor" />
     <origin xyz="-0.04 -0.18 0.01" rpy="0 0 0" />
   </joint>
-<!-- Rear UR Control Box -->
-  <link name="rear_ur_control_box">
+  <!-- Rear UR Control Box -->
+  <link name="${tf_prefix}rear_ur_control_box">
     <visual>
       <geometry>
@@ -169,11 +184,11 @@
     </collision>
   </link>
-  <joint name="rear_ur_control_box_joint" type="fixed">
-    <parent link="default_mount" />
-    <child link="rear_ur_control_box" />
+  <joint name="${tf_prefix}rear_ur_control_box_joint" type="fixed">
+    <parent link="${tf_prefix}default_mount" />
+    <child link="${tf_prefix}rear_ur_control_box" />
     <origin xyz="-0.44274 0.13 0" rpy="0 0 0" />
   </joint>
-<!-- Front UR Control Box -->
-  <link name="front_ur_control_box">
+  <!-- Front UR Control Box -->
+  <link name="${tf_prefix}front_ur_control_box">
     <visual>
       <geometry>
@@ -190,11 +205,11 @@
     </collision>
   </link>
-  <joint name="front_ur_control_box_joint" type="fixed">
-    <parent link="default_mount" />
-    <child link="front_ur_control_box" />
+  <joint name="${tf_prefix}front_ur_control_box_joint" type="fixed">
+    <parent link="${tf_prefix}default_mount" />
+    <child link="${tf_prefix}front_ur_control_box" />
     <origin xyz="0.44274 -0.13 0" rpy="0 0 ${pi}" />
   </joint>
-<!-- Rear Ewellix SCU -->
-  <link name="rear_scu">
+  <!-- Rear Ewellix SCU -->
+  <link name="${tf_prefix}rear_scu">
     <visual>
       <geometry>
@@ -211,11 +226,11 @@
     </collision>
   </link>
-  <joint name="rear_scu_joint" type="fixed">
-    <parent link="default_mount" />
-    <child link="rear_scu" />
+  <joint name="${tf_prefix}rear_scu_joint" type="fixed">
+    <parent link="${tf_prefix}default_mount" />
+    <child link="${tf_prefix}rear_scu" />
     <origin xyz="-0.18187 0 0" rpy="0 0 0" />
   </joint>
-<!-- Front Ewellix SCU -->
-  <link name="front_scu">
+  <!-- Front Ewellix SCU -->
+  <link name="${tf_prefix}front_scu">
     <visual>
       <geometry>
@@ -232,11 +247,11 @@
     </collision>
   </link>
-  <joint name="front_scu_joint" type="fixed">
-    <parent link="default_mount" />
-    <child link="front_scu" />
+  <joint name="${tf_prefix}front_scu_joint" type="fixed">
+    <parent link="${tf_prefix}default_mount" />
+    <child link="${tf_prefix}front_scu" />
     <origin xyz="0.18187 0 0" rpy="0 0 ${pi}" />
   </joint>
-<!-- Autec wireless e-stop MVRCAN receiver -->
-  <link name="autec_receiver">
+  <!-- Autec wireless e-stop MVRCAN receiver -->
+  <link name="${tf_prefix}autec_receiver">
     <visual>
       <geometry>
@@ -253,11 +268,11 @@
     </collision>
   </link>
-  <joint name="autec_receiver_joint" type="fixed">
-    <parent link="default_mount" />
-    <child link="autec_receiver" />
+  <joint name="${tf_prefix}autec_receiver_joint" type="fixed">
+    <parent link="${tf_prefix}default_mount" />
+    <child link="${tf_prefix}autec_receiver" />
     <origin xyz="-0.26 -0.29909 0" rpy="0 0 0" />
   </joint>
-<!-- Right wifi antenna -->
-  <link name="right_wifi_antenna">
+  <!-- Right wifi antenna -->
+  <link name="${tf_prefix}right_wifi_antenna">
     <visual>
       <geometry>
@@ -274,11 +289,11 @@
     </collision>
   </link>
-  <joint name="right_wifi_antenna_joint" type="fixed">
-    <parent link="default_mount" />
-    <child link="right_wifi_antenna" />
+  <joint name="${tf_prefix}right_wifi_antenna_joint" type="fixed">
+    <parent link="${tf_prefix}default_mount" />
+    <child link="${tf_prefix}right_wifi_antenna" />
     <origin xyz="-0.086 -0.384 0.22" rpy="0 0 0" />
   </joint>
-<!-- Left wifi antenna -->
-  <link name="left_wifi_antenna">
+  <!-- Left wifi antenna -->
+  <link name="${tf_prefix}left_wifi_antenna">
     <visual>
       <geometry>
@@ -295,11 +310,11 @@
     </collision>
   </link>
-  <joint name="left_wifi_antenna_joint" type="fixed">
-    <parent link="default_mount" />
-    <child link="left_wifi_antenna" />
+  <joint name="${tf_prefix}left_wifi_antenna_joint" type="fixed">
+    <parent link="${tf_prefix}default_mount" />
+    <child link="${tf_prefix}left_wifi_antenna" />
     <origin xyz="-0.086 0.384 0.22" rpy="0 0 0" />
   </joint>
-<!-- Autec wireless e-stop antenna -->
-  <link name="autec_antenna">
+  <!-- Autec wireless e-stop antenna -->
+  <link name="${tf_prefix}autec_antenna">
     <visual>
       <geometry>
@@ -316,11 +331,11 @@
     </collision>
   </link>
-  <joint name="autec_antenna_joint" type="fixed">
-    <parent link="default_mount" />
-    <child link="autec_antenna" />
+  <joint name="${tf_prefix}autec_antenna_joint" type="fixed">
+    <parent link="${tf_prefix}default_mount" />
+    <child link="${tf_prefix}autec_antenna" />
     <origin xyz="0.0845 -0.384 0.22" rpy="0 0 0" />
   </joint>
-<!-- Left Ewellix mounting flange -->
-  <link name="left_ewellix_mount_flange_link">
+  <!-- Left Ewellix mounting flange -->
+  <link name="${tf_prefix}left_ewellix_mount_flange_link">
     <visual>
       <geometry>
@@ -337,11 +352,11 @@
     </collision>
   </link>
-  <joint name="left_ewellix_mount_flange_joint" type="fixed">
-    <parent link="default_mount"/>
-    <child link="left_ewellix_mount_flange_link"/>
+  <joint name="${tf_prefix}left_ewellix_mount_flange_joint" type="fixed">
+    <parent link="${tf_prefix}default_mount"/>
+    <child link="${tf_prefix}left_ewellix_mount_flange_link"/>
     <origin xyz="0 $(optenv LEFT_LIFT_Y 0.2) 0.04" rpy="0 0 0" />
   </joint>
-<!-- Right Ewellix mounting flange -->
-  <link name="right_ewellix_mount_flange_link">
+  <!-- Right Ewellix mounting flange -->
+  <link name="${tf_prefix}right_ewellix_mount_flange_link">
     <visual>
       <geometry>
@@ -358,59 +373,41 @@
     </collision>
   </link>
-  <joint name="right_ewellix_mount_flange_joint" type="fixed">
-    <parent link="default_mount"/>
-    <child link="right_ewellix_mount_flange_link"/>
+  <joint name="${tf_prefix}right_ewellix_mount_flange_joint" type="fixed">
+    <parent link="${tf_prefix}default_mount"/>
+    <child link="${tf_prefix}right_ewellix_mount_flange_link"/>
     <origin xyz="0 -$(optenv RIGHT_LIFT_Y 0.2) 0.04" rpy="0 0 0" />
   </joint>
 <!-- Ewellix lift column xacro -->
-  <!-- OLD VERSION -->
-  <!-- <xacro:include filename="$(find ewellix_lift)/urdf/ewellix_lift_500mm.urdf.xacro" />
-  <xacro:ewellix_lift_500mm prefix="left_" parent="left_ewellix_mount_flange_link" cut_model="1">
-    <origin xyz="0.0 0.0 0.015" rpy="0 0 0" />
-  </xacro:ewellix_lift_500mm>
-  <xacro:ewellix_lift_500mm prefix="right_" parent="right_ewellix_mount_flange_link" cut_model="1">
-    <origin xyz="0.0 0.0 0.015" rpy="0 0 0" />
-  </xacro:ewellix_lift_500mm> -->
-  <!-- end OLD VERSION -->
-  <!-- clearpath ewellix -->
-  <xacro:include filename="$(find clearpath_manipulators_description)/urdf/lift/ewellix.urdf.xacro"/>
-  <xacro:ewellix name="left" parent_link="left_ewellix_mount_flange_link" add_plate="false">
-    <origin xyz="0.0 0.0 0.015" rpy="0 0 0"/>
-  </xacro:ewellix>
-  <xacro:ewellix name="right" parent_link="right_ewellix_mount_flange_link" add_plate="false">
-    <origin xyz="0.0 0.0 0.015" rpy="0 0 0"/>
-  </xacro:ewellix>
-  <!-- end clearpath ewellix -->
-  <!-- our_ewellix -->
-  <!-- use_fake_hardware="$(arg use_fake_hardware)"
-  com_port="$(arg com_port)" -->
-  <!-- base is 0.015 from clearpath description. 0.2457 is from ewellix_lift.xacro -->
-  <!-- <xacro:include filename="$(find ewellix_liftkit_description)/urdf/ewellix_lift.xacro"/>
+  <!-- base is 0.075 (0.015/2) from clearpath description. 0.2457 is from DRT's ewellix_lift.xacro -->
+  <xacro:include filename="$(find ewellix_liftkit_description)/urdf/ewellix_lift.xacro"/>
   <xacro:include filename="$(find ewellix_liftkit_description)/urdf/properties.xacro"/>
   <xacro:ewellix_lift
-    name="left_ewellix"
+    name="${tf_prefix}left_ewellix"
     is_700="false"
     is_500="true"
-    tf_prefix="left_"
-    parent="left_ewellix_mount_flange_link"
+    tf_prefix="${tf_prefix}left_"
+    parent="${tf_prefix}left_ewellix_mount_flange_link"
     height_limit="0.5"
     omit_plates="true"
+    use_fake_hardware="${use_fake_hardware}"
+    com_port="${left_ewellix_com_port}"
   >
     <origin xyz="0 0 ${0.0075+0.2457}" rpy="0 0 0"/>
   </xacro:ewellix_lift>
   <xacro:ewellix_lift
-    name="right_ewellix"
+    name="${tf_prefix}right_ewellix"
     is_700="false"
     is_500="true"
-    tf_prefix="right_"
-    parent="right_ewellix_mount_flange_link"
+    tf_prefix="${tf_prefix}right_"
+    parent="${tf_prefix}right_ewellix_mount_flange_link"
     height_limit="0.5"
     omit_plates="true"
+    use_fake_hardware="${use_fake_hardware}"
+    com_port="${right_ewellix_com_port}"
   >
     <origin xyz="0 0 ${0.0075+0.2457}" rpy="0 0 0"/>
-  </xacro:ewellix_lift> -->
-  <!-- end our_ewellix -->
-<!-- Left arm mount plate -->
-  <link name="left_arm_mount_plate">
+  </xacro:ewellix_lift>
+  <!-- Left arm mount plate -->
+  <link name="${tf_prefix}left_arm_mount_plate">
     <visual>
       <geometry>
@@ -425,12 +422,11 @@
     </collision>
   </link>
-  <joint name="left_arm_mount_plate_joint" type="fixed">
-    <parent link="left_mount" />
-    <!-- <parent link="left_ewellix_lift_tip_link" /> -->
-    <child link="left_arm_mount_plate" />
+  <joint name="${tf_prefix}left_arm_mount_plate_joint" type="fixed">
+    <parent link="${tf_prefix}left_ewellix_lift_tip_link" />
+    <child link="${tf_prefix}left_arm_mount_plate" />
     <origin xyz="0 0 0" rpy="0 0 0" />
   </joint>
-<!-- Right arm mount plate -->
-  <link name="right_arm_mount_plate">
+  <!-- Right arm mount plate -->
+  <link name="${tf_prefix}right_arm_mount_plate">
     <visual>
       <geometry>
@@ -445,105 +441,77 @@
     </collision>
   </link>
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
File: phoebe_description/urdf/phoebe.urdf.xacro (robot description, xacro)
@@ -3,6 +3,13 @@
     <xacro:arg name="tf_prefix" default="" />
     <xacro:arg name="ns" default="" />
-    <xacro:arg name="is_sim" default="true" />
-    <xacro:arg name="parent" default="world" />
+    <xacro:arg name="is_sim" default="false" />
+    <xacro:arg name="sim_ignition" default="false" />
+    <xacro:arg name="use_fake_hardware" default="false" />
+    <xacro:arg name="left_ewellix_com_port" default="/dev/ttyUSB0" />
+    <xacro:arg name="right_ewellix_com_port" default="/dev/ttyUSB1" />
+    <xacro:arg name="left_ur_ip_addr" default="192.168.131.40" />
+    <xacro:arg name="right_ur_ip_addr" default="192.168.131.41" />
+    <xacro:arg name="left_ur_kinematics_file" default="$(find ur_description)/config/ur5e/default_kinematics.yaml" />
+    <xacro:arg name="right_ur_kinematics_file" default="$(find ur_description)/config/ur5e/default_kinematics.yaml" />
     <!-- Includes -->
     <xacro:include filename="$(find clearpath_platform_description)/urdf/common.urdf.xacro" />
@@ -14,4 +21,14 @@
     />
     <xacro:include filename="$(find phoebe_description)/urdf/jaco01_customization.urdf.xacro" />
-    <xacro:jaco01_customization/>
+    <xacro:jaco01_customization
+        tf_prefix="$(arg tf_prefix)"
+        use_fake_hardware="$(arg is_sim)"
+        sim_ignition="$(arg sim_ignition)"
+        left_ewellix_com_port="$(arg left_ewellix_com_port)"
+        right_ewellix_com_port="$(arg right_ewellix_com_port)"
+        left_ur_ip_addr="$(arg left_ur_ip_addr)"
+        right_ur_ip_addr="$(arg right_ur_ip_addr)"
+        left_ur_kinematics_file="$(arg left_ur_kinematics_file)"
+        right_ur_kinematics_file="$(arg right_ur_kinematics_file)"
+    />
 </robot>
