Commit message: adding camera models and launch

File: phoebe_description/urdf/ee_interface.xacro (robot description, xacro)
@@ -42,4 +42,30 @@
         </collision>
     </link>
+    <joint name="${tf_prefix}mtc_effector_side_to_realsense_mount" type="fixed">
+        <parent link="${tf_prefix}mtc_effector_side"/>
+        <child link="${tf_prefix}ur_realsense_mount"/>
+        <origin xyz="0 0 0.024" rpy="0 0 0"/>
+    </joint>
+    <link name="${tf_prefix}ur_realsense_mount">
+        <visual>
+            <geometry>
+                <mesh filename= "package://phoebe_description/meshes/visual/ur_realsense_short_mount_tube.stl"/>
+            </geometry>
+            <material name="${tf_prefix}ur_realsense_mount">
+                <color rgba="0.1 0.1 0.1 1.0"/>
+            </material>
+        </visual>
+        <collision>
+            <geometry>
+                <mesh filename= "package://phoebe_description/meshes/visual/ur_realsense_short_mount_tube.stl"/>
+            </geometry>
+        </collision>
+    </link>
+    <!-- Realsense camera -->
+    <xacro:property name="realsense_materials_defined" value="true" />
+    <xacro:include filename="$(find realsense2_description)/urdf/_d435.urdf.xacro"/>
+    <xacro:sensor_d435 parent="${tf_prefix}ur_realsense_mount" use_nominal_extrinsics="true" use_mesh="true" name="${tf_prefix}wrist_mounted_camera">
+        <origin xyz="-0.064 -0.003 0.016" rpy="0.136 -1.429 -0.128"/>
+    </xacro:sensor_d435>
     </xacro:macro>
 </robot>

File: phoebe_description/urdf/phoebe_macro.xacro (robot description, xacro)
@@ -605,7 +605,7 @@
       name="${tf_prefix}right_dextivr_hande"
       tf_prefix="${tf_prefix}right_"
-      parent="${tf_prefix}right_mtc_effector_side"
+      parent="${tf_prefix}right_ur_realsense_mount"
       finger_xacro="fngr_original">
-      <origin xyz="0 0 0.024" rpy="0 0 ${pi}"/>
+      <origin xyz="0 0 0.008" rpy="0 0 ${pi}"/>
     </xacro:dextivr_hande>
     <xacro:dextivr_hande
@@ -614,7 +614,7 @@
       name="${tf_prefix}left_dextivr_hande"
       tf_prefix="${tf_prefix}left_"
-      parent="${tf_prefix}left_mtc_effector_side"
+      parent="${tf_prefix}left_ur_realsense_mount"
       finger_xacro="fngr_original">
-      <origin xyz="0 0 0.024" rpy="0 0 ${pi}"/>
+      <origin xyz="0 0 0.008" rpy="0 0 ${pi}"/>
     </xacro:dextivr_hande>
   </xacro:unless>

Commit message: updating for new camera mount

File: phoebe_description/urdf/ee_interface.xacro (robot description, xacro)
@@ -50,5 +50,5 @@
         <visual>
             <geometry>
-                <mesh filename= "package://phoebe_description/meshes/visual/ur_realsense_short_mount_tube.stl"/>
+                <mesh filename= "package://phoebe_description/meshes/visual/ich-005_realsense_cable_mount_corr.stl" scale="0.0254 0.0254 0.0254"/>
             </geometry>
             <material name="${tf_prefix}ur_realsense_mount">
@@ -58,14 +58,8 @@
         <collision>
             <geometry>
-                <mesh filename= "package://phoebe_description/meshes/visual/ur_realsense_short_mount_tube.stl"/>
+                <mesh filename= "package://phoebe_description/meshes/visual/ich-005_realsense_cable_mount_corr.stl" scale="0.0254 0.0254 0.0254"/>
             </geometry>
         </collision>
     </link>
-    <!-- Realsense camera -->
-    <xacro:property name="realsense_materials_defined" value="true" />
-    <xacro:include filename="$(find realsense2_description)/urdf/_d435.urdf.xacro"/>
-    <xacro:sensor_d435 parent="${tf_prefix}ur_realsense_mount" use_nominal_extrinsics="true" use_mesh="true" name="${tf_prefix}wrist_mounted_camera">
-        <origin xyz="-0.064 -0.003 0.016" rpy="0.136 -1.429 -0.128"/>
-    </xacro:sensor_d435>
     </xacro:macro>
 </robot>

File: phoebe_description/urdf/phoebe_macro.xacro (robot description, xacro)
@@ -546,15 +546,48 @@
   </xacro:ur_robot>
   <!-- end effector interface stack -->
-  <xacro:include filename="$(find phoebe_description)/urdf/ee_interface.xacro"/>
-  <xacro:ee_interface
-    tf_prefix="${tf_prefix}right_"
-    parent="${tf_prefix}right_ur_arm_tool0">
-    <origin xyz="0 0 0.0" rpy="0 0 ${pi}"/>
-  </xacro:ee_interface>
-  <xacro:ee_interface
-    tf_prefix="${tf_prefix}left_"
-    parent="${tf_prefix}left_ur_arm_tool0">
-    <origin xyz="0 0 0.0" rpy="0 0 ${pi}"/>
-  </xacro:ee_interface>
+  <xacro:unless value="${calibration_mode}">
+    <xacro:include filename="$(find phoebe_description)/urdf/ee_interface.xacro"/>
+    <xacro:ee_interface
+      tf_prefix="${tf_prefix}right_"
+      parent="${tf_prefix}right_ur_arm_tool0">
+      <origin xyz="0 0 0.0" rpy="0 0 ${pi}"/>
+    </xacro:ee_interface>
+    <xacro:ee_interface
+      tf_prefix="${tf_prefix}left_"
+      parent="${tf_prefix}left_ur_arm_tool0">
+      <origin xyz="0 0 0.0" rpy="0 0 ${pi}"/>
+    </xacro:ee_interface>
+    <!-- Realsense camera -->
+    <xacro:property name="realsense_materials_defined" value="true" />
+    <xacro:include filename="$(find realsense2_description)/urdf/_d435.urdf.xacro"/>
+    <!-- right camera -->
+    <xacro:sensor_d435 parent="${tf_prefix}right_ur_realsense_mount" use_nominal_extrinsics="true" use_mesh="true" name="${tf_prefix}right_wrist_mounted_camera">
+      <origin xyz="-0.064 -0.003 0.016" rpy="0.136 -1.429 -0.128"/>
+    </xacro:sensor_d435>
+    <!-- left camera -->
+    <xacro:sensor_d435 parent="${tf_prefix}left_ur_realsense_mount" use_nominal_extrinsics="true" use_mesh="true" name="${tf_prefix}left_wrist_mounted_camera">
+      <origin xyz="-0.064 -0.003 0.016" rpy="0.136 -1.429 -0.128"/>
+    </xacro:sensor_d435>
+    <!-- Hand-E Grippers -->
+    <xacro:include filename="$(find dextivr_hande_description)/urdf/dextivr_hande.xacro"/>
+    <xacro:dextivr_hande
+      com_port="${right_hande_com_port}"
+      use_fake_hardware="${use_fake_hardware}"
+      name="${tf_prefix}right_dextivr_hande"
+      tf_prefix="${tf_prefix}right_"
+      parent="${tf_prefix}right_ur_realsense_mount"
+      finger_xacro="fngr_original">
+      <origin xyz="0 0 0.008" rpy="0 0 ${pi}"/>
+    </xacro:dextivr_hande>
+    <xacro:dextivr_hande
+      com_port="${left_hande_com_port}"
+      use_fake_hardware="${use_fake_hardware}"
+      name="${tf_prefix}left_dextivr_hande"
+      tf_prefix="${tf_prefix}left_"
+      parent="${tf_prefix}left_ur_realsense_mount"
+      finger_xacro="fngr_original">
+      <origin xyz="0 0 0.008" rpy="0 0 ${pi}"/>
+    </xacro:dextivr_hande>
+  </xacro:unless>
   <!-- Calibration HW -->
   <xacro:if value="${calibration_mode}">
@@ -597,26 +630,4 @@
     <link name="${tf_prefix}calibration_face_target_side"/>
   </xacro:if>
-  <!-- Hand-E Grippers -->
-  <xacro:unless value="${calibration_mode}">
-    <xacro:include filename="$(find dextivr_hande_description)/urdf/dextivr_hande.xacro"/>
-    <xacro:dextivr_hande
-      com_port="${right_hande_com_port}"
-      use_fake_hardware="${use_fake_hardware}"
-      name="${tf_prefix}right_dextivr_hande"
-      tf_prefix="${tf_prefix}right_"
-      parent="${tf_prefix}right_ur_realsense_mount"
-      finger_xacro="fngr_original">
-      <origin xyz="0 0 0.008" rpy="0 0 ${pi}"/>
-    </xacro:dextivr_hande>
-    <xacro:dextivr_hande
-      com_port="${left_hande_com_port}"
-      use_fake_hardware="${use_fake_hardware}"
-      name="${tf_prefix}left_dextivr_hande"
-      tf_prefix="${tf_prefix}left_"
-      parent="${tf_prefix}left_ur_realsense_mount"
-      finger_xacro="fngr_original">
-      <origin xyz="0 0 0.008" rpy="0 0 ${pi}"/>
-    </xacro:dextivr_hande>
-  </xacro:unless>
   </xacro:macro>
 </robot>

Commit message: rotating ee stack to be correct

File: phoebe_description/urdf/ee_interface.xacro (robot description, xacro)
@@ -45,5 +45,5 @@
         <parent link="${tf_prefix}mtc_effector_side"/>
         <child link="${tf_prefix}ur_realsense_mount"/>
-        <origin xyz="0 0 0.024" rpy="0 0 0"/>
+        <origin xyz="0 0 0.024" rpy="0 0 ${radians(90)}"/>
     </joint>
     <link name="${tf_prefix}ur_realsense_mount">

File: phoebe_description/urdf/phoebe_macro.xacro (robot description, xacro)
@@ -578,5 +578,5 @@
       parent="${tf_prefix}right_ur_realsense_mount"
       finger_xacro="fngr_original">
-      <origin xyz="0 0 0.008" rpy="0 0 ${pi}"/>
+      <origin xyz="0 0 0.008" rpy="0 0 ${pi/2}"/>
     </xacro:dextivr_hande>
     <xacro:dextivr_hande
@@ -587,5 +587,5 @@
       parent="${tf_prefix}left_ur_realsense_mount"
       finger_xacro="fngr_original">
-      <origin xyz="0 0 0.008" rpy="0 0 ${pi}"/>
+      <origin xyz="0 0 0.008" rpy="0 0 ${pi/2}"/>
     </xacro:dextivr_hande>
   </xacro:unless>
