Commit message: Added cylinder and cylinder jig into the environment urdf. Made a new rviz config file for the environment.

File: phoebe_description/urdf/phoebe_environment.xacro (robot description, xacro)
@@ -1,5 +1,5 @@
 <?xml version="1.0"?>
 <robot xmlns:xacro="http://wiki.ros.org/xacro" name="phoebe_environment">
-  <!-- ===================== MATERIALS ===================== -->
+  <!-- ===================== MATERIALS/COLORS ===================== -->
   <material name="black">
     <color rgba="0.1 0.1 0.1 1"/>
@@ -13,4 +13,7 @@
   <material name="gray">
     <color rgba="0.7 0.7 0.7 1"/>
+  </material>
+  <material name="bottle_blue">
+    <color rgba="0.1 0.4 0.9 1"/>
   </material>
   <!-- ===================== MACRO ===================== -->
@@ -156,4 +159,38 @@
     </joint>
   </xacro:macro>
+  <!-- ===================== CYLINDER ===================== -->
+    <link name="cylinder">
+     <visual>
+        <origin xyz="2.75 -0.666 0.665"/>
+        <geometry>
+            <mesh filename="package://phoebe_description/meshes/visual/cylinder/cylinder_mockup_full_length.stl" scale="0.001 0.001 0.001"/>
+        </geometry>
+        <material name="bottle_blue"/>
+     </visual>
+     <collision>
+        <origin xyz="2.75 -0.666 0.665"/>
+        <geometry>
+            <mesh filename="package://phoebe_description/meshes/visual/cylinder/cylinder_mockup_full_length.stl" scale="0.001 0.001 0.001"/>
+        </geometry>
+     </collision>
+    </link>
+    <joint name="world_to_cylinder" type="fixed">
+      <parent link="world"/>
+      <child link="cylinder"/>
+  </joint>
+  <!-- ===================== CYLINDER JIG ===================== -->
+  <link name="cylinder_jig">
+    <visual>
+      <origin xyz="-2.1 -0.666 0.667" rpy="-1.57 3.14 -1.57"/>
+      <geometry>
+        <mesh filename="package://phoebe_description/meshes/visual/cylinder/cylinder_jig/cylinder_jig.obj" scale="0.001 0.001 0.001"/>
+      </geometry>
+      <material name="black"/>
+    </visual>
+  </link>
+  <joint name="world_to_cylinder_jig" type="fixed">
+    <parent link="world"/>
+    <child link="cylinder_jig"/>
+  </joint>
   <!-- ===================== INSTANTIATE MACRO ===================== -->
   <xacro:phoebe_environment/>

Commit message: Replaced cylinder jig mesh obj file with stl file in the environment urdf. Plus general clean up and pre-commit.

File: phoebe_description/urdf/phoebe_environment.xacro (robot description, xacro)
@@ -182,7 +182,7 @@
   <link name="cylinder_jig">
     <visual>
-      <origin xyz="-2.1 -0.666 0.667" rpy="-1.57 3.14 -1.57"/>
+      <origin xyz="-2.1 -0.666 0.667" rpy="3.14 3.14 0"/>
       <geometry>
-        <mesh filename="package://phoebe_description/meshes/visual/cylinder/cylinder_jig/cylinder_jig.obj" scale="0.001 0.001 0.001"/>
+        <mesh filename="package://phoebe_description/meshes/visual/cylinder/cylinder_jig/cylinder_jig.stl" scale="0.001 0.001 0.001"/>
       </geometry>
       <material name="black"/>
