Commit message: File structure update. Made a seperate color xacro.

File: phoebe_description/urdf/phoebe_environment_macro.xacro (robot description, xacro)
@@ -1,42 +1,9 @@
 <?xml version="1.0"?>
 <robot xmlns:xacro="http://wiki.ros.org/xacro" name="phoebe_environment">
-  <!-- ===================== MATERIALS/COLORS ===================== -->
-  <material name="black">
-    <color rgba="0.1 0.1 0.1 1"/>
-  </material>
-  <material name="blue">
-    <color rgba="0.1 0.1 0.3 1"/>
-  </material>
-  <material name="brown">
-    <color rgba="0.42 0.22 0.16 1"/>
-  </material>
-  <material name="gray">
-    <color rgba="0.7 0.7 0.7 1"/>
-  </material>
-  <material name="bottle_blue">
-    <color rgba="0.1 0.4 0.9 1"/>
-  </material>
-  <!-- ===================== MACRO ===================== -->
   <xacro:macro name="phoebe_environment">
+  <!-- Include color xacro -->
+  <xacro:include filename="$(find phoebe_description)/urdf/phoebe_environment_colors.xacro"/>
     <!-- WORLD -->
     <link name="world"/>
-    <!-- ===================== FLOOR ===================== -->
-    <link name="floor">
-      <visual>
-        <geometry>
-          <plane normal="0 0 1"/>
-        </geometry>
-        <material name="gray"/>
-      </visual>
-      <collision>
-        <geometry>
-          <plane normal="0 0 1"/>
-        </geometry>
-      </collision>
-    </link>
-    <joint name="world_to_floor" type="fixed">
-      <parent link="world"/>
-      <child link="floor"/>
-    </joint>
     <!-- ===================== BOOKSHELVES (CABINETS) ===================== -->
     <link name="bookshelves">
@@ -47,5 +14,5 @@
           <box size="3.0 0.5 1.5"/>
         </geometry>
-        <material name="black"/>
+        <material name="phoebe_environment_black"/>
       </visual>
       <collision>
@@ -61,5 +28,5 @@
           <box size="3.0 0.5 1.5"/>
         </geometry>
-        <material name="black"/>
+        <material name="phoebe_environment_black"/>
       </visual>
       <collision>
@@ -82,5 +49,5 @@
           <box size="0.666 1.332 0.666"/>
         </geometry>
-        <material name="blue"/>
+        <material name="phoebe_environment_blue"/>
       </visual>
       <collision>
@@ -96,5 +63,5 @@
           <box size="0.666 0.666 0.666"/>
         </geometry>
-        <material name="blue"/>
+        <material name="phoebe_environment_blue"/>
       </visual>
       <collision>
@@ -117,5 +84,5 @@
           <box size="0.666 1.332 0.666"/>
         </geometry>
-        <material name="brown"/>
+        <material name="phoebe_environment_brown"/>
       </visual>
       <collision>
@@ -131,5 +98,5 @@
           <box size="0.666 1.332 0.666"/>
         </geometry>
-        <material name="brown"/>
+        <material name="phoebe_environment_brown"/>
       </visual>
       <collision>
@@ -145,5 +112,5 @@
           <box size="0.666 2.5 0.666"/>
         </geometry>
-        <material name="brown"/>
+        <material name="phoebe_environment_brown"/>
       </visual>
       <collision>
@@ -160,5 +127,5 @@
   </xacro:macro>
   <!-- ===================== CYLINDER ===================== -->
-    <link name="cylinder">
+  <link name="cylinder">
      <visual>
         <origin xyz="2.75 -0.666 0.665"/>
@@ -166,5 +133,5 @@
             <mesh filename="package://phoebe_description/meshes/visual/cylinder/cylinder_mockup_full_length.stl" scale="0.001 0.001 0.001"/>
         </geometry>
-        <material name="bottle_blue"/>
+        <material name="cylinder_bottle_blue"/>
      </visual>
      <collision>
@@ -174,8 +141,8 @@
         </geometry>
      </collision>
-    </link>
-    <joint name="world_to_cylinder" type="fixed">
-      <parent link="world"/>
-      <child link="cylinder"/>
+  </link>
+  <joint name="world_to_cylinder" type="fixed">
+    <parent link="world"/>
+    <child link="cylinder"/>
   </joint>
   <!-- ===================== CYLINDER JIG ===================== -->
@@ -186,5 +153,5 @@
         <mesh filename="package://phoebe_description/meshes/visual/cylinder/cylinder_jig/cylinder_jig.stl" scale="0.001 0.001 0.001"/>
       </geometry>
-      <material name="black"/>
+      <material name="phoebe_environment_black"/>
     </visual>
   </link>

Commit message: Updated the parent as a parameter in the macro,, updated urdf xacro file. More clean-up.

File: phoebe_description/urdf/phoebe_environment_macro.xacro (robot description, xacro)
@@ -1,9 +1,7 @@
 <?xml version="1.0"?>
 <robot xmlns:xacro="http://wiki.ros.org/xacro" name="phoebe_environment">
-  <xacro:macro name="phoebe_environment">
-  <!-- Include color xacro -->
-  <xacro:include filename="$(find phoebe_description)/urdf/phoebe_environment_colors.xacro"/>
-    <!-- WORLD -->
-    <link name="world"/>
+  <xacro:macro name="phoebe_environment" params="parent">
+    <!-- Include color xacro -->
+    <xacro:include filename="$(find phoebe_description)/urdf/phoebe_environment_colors.xacro"/>
     <!-- ===================== BOOKSHELVES (CABINETS) ===================== -->
     <link name="bookshelves">
@@ -37,6 +35,6 @@
       </collision>
     </link>
-    <joint name="world_to_bookshelves" type="fixed">
-      <parent link="world"/>
+    <joint name="${parent}_to_bookshelves" type="fixed">
+      <parent link="${parent}"/>
       <child link="bookshelves"/>
     </joint>
@@ -72,6 +70,6 @@
       </collision>
     </link>
-    <joint name="world_to_tables" type="fixed">
-      <parent link="world"/>
+    <joint name="${parent}_to_tables" type="fixed">
+      <parent link="${parent}"/>
       <child link="tables"/>
     </joint>
@@ -121,44 +119,42 @@
       </collision>
     </link>
-    <joint name="world_to_desks" type="fixed">
-      <parent link="world"/>
+    <joint name="${parent}_to_desks" type="fixed">
+      <parent link="${parent}"/>
       <child link="desks"/>
     </joint>
+    <!-- ===================== CYLINDER ===================== -->
+    <link name="cylinder">
+       <visual>
+          <origin xyz="2.75 -0.666 0.665"/>
+          <geometry>
+              <mesh filename="package://phoebe_description/meshes/visual/cylinder/cylinder_mockup_full_length.stl" scale="0.001 0.001 0.001"/>
+          </geometry>
+          <material name="cylinder_bottle_blue"/>
+       </visual>
+       <collision>
+          <origin xyz="2.75 -0.666 0.665"/>
+          <geometry>
+              <mesh filename="package://phoebe_description/meshes/visual/cylinder/cylinder_mockup_full_length.stl" scale="0.001 0.001 0.001"/>
+          </geometry>
+       </collision>
+    </link>
+    <joint name="${parent}_to_cylinder" type="fixed">
+      <parent link="${parent}"/>
+      <child link="cylinder"/>
+    </joint>
+    <!-- ===================== CYLINDER JIG ===================== -->
+    <link name="cylinder_jig">
+      <visual>
+        <origin xyz="-2.1 -0.666 0.667" rpy="3.14 3.14 0"/>
+        <geometry>
+          <mesh filename="package://phoebe_description/meshes/visual/cylinder/cylinder_jig/cylinder_jig.stl" scale="0.001 0.001 0.001"/>
+        </geometry>
+        <material name="phoebe_environment_black"/>
+      </visual>
+    </link>
+    <joint name="${parent}_to_cylinder_jig" type="fixed">
+      <parent link="${parent}"/>
+      <child link="cylinder_jig"/>
+    </joint>
   </xacro:macro>
-  <!-- ===================== CYLINDER ===================== -->
-  <link name="cylinder">
-     <visual>
-        <origin xyz="2.75 -0.666 0.665"/>
-        <geometry>
-            <mesh filename="package://phoebe_description/meshes/visual/cylinder/cylinder_mockup_full_length.stl" scale="0.001 0.001 0.001"/>
-        </geometry>
-        <material name="cylinder_bottle_blue"/>
-     </visual>
-     <collision>
-        <origin xyz="2.75 -0.666 0.665"/>
-        <geometry>
-            <mesh filename="package://phoebe_description/meshes/visual/cylinder/cylinder_mockup_full_length.stl" scale="0.001 0.001 0.001"/>
-        </geometry>
-     </collision>
-  </link>
-  <joint name="world_to_cylinder" type="fixed">
-    <parent link="world"/>
-    <child link="cylinder"/>
-  </joint>
-  <!-- ===================== CYLINDER JIG ===================== -->
-  <link name="cylinder_jig">
-    <visual>
-      <origin xyz="-2.1 -0.666 0.667" rpy="3.14 3.14 0"/>
-      <geometry>
-        <mesh filename="package://phoebe_description/meshes/visual/cylinder/cylinder_jig/cylinder_jig.stl" scale="0.001 0.001 0.001"/>
-      </geometry>
-      <material name="phoebe_environment_black"/>
-    </visual>
-  </link>
-  <joint name="world_to_cylinder_jig" type="fixed">
-    <parent link="world"/>
-    <child link="cylinder_jig"/>
-  </joint>
-  <!-- ===================== INSTANTIATE MACRO ===================== -->
-  <xacro:phoebe_environment/>
 </robot>
