Commit message: fixing orientation of urs and grippers

File: phoebe_description/urdf/phoebe_macro.xacro (robot description, xacro)
@@ -491,5 +491,5 @@
     output_recipe_filename="$(find ur_robot_driver)/resources/rtde_output_recipe.txt"
     >
-    <origin xyz="0 0 0" rpy="0 0 0" />
+    <origin xyz="0 0 0" rpy="0 0 ${5*pi/4}" />
   </xacro:ur_robot>
   <xacro:ur_robot
@@ -514,5 +514,5 @@
     output_recipe_filename="$(find ur_robot_driver)/resources/rtde_output_recipe.txt"
     >
-    <origin xyz="0 0 0" rpy="0 0 0" /> <!-- TODO: need to integrate the OPTENV RIGEBACK_RIGHT_UR_XYZ stuff-->
+    <origin xyz="0 0 0" rpy="0 0 ${-pi/4}" /> <!-- TODO: need to integrate the OPTENV RIGEBACK_RIGHT_UR_XYZ stuff-->
   </xacro:ur_robot>
   <!-- Hand-E Grippers -->
@@ -525,5 +525,5 @@
     parent="${tf_prefix}right_ur_arm_tool0"
     finger_xacro="fngr_original">
-    <origin xyz="0 0 0" rpy="0 0 ${radians(-90)}"/>
+    <origin xyz="0 0 0" rpy="0 0 0"/>
   </xacro:dextivr_hande>
   <xacro:dextivr_hande
@@ -534,5 +534,5 @@
     parent="${tf_prefix}left_ur_arm_tool0"
     finger_xacro="fngr_original">
-    <origin xyz="0 0 0" rpy="0 0 ${radians(-90)}"/>
+    <origin xyz="0 0 0" rpy="0 0 0"/>
   </xacro:dextivr_hande>
   </xacro:macro>

Commit message: adding in the EE stack with quick disconnect

File: phoebe_description/urdf/phoebe_macro.xacro (robot description, xacro)
@@ -530,4 +530,16 @@
     <origin xyz="0 0 0" rpy="0 0 ${-pi/4}" /> <!-- TODO: need to integrate the OPTENV RIGEBACK_RIGHT_UR_XYZ stuff-->
   </xacro:ur_robot>
+  <!-- end effector interface stack -->
+  <xacro:include filename="$(find phoebe_description)/urdf/ee_interface.xacro"/>
+  <xacro:ee_interface
+    tf_prefix="${tf_prefix}right_"
+    parent="${tf_prefix}right_ur_arm_tool0">
+    <origin xyz="0 0 0.0" rpy="0 0 ${pi}"/>
+  </xacro:ee_interface>
+  <xacro:ee_interface
+    tf_prefix="${tf_prefix}left_"
+    parent="${tf_prefix}left_ur_arm_tool0">
+    <origin xyz="0 0 0.0" rpy="0 0 ${pi}"/>
+  </xacro:ee_interface>
   <!-- Hand-E Grippers -->
   <xacro:include filename="$(find dextivr_hande_description)/urdf/dextivr_hande.xacro"/>
@@ -537,7 +549,7 @@
     name="${tf_prefix}right_dextivr_hande"
     tf_prefix="${tf_prefix}right_"
-    parent="${tf_prefix}right_ur_arm_tool0"
+    parent="${tf_prefix}right_mtc_effector_side"
     finger_xacro="fngr_original">
-    <origin xyz="0 0 0" rpy="0 0 0"/>
+    <origin xyz="0 0 0.024" rpy="0 0 ${pi}"/>
   </xacro:dextivr_hande>
   <xacro:dextivr_hande
@@ -546,7 +558,7 @@
     name="${tf_prefix}left_dextivr_hande"
     tf_prefix="${tf_prefix}left_"
-    parent="${tf_prefix}left_ur_arm_tool0"
+    parent="${tf_prefix}left_mtc_effector_side"
     finger_xacro="fngr_original">
-    <origin xyz="0 0 0" rpy="0 0 0"/>
+    <origin xyz="0 0 0.024" rpy="0 0 ${pi}"/>
   </xacro:dextivr_hande>
   </xacro:macro>

Commit message: adding calibration link info and bumping up ewellix

File: phoebe_description/urdf/phoebe_macro.xacro (robot description, xacro)
@@ -446,5 +446,5 @@
     <parent link="${tf_prefix}left_ewellix_lift_tip_link" />
     <child link="${tf_prefix}left_arm_mount_plate" />
-    <origin xyz="0 0 0" rpy="0 0 0" />
+    <origin xyz="0 0 0.03" rpy="0 0 0" />
   </joint>
   <!-- Right arm mount plate -->
@@ -465,5 +465,5 @@
     <parent link="${tf_prefix}right_ewellix_lift_tip_link" />
     <child link="${tf_prefix}right_arm_mount_plate" />
-    <origin xyz="0 0 0" rpy="0 0 ${pi}" />
+    <origin xyz="0 0 0.03" rpy="0 0 ${pi}" />
   </joint>
   <!-- calibration links -->
@@ -472,5 +472,5 @@
     <parent link="${tf_prefix}left_arm_mount_plate" />
     <child link="${tf_prefix}left_arm_cal_link" />
-    <origin xyz="0 0 0" rpy="0 0 0"/>
+    <origin xyz="0.00807 -0.00363 0.01019" rpy="0.01529 0.01951 -0.00426"/>
   </joint>
   <link name="${tf_prefix}right_arm_cal_link"> </link>
@@ -478,5 +478,5 @@
     <parent link="${tf_prefix}right_arm_mount_plate" />
     <child link="${tf_prefix}right_arm_cal_link" />
-    <origin xyz="0 0 0" rpy="0 0 0"/>
+    <origin xyz="-0.00878 -0.00039 0.00881" rpy="0.01118 -0.02966 -0.00119"/>
   </joint>
   <!-- end calibration links -->

Commit message: removing the 0.03 offset

File: phoebe_description/urdf/phoebe_macro.xacro (robot description, xacro)
@@ -446,5 +446,5 @@
     <parent link="${tf_prefix}left_ewellix_lift_tip_link" />
     <child link="${tf_prefix}left_arm_mount_plate" />
-    <origin xyz="0 0 0.03" rpy="0 0 0" />
+    <origin xyz="0 0 0" rpy="0 0 0" />
   </joint>
   <!-- Right arm mount plate -->
@@ -465,5 +465,5 @@
     <parent link="${tf_prefix}right_ewellix_lift_tip_link" />
     <child link="${tf_prefix}right_arm_mount_plate" />
-    <origin xyz="0 0 0.03" rpy="0 0 ${pi}" />
+    <origin xyz="0 0 0" rpy="0 0 ${pi}" />
   </joint>
   <!-- calibration links -->

Commit message: switching to trac_ik and updating for camera calibration

File: phoebe_description/urdf/phoebe_macro.xacro (robot description, xacro)
@@ -567,5 +567,6 @@
     <!-- left camera -->
     <xacro:sensor_d435 parent="${tf_prefix}left_ur_realsense_mount" use_nominal_extrinsics="true" use_mesh="true" name="${tf_prefix}left_wrist_mounted_camera">
-      <origin xyz="-0.064 -0.003 0.016" rpy="0.136 -1.429 -0.128"/>
+      <!-- <origin xyz="-0.064 -0.003 0.016" rpy="0.136 -1.429 -0.128"/> -->
+      <origin xyz="-6.3398954689359577e-02 1.0843610275642415e-03 1.0771886573701910e-02" rpy="-3.3291953701393887e-02 -1.4542171203396566e+00 3.8217188478749678e-02"/>
     </xacro:sensor_d435>
     <!-- Hand-E Grippers -->

Commit message: big commit for general features of demo working with action pipeline

File: phoebe_description/urdf/phoebe_macro.xacro (robot description, xacro)
@@ -180,10 +180,10 @@
   <!-- Rear UR Control Box -->
   <link name="${tf_prefix}rear_ur_control_box">
-    <visual>
+    <!-- <visual>
       <geometry>
         <mesh filename="package://phoebe_description/meshes/visual/jaco01_meshes/ur_control_box.STL"/>
       </geometry>
       <material name="clearpath_aluminum" />
-    </visual>
+    </visual> -->
     <collision>
       <origin xyz="0.090 -0.107 0.098"/>
@@ -201,10 +201,10 @@
   <!-- Front UR Control Box -->
   <link name="${tf_prefix}front_ur_control_box">
-    <visual>
+    <!-- <visual>
       <geometry>
         <mesh filename="package://phoebe_description/meshes/visual/jaco01_meshes/ur_control_box.STL"/>
       </geometry>
       <material name="clearpath_aluminum" />
-    </visual>
+    </visual> -->
     <collision>
       <origin xyz="0.090 -0.107 0.098"/>
@@ -563,10 +563,17 @@
     <!-- right camera -->
     <xacro:sensor_d435 parent="${tf_prefix}right_ur_realsense_mount" use_nominal_extrinsics="true" use_mesh="true" name="${tf_prefix}right_wrist_mounted_camera">
-      <origin xyz="-0.064 -0.003 0.016" rpy="0.136 -1.429 -0.128"/>
+      <!-- original -->
+      <!-- <origin xyz="-0.064 -0.003 0.016" rpy="0.136 -1.429 -0.128"/> -->
+      <!-- first cal ~2.3 px reproj error -->
+      <origin xyz="-6.1788056476961728e-02 -2.4867707148071745e-03 1.2036970069250407e-02" rpy="-5.2776889304282960e-03 -1.4500635837943188e+00 2.5519090344067272e-02"/>
     </xacro:sensor_d435>
     <!-- left camera -->
     <xacro:sensor_d435 parent="${tf_prefix}left_ur_realsense_mount" use_nominal_extrinsics="true" use_mesh="true" name="${tf_prefix}left_wrist_mounted_camera">
+      <!-- original -->
       <!-- <origin xyz="-0.064 -0.003 0.016" rpy="0.136 -1.429 -0.128"/> -->
-      <origin xyz="-6.3398954689359577e-02 1.0843610275642415e-03 1.0771886573701910e-02" rpy="-3.3291953701393887e-02 -1.4542171203396566e+00 3.8217188478749678e-02"/>
+      <!-- first cal ~4 px reproj error -->
+      <!-- <origin xyz="-6.3398954689359577e-02 1.0843610275642415e-03 1.0771886573701910e-02" rpy="-3.3291953701393887e-02 -1.4542171203396566e+00 3.8217188478749678e-02"/> -->
+      <!-- second cal ~2.4 px reproj error -->
+      <origin xyz="-6.4777232475001029e-02 1.1461581058038600e-04 1.2884814853441564e-02" rpy="-9.9487205554735336e-02 -1.4520756449714673e+00 1.0569277772629829e-01"/>
     </xacro:sensor_d435>
     <!-- Hand-E Grippers -->
@@ -579,5 +586,5 @@
       parent="${tf_prefix}right_ur_realsense_mount"
       finger_xacro="fngr_original">
-      <origin xyz="0 0 0.008" rpy="0 0 ${pi/2}"/>
+      <origin xyz="0 0 0.003" rpy="0 0 ${pi/2}"/>
     </xacro:dextivr_hande>
     <xacro:dextivr_hande
@@ -588,5 +595,5 @@
       parent="${tf_prefix}left_ur_realsense_mount"
       finger_xacro="fngr_original">
-      <origin xyz="0 0 0.008" rpy="0 0 ${pi/2}"/>
+      <origin xyz="0 0 0.003" rpy="0 0 ${pi/2}"/>
     </xacro:dextivr_hande>
   </xacro:unless>

Commit message: updates with improved processing for full phoebe conversion

File: phoebe_description/urdf/phoebe_macro.xacro (robot description, xacro)
@@ -587,4 +587,5 @@
       tf_prefix="${tf_prefix}right_"
       parent="${tf_prefix}right_ur_realsense_mount"
+      generate_ros2_control_tag="${generate_ros2_control_tag}"
       finger_xacro="fngr_original">
       <origin xyz="0 0 0.003" rpy="0 0 ${pi/2}"/>
@@ -596,4 +597,5 @@
       tf_prefix="${tf_prefix}left_"
       parent="${tf_prefix}left_ur_realsense_mount"
+      generate_ros2_control_tag="${generate_ros2_control_tag}"
       finger_xacro="fngr_original">
       <origin xyz="0 0 0.003" rpy="0 0 ${pi/2}"/>
@@ -640,33 +642,4 @@
     <link name="${tf_prefix}calibration_face_target_side"/>
   </xacro:if>
-<<<<<<< HEAD
-  <!-- Hand-E Grippers -->
-  <xacro:unless value="${calibration_mode}">
-    <xacro:include filename="$(find dextivr_hande_description)/urdf/dextivr_hande.xacro"/>
-    <xacro:dextivr_hande
-      com_port="${right_hande_com_port}"
-      use_fake_hardware="${use_fake_hardware}"
-      name="${tf_prefix}right_dextivr_hande"
-      tf_prefix="${tf_prefix}right_"
-      parent="${tf_prefix}right_ur_realsense_mount"
-      finger_xacro="fngr_original"
-      generate_ros2_control_tag="${generate_ros2_control_tag}"
-    >
-      <origin xyz="0 0 0.008" rpy="0 0 ${pi}"/>
-    </xacro:dextivr_hande>
-    <xacro:dextivr_hande
-      com_port="${left_hande_com_port}"
-      use_fake_hardware="${use_fake_hardware}"
-      name="${tf_prefix}left_dextivr_hande"
-      tf_prefix="${tf_prefix}left_"
-      parent="${tf_prefix}left_ur_realsense_mount"
-      finger_xacro="fngr_original"
-      generate_ros2_control_tag="${generate_ros2_control_tag}"
-    >
-      <origin xyz="0 0 0.008" rpy="0 0 ${pi}"/>
-    </xacro:dextivr_hande>
-  </xacro:unless>
-=======
->>>>>>> humble-feature/nav2-go
   </xacro:macro>
 </robot>

Commit message: World frame WIP

File: phoebe_description/urdf/phoebe_macro.xacro (robot description, xacro)
@@ -9,4 +9,5 @@
       use_fake_hardware:='false'
       sim_ignition:='false'
+      include_world_frame:='false'
       calibration_mode:='false'
       left_ewellix_com_port:='/dev/ewellix_left'
@@ -28,4 +29,14 @@
   <xacro:include filename="$(find clearpath_platform_description)/urdf/common.urdf.xacro" />
   <xacro:include filename="$(find phoebe_description)/urdf/r100/r100_macro.xacro" />
+  <!-- Moveit Pro explicity requires a world frame in the description, so we conditionally ad it here. -->
+  <xacro:if value="${include_world_frame}">
+    <link name="world"/>
+    <!-- Add a floating joint so that it can freely move in the world -->
+    <joint name="world_to_base_link" type="floating">
+      <parent link="world"/>
+      <child link="${tf_prefix}base_link"/>
+      <origin xyz="0 0 0" rpy="0 0 0"/>
+    </joint>
+  </xacro:if>
   <xacro:r100
       tf_prefix="${tf_prefix}"

Commit message: Update the world joints

File: phoebe_description/urdf/phoebe_macro.xacro (robot description, xacro)
@@ -9,5 +9,5 @@
       use_fake_hardware:='false'
       sim_ignition:='false'
-      include_world_frame:='false'
+      include_world_joints:='false'
       calibration_mode:='false'
       left_ewellix_com_port:='/dev/ewellix_left'
@@ -29,12 +29,34 @@
   <xacro:include filename="$(find clearpath_platform_description)/urdf/common.urdf.xacro" />
   <xacro:include filename="$(find phoebe_description)/urdf/r100/r100_macro.xacro" />
-  <!-- Moveit Pro explicity requires a world frame in the description, so we conditionally ad it here. -->
-  <xacro:if value="${include_world_frame}">
+  <!-- Conditionally attach the world to the base_link with a x, y, and yaw joints. -->
+  <!-- This is necessary for moveit pro integration and for whole body motion planning and execution. -->
+  <!-- However, as this is non-standare for other applications we do not necessarily want it by default. -->
+  <xacro:if value="${include_world_joints}">
     <link name="world"/>
-    <!-- Add a floating joint so that it can freely move in the world -->
-    <joint name="world_to_base_link" type="floating">
-      <parent link="world"/>
+    <link name="virtual_rail_link_1"/>
+    <joint name="linear_x_joint" type="prismatic">
+      <axis xyz="1 0 0"/>
+      <parent link="world" />
+      <child link="virtual_rail_link_1" />
+      <origin xyz="0 0 0" rpy="0 0 0" />
+      <limit effort="1000.0" lower="-20.0" upper="20.0" velocity="0.175" acceleration="10.0"/>
+      <dynamics damping="20.0" friction="500.0" />
+    </joint>
+    <link name="virtual_rail_link_2"/>
+    <joint name="linear_y_joint" type="prismatic">
+      <axis xyz="0 1 0"/>
+      <parent link="virtual_rail_link_1" />
+      <child link="virtual_rail_link_2" />
+      <origin xyz="0 0 0" rpy="0 0 0" />
+      <limit effort="1000.0" lower="-5.0" upper="55.0" velocity="0.175" acceleration="10.0"/>
+      <dynamics damping="20.0" friction="500.0" />
+    </joint>
+    <joint name="rotational_yaw_joint" type="continuous">
+      <axis xyz="0 0 1"/>
+      <parent link="virtual_rail_link_2"/>
       <child link="${tf_prefix}base_link"/>
-      <origin xyz="0 0 0" rpy="0 0 0"/>
+      <origin rpy="0 0 0" xyz="0 0 0"/>
+      <limit effort="150.0" velocity="0.5235987755982988"/>
+      <dynamics damping="0" friction="0"/>
     </joint>
   </xacro:if>

Commit message: TEMP: Static map and odom

File: phoebe_description/urdf/phoebe_macro.xacro (robot description, xacro)
@@ -34,4 +34,18 @@
   <xacro:if value="${include_world_joints}">
     <link name="world"/>
+    <!-- For nav2 compatibility we affix map and odom to the world frame. -->
+    <!-- All odometry/world transforms are converted to joint states for the virtual joints manually. -->
+    <link name="map"/>
+    <joint name="world_to_map" type="fixed">
+      <parent link="world"/>
+      <child link="map"/>
+      <origin xyz="0 0 0" rpy="0 0 0"/>
+    </joint>
+    <link name="odom"/>
+    <joint name="map_to_odom" type="fixed">
+      <parent link="map"/>
+      <child link="odom"/>
+      <origin xyz="0 0 0" rpy="0 0 0"/>
+    </joint>
     <link name="virtual_rail_link_1"/>
     <joint name="linear_x_joint" type="prismatic">

Commit message: Connect odom to base

File: phoebe_description/urdf/phoebe_macro.xacro (robot description, xacro)
@@ -33,13 +33,8 @@
   <!-- However, as this is non-standard for other applications we do not want it by default. -->
   <xacro:if value="${include_world_joints}">
-    <link name="world"/>
     <!-- For nav2 compatibility we affix map and odom to the world frame. -->
+    <!-- The map pose in the world frame must be set manually from the world publisher. -->
     <!-- All odometry/world transforms are converted to joint states for the virtual joints manually. -->
     <link name="map"/>
-    <joint name="world_to_map" type="fixed">
-      <parent link="world"/>
-      <child link="map"/>
-      <origin xyz="0 0 0" rpy="0 0 0"/>
-    </joint>
     <link name="odom"/>
     <joint name="map_to_odom" type="fixed">
@@ -49,7 +44,8 @@
     </joint>
     <link name="virtual_rail_link_1"/>
+    <!-- Connecting to odometry will enable the map -> world xform to be updated without distruption. -->
     <joint name="linear_x_joint" type="prismatic">
       <axis xyz="1 0 0"/>
-      <parent link="world" />
+      <parent link="odom" />
       <child link="virtual_rail_link_1" />
       <origin xyz="0 0 0" rpy="0 0 0" />

Commit message: adding second 2f85

File: phoebe_description/urdf/phoebe_macro.xacro (robot description, xacro)
@@ -629,5 +629,5 @@
     </xacro:robotiq_2f_85>
     <!-- Left gripper - Hand-E -->
-    <xacro:include filename="$(find dextivr_hande_description)/urdf/dextivr_hande.xacro"/>
+    <!-- <xacro:include filename="$(find dextivr_hande_description)/urdf/dextivr_hande.xacro"/>
     <xacro:dextivr_hande
       com_port="${left_hande_com_port}"
@@ -640,5 +640,16 @@
       finger_xacro="fngr_original">
       <origin xyz="0 0 0.003" rpy="0 0 ${pi/2}"/>
-    </xacro:dextivr_hande>
+    </xacro:dextivr_hande> -->
+    <!-- Left gripper - 2F-85 -->
+    <xacro:robotiq_2f_85
+      com_port="${left_hande_com_port}"
+      use_fake_hardware="${use_fake_hardware}"
+      name="${tf_prefix}left_dextivr_hande"
+      tf_prefix="${tf_prefix}left_"
+      parent="${tf_prefix}left_ur_realsense_mount"
+      generate_ros2_control_tag="${generate_ros2_control_tag}"
+      add_grasp_push_frames="${add_grasp_push_frames}">
+      <origin xyz="0 0 0.003" rpy="0 0 ${pi/2}"/>
+    </xacro:robotiq_2f_85>
   </xacro:unless>
   <!-- Calibration HW -->

File: phoebe_description/urdf/robotiq_2f_85_macro.xacro (robot description, xacro)
@@ -53,5 +53,5 @@
     <xacro:include filename="$(find robotiq_description)/urdf/robotiq_2f_85_macro.urdf.xacro"/>
     <xacro:robotiq_gripper
-      com_port="${right_hande_com_port}"
+      com_port="${com_port}"
       use_fake_hardware="${use_fake_hardware}"
       name="${name}"
