Commit message: Added launch and xacro argument for replacing the left Ewellix liftkit with the static pedestal. Modified urdf and xacro files accordingly.

File: phoebe_description/urdf/phoebe_macro.xacro (robot description, xacro)
@@ -25,4 +25,5 @@
       add_grasp_push_frames:='true'
       use_camera_mesh:='true'
+      use_left_static_pedestal:='false'
     "
   >
@@ -392,30 +393,52 @@
   </joint>
   <!-- Left Ewellix mounting flange -->
-  <link name="${tf_prefix}left_ewellix_mount_flange_link">
-    <visual>
-      <geometry>
-        <box size="0.2 0.2 0.015"/>
-      </geometry>
-      <material name="clearpath_aluminum"/>
-      <origin rpy="0 0 0" xyz="0 0 0.0075"/>
-    </visual>
-    <collision>
-      <geometry>
-        <box size="0.2 0.2 0.015"/>
-      </geometry>
-      <origin rpy="0 0 0" xyz="0 0 0.0075"/>
-    </collision>
-  </link>
   <!-- load the liftkit mount calibration -->
-  <xacro:property name="liftkit_mount_calibration" value="${xacro.load_yaml(liftkit_mount_calibration_file)}"/>
-  <xacro:property name="left_edge_aligned_distance" value="${liftkit_mount_calibration['left_edge_aligned_distance']}"/>
-  <xacro:property name="right_edge_aligned_distance" value="${liftkit_mount_calibration['right_edge_aligned_distance']}"/>
-  <xacro:property name="left_liftkit_dist_from_edge" value="${liftkit_mount_calibration['left_liftkit_dist_from_edge']}"/>
-  <xacro:property name="right_liftkit_dist_from_edge" value="${liftkit_mount_calibration['right_liftkit_dist_from_edge']}"/>
-  <joint name="${tf_prefix}left_ewellix_mount_flange_joint" type="fixed">
-    <parent link="${tf_prefix}default_mount"/>
-    <child link="${tf_prefix}left_ewellix_mount_flange_link"/>
-    <origin xyz="0 ${left_edge_aligned_distance-left_liftkit_dist_from_edge} 0.04" rpy="0 0 0" />
-  </joint>
+    <xacro:property name="liftkit_mount_calibration" value="${xacro.load_yaml(liftkit_mount_calibration_file)}"/>
+    <xacro:property name="left_edge_aligned_distance" value="${liftkit_mount_calibration['left_edge_aligned_distance']}"/>
+    <xacro:property name="right_edge_aligned_distance" value="${liftkit_mount_calibration['right_edge_aligned_distance']}"/>
+    <xacro:property name="left_liftkit_dist_from_edge" value="${liftkit_mount_calibration['left_liftkit_dist_from_edge']}"/>
+    <xacro:property name="right_liftkit_dist_from_edge" value="${liftkit_mount_calibration['right_liftkit_dist_from_edge']}"/>
+  <xacro:unless value="${use_left_static_pedestal}">
+    <link name="${tf_prefix}left_ewellix_mount_flange_link">
+      <visual>
+        <geometry>
+          <box size="0.2 0.2 0.015"/>
+        </geometry>
+        <material name="clearpath_aluminum"/>
+        <origin rpy="0 0 0" xyz="0 0 0.0075"/>
+      </visual>
+      <collision>
+        <geometry>
+          <box size="0.2 0.2 0.015"/>
+        </geometry>
+        <origin rpy="0 0 0" xyz="0 0 0.0075"/>
+      </collision>
+    </link>
+    <joint name="${tf_prefix}left_ewellix_mount_flange_joint" type="fixed">
+      <parent link="${tf_prefix}default_mount"/>
+      <child link="${tf_prefix}left_ewellix_mount_flange_link"/>
+      <origin xyz="0 ${left_edge_aligned_distance-left_liftkit_dist_from_edge} 0.04" rpy="0 0 0" />
+    </joint>
+  </xacro:unless>
+  <xacro:if value="${use_left_static_pedestal}">
+    <link name="${tf_prefix}left_static_pedestal_link">
+      <visual>
+        <geometry>
+          <mesh filename="package://phoebe_description/meshes/visual/static_pedestal.stl" scale="0.0254 0.0254 0.0254"/>
+        </geometry>
+        <material name="clearpath_aluminum"/>
+      </visual>
+      <collision>
+        <geometry>
+          <mesh filename="package://phoebe_description/meshes/visual/static_pedestal.stl" scale="0.0254 0.0254 0.0254"/>
+        </geometry>
+      </collision>
+    </link>
+    <joint name="${tf_prefix}left_ewellix_pedestal_link_joint" type="fixed">
+      <parent link="${tf_prefix}default_mount"/>
+      <child link="${tf_prefix}left_static_pedestal_link"/>
+      <origin xyz="0 ${left_edge_aligned_distance-left_liftkit_dist_from_edge} 0.04" rpy="0 0 0" />
+    </joint>
+  </xacro:if>
   <!-- Right Ewellix mounting flange -->
   <link name="${tf_prefix}right_ewellix_mount_flange_link">
@@ -446,53 +469,83 @@
   <!-- <xacro:property name="left_liftkit_calibration_file" value="${left_liftkit_calibration_file}"/>
   <xacro:property name="right_liftkit_calibration_file" value="${right_liftkit_calibration_file}"/> -->
+  <xacro:unless value="${use_left_static_pedestal}">
+    <xacro:ewellix_lift
+      name="${tf_prefix}left_ewellix"
+      is_700="false"
+      is_500="true"
+      tf_prefix="${tf_prefix}left_"
+      parent="${tf_prefix}left_ewellix_mount_flange_link"
+      height_limit="0.5"
+      initial_value="0.26644069061695785"
+      omit_plates="true"
+      use_fake_hardware="${use_fake_hardware}"
+      com_port="${left_ewellix_com_port}"
+      generate_ros2_control_tag="${generate_ros2_control_tag}"
+    >
+      <origin xyz="0 0 ${0.0075+0.2457}" rpy="0 0 0"/>
+    </xacro:ewellix_lift>
+    <!-- Left arm mount plate -->
+    <link name="${tf_prefix}left_arm_mount_plate">
+      <visual>
+        <geometry>
+          <mesh filename="package://phoebe_description/meshes/visual/jaco01_meshes/arm_mount.STL"/>
+        </geometry>
+        <material name="clearpath_black" />
+      </visual>
+      <collision>
+        <geometry>
+          <mesh filename="package://phoebe_description/meshes/visual/jaco01_meshes/arm_mount_collision.STL"/>
+        </geometry>
+      </collision>
+    </link>
+    <joint name="${tf_prefix}left_arm_mount_plate_joint" type="fixed">
+      <parent link="${tf_prefix}left_ewellix_lift_tip_link" />
+      <child link="${tf_prefix}left_arm_mount_plate" />
+      <origin xyz="0 0 0" rpy="0 0 0" />
+    </joint>
+  </xacro:unless>
+  <xacro:if value="${use_left_static_pedestal}">
+     <link name="${tf_prefix}left_ewellix_lift_tip_link">
+     </link>
+     <joint name="${tf_prefix}ewellix_lift_tip_joint" type="fixed">
+      <parent link="${tf_prefix}left_static_pedestal_link"/>
+      <child link="${tf_prefix}left_ewellix_lift_tip_link"/>
+      <origin xyz="0 0 0.6096" rpy="0 0 0"/>
+    </joint>
+    <!-- Left arm mount plate -->
+    <link name="${tf_prefix}left_arm_mount_plate">
+      <visual>
+        <geometry>
+          <mesh filename="package://phoebe_description/meshes/visual/jaco01_meshes/arm_mount.STL"/>
+        </geometry>
+        <material name="clearpath_black" />
+      </visual>
+      <collision>
+        <geometry>
+          <mesh filename="package://phoebe_description/meshes/visual/jaco01_meshes/arm_mount_collision.STL"/>
+        </geometry>
+      </collision>
+    </link>
+    <joint name="${tf_prefix}left_arm_mount_plate_joint" type="fixed">
+      <parent link="${tf_prefix}left_ewellix_lift_tip_link" />
+      <child link="${tf_prefix}left_arm_mount_plate" />
+      <origin xyz="0 0 0" rpy="0 0 0" />
+    </joint>
+  </xacro:if>
   <xacro:ewellix_lift
-    name="${tf_prefix}left_ewellix"
-    is_700="false"
-    is_500="true"
-    tf_prefix="${tf_prefix}left_"
-    parent="${tf_prefix}left_ewellix_mount_flange_link"
-    height_limit="0.5"
-    initial_value="0.26644069061695785"
-    omit_plates="true"
-    use_fake_hardware="${use_fake_hardware}"
-    com_port="${left_ewellix_com_port}"
-    generate_ros2_control_tag="${generate_ros2_control_tag}"
-  >
-    <origin xyz="0 0 ${0.0075+0.2457}" rpy="0 0 0"/>
+      name="${tf_prefix}right_ewellix"
+      is_700="false"
+      is_500="true"
+      tf_prefix="${tf_prefix}right_"
+      parent="${tf_prefix}right_ewellix_mount_flange_link"
+      height_limit="0.5"
+      initial_value="0.259764889515653"
+      omit_plates="true"
+      use_fake_hardware="${use_fake_hardware}"
+      com_port="${right_ewellix_com_port}"
+      generate_ros2_control_tag="${generate_ros2_control_tag}"
+    >
+      <origin xyz="0 0 ${0.0075+0.2457}" rpy="0 0 0"/>
   </xacro:ewellix_lift>
-  <xacro:ewellix_lift
-    name="${tf_prefix}right_ewellix"
-    is_700="false"
-    is_500="true"
-    tf_prefix="${tf_prefix}right_"
-    parent="${tf_prefix}right_ewellix_mount_flange_link"
-    height_limit="0.5"
-    initial_value="0.259764889515653"
-    omit_plates="true"
-    use_fake_hardware="${use_fake_hardware}"
-    com_port="${right_ewellix_com_port}"
-    generate_ros2_control_tag="${generate_ros2_control_tag}"
-  >
-    <origin xyz="0 0 ${0.0075+0.2457}" rpy="0 0 0"/>
-  </xacro:ewellix_lift>
-  <!-- Left arm mount plate -->
-  <link name="${tf_prefix}left_arm_mount_plate">
-    <visual>
-      <geometry>
-        <mesh filename="package://phoebe_description/meshes/visual/jaco01_meshes/arm_mount.STL"/>
-      </geometry>
-      <material name="clearpath_black" />
-    </visual>
-    <collision>
-      <geometry>
-        <mesh filename="package://phoebe_description/meshes/visual/jaco01_meshes/arm_mount_collision.STL"/>
-      </geometry>
-    </collision>
-  </link>
-  <joint name="${tf_prefix}left_arm_mount_plate_joint" type="fixed">
-    <parent link="${tf_prefix}left_ewellix_lift_tip_link" />
-    <child link="${tf_prefix}left_arm_mount_plate" />
-    <origin xyz="0 0 0" rpy="0 0 0" />
-  </joint>
   <!-- Right arm mount plate -->
   <link name="${tf_prefix}right_arm_mount_plate">

Commit message: Modified URDF to reflect updated static pedestal mounting config on hardware.

File: phoebe_description/urdf/phoebe_macro.xacro (robot description, xacro)
@@ -425,5 +425,5 @@
       <visual>
         <geometry>
-          <mesh filename="package://phoebe_description/meshes/visual/static_pedestal.stl" scale="0.0254 0.0254 0.0254"/>
+          <mesh filename="package://phoebe_description/meshes/visual/static_pedestal_with_mount.stl" scale="0.0254 0.0254 0.0254"/>
         </geometry>
         <material name="clearpath_aluminum"/>
@@ -431,5 +431,5 @@
       <collision>
         <geometry>
-          <mesh filename="package://phoebe_description/meshes/visual/static_pedestal.stl" scale="0.0254 0.0254 0.0254"/>
+          <mesh filename="package://phoebe_description/meshes/visual/static_pedestal_with_mount.stl" scale="0.0254 0.0254 0.0254"/>
         </geometry>
       </collision>
@@ -438,5 +438,5 @@
       <parent link="${tf_prefix}default_mount"/>
       <child link="${tf_prefix}left_static_pedestal_link"/>
-      <origin xyz="0 ${left_edge_aligned_distance-left_liftkit_dist_from_edge} 0.04" rpy="0 0 0" />
+      <origin xyz="0 ${left_edge_aligned_distance-left_liftkit_dist_from_edge} 0.04" rpy="0 0 1.5707963" />
     </joint>
   </xacro:if>
@@ -514,5 +514,5 @@
     </joint>
     <!-- Left arm mount plate -->
-    <link name="${tf_prefix}left_arm_mount_plate">
+    <!-- <link name="${tf_prefix}left_arm_mount_plate">
       <visual>
         <geometry>
@@ -531,5 +531,5 @@
       <child link="${tf_prefix}left_arm_mount_plate" />
       <origin xyz="0 0 0" rpy="0 0 0" />
-    </joint>
+    </joint> -->
   </xacro:if>
   <xacro:ewellix_lift
@@ -568,10 +568,20 @@
   </joint>
   <!-- calibration links -->
-  <link name="${tf_prefix}left_arm_cal_link"> </link>
-  <joint name="${tf_prefix}left_arm_cal_joint" type="fixed">
-    <parent link="${tf_prefix}left_arm_mount_plate" />
-    <child link="${tf_prefix}left_arm_cal_link" />
-    <origin xyz="0.00807 -0.00363 0.01019" rpy="0.01529 0.01951 -0.00426"/>
-  </joint>
+  <xacro:unless value="${use_left_static_pedestal}">
+    <link name="${tf_prefix}left_arm_cal_link"> </link>
+    <joint name="${tf_prefix}left_arm_cal_joint" type="fixed">
+      <parent link="${tf_prefix}left_arm_mount_plate" />
+      <child link="${tf_prefix}left_arm_cal_link" />
+      <origin xyz="0.00807 -0.00363 0.01019" rpy="0.01529 0.01951 -0.00426"/>
+    </joint>
+  </xacro:unless>
+  <xacro:if value="${use_left_static_pedestal}">
+    <link name="${tf_prefix}left_arm_cal_link"> </link>
+    <joint name="${tf_prefix}left_arm_cal_joint" type="fixed">
+      <parent link="${tf_prefix}left_static_pedestal_link" />
+      <child link="${tf_prefix}left_arm_cal_link" />
+      <origin xyz="0 0 0" rpy="0 0 0"/>
+    </joint>
+  </xacro:if>
   <link name="${tf_prefix}right_arm_cal_link"> </link>
   <joint name="${tf_prefix}right_arm_cal_joint" type="fixed">

Commit message: Modified URDF to reflect updated static pedestal mounting config on hardware.

File: phoebe_description/urdf/phoebe_macro.xacro (robot description, xacro)
@@ -425,5 +425,5 @@
       <visual>
         <geometry>
-          <mesh filename="package://phoebe_description/meshes/visual/static_pedestal.stl" scale="0.0254 0.0254 0.0254"/>
+          <mesh filename="package://phoebe_description/meshes/visual/static_pedestal_with_mount.stl" scale="0.0254 0.0254 0.0254"/>
         </geometry>
         <material name="clearpath_aluminum"/>
@@ -431,5 +431,5 @@
       <collision>
         <geometry>
-          <mesh filename="package://phoebe_description/meshes/visual/static_pedestal.stl" scale="0.0254 0.0254 0.0254"/>
+          <mesh filename="package://phoebe_description/meshes/visual/static_pedestal_with_mount.stl" scale="0.0254 0.0254 0.0254"/>
         </geometry>
       </collision>
@@ -438,5 +438,5 @@
       <parent link="${tf_prefix}default_mount"/>
       <child link="${tf_prefix}left_static_pedestal_link"/>
-      <origin xyz="0 ${left_edge_aligned_distance-left_liftkit_dist_from_edge} 0.04" rpy="0 0 0" />
+      <origin xyz="0 ${left_edge_aligned_distance-left_liftkit_dist_from_edge} 0.04" rpy="0 0 1.5707963" />
     </joint>
   </xacro:if>
@@ -514,5 +514,5 @@
     </joint>
     <!-- Left arm mount plate -->
-    <link name="${tf_prefix}left_arm_mount_plate">
+    <!-- <link name="${tf_prefix}left_arm_mount_plate">
       <visual>
         <geometry>
@@ -531,5 +531,5 @@
       <child link="${tf_prefix}left_arm_mount_plate" />
       <origin xyz="0 0 0" rpy="0 0 0" />
-    </joint>
+    </joint> -->
   </xacro:if>
   <xacro:ewellix_lift
@@ -568,10 +568,20 @@
   </joint>
   <!-- calibration links -->
-  <link name="${tf_prefix}left_arm_cal_link"> </link>
-  <joint name="${tf_prefix}left_arm_cal_joint" type="fixed">
-    <parent link="${tf_prefix}left_arm_mount_plate" />
-    <child link="${tf_prefix}left_arm_cal_link" />
-    <origin xyz="0.00807 -0.00363 0.01019" rpy="0.01529 0.01951 -0.00426"/>
-  </joint>
+  <xacro:unless value="${use_left_static_pedestal}">
+    <link name="${tf_prefix}left_arm_cal_link"> </link>
+    <joint name="${tf_prefix}left_arm_cal_joint" type="fixed">
+      <parent link="${tf_prefix}left_arm_mount_plate" />
+      <child link="${tf_prefix}left_arm_cal_link" />
+      <origin xyz="0.00807 -0.00363 0.01019" rpy="0.01529 0.01951 -0.00426"/>
+    </joint>
+  </xacro:unless>
+  <xacro:if value="${use_left_static_pedestal}">
+    <link name="${tf_prefix}left_arm_cal_link"> </link>
+    <joint name="${tf_prefix}left_arm_cal_joint" type="fixed">
+      <parent link="${tf_prefix}left_static_pedestal_link" />
+      <child link="${tf_prefix}left_arm_cal_link" />
+      <origin xyz="0 0 0" rpy="0 0 0"/>
+    </joint>
+  </xacro:if>
   <link name="${tf_prefix}right_arm_cal_link"> </link>
   <joint name="${tf_prefix}right_arm_cal_joint" type="fixed">
@@ -599,4 +609,5 @@
   <!-- TODO: need to integrate the motion on the rails. this used to be done like below -->
   <!-- <origin xyz="$(optenv RIDGEBACK_RIGHT_UR_XYZ 0 0 0)" rpy="$(optenv RIDGEBACK_RIGHT_UR_RPY 0 0 0)" /> -->
+  <!-- RIGHT ARM -->
   <xacro:ur_robot
     name="${tf_prefix}right_ur5e"
@@ -623,28 +634,57 @@
     <origin xyz="0 0 0" rpy="0 0 ${5*pi/4}" />
   </xacro:ur_robot>
-  <xacro:ur_robot
-    name="${tf_prefix}left_ur5e"
-    tf_prefix="${tf_prefix}left_ur_arm_"
-    parent="${tf_prefix}left_arm_mount_plate_2"
-    kinematics_parameters_file="${left_ur_kinematics_file}"
-    joint_limits_parameters_file="$(find ur_description)/config/ur5e/joint_limits.yaml"
-    physical_parameters_file="$(find ur_description)/config/ur5e/physical_parameters.yaml"
-    visual_parameters_file="$(find ur_description)/config/ur5e/visual_parameters.yaml"
-    initial_positions="${xacro.load_yaml(initial_positions_file_left)}"
-    use_fake_hardware="${use_fake_hardware}"
-    sim_ignition="${sim_ignition}"
-    robot_ip="${left_ur_ip_addr}"
-    reverse_port="50001"
-    script_sender_port="50002"
-    script_command_port="50004"
-    trajectory_port="50003"
-    use_tool_communication="false"
-    script_filename="$(find ur_client_library)/resources/external_control.urscript"
-    input_recipe_filename="$(find ur_robot_driver)/resources/rtde_input_recipe.txt"
-    output_recipe_filename="$(find ur_robot_driver)/resources/rtde_output_recipe.txt"
-    generate_ros2_control_tag="${generate_ros2_control_tag}"
-    >
-    <origin xyz="0 0 0" rpy="0 0 ${-pi/4}" /> <!-- TODO: need to integrate the OPTENV RIGEBACK_RIGHT_UR_XYZ stuff-->
-  </xacro:ur_robot>
+  <!-- LEFT ARM  -->
+  <xacro:unless value="${use_left_static_pedestal}">
+    <xacro:ur_robot
+      name="${tf_prefix}left_ur5e"
+      tf_prefix="${tf_prefix}left_ur_arm_"
+      parent="${tf_prefix}left_arm_mount_plate_2"
+      kinematics_parameters_file="${left_ur_kinematics_file}"
+      joint_limits_parameters_file="$(find ur_description)/config/ur5e/joint_limits.yaml"
+      physical_parameters_file="$(find ur_description)/config/ur5e/physical_parameters.yaml"
+      visual_parameters_file="$(find ur_description)/config/ur5e/visual_parameters.yaml"
+      initial_positions="${xacro.load_yaml(initial_positions_file_left)}"
+      use_fake_hardware="${use_fake_hardware}"
+      sim_ignition="${sim_ignition}"
+      robot_ip="${left_ur_ip_addr}"
+      reverse_port="50001"
+      script_sender_port="50002"
+      script_command_port="50004"
+      trajectory_port="50003"
+      use_tool_communication="false"
+      script_filename="$(find ur_client_library)/resources/external_control.urscript"
+      input_recipe_filename="$(find ur_robot_driver)/resources/rtde_input_recipe.txt"
+      output_recipe_filename="$(find ur_robot_driver)/resources/rtde_output_recipe.txt"
+      generate_ros2_control_tag="${generate_ros2_control_tag}"
+      >
+      <origin xyz="0 0 0" rpy="0 0 ${-pi/4}" />
+    </xacro:ur_robot>
+  </xacro:unless>
+  <xacro:if value="${use_left_static_pedestal}">
+    <xacro:ur_robot
+      name="${tf_prefix}left_ur5e"
+      tf_prefix="${tf_prefix}left_ur_arm_"
+      parent="${tf_prefix}left_arm_cal_link"
+      kinematics_parameters_file="${left_ur_kinematics_file}"
+      joint_limits_parameters_file="$(find ur_description)/config/ur5e/joint_limits.yaml"
+      physical_parameters_file="$(find ur_description)/config/ur5e/physical_parameters.yaml"
+      visual_parameters_file="$(find ur_description)/config/ur5e/visual_parameters.yaml"
+      initial_positions="${xacro.load_yaml(initial_positions_file_left)}"
+      use_fake_hardware="${use_fake_hardware}"
+      sim_ignition="${sim_ignition}"
+      robot_ip="${left_ur_ip_addr}"
+      reverse_port="50001"
+      script_sender_port="50002"
+      script_command_port="50004"
+      trajectory_port="50003"
+      use_tool_communication="false"
+      script_filename="$(find ur_client_library)/resources/external_control.urscript"
+      input_recipe_filename="$(find ur_robot_driver)/resources/rtde_input_recipe.txt"
+      output_recipe_filename="$(find ur_robot_driver)/resources/rtde_output_recipe.txt"
+      generate_ros2_control_tag="${generate_ros2_control_tag}"
+      >
+      <origin xyz="0 0 0.649605" rpy="0 0 0" /> <!-- TODO: need to integrate the OPTENV RIGEBACK_RIGHT_UR_XYZ stuff-->
+    </xacro:ur_robot>
+  </xacro:if>
   <!-- end effector interface stack -->
   <xacro:unless value="${calibration_mode}">
