Commit message: Deleted mesh of static pedestal without mounting and cleaned up urdf.

File: phoebe_description/urdf/phoebe_macro.xacro (robot description, xacro)
@@ -392,11 +392,10 @@
     <origin xyz="0.0845 -0.384 0.22" rpy="0 0 0" />
   </joint>
-  <!-- Left Ewellix mounting flange -->
   <!-- load the liftkit mount calibration -->
-    <xacro:property name="liftkit_mount_calibration" value="${xacro.load_yaml(liftkit_mount_calibration_file)}"/>
-    <xacro:property name="left_edge_aligned_distance" value="${liftkit_mount_calibration['left_edge_aligned_distance']}"/>
-    <xacro:property name="right_edge_aligned_distance" value="${liftkit_mount_calibration['right_edge_aligned_distance']}"/>
-    <xacro:property name="left_liftkit_dist_from_edge" value="${liftkit_mount_calibration['left_liftkit_dist_from_edge']}"/>
-    <xacro:property name="right_liftkit_dist_from_edge" value="${liftkit_mount_calibration['right_liftkit_dist_from_edge']}"/>
+  <xacro:property name="liftkit_mount_calibration" value="${xacro.load_yaml(liftkit_mount_calibration_file)}"/>
+  <xacro:property name="left_edge_aligned_distance" value="${liftkit_mount_calibration['left_edge_aligned_distance']}"/>
+  <xacro:property name="right_edge_aligned_distance" value="${liftkit_mount_calibration['right_edge_aligned_distance']}"/>
+  <xacro:property name="left_liftkit_dist_from_edge" value="${liftkit_mount_calibration['left_liftkit_dist_from_edge']}"/>
+  <xacro:property name="right_liftkit_dist_from_edge" value="${liftkit_mount_calibration['right_liftkit_dist_from_edge']}"/>
   <xacro:unless value="${use_left_static_pedestal}">
     <link name="${tf_prefix}left_ewellix_mount_flange_link">
@@ -636,55 +635,37 @@
   <!-- LEFT ARM  -->
   <xacro:unless value="${use_left_static_pedestal}">
-    <xacro:ur_robot
-      name="${tf_prefix}left_ur5e"
-      tf_prefix="${tf_prefix}left_ur_arm_"
-      parent="${tf_prefix}left_arm_mount_plate_2"
-      kinematics_parameters_file="${left_ur_kinematics_file}"
-      joint_limits_parameters_file="$(find ur_description)/config/ur5e/joint_limits.yaml"
-      physical_parameters_file="$(find ur_description)/config/ur5e/physical_parameters.yaml"
-      visual_parameters_file="$(find ur_description)/config/ur5e/visual_parameters.yaml"
-      initial_positions="${xacro.load_yaml(initial_positions_file_left)}"
-      use_fake_hardware="${use_fake_hardware}"
-      sim_ignition="${sim_ignition}"
-      robot_ip="${left_ur_ip_addr}"
-      reverse_port="50001"
-      script_sender_port="50002"
-      script_command_port="50004"
-      trajectory_port="50003"
-      use_tool_communication="false"
-      script_filename="$(find ur_client_library)/resources/external_control.urscript"
-      input_recipe_filename="$(find ur_robot_driver)/resources/rtde_input_recipe.txt"
-      output_recipe_filename="$(find ur_robot_driver)/resources/rtde_output_recipe.txt"
-      generate_ros2_control_tag="${generate_ros2_control_tag}"
-      >
-      <origin xyz="0 0 0" rpy="0 0 ${-pi/4}" />
-    </xacro:ur_robot>
+    <xacro:property name="parent" value="${tf_prefix}left_arm_mount_plate_2"/>
+    <xacro:property name="origin_xyz" value="0 0 0"/>
+    <xacro:property name="origin_rpy" value="0 0 ${-pi/4}"/>
   </xacro:unless>
-  <xacro:if value="${use_left_static_pedestal}">
-    <xacro:ur_robot
-      name="${tf_prefix}left_ur5e"
-      tf_prefix="${tf_prefix}left_ur_arm_"
-      parent="${tf_prefix}left_arm_cal_link"
-      kinematics_parameters_file="${left_ur_kinematics_file}"
-      joint_limits_parameters_file="$(find ur_description)/config/ur5e/joint_limits.yaml"
-      physical_parameters_file="$(find ur_description)/config/ur5e/physical_parameters.yaml"
-      visual_parameters_file="$(find ur_description)/config/ur5e/visual_parameters.yaml"
-      initial_positions="${xacro.load_yaml(initial_positions_file_left)}"
-      use_fake_hardware="${use_fake_hardware}"
-      sim_ignition="${sim_ignition}"
-      robot_ip="${left_ur_ip_addr}"
-      reverse_port="50001"
-      script_sender_port="50002"
-      script_command_port="50004"
-      trajectory_port="50003"
-      use_tool_communication="false"
-      script_filename="$(find ur_client_library)/resources/external_control.urscript"
-      input_recipe_filename="$(find ur_robot_driver)/resources/rtde_input_recipe.txt"
-      output_recipe_filename="$(find ur_robot_driver)/resources/rtde_output_recipe.txt"
-      generate_ros2_control_tag="${generate_ros2_control_tag}"
-      >
-      <origin xyz="0 0 0.649605" rpy="0 0 0" /> <!-- TODO: need to integrate the OPTENV RIGEBACK_RIGHT_UR_XYZ stuff-->
-    </xacro:ur_robot>
+   <xacro:if value="${use_left_static_pedestal}">
+    <xacro:property name="parent" value="${tf_prefix}left_arm_cal_link"/>
+    <xacro:property name="origin_xyz" value="0 0 0.649605"/>
+    <xacro:property name="origin_rpy" value="0 0 0"/>
   </xacro:if>
+  <xacro:ur_robot
+    name="${tf_prefix}left_ur5e"
+    tf_prefix="${tf_prefix}left_ur_arm_"
+    parent="${parent}"
+    kinematics_parameters_file="${left_ur_kinematics_file}"
+    joint_limits_parameters_file="$(find ur_description)/config/ur5e/joint_limits.yaml"
+    physical_parameters_file="$(find ur_description)/config/ur5e/physical_parameters.yaml"
+    visual_parameters_file="$(find ur_description)/config/ur5e/visual_parameters.yaml"
+    initial_positions="${xacro.load_yaml(initial_positions_file_left)}"
+    use_fake_hardware="${use_fake_hardware}"
+    sim_ignition="${sim_ignition}"
+    robot_ip="${left_ur_ip_addr}"
+    reverse_port="50001"
+    script_sender_port="50002"
+    script_command_port="50004"
+    trajectory_port="50003"
+    use_tool_communication="false"
+    script_filename="$(find ur_client_library)/resources/external_control.urscript"
+    input_recipe_filename="$(find ur_robot_driver)/resources/rtde_input_recipe.txt"
+    output_recipe_filename="$(find ur_robot_driver)/resources/rtde_output_recipe.txt"
+    generate_ros2_control_tag="${generate_ros2_control_tag}"
+    >
+    <origin xyz="${origin_xyz}" rpy="${origin_rpy}" />
+  </xacro:ur_robot>
   <!-- end effector interface stack -->
   <xacro:unless value="${calibration_mode}">

Commit message: Deleted mesh of static pedestal without mounting and cleaned up urdf.

File: phoebe_description/urdf/phoebe_macro.xacro (robot description, xacro)
@@ -392,11 +392,10 @@
     <origin xyz="0.0845 -0.384 0.22" rpy="0 0 0" />
   </joint>
-  <!-- Left Ewellix mounting flange -->
   <!-- load the liftkit mount calibration -->
-    <xacro:property name="liftkit_mount_calibration" value="${xacro.load_yaml(liftkit_mount_calibration_file)}"/>
-    <xacro:property name="left_edge_aligned_distance" value="${liftkit_mount_calibration['left_edge_aligned_distance']}"/>
-    <xacro:property name="right_edge_aligned_distance" value="${liftkit_mount_calibration['right_edge_aligned_distance']}"/>
-    <xacro:property name="left_liftkit_dist_from_edge" value="${liftkit_mount_calibration['left_liftkit_dist_from_edge']}"/>
-    <xacro:property name="right_liftkit_dist_from_edge" value="${liftkit_mount_calibration['right_liftkit_dist_from_edge']}"/>
+  <xacro:property name="liftkit_mount_calibration" value="${xacro.load_yaml(liftkit_mount_calibration_file)}"/>
+  <xacro:property name="left_edge_aligned_distance" value="${liftkit_mount_calibration['left_edge_aligned_distance']}"/>
+  <xacro:property name="right_edge_aligned_distance" value="${liftkit_mount_calibration['right_edge_aligned_distance']}"/>
+  <xacro:property name="left_liftkit_dist_from_edge" value="${liftkit_mount_calibration['left_liftkit_dist_from_edge']}"/>
+  <xacro:property name="right_liftkit_dist_from_edge" value="${liftkit_mount_calibration['right_liftkit_dist_from_edge']}"/>
   <xacro:unless value="${use_left_static_pedestal}">
     <link name="${tf_prefix}left_ewellix_mount_flange_link">
@@ -644,8 +643,18 @@
   </xacro:if>
   <!-- left ur -->
+  <xacro:unless value="${use_left_static_pedestal}">
+    <xacro:property name="parent" value="${tf_prefix}left_arm_mount_plate_2"/>
+    <xacro:property name="origin_xyz" value="0 0 0"/>
+    <xacro:property name="origin_rpy" value="0 0 ${-pi/4}"/>
+  </xacro:unless>
+  <xacro:if value="${use_left_static_pedestal}">
+    <xacro:property name="parent" value="${tf_prefix}left_arm_cal_link"/>
+    <xacro:property name="origin_xyz" value="0 0 0.649605"/>
+    <xacro:property name="origin_rpy" value="0 0 0"/>
+  </xacro:if>
   <xacro:ur_robot
     name="${tf_prefix}left_ur5e"
     tf_prefix="${tf_prefix}left_ur_arm_"
-    parent="${tf_prefix}left_arm_mount_plate_2"
+    parent="${parent}"
     kinematics_parameters_file="${left_ur_kinematics_file}"
     joint_limits_parameters_file="$(find ur_description)/config/ur5e/joint_limits.yaml"
@@ -656,5 +665,5 @@
     safety_k_position="20"
     >
-    <origin xyz="0 0 0" rpy="0 0 ${-pi/4}" /> <!-- TODO: need to integrate the OPTENV RIGEBACK_RIGHT_UR_XYZ stuff-->
+    <origin xyz="${origin_xyz}" rpy="${origin_rpy}" />
   </xacro:ur_robot>
   <xacro:if value="${generate_ros2_control_tag}">

Commit message: ModifiedURDF to reflect new arm mount for the static pedestal, and added mesh file.

File: phoebe_description/urdf/phoebe_macro.xacro (robot description, xacro)
@@ -510,11 +510,11 @@
       <parent link="${tf_prefix}left_static_pedestal_link"/>
       <child link="${tf_prefix}left_ewellix_lift_tip_link"/>
-      <origin xyz="0 0 0.6096" rpy="0 0 0"/>
+      <origin xyz="0 0 0.6496" rpy="0 0 0"/>
     </joint>
     <!-- Left arm mount plate -->
-    <!-- <link name="${tf_prefix}left_arm_mount_plate">
+    <link name="${tf_prefix}left_arm_mount_plate">
       <visual>
         <geometry>
-          <mesh filename="package://phoebe_description/meshes/visual/jaco01_meshes/arm_mount.STL"/>
+          <mesh filename="package://phoebe_description/meshes/visual/jaco01_meshes/arm_mount_swivellink_new.stl" scale="0.0254 0.0254 0.0254"/>
         </geometry>
         <material name="clearpath_black" />
@@ -522,5 +522,5 @@
       <collision>
         <geometry>
-          <mesh filename="package://phoebe_description/meshes/visual/jaco01_meshes/arm_mount_collision.STL"/>
+          <mesh filename="package://phoebe_description/meshes/visual/jaco01_meshes/arm_mount_swivellink_new.stl" scale="0.0254 0.0254 0.0254"/>
         </geometry>
       </collision>
@@ -530,5 +530,5 @@
       <child link="${tf_prefix}left_arm_mount_plate" />
       <origin xyz="0 0 0" rpy="0 0 0" />
-    </joint> -->
+    </joint>
   </xacro:if>
   <xacro:ewellix_lift
@@ -567,20 +567,12 @@
   </joint>
   <!-- calibration links -->
-  <xacro:unless value="${use_left_static_pedestal}">
-    <link name="${tf_prefix}left_arm_cal_link"> </link>
-    <joint name="${tf_prefix}left_arm_cal_joint" type="fixed">
-      <parent link="${tf_prefix}left_arm_mount_plate" />
-      <child link="${tf_prefix}left_arm_cal_link" />
-      <origin xyz="0.00807 -0.00363 0.01019" rpy="0.01529 0.01951 -0.00426"/>
-    </joint>
-  </xacro:unless>
-  <xacro:if value="${use_left_static_pedestal}">
-    <link name="${tf_prefix}left_arm_cal_link"> </link>
-    <joint name="${tf_prefix}left_arm_cal_joint" type="fixed">
-      <parent link="${tf_prefix}left_static_pedestal_link" />
-      <child link="${tf_prefix}left_arm_cal_link" />
-      <origin xyz="0 0 0" rpy="0 0 0"/>
-    </joint>
-  </xacro:if>
+  <!-- LEFT -->
+  <link name="${tf_prefix}left_arm_cal_link"> </link>
+  <joint name="${tf_prefix}left_arm_cal_joint" type="fixed">
+    <parent link="${tf_prefix}left_arm_mount_plate" />
+    <child link="${tf_prefix}left_arm_cal_link" />
+    <origin xyz="0.00807 -0.00363 0.01019" rpy="0.01529 0.01951 -0.00426"/>
+  </joint>
+  <!-- RIGHT -->
   <link name="${tf_prefix}right_arm_cal_link"> </link>
   <joint name="${tf_prefix}right_arm_cal_joint" type="fixed">
@@ -590,4 +582,5 @@
   </joint>
   <!-- end calibration links -->
+  <!-- LEFT -->
   <link name="${tf_prefix}left_arm_mount_plate_2"> </link>
   <joint name="${tf_prefix}left_arm_mount_joint" type="fixed">
@@ -596,4 +589,5 @@
     <origin xyz="0 0.01628 0.09117" rpy="-${pi/4} 0 0"/>
   </joint>
+  <!-- RIGHT -->
   <link name="${tf_prefix}right_arm_mount_plate_2"> </link>
   <joint name="${tf_prefix}right_arm_mount_joint" type="fixed">
@@ -639,8 +633,8 @@
     <xacro:property name="origin_rpy" value="0 0 ${-pi/4}"/>
   </xacro:unless>
-   <xacro:if value="${use_left_static_pedestal}">
-    <xacro:property name="parent" value="${tf_prefix}left_arm_cal_link"/>
-    <xacro:property name="origin_xyz" value="0 0 0.649605"/>
-    <xacro:property name="origin_rpy" value="0 0 0"/>
+  <xacro:if value="${use_left_static_pedestal}">
+    <xacro:property name="parent" value="${tf_prefix}left_arm_mount_plate"/>
+    <xacro:property name="origin_xyz" value="${1.8957*0.0254} 0 ${5.2763*0.0254}"/>
+    <xacro:property name="origin_rpy" value="0.7853 0 1.5708"/>
   </xacro:if>
   <xacro:ur_robot

Commit message: ModifiedURDF to reflect new arm mount for the static pedestal, and added mesh file.

File: phoebe_description/urdf/phoebe_macro.xacro (robot description, xacro)
@@ -510,11 +510,11 @@
       <parent link="${tf_prefix}left_static_pedestal_link"/>
       <child link="${tf_prefix}left_ewellix_lift_tip_link"/>
-      <origin xyz="0 0 0.6096" rpy="0 0 0"/>
+      <origin xyz="0 0 0.6496" rpy="0 0 0"/>
     </joint>
     <!-- Left arm mount plate -->
-    <!-- <link name="${tf_prefix}left_arm_mount_plate">
+    <link name="${tf_prefix}left_arm_mount_plate">
       <visual>
         <geometry>
-          <mesh filename="package://phoebe_description/meshes/visual/jaco01_meshes/arm_mount.STL"/>
+          <mesh filename="package://phoebe_description/meshes/visual/jaco01_meshes/arm_mount_swivellink_new.stl" scale="0.0254 0.0254 0.0254"/>
         </geometry>
         <material name="clearpath_black" />
@@ -522,5 +522,5 @@
       <collision>
         <geometry>
-          <mesh filename="package://phoebe_description/meshes/visual/jaco01_meshes/arm_mount_collision.STL"/>
+          <mesh filename="package://phoebe_description/meshes/visual/jaco01_meshes/arm_mount_swivellink_new.stl" scale="0.0254 0.0254 0.0254"/>
         </geometry>
       </collision>
@@ -530,5 +530,5 @@
       <child link="${tf_prefix}left_arm_mount_plate" />
       <origin xyz="0 0 0" rpy="0 0 0" />
-    </joint> -->
+    </joint>
   </xacro:if>
   <xacro:ewellix_lift
@@ -567,20 +567,12 @@
   </joint>
   <!-- calibration links -->
-  <xacro:unless value="${use_left_static_pedestal}">
-    <link name="${tf_prefix}left_arm_cal_link"> </link>
-    <joint name="${tf_prefix}left_arm_cal_joint" type="fixed">
-      <parent link="${tf_prefix}left_arm_mount_plate" />
-      <child link="${tf_prefix}left_arm_cal_link" />
-      <origin xyz="0.00807 -0.00363 0.01019" rpy="0.01529 0.01951 -0.00426"/>
-    </joint>
-  </xacro:unless>
-  <xacro:if value="${use_left_static_pedestal}">
-    <link name="${tf_prefix}left_arm_cal_link"> </link>
-    <joint name="${tf_prefix}left_arm_cal_joint" type="fixed">
-      <parent link="${tf_prefix}left_static_pedestal_link" />
-      <child link="${tf_prefix}left_arm_cal_link" />
-      <origin xyz="0 0 0" rpy="0 0 0"/>
-    </joint>
-  </xacro:if>
+  <!-- LEFT -->
+  <link name="${tf_prefix}left_arm_cal_link"> </link>
+  <joint name="${tf_prefix}left_arm_cal_joint" type="fixed">
+    <parent link="${tf_prefix}left_arm_mount_plate" />
+    <child link="${tf_prefix}left_arm_cal_link" />
+    <origin xyz="0.00807 -0.00363 0.01019" rpy="0.01529 0.01951 -0.00426"/>
+  </joint>
+  <!-- RIGHT -->
   <link name="${tf_prefix}right_arm_cal_link"> </link>
   <joint name="${tf_prefix}right_arm_cal_joint" type="fixed">
@@ -590,4 +582,5 @@
   </joint>
   <!-- end calibration links -->
+  <!-- LEFT -->
   <link name="${tf_prefix}left_arm_mount_plate_2"> </link>
   <joint name="${tf_prefix}left_arm_mount_joint" type="fixed">
@@ -596,4 +589,5 @@
     <origin xyz="0 0.01628 0.09117" rpy="-${pi/4} 0 0"/>
   </joint>
+  <!-- RIGHT -->
   <link name="${tf_prefix}right_arm_mount_plate_2"> </link>
   <joint name="${tf_prefix}right_arm_mount_joint" type="fixed">
@@ -649,7 +643,7 @@
   </xacro:unless>
   <xacro:if value="${use_left_static_pedestal}">
-    <xacro:property name="parent" value="${tf_prefix}left_arm_cal_link"/>
-    <xacro:property name="origin_xyz" value="0 0 0.649605"/>
-    <xacro:property name="origin_rpy" value="0 0 0"/>
+    <xacro:property name="parent" value="${tf_prefix}left_arm_mount_plate"/>
+    <xacro:property name="origin_xyz" value="${1.8957*0.0254} 0 ${5.2763*0.0254}"/>
+    <xacro:property name="origin_rpy" value="0.7853 0 1.5708"/>
   </xacro:if>
   <xacro:ur_robot

Commit message: Modified origin of left ur based on hardware. Disabled collisions involving pedestal.

File: phoebe_description/urdf/phoebe_macro.xacro (robot description, xacro)
@@ -645,5 +645,5 @@
     <xacro:property name="parent" value="${tf_prefix}left_arm_mount_plate"/>
     <xacro:property name="origin_xyz" value="${1.8957*0.0254} 0 ${5.2763*0.0254}"/>
-    <xacro:property name="origin_rpy" value="0.7853 0 1.5708"/>
+    <xacro:property name="origin_rpy" value="0 -0.7853 ${pi}"/>
   </xacro:if>
   <xacro:ur_robot

Commit message: Modified origin of left ur based on hardware. Disabled collisions involving pedestal.

File: phoebe_description/urdf/phoebe_macro.xacro (robot description, xacro)
@@ -636,5 +636,5 @@
     <xacro:property name="parent" value="${tf_prefix}left_arm_mount_plate"/>
     <xacro:property name="origin_xyz" value="${1.8957*0.0254} 0 ${5.2763*0.0254}"/>
-    <xacro:property name="origin_rpy" value="0.7853 0 1.5708"/>
+    <xacro:property name="origin_rpy" value="0 -0.7853 ${pi}"/>
   </xacro:if>
   <xacro:ur_robot

Commit message: breaking out ur description macro

File: phoebe_description/urdf/phoebe_macro.xacro (robot description, xacro)
@@ -544,6 +544,5 @@
   <xacro:property name="initial_positions_file_left" default="$(find phoebe_description)/config/left_ur_initial_positions.yaml"/>
   <xacro:property name="initial_positions_file_right" default="$(find phoebe_description)/config/right_ur_initial_positions.yaml"/>
-  <!-- TODO: need to integrate the motion on the rails. this used to be done like below -->
-  <!-- <origin xyz="$(optenv RIDGEBACK_RIGHT_UR_XYZ 0 0 0)" rpy="$(optenv RIDGEBACK_RIGHT_UR_RPY 0 0 0)" /> -->
+  <!-- right ur -->
   <xacro:ur_robot
     name="${tf_prefix}right_ur5e"
@@ -554,20 +553,32 @@
     physical_parameters_file="$(find ur_description)/config/ur5e/physical_parameters.yaml"
     visual_parameters_file="$(find ur_description)/config/ur5e/visual_parameters.yaml"
-    initial_positions="${xacro.load_yaml(initial_positions_file_right)}"
-    use_fake_hardware="${use_fake_hardware}"
-    sim_ignition="${sim_ignition}"
-    robot_ip="${right_ur_ip_addr}"
-    reverse_port="60001"
-    script_sender_port="60002"
-    script_command_port="60004"
-    trajectory_port="60003"
-    use_tool_communication="false"
-    script_filename="$(find ur_client_library)/resources/external_control.urscript"
-    input_recipe_filename="$(find ur_robot_driver)/resources/rtde_input_recipe.txt"
-    output_recipe_filename="$(find ur_robot_driver)/resources/rtde_output_recipe.txt"
-    generate_ros2_control_tag="${generate_ros2_control_tag}"
+    safety_limits="false"
+    safety_pos_margin="0.15"
+    safety_k_position="20"
     >
     <origin xyz="0 0 0" rpy="0 0 ${5*pi/4}" />
   </xacro:ur_robot>
+  <xacro:if value="${generate_ros2_control_tag}">
+    <!-- only including the ros2_control files in this first UR block -->
+    <xacro:include filename="$(find ur_robot_driver)/urdf/ur.ros2_control.xacro" />
+    <xacro:include filename="$(find ur_description)/urdf/inc/ur_transmissions.xacro" />
+    <xacro:ur_ros2_control
+      name="${tf_prefix}right_ur5e_ros2_control"
+      tf_prefix="${tf_prefix}right_ur_arm_"
+      kinematics_parameters_file="${right_ur_kinematics_file}"
+      use_mock_hardware="${use_fake_hardware}"
+      mock_sensor_commands="${use_fake_hardware}"
+      initial_positions="${xacro.load_yaml(initial_positions_file_right)}"
+      robot_ip="${right_ur_ip_addr}"
+      script_filename="$(find ur_client_library)/resources/external_control.urscript"
+      output_recipe_filename="$(find ur_robot_driver)/resources/rtde_output_recipe.txt"
+      input_recipe_filename="$(find ur_robot_driver)/resources/rtde_input_recipe.txt"
+      reverse_port="60001"
+      script_sender_port="60002"
+      trajectory_port="60003"
+      script_command_port="60004"
+    />
+  </xacro:if>
+  <!-- left ur -->
   <xacro:ur_robot
     name="${tf_prefix}left_ur5e"
@@ -578,20 +589,28 @@
     physical_parameters_file="$(find ur_description)/config/ur5e/physical_parameters.yaml"
     visual_parameters_file="$(find ur_description)/config/ur5e/visual_parameters.yaml"
-    initial_positions="${xacro.load_yaml(initial_positions_file_left)}"
-    use_fake_hardware="${use_fake_hardware}"
-    sim_ignition="${sim_ignition}"
-    robot_ip="${left_ur_ip_addr}"
-    reverse_port="50001"
-    script_sender_port="50002"
-    script_command_port="50004"
-    trajectory_port="50003"
-    use_tool_communication="false"
-    script_filename="$(find ur_client_library)/resources/external_control.urscript"
-    input_recipe_filename="$(find ur_robot_driver)/resources/rtde_input_recipe.txt"
-    output_recipe_filename="$(find ur_robot_driver)/resources/rtde_output_recipe.txt"
-    generate_ros2_control_tag="${generate_ros2_control_tag}"
+    safety_limits="false"
+    safety_pos_margin="0.15"
+    safety_k_position="20"
     >
     <origin xyz="0 0 0" rpy="0 0 ${-pi/4}" /> <!-- TODO: need to integrate the OPTENV RIGEBACK_RIGHT_UR_XYZ stuff-->
   </xacro:ur_robot>
+  <xacro:if value="${generate_ros2_control_tag}">
+    <xacro:ur_ros2_control
+      name="${tf_prefix}left_ur5e_ros2_control"
+      tf_prefix="${tf_prefix}left_ur_arm_"
+      kinematics_parameters_file="${left_ur_kinematics_file}"
+      use_mock_hardware="${use_fake_hardware}"
+      mock_sensor_commands="${use_fake_hardware}"
+      initial_positions="${xacro.load_yaml(initial_positions_file_left)}"
+      robot_ip="${left_ur_ip_addr}"
+      script_filename="$(find ur_client_library)/resources/external_control.urscript"
+      output_recipe_filename="$(find ur_robot_driver)/resources/rtde_output_recipe.txt"
+      input_recipe_filename="$(find ur_robot_driver)/resources/rtde_input_recipe.txt"
+      reverse_port="50001"
+      script_sender_port="50002"
+      script_command_port="50004"
+      trajectory_port="50003"
+    />
+  </xacro:if>
   <!-- end effector interface stack -->
   <xacro:unless value="${calibration_mode}">
