Commit message: added some missing prefixes

File: phoebe_description/urdf/phoebe_macro.xacro (robot description, xacro)
@@ -44,26 +44,26 @@
       <origin xyz="0 0 0" rpy="0 0 0"/>
     </joint>
-    <link name="virtual_rail_link_1"/>
+    <link name="${tf_prefix}virtual_rail_link_1"/>
     <!-- Connecting to odometry will enable the map -> world xform to be updated without distruption. -->
-    <joint name="linear_x_joint" type="prismatic">
+    <joint name="${tf_prefix}linear_x_joint" type="prismatic">
       <axis xyz="1 0 0"/>
       <parent link="odom" />
-      <child link="virtual_rail_link_1" />
+      <child link="${tf_prefix}virtual_rail_link_1" />
       <origin xyz="0 0 0" rpy="0 0 0" />
       <limit effort="1000.0" lower="-20.0" upper="20.0" velocity="0.175" acceleration="10.0"/>
       <dynamics damping="20.0" friction="500.0" />
     </joint>
-    <link name="virtual_rail_link_2"/>
-    <joint name="linear_y_joint" type="prismatic">
+    <link name="${tf_prefix}virtual_rail_link_2"/>
+    <joint name="${tf_prefix}linear_y_joint" type="prismatic">
       <axis xyz="0 1 0"/>
-      <parent link="virtual_rail_link_1" />
-      <child link="virtual_rail_link_2" />
+      <parent link="${tf_prefix}virtual_rail_link_1" />
+      <child link="${tf_prefix}virtual_rail_link_2" />
       <origin xyz="0 0 0" rpy="0 0 0" />
       <limit effort="1000.0" lower="-5.0" upper="55.0" velocity="0.175" acceleration="10.0"/>
       <dynamics damping="20.0" friction="500.0" />
     </joint>
-    <joint name="rotational_yaw_joint" type="continuous">
+    <joint name="${tf_prefix}rotational_yaw_joint" type="continuous">
       <axis xyz="0 0 1"/>
-      <parent link="virtual_rail_link_2"/>
+      <parent link="${tf_prefix}virtual_rail_link_2"/>
       <child link="${tf_prefix}base_link"/>
       <origin rpy="0 0 0" xyz="0 0 0"/>

Commit message: Add options to swap out grippers

File: phoebe_description/urdf/phoebe_macro.xacro (robot description, xacro)
@@ -14,5 +14,7 @@
       left_ewellix_com_port:='/dev/ewellix_left'
       right_ewellix_com_port:='/dev/ewellix_right'
+      left_end_effector:='hande'
       left_hande_com_port:='/tmp/hande_left'
+      right_end_effector:='2f-85'
       right_hande_com_port:='/tmp/hande_right'
       left_ur_ip_addr:='192.168.131.40'
@@ -712,29 +714,60 @@
       <origin xyz="-6.4777232475001029e-02 1.1461581058038600e-04 1.2884814853441564e-02" rpy="-9.9487205554735336e-02 -1.4520756449714673e+00 1.0569277772629829e-01"/>
     </xacro:sensor_d435>
-    <!-- right gripper - 2F-85 -->
-    <xacro:include filename="$(find phoebe_description)/urdf/robotiq_2f_85_macro.xacro"/>
-    <xacro:robotiq_2f_85
-      com_port="${right_hande_com_port}"
-      use_fake_hardware="${use_fake_hardware}"
-      name="${tf_prefix}right_dextivr_hande"
-      tf_prefix="${tf_prefix}right_"
-      parent="${tf_prefix}right_ur_realsense_mount"
-      generate_ros2_control_tag="${generate_ros2_control_tag}"
-      add_grasp_push_frames="${add_grasp_push_frames}">
-      <origin xyz="0 0 0.003" rpy="0 0 ${pi/2}"/>
-    </xacro:robotiq_2f_85>
-    <!-- Left gripper - Hand-E -->
-    <xacro:include filename="$(find dextivr_hande_description)/urdf/dextivr_hande.xacro"/>
-    <xacro:dextivr_hande
-      com_port="${left_hande_com_port}"
-      use_fake_hardware="${use_fake_hardware}"
-      name="${tf_prefix}left_dextivr_hande"
-      tf_prefix="${tf_prefix}left_"
-      parent="${tf_prefix}left_ur_realsense_mount"
-      generate_ros2_control_tag="${generate_ros2_control_tag}"
-      add_grasp_push_frames="${add_grasp_push_frames}"
-      finger_xacro="fngr_original">
-      <origin xyz="0 0 0.003" rpy="0 0 ${pi/2}"/>
-    </xacro:dextivr_hande>
+    <!-- Right gripper -->
+    <xacro:if value="${right_end_effector == 'hande'}">
+      <xacro:include filename="$(find dextivr_hande_description)/urdf/dextivr_hande.xacro"/>
+      <xacro:dextivr_hande
+        com_port="${right_hande_com_port}"
+        use_fake_hardware="${use_fake_hardware}"
+        name="${tf_prefix}right_dextivr_hande"
+        tf_prefix="${tf_prefix}right_"
+        parent="${tf_prefix}right_ur_realsense_mount"
+        generate_ros2_control_tag="${generate_ros2_control_tag}"
+        add_grasp_push_frames="${add_grasp_push_frames}"
+        finger_xacro="fngr_original">
+        <origin xyz="0 0 0.003" rpy="0 0 ${pi/2}"/>
+      </xacro:dextivr_hande>
+    </xacro:if>
+    <xacro:if value="${right_end_effector == '2f-85'}">
+      <xacro:include filename="$(find phoebe_description)/urdf/robotiq_2f_85_macro.xacro"/>
+      <xacro:robotiq_2f_85
+        com_port="${right_hande_com_port}"
+        use_fake_hardware="${use_fake_hardware}"
+        name="${tf_prefix}right_dextivr_hande"
+        tf_prefix="${tf_prefix}right_"
+        parent="${tf_prefix}right_ur_realsense_mount"
+        generate_ros2_control_tag="${generate_ros2_control_tag}"
+        add_grasp_push_frames="${add_grasp_push_frames}">
+        <origin xyz="0 0 0.003" rpy="0 0 ${pi/2}"/>
+      </xacro:robotiq_2f_85>
+    </xacro:if>
+    <!-- Left gripper -->
+    <xacro:if value="${left_end_effector == 'hande'}">
+      <xacro:include filename="$(find dextivr_hande_description)/urdf/dextivr_hande.xacro"/>
+      <xacro:dextivr_hande
+        com_port="${left_hande_com_port}"
+        use_fake_hardware="${use_fake_hardware}"
+        name="${tf_prefix}left_dextivr_hande"
+        tf_prefix="${tf_prefix}left_"
+        parent="${tf_prefix}left_ur_realsense_mount"
+        generate_ros2_control_tag="${generate_ros2_control_tag}"
+        add_grasp_push_frames="${add_grasp_push_frames}"
+        finger_xacro="fngr_original">
+        <origin xyz="0 0 0.003" rpy="0 0 ${pi/2}"/>
+      </xacro:dextivr_hande>
+    </xacro:if>
+    <xacro:if value="${left_end_effector == '2f-85'}">
+      <xacro:include filename="$(find phoebe_description)/urdf/robotiq_2f_85_macro.xacro"/>
+      <xacro:robotiq_2f_85
+        com_port="${left_hande_com_port}"
+        use_fake_hardware="${use_fake_hardware}"
+        name="${tf_prefix}left_dextivr_hande"
+        tf_prefix="${tf_prefix}left_"
+        parent="${tf_prefix}left_ur_realsense_mount"
+        generate_ros2_control_tag="${generate_ros2_control_tag}"
+        add_grasp_push_frames="${add_grasp_push_frames}">
+        <origin xyz="0 0 0.003" rpy="0 0 ${pi/2}"/>
+      </xacro:robotiq_2f_85>
+    </xacro:if>
   </xacro:unless>
   <!-- Calibration HW -->
