Commit message: Parameterize generation files for a magic carpet version of PB

File: phoebe_description/urdf/phoebe_macro.xacro (robot description, xacro)
@@ -49,5 +49,11 @@
       <origin xyz="0 0 0" rpy="0 0 0"/>
     </joint>
-    <link name="${tf_prefix}virtual_rail_link_1"/>
+    <link name="${tf_prefix}virtual_rail_link_1">
+      <inertial>
+        <mass value="0.01"/>
+        <origin xyz="0 0 0"/>
+        <inertia ixx="1e-6" ixy="0" ixz="0" iyy="1e-6" iyz="0" izz="1e-6"/>
+      </inertial>
+    </link>
     <!-- Connecting to odometry will enable the map -> world xform to be updated without distruption. -->
     <joint name="${tf_prefix}linear_x_joint" type="prismatic">
@@ -56,8 +62,14 @@
       <child link="${tf_prefix}virtual_rail_link_1" />
       <origin xyz="0 0 0" rpy="0 0 0" />
-      <limit effort="1000.0" lower="-20.0" upper="20.0" velocity="0.175" acceleration="10.0"/>
+      <limit effort="1000.0" lower="-100.0" upper="100.0" velocity="0.175" acceleration="10.0"/>
       <dynamics damping="20.0" friction="500.0" />
     </joint>
-    <link name="${tf_prefix}virtual_rail_link_2"/>
+    <link name="${tf_prefix}virtual_rail_link_2">
+      <inertial>
+        <mass value="0.01"/>
+        <origin xyz="0 0 0"/>
+        <inertia ixx="1e-6" ixy="0" ixz="0" iyy="1e-6" iyz="0" izz="1e-6"/>
+      </inertial>
+    </link>
     <joint name="${tf_prefix}linear_y_joint" type="prismatic">
       <axis xyz="0 1 0"/>
@@ -65,5 +77,5 @@
       <child link="${tf_prefix}virtual_rail_link_2" />
       <origin xyz="0 0 0" rpy="0 0 0" />
-      <limit effort="1000.0" lower="-5.0" upper="55.0" velocity="0.175" acceleration="10.0"/>
+      <limit effort="1000.0" lower="-100.0" upper="100.0" velocity="0.175" acceleration="10.0"/>
       <dynamics damping="20.0" friction="500.0" />
     </joint>

File: phoebe_mujoco_config/urdf/phoebe_mujoco_raw_inputs.xacro (robot description, xacro)
@@ -7,4 +7,5 @@
     right_hand_type:='hande'
     defaults_prefix:=''
+    include_world_joints:=false
   ">
     <option integrator="implicitfast" impratio="20" cone="elliptic" noslip_iterations="5">
@@ -86,10 +87,19 @@
         <general class="size2" name="${tf_prefix}right_ur_arm_wrist_2_joint" joint="${tf_prefix}right_ur_arm_wrist_2_joint"/>
         <general class="size2" name="${tf_prefix}right_ur_arm_wrist_3_joint" joint="${tf_prefix}right_ur_arm_wrist_3_joint"/>
-        <velocity name="${tf_prefix}front_right_wheel_joint" joint="${tf_prefix}front_right_wheel_joint" ctrlrange="-15 15" kv="50"/>
-        <velocity name="${tf_prefix}front_left_wheel_joint" joint="${tf_prefix}front_left_wheel_joint" ctrlrange="-15 15" kv="50"/>
-        <velocity name="${tf_prefix}rear_right_wheel_joint" joint="${tf_prefix}rear_right_wheel_joint" ctrlrange="-15 15" kv="50"/>
-        <velocity name="${tf_prefix}rear_left_wheel_joint" joint="${tf_prefix}rear_left_wheel_joint" ctrlrange="-15 15" kv="50"/>
+        <!-- Nominally include the wheels -->
+        <xacro:unless value="${include_world_joints}">
+            <velocity name="${tf_prefix}front_right_wheel_joint" joint="${tf_prefix}front_right_wheel_joint" ctrlrange="-15 15" kv="50"/>
+            <velocity name="${tf_prefix}front_left_wheel_joint" joint="${tf_prefix}front_left_wheel_joint" ctrlrange="-15 15" kv="50"/>
+            <velocity name="${tf_prefix}rear_right_wheel_joint" joint="${tf_prefix}rear_right_wheel_joint" ctrlrange="-15 15" kv="50"/>
+            <velocity name="${tf_prefix}rear_left_wheel_joint" joint="${tf_prefix}rear_left_wheel_joint" ctrlrange="-15 15" kv="50"/>
+        </xacro:unless>
+         <!-- Otherwise it's magic carpet mode -->
+        <xacro:if value="${include_world_joints}">
+            <position joint="${tf_prefix}linear_x_joint" name="${tf_prefix}linear_x_joint" kp="5000" dampratio="1.0" ctrlrange="-10.0 10.0"/>
+            <position joint="${tf_prefix}linear_y_joint" name="${tf_prefix}linear_y_joint" kp="5000" dampratio="1.0" ctrlrange="-10.0 10.0"/>
+            <position joint="${tf_prefix}rotational_yaw_joint" name="${tf_prefix}rotational_yaw_joint" kp="5000" dampratio="1.0"/>
+        </xacro:if>
     </actuator>
-    <contact>
+        <contact>
         <xacro:unless value="${use_left_static_pedestal}">
             <exclude body1="${tf_prefix}base_link" body2="${tf_prefix}left_ewellix_lift_higher_link"/>
@@ -98,40 +108,51 @@
         <exclude body1="${tf_prefix}base_link" body2="${tf_prefix}right_ewellix_lift_higher_link"/>
         <exclude body1="${tf_prefix}base_link" body2="${tf_prefix}right_ewellix_lift_middle_link"/>
-        <exclude body1="${tf_prefix}base_link" body2="${tf_prefix}rear_left_wheel_link"/>
-        <exclude body1="${tf_prefix}base_link" body2="${tf_prefix}rear_left_wheel_roller_0_link"/>
-        <exclude body1="${tf_prefix}base_link" body2="${tf_prefix}rear_left_wheel_roller_1_link"/>
-        <exclude body1="${tf_prefix}base_link" body2="${tf_prefix}rear_left_wheel_roller_2_link"/>
-        <exclude body1="${tf_prefix}base_link" body2="${tf_prefix}rear_left_wheel_roller_3_link"/>
-        <exclude body1="${tf_prefix}base_link" body2="${tf_prefix}rear_left_wheel_roller_4_link"/>
-        <exclude body1="${tf_prefix}base_link" body2="${tf_prefix}rear_left_wheel_roller_5_link"/>
-        <exclude body1="${tf_prefix}base_link" body2="${tf_prefix}rear_left_wheel_roller_6_link"/>
-        <exclude body1="${tf_prefix}base_link" body2="${tf_prefix}rear_left_wheel_roller_7_link"/>
-        <exclude body1="${tf_prefix}base_link" body2="${tf_prefix}rear_right_wheel_link"/>
-        <exclude body1="${tf_prefix}base_link" body2="${tf_prefix}rear_right_wheel_roller_0_link"/>
-        <exclude body1="${tf_prefix}base_link" body2="${tf_prefix}rear_right_wheel_roller_1_link"/>
-        <exclude body1="${tf_prefix}base_link" body2="${tf_prefix}rear_right_wheel_roller_2_link"/>
-        <exclude body1="${tf_prefix}base_link" body2="${tf_prefix}rear_right_wheel_roller_3_link"/>
-        <exclude body1="${tf_prefix}base_link" body2="${tf_prefix}rear_right_wheel_roller_4_link"/>
-        <exclude body1="${tf_prefix}base_link" body2="${tf_prefix}rear_right_wheel_roller_5_link"/>
-        <exclude body1="${tf_prefix}base_link" body2="${tf_prefix}rear_right_wheel_roller_6_link"/>
-        <exclude body1="${tf_prefix}base_link" body2="${tf_prefix}rear_right_wheel_roller_7_link"/>
-        <exclude body1="${tf_prefix}base_link" body2="${tf_prefix}front_left_wheel_link"/>
-        <exclude body1="${tf_prefix}base_link" body2="${tf_prefix}front_left_wheel_roller_0_link"/>
-        <exclude body1="${tf_prefix}base_link" body2="${tf_prefix}front_left_wheel_roller_1_link"/>
-        <exclude body1="${tf_prefix}base_link" body2="${tf_prefix}front_left_wheel_roller_2_link"/>
-        <exclude body1="${tf_prefix}base_link" body2="${tf_prefix}front_left_wheel_roller_3_link"/>
-        <exclude body1="${tf_prefix}base_link" body2="${tf_prefix}front_left_wheel_roller_4_link"/>
-        <exclude body1="${tf_prefix}base_link" body2="${tf_prefix}front_left_wheel_roller_5_link"/>
-        <exclude body1="${tf_prefix}base_link" body2="${tf_prefix}front_left_wheel_roller_6_link"/>
-        <exclude body1="${tf_prefix}base_link" body2="${tf_prefix}front_left_wheel_roller_7_link"/>
-        <exclude body1="${tf_prefix}base_link" body2="${tf_prefix}front_right_wheel_link"/>
-        <exclude body1="${tf_prefix}base_link" body2="${tf_prefix}front_right_wheel_roller_0_link"/>
-        <exclude body1="${tf_prefix}base_link" body2="${tf_prefix}front_right_wheel_roller_1_link"/>
-        <exclude body1="${tf_prefix}base_link" body2="${tf_prefix}front_right_wheel_roller_2_link"/>
-        <exclude body1="${tf_prefix}base_link" body2="${tf_prefix}front_right_wheel_roller_3_link"/>
-        <exclude body1="${tf_prefix}base_link" body2="${tf_prefix}front_right_wheel_roller_4_link"/>
-        <exclude body1="${tf_prefix}base_link" body2="${tf_prefix}front_right_wheel_roller_5_link"/>
-        <exclude body1="${tf_prefix}base_link" body2="${tf_prefix}front_right_wheel_roller_6_link"/>
-        <exclude body1="${tf_prefix}base_link" body2="${tf_prefix}front_right_wheel_roller_7_link"/>
+        <xacro:unless value="${include_world_joints}">
+            <exclude body1="${tf_prefix}base_link" body2="${tf_prefix}rear_left_wheel_link"/>
+            <exclude body1="${tf_prefix}base_link" body2="${tf_prefix}rear_left_wheel_roller_0_link"/>
+            <exclude body1="${tf_prefix}base_link" body2="${tf_prefix}rear_left_wheel_roller_1_link"/>
+            <exclude body1="${tf_prefix}base_link" body2="${tf_prefix}rear_left_wheel_roller_2_link"/>
+            <exclude body1="${tf_prefix}base_link" body2="${tf_prefix}rear_left_wheel_roller_3_link"/>
+            <exclude body1="${tf_prefix}base_link" body2="${tf_prefix}rear_left_wheel_roller_4_link"/>
+            <exclude body1="${tf_prefix}base_link" body2="${tf_prefix}rear_left_wheel_roller_5_link"/>
+            <exclude body1="${tf_prefix}base_link" body2="${tf_prefix}rear_left_wheel_roller_6_link"/>
+            <exclude body1="${tf_prefix}base_link" body2="${tf_prefix}rear_left_wheel_roller_7_link"/>
+            <exclude body1="${tf_prefix}base_link" body2="${tf_prefix}rear_right_wheel_link"/>
+            <exclude body1="${tf_prefix}base_link" body2="${tf_prefix}rear_right_wheel_roller_0_link"/>
+            <exclude body1="${tf_prefix}base_link" body2="${tf_prefix}rear_right_wheel_roller_1_link"/>
+            <exclude body1="${tf_prefix}base_link" body2="${tf_prefix}rear_right_wheel_roller_2_link"/>
+            <exclude body1="${tf_prefix}base_link" body2="${tf_prefix}rear_right_wheel_roller_3_link"/>
+            <exclude body1="${tf_prefix}base_link" body2="${tf_prefix}rear_right_wheel_roller_4_link"/>
+            <exclude body1="${tf_prefix}base_link" body2="${tf_prefix}rear_right_wheel_roller_5_link"/>
+            <exclude body1="${tf_prefix}base_link" body2="${tf_prefix}rear_right_wheel_roller_6_link"/>
+            <exclude body1="${tf_prefix}base_link" body2="${tf_prefix}rear_right_wheel_roller_7_link"/>
+            <exclude body1="${tf_prefix}base_link" body2="${tf_prefix}front_left_wheel_link"/>
+            <exclude body1="${tf_prefix}base_link" body2="${tf_prefix}front_left_wheel_roller_0_link"/>
+            <exclude body1="${tf_prefix}base_link" body2="${tf_prefix}front_left_wheel_roller_1_link"/>
+            <exclude body1="${tf_prefix}base_link" body2="${tf_prefix}front_left_wheel_roller_2_link"/>
+            <exclude body1="${tf_prefix}base_link" body2="${tf_prefix}front_left_wheel_roller_3_link"/>
+            <exclude body1="${tf_prefix}base_link" body2="${tf_prefix}front_left_wheel_roller_4_link"/>
+            <exclude body1="${tf_prefix}base_link" body2="${tf_prefix}front_left_wheel_roller_5_link"/>
+            <exclude body1="${tf_prefix}base_link" body2="${tf_prefix}front_left_wheel_roller_6_link"/>
+            <exclude body1="${tf_prefix}base_link" body2="${tf_prefix}front_left_wheel_roller_7_link"/>
+            <exclude body1="${tf_prefix}base_link" body2="${tf_prefix}front_right_wheel_link"/>
+            <exclude body1="${tf_prefix}base_link" body2="${tf_prefix}front_right_wheel_roller_0_link"/>
+            <exclude body1="${tf_prefix}base_link" body2="${tf_prefix}front_right_wheel_roller_1_link"/>
+            <exclude body1="${tf_prefix}base_link" body2="${tf_prefix}front_right_wheel_roller_2_link"/>
+            <exclude body1="${tf_prefix}base_link" body2="${tf_prefix}front_right_wheel_roller_3_link"/>
+            <exclude body1="${tf_prefix}base_link" body2="${tf_prefix}front_right_wheel_roller_4_link"/>
+            <exclude body1="${tf_prefix}base_link" body2="${tf_prefix}front_right_wheel_roller_5_link"/>
+            <exclude body1="${tf_prefix}base_link" body2="${tf_prefix}front_right_wheel_roller_6_link"/>
+            <exclude body1="${tf_prefix}base_link" body2="${tf_prefix}front_right_wheel_roller_7_link"/>
+        </xacro:unless>
+        <xacro:if value="${include_world_joints}">
+            <exclude body1="world" body2="${tf_prefix}base_link"/>
+            <exclude body1="world" body2="${tf_prefix}virtual_rail_link_1"/>
+            <exclude body1="world" body2="${tf_prefix}virtual_rail_link_2"/>
+            <exclude body1="world" body2="${tf_prefix}front_left_wheel_link"/>
+            <exclude body1="world" body2="${tf_prefix}front_right_wheel_link"/>
+            <exclude body1="world" body2="${tf_prefix}rear_left_wheel_link"/>
+            <exclude body1="world" body2="${tf_prefix}rear_right_wheel_link"/>
+        </xacro:if>
     </contact>
     <!-- left hand - hande or 2f85 -->

File: phoebe_mujoco_config/urdf/phoebe_mujoco_ros2_control_macros.xacro (robot description, xacro)
@@ -44,4 +44,5 @@
     right_hand_type:='hande'
     use_left_static_pedestal:=false
+    include_world_joints:=false
   ">
     <xacro:unless value="${use_left_static_pedestal}">
@@ -204,36 +205,66 @@
       <state_interface name="effort"/>
     </joint>
-    <joint name="${tf_prefix}front_left_wheel_joint">
-      <command_interface name="velocity"/>
-      <state_interface name="position">
-        <param name="initial_value">0.0</param>
-      </state_interface>
-      <state_interface name="velocity"/>
-      <state_interface name="effort"/>
-    </joint>
-    <joint name="${tf_prefix}front_right_wheel_joint">
-      <command_interface name="velocity"/>
-      <state_interface name="position">
-        <param name="initial_value">0.0</param>
-      </state_interface>
-      <state_interface name="velocity"/>
-      <state_interface name="effort"/>
-    </joint>
-    <joint name="${tf_prefix}rear_left_wheel_joint">
-      <command_interface name="velocity"/>
-      <state_interface name="position">
-        <param name="initial_value">0.0</param>
-      </state_interface>
-      <state_interface name="velocity"/>
-      <state_interface name="effort"/>
-    </joint>
-    <joint name="${tf_prefix}rear_right_wheel_joint">
-      <command_interface name="velocity"/>
-      <state_interface name="position">
-        <param name="initial_value">0.0</param>
-      </state_interface>
-      <state_interface name="velocity"/>
-      <state_interface name="effort"/>
-    </joint>
+    <!-- In normal modes we command the wheel joints directly -->
+    <xacro:unless value="${include_world_joints}">
+      <joint name="${tf_prefix}front_left_wheel_joint">
+        <command_interface name="velocity"/>
+        <state_interface name="position">
+          <param name="initial_value">0.0</param>
+        </state_interface>
+        <state_interface name="velocity"/>
+        <state_interface name="effort"/>
+      </joint>
+      <joint name="${tf_prefix}front_right_wheel_joint">
+        <command_interface name="velocity"/>
+        <state_interface name="position">
+          <param name="initial_value">0.0</param>
+        </state_interface>
+        <state_interface name="velocity"/>
+        <state_interface name="effort"/>
+      </joint>
+      <joint name="${tf_prefix}rear_left_wheel_joint">
+        <command_interface name="velocity"/>
+        <state_interface name="position">
+          <param name="initial_value">0.0</param>
+        </state_interface>
+        <state_interface name="velocity"/>
+        <state_interface name="effort"/>
+      </joint>
+      <joint name="${tf_prefix}rear_right_wheel_joint">
+        <command_interface name="velocity"/>
+        <state_interface name="position">
+          <param name="initial_value">0.0</param>
+        </state_interface>
+        <state_interface name="velocity"/>
+        <state_interface name="effort"/>
+      </joint>
+    </xacro:unless>
+    <!-- Some simulation environments may use a magic carpet, and we should include those joints -->
+    <xacro:if value="${include_world_joints}">
+      <joint name="${tf_prefix}linear_x_joint">
+        <command_interface name="position"/>
+        <state_interface name="position">
+          <param name="initial_value">0.0</param>
+        </state_interface>
+        <state_interface name="velocity"/>
+        <state_interface name="effort"/>
+      </joint>
+      <joint name="${tf_prefix}linear_y_joint">
+        <command_interface name="position"/>
+        <state_interface name="position">
+          <param name="initial_value">0.0</param>
+        </state_interface>
+        <state_interface name="velocity"/>
+        <state_interface name="effort"/>
+      </joint>
+      <joint name="${tf_prefix}rotational_yaw_joint">
+        <command_interface name="position"/>
+        <state_interface name="position">
+          <param name="initial_value">0.0</param>
+        </state_interface>
+        <state_interface name="velocity"/>
+        <state_interface name="effort"/>
+      </joint>
+    </xacro:if>
   </xacro:macro>
 </robot>

File: phoebe_mujoco_config/urdf/phoebe_mujoco_xacro.urdf (robot description, URDF)
Before this commit: robot phoebe, 1 links, 1 joints
Joints:
- removed joint floating_base_joint

Commit message: Lift Phoebe when on a magic carpet

File: phoebe_description/urdf/phoebe_macro.xacro (robot description, xacro)
@@ -84,5 +84,6 @@
       <parent link="${tf_prefix}virtual_rail_link_2"/>
       <child link="${tf_prefix}base_link"/>
-      <origin rpy="0 0 0" xyz="0 0 0"/>
+      <!-- Wheel axle is 0.05 above base_link with a 0.0759 radius, lift so the wheels "rest" on the floor. -->
+      <origin rpy="0 0 0" xyz="0 0 0.0259"/>
       <limit effort="150.0" velocity="0.5235987755982988"/>
       <dynamics damping="0" friction="0"/>

File: phoebe_mujoco_config/urdf/phoebe_mujoco_raw_inputs.xacro (robot description, xacro)
@@ -147,4 +147,5 @@
             <exclude body1="${tf_prefix}base_link" body2="${tf_prefix}front_right_wheel_roller_7_link"/>
         </xacro:unless>
+        <!-- If phoebe is on a carpet, the wheels will not interact with anything -->
         <xacro:if value="${include_world_joints}">
             <exclude body1="world" body2="${tf_prefix}base_link"/>

Commit message: readding liftkit cal

File: phoebe_description/urdf/phoebe_macro.xacro (robot description, xacro)
@@ -484,7 +484,4 @@
   <xacro:include filename="$(find ewellix_liftkit_description)/urdf/ewellix_lift.xacro"/>
   <xacro:include filename="$(find ewellix_liftkit_description)/urdf/properties.xacro"/>
-  <!-- convert the arg into a property to be usable by the xacro -->
-  <!-- <xacro:property name="left_liftkit_calibration_file" value="${left_liftkit_calibration_file}"/>
-  <xacro:property name="right_liftkit_calibration_file" value="${right_liftkit_calibration_file}"/> -->
   <xacro:unless value="${use_left_static_pedestal}">
     <xacro:ewellix_lift
@@ -499,4 +496,5 @@
       use_fake_hardware="${use_fake_hardware}"
       com_port="${left_ewellix_com_port}"
+      hw_calibration="${xacro.load_yaml(left_liftkit_calibration_file)}"
       generate_ros2_control_tag="${generate_ros2_control_tag}"
     >
@@ -562,4 +560,5 @@
       use_fake_hardware="${use_fake_hardware}"
       com_port="${right_ewellix_com_port}"
+      hw_calibration="${xacro.load_yaml(right_liftkit_calibration_file)}"
       generate_ros2_control_tag="${generate_ros2_control_tag}"
     >
