Commit message: adding tf_prefix to joints

File: phoebe_description/urdf/phoebe.urdf.xacro (robot description, xacro)
@@ -3,7 +3,12 @@
     <xacro:arg name="namespace" default="" />
     <xacro:arg name="is_sim" default="true" />
+    <xacro:arg name="tf_prefix" default="''" />
+    <xacro:arg name="parent" default="world" />
     <!-- Includes -->
     <xacro:include filename="$(find clearpath_platform_description)/urdf/common.urdf.xacro" />
     <xacro:include filename="$(find phoebe_description)/urdf/r100.urdf.xacro" />
-    <xacro:r100 />
+    <xacro:r100
+        tf_prefix="$(arg tf_prefix)"
+        is_sim="$(arg is_sim)"
+    />
 </robot>

File: phoebe_description/urdf/r100.urdf.xacro (robot description, xacro)
@@ -1,6 +1,4 @@
 <?xml version="1.0"?>
 <robot xmlns:xacro="http://ros.org/wiki/xacro">
-    <xacro:arg name="namespace" default="" />
-    <xacro:arg name="is_sim" default="false" />
     <xacro:arg name="gazebo_controllers"
         default="$(find phoebe_deploy)/config/control.yaml" />
@@ -10,5 +8,8 @@
     <xacro:include filename="$(find phoebe_description)/urdf/rocker.urdf.xacro" />
     <!-- R100 Platform Macro -->
-    <xacro:macro name="r100" params="wheel:='default'">
+    <xacro:macro name="r100"
+        params="wheel:='default'
+                tf_prefix:=''
+                is_sim:=false">
         <!-- Variables -->
         <xacro:property name="wheel_radius" value="0.0759" />
@@ -29,11 +30,11 @@
         <xacro:property name="dummy_inertia" value="1e-09" />
         <!-- Chassis -->
-        <link name="base_link"></link>
-        <joint name="base_link_joint" type="fixed">
-            <origin xyz="0 0 0" rpy="0 0 0" />
-            <parent link="base_link" />
-            <child link="chassis_link" />
-        </joint>
-        <link name="chassis_link">
+        <link name="${tf_prefix}base_link"></link>
+        <joint name="${tf_prefix}base_link_joint" type="fixed">
+            <origin xyz="0 0 0" rpy="0 0 0" />
+            <parent link="${tf_prefix}base_link" />
+            <child link="${tf_prefix}chassis_link" />
+        </joint>
+        <link name="${tf_prefix}chassis_link">
             <visual>
                 <origin xyz="0 0 0" rpy="0 0 0" />
@@ -59,15 +60,15 @@
         </link>
         <!-- Covers -->
-        <joint name="right_side_cover_link_joint" type="fixed">
-            <origin xyz="0 0 0" rpy="0 0 0" />
-            <parent link="chassis_link" />
-            <child link="right_side_cover_link" />
-        </joint>
-        <joint name="left_side_cover_link_joint" type="fixed">
-            <origin xyz="0 0 0" rpy="0 0 0" />
-            <parent link="chassis_link" />
-            <child link="left_side_cover_link" />
-        </joint>
-        <link name="left_side_cover_link">
+        <joint name="${tf_prefix}right_side_cover_link_joint" type="fixed">
+            <origin xyz="0 0 0" rpy="0 0 0" />
+            <parent link="${tf_prefix}chassis_link" />
+            <child link="${tf_prefix}right_side_cover_link" />
+        </joint>
+        <joint name="${tf_prefix}left_side_cover_link_joint" type="fixed">
+            <origin xyz="0 0 0" rpy="0 0 0" />
+            <parent link="${tf_prefix}chassis_link" />
+            <child link="${tf_prefix}left_side_cover_link" />
+        </joint>
+        <link name="${tf_prefix}left_side_cover_link">
             <visual>
                 <origin xyz="0 0 0" rpy="0 0 ${math.pi}" />
@@ -78,5 +79,5 @@
             </visual>
         </link>
-        <link name="right_side_cover_link">
+        <link name="${tf_prefix}right_side_cover_link">
             <visual>
                 <origin xyz="0 0 0" rpy="0 0 0" />
@@ -87,10 +88,10 @@
             </visual>
         </link>
-        <joint name="front_cover_link_joint" type="fixed">
-            <origin xyz="0 0 0" rpy="0 0 0" />
-            <parent link="chassis_link" />
-            <child link="front_cover_link" />
-        </joint>
-        <link name="front_cover_link">
+        <joint name="${tf_prefix}front_cover_link_joint" type="fixed">
+            <origin xyz="0 0 0" rpy="0 0 0" />
+            <parent link="${tf_prefix}chassis_link" />
+            <child link="${tf_prefix}front_cover_link" />
+        </joint>
+        <link name="${tf_prefix}front_cover_link">
             <visual>
                 <origin xyz="0 0 0" rpy="0 0 0" />
@@ -101,10 +102,10 @@
             </visual>
         </link>
-        <joint name="rear_cover_link_joint" type="fixed">
-            <origin xyz="0 0 0" rpy="0 0 0" />
-            <parent link="chassis_link" />
-            <child link="rear_cover_link" />
-        </joint>
-        <link name="rear_cover_link">
+        <joint name="${tf_prefix}rear_cover_link_joint" type="fixed">
+            <origin xyz="0 0 0" rpy="0 0 0" />
+            <parent link="${tf_prefix}chassis_link" />
+            <child link="${tf_prefix}rear_cover_link" />
+        </joint>
+        <link name="${tf_prefix}rear_cover_link">
             <visual>
                 <origin xyz="0 0 0" rpy="0 0 ${math.pi}" />
@@ -116,15 +117,15 @@
         </link>
         <!-- Lights -->
-        <joint name="front_lights_link_joint" type="fixed">
-            <origin xyz="0 0 0" rpy="0 0 0" />
-            <parent link="chassis_link" />
-            <child link="front_lights_link" />
-        </joint>
-        <joint name="rear_lights_link_joint" type="fixed">
-            <origin xyz="0 0 0" rpy="0 0 0" />
-            <parent link="chassis_link" />
-            <child link="rear_lights_link" />
-        </joint>
-        <link name="front_lights_link">
+        <joint name="${tf_prefix}front_lights_link_joint" type="fixed">
+            <origin xyz="0 0 0" rpy="0 0 0" />
+            <parent link="${tf_prefix}chassis_link" />
+            <child link="${tf_prefix}front_lights_link" />
+        </joint>
+        <joint name="${tf_prefix}rear_lights_link_joint" type="fixed">
+            <origin xyz="0 0 0" rpy="0 0 0" />
+            <parent link="${tf_prefix}chassis_link" />
+            <child link="${tf_prefix}rear_lights_link" />
+        </joint>
+        <link name="${tf_prefix}front_lights_link">
             <visual>
                 <origin xyz="0 0 0" rpy="0 0 0" />
@@ -135,5 +136,5 @@
             </visual>
         </link>
-        <link name="rear_lights_link">
+        <link name="${tf_prefix}rear_lights_link">
             <visual>
                 <origin xyz="0 0 0" rpy="0 0 ${math.pi}" />
@@ -145,10 +146,10 @@
         </link>
         <!-- Axle -->
-        <joint name="axle_joint" type="fixed">
+        <joint name="${tf_prefix}axle_joint" type="fixed">
             <origin xyz="0 0 ${axle_offset}" rpy="0 0 0" />
-            <parent link="chassis_link" />
-            <child link="axle_link" />
-        </joint>
-        <link name="axle_link">
+            <parent link="${tf_prefix}chassis_link" />
+            <child link="${tf_prefix}axle_link" />
+        </joint>
+        <link name="${tf_prefix}axle_link">
             <visual>
                 <origin xyz="0 0 0" rpy="0 ${math.pi/2} 0" />
@@ -160,10 +161,10 @@
         </link>
         <!-- Riser -->
-        <joint name="riser_link_joint" type="fixed">
+        <joint name="${tf_prefix}riser_link_joint" type="fixed">
             <origin xyz="0 0 ${0.225 - deck_thickness}" rpy="0 0 0" />
-            <parent link="chassis_link" />
-            <child link="riser_link" />
-        </joint>
-        <link name="riser_link">
+            <parent link="${tf_prefix}chassis_link" />
+            <child link="${tf_prefix}riser_link" />
+        </joint>
+        <link name="${tf_prefix}riser_link">
             <visual>
                 <origin xyz="0 0 ${riser_height/2}" rpy="0 0 ${pi/4}" />
@@ -181,10 +182,10 @@
         </link>
         <!-- Top Plate -->
-        <joint name="top_link_joint" type="fixed">
+        <joint name="${tf_prefix}top_link_joint" type="fixed">
             <origin xyz="0 0 ${riser_height-deck_height+deck_thickness}" rpy="0 0 0" />
-            <parent link="riser_link" />
-            <child link="top_link" />
-        </joint>
-        <link name="top_link">
+            <parent link="${tf_prefix}riser_link" />
+            <child link="${tf_prefix}top_link" />
+        </joint>
+        <link name="${tf_prefix}top_link">
             <visual>
                 <origin xyz="0 0 0" rpy="0 0 0" />
@@ -202,8 +203,8 @@
         </link>
         <!-- Rocker -->
-        <xacro:r100_rocker prefix="front" joint_type="fixed" location="1">
+        <xacro:r100_rocker prefix="front" joint_type="fixed" location="1" tf_prefix="${tf_prefix}">
             <limit lower="-0.08726" upper="0.08726" effort="0" velocity="0" />
         </xacro:r100_rocker>
-        <xacro:r100_rocker prefix="rear" joint_type="fixed" location="-1">
+        <xacro:r100_rocker prefix="rear" joint_type="fixed" location="-1" tf_prefix="${tf_prefix}">
             <limit effort="0" velocity="0" />
         </xacro:r100_rocker>
@@ -211,5 +212,5 @@
             <plugin filename="libignition-gazebo-wheel-slip-system.so"
                 name="ignition::gazebo::systems::WheelSlip">
-                <wheel link_name="front_left_wheel_link">
+                <wheel link_name="${tf_prefix}front_left_wheel_link">
                     <slip_compliance_lateral>1.0</slip_compliance_lateral>
                     <slip_compliance_longitudinal>1.0</slip_compliance_longitudinal>
@@ -217,5 +218,5 @@
                     <wheel_radius>${wheel_radius}</wheel_radius>
                 </wheel>
-                <wheel link_name="front_right_wheel_link">
+                <wheel link_name="${tf_prefix}front_right_wheel_link">
                     <slip_compliance_lateral>1.0</slip_compliance_lateral>
                     <slip_compliance_longitudinal>1.0</slip_compliance_longitudinal>
@@ -223,5 +224,5 @@
                     <wheel_radius>${wheel_radius}</wheel_radius>
                 </wheel>
-                <wheel link_name="rear_left_wheel_link">
+                <wheel link_name="${tf_prefix}rear_left_wheel_link">
                     <slip_compliance_lateral>1.0</slip_compliance_lateral>
                     <slip_compliance_longitudinal>1.0</slip_compliance_longitudinal>
@@ -229,5 +230,5 @@
                     <wheel_radius>${wheel_radius}</wheel_radius>
                 </wheel>
-                <wheel link_name="rear_right_wheel_link">
+                <wheel link_name="${tf_prefix}rear_right_wheel_link">
                     <slip_compliance_lateral>1.0</slip_compliance_lateral>
                     <slip_compliance_longitudinal>1.0</slip_compliance_longitudinal>
@@ -238,5 +239,5 @@
         </gazebo>
         <!-- Internal IMU -->
-        <link name="imu_0_link">
+        <link name="${tf_prefix}imu_0_link">
             <inertial>
                 <mass value="0.001" />
@@ -246,10 +247,10 @@
             </inertial>
         </link>
-        <joint name="imu_0_joint" type="fixed">
-            <parent link="chassis_link" />
-            <child link="imu_0_link" />
+        <joint name="${tf_prefix}imu_0_joint" type="fixed">
+            <parent link="${tf_prefix}chassis_link" />
+            <child link="${tf_prefix}imu_0_link" />
             <origin xyz="${imu_offset_x} ${imu_offset_y} ${imu_offset_z}" rpy="0 0 0" />
         </joint>
-        <gazebo reference="imu_0_link">
+        <gazebo reference="${tf_prefix}imu_0_link">
             <sensor type="imu" name="imu_0">
                 <always_on>true</always_on>
@@ -260,8 +261,8 @@
         </gazebo>
         <!-- Mounting Hardpoints -->
-        <link name="default_mount" />
-        <joint name="default_mount_joint" type="fixed">
-            <parent link="riser_link" />
-            <child link="default_mount" />
+        <link name="${tf_prefix}default_mount" />
+        <joint name="${tf_prefix}default_mount_joint" type="fixed">
+            <parent link="${tf_prefix}riser_link" />
+            <child link="${tf_prefix}default_mount" />
             <origin xyz="0 0 ${riser_height + deck_thickness}" rpy="0 0 0" />
         </joint>
@@ -278,20 +279,20 @@
                 </xacro:unless>
             </hardware>
-            <joint name="front_left_wheel_joint">
+            <joint name="${tf_prefix}front_left_wheel_joint">
                 <command_interface name="velocity" />
                 <state_interface name="position" />
                 <state_interface name="velocity" />
             </joint>
-            <joint name="front_right_wheel_joint">
+            <joint name="${tf_prefix}front_right_wheel_joint">
                 <command_interface name="velocity" />
                 <state_interface name="position" />
                 <state_interface name="velocity" />
             </joint>
-            <joint name="rear_left_wheel_joint">
+            <joint name="${tf_prefix}rear_left_wheel_joint">
                 <command_interface name="velocity" />
                 <state_interface name="position" />
                 <state_interface name="velocity" />
             </joint>
-            <joint name="rear_right_wheel_joint">
+            <joint name="${tf_prefix}rear_right_wheel_joint">
                 <command_interface name="velocity" />
                 <state_interface name="position" />

File: phoebe_description/urdf/rocker.urdf.xacro (robot description, xacro)
@@ -2,6 +2,6 @@
 <robot xmlns:xacro="http://ros.org/wiki/xacro" name="r100_rocker">
   <xacro:include filename="$(find phoebe_description)/urdf/wheels/wheel.urdf.xacro" />
-  <xacro:macro name="r100_rocker" params="prefix joint_type location *joint_limits">
-    <link name="${prefix}_rocker_link">
+  <xacro:macro name="r100_rocker" params="prefix joint_type location tf_prefix *joint_limits">
+    <link name="${tf_prefix}${prefix}_rocker_link">
       <visual>
         <origin xyz="0 0 0" rpy="${math.pi/2} 0 ${math.pi/2}" />
@@ -20,15 +20,17 @@
       </inertial>
     </link>
-    <joint name="${prefix}_rocker" type="${joint_type}">
-      <parent link="axle_link" />
-      <child link="${prefix}_rocker_link" />
+    <joint name="${tf_prefix}${prefix}_rocker" type="${joint_type}">
+      <parent link="${tf_prefix}axle_link" />
+      <child link="${tf_prefix}${prefix}_rocker_link" />
       <origin xyz="${location*rocker_offset} 0 0" rpy="0 0 0" />
       <axis xyz="1 0 0" />
       <xacro:insert_block name="joint_limits" />
     </joint>
-    <xacro:r100_wheel parent="${prefix}_rocker_link" prefix="${prefix}_left" side="${-location}">
+    <xacro:r100_wheel parent="${tf_prefix}${prefix}_rocker_link" prefix="${prefix}_left"
+      side="${-location}" tf_prefix="${tf_prefix}">
       <origin xyz="0 ${rocker_width/2 + wheel_width/2} 0" rpy="0 0 0" />
     </xacro:r100_wheel>
-    <xacro:r100_wheel parent="${prefix}_rocker_link" prefix="${prefix}_right" side="${location}">
+    <xacro:r100_wheel parent="${tf_prefix}${prefix}_rocker_link" prefix="${prefix}_right"
+      side="${location}" tf_prefix="${tf_prefix}">
       <origin xyz="0 ${-(rocker_width/2 + wheel_width/2)} 0" rpy="0 0 0" />
     </xacro:r100_wheel>

File: phoebe_description/urdf/wheels/wheel.urdf.xacro (robot description, xacro)
@@ -2,6 +2,6 @@
 <robot xmlns:xacro="http://ros.org/wiki/xacro" xmlns:ignition="http://gazebosim.org/schema"
   name="r100_wheel">
-  <xacro:macro name="r100_wheel" params="parent prefix side *joint_pose">
-    <link name="${prefix}_wheel_link">
+  <xacro:macro name="r100_wheel" params="parent prefix side tf_prefix *joint_pose">
+    <link name="${tf_prefix}${prefix}_wheel_link">
       <visual>
         <origin xyz="0 0 0" rpy="${math.pi/2} 0 0" />
@@ -27,5 +27,5 @@
       </inertial>
     </link>
-    <gazebo reference="${prefix}_wheel_link">
+    <gazebo reference="${tf_prefix}${prefix}_wheel_link">
       <collision>
         <surface>
@@ -34,5 +34,5 @@
               <mu>1.0</mu>
               <mu2>0.0</mu2>
-              <fdir1 ignition:expressed_in="base_link">1 ${side} 0</fdir1>
+              <fdir1 ignition:expressed_in="${tf_prefix}base_link">1 ${side} 0</fdir1>
             </ode>
           </friction>
@@ -40,7 +40,7 @@
       </collision>
     </gazebo>
-    <joint name="${prefix}_wheel_joint" type="continuous">
+    <joint name="${tf_prefix}${prefix}_wheel_joint" type="continuous">
       <parent link="${parent}" />
-      <child link="${prefix}_wheel_link" />
+      <child link="${tf_prefix}${prefix}_wheel_link" />
       <xacro:insert_block name="joint_pose" />
       <axis xyz="0 1 0" />
