Commit message: adding a separate r100 urdf folder and making phoebe a macro itself

File: phoebe_description/urdf/phoebe.urdf.xacro (robot description, xacro)
@@ -3,7 +3,6 @@
     <xacro:arg name="tf_prefix" default="" />
     <xacro:arg name="ns" default="" />
-    <xacro:arg name="is_sim" default="false" />
+    <xacro:arg name="use_fake_hardware" default="false" />
     <xacro:arg name="sim_ignition" default="false" />
-    <xacro:arg name="use_fake_hardware" default="false" />
     <xacro:arg name="left_ewellix_com_port" default="/dev/ttyUSB0" />
     <xacro:arg name="right_ewellix_com_port" default="/dev/ttyUSB1" />
@@ -13,13 +12,7 @@
     <xacro:arg name="right_ur_kinematics_file" default="$(find ur_description)/config/ur5e/default_kinematics.yaml" />
     <!-- Includes -->
-    <xacro:include filename="$(find clearpath_platform_description)/urdf/common.urdf.xacro" />
-    <xacro:include filename="$(find phoebe_description)/urdf/r100.urdf.xacro" />
-    <xacro:r100
-        tf_prefix="$(arg tf_prefix)"
-        is_sim="$(arg is_sim)"
+    <xacro:include filename="$(find phoebe_description)/urdf/phoebe_macro.urdf.xacro" />
+    <xacro:phoebe
         ns="$(arg ns)"
-    />
-    <xacro:include filename="$(find phoebe_description)/urdf/jaco01_customization.urdf.xacro" />
-    <xacro:jaco01_customization
         tf_prefix="$(arg tf_prefix)"
         use_fake_hardware="$(arg is_sim)"

File: phoebe_description/urdf/phoebe_macro.urdf.xacro (robot description, xacro)
@@ -3,9 +3,10 @@
   <!-- Macro for phoebe customization -->
   <xacro:macro
-    name="jaco01_customization"
+    name="phoebe"
     params="
+      ns:=''
+      tf_prefix:=''
       use_fake_hardware:='false'
       sim_ignition:='false'
-      tf_prefix:=''
       left_ewellix_com_port:='/dev/ttyUSB0'
       right_ewellix_com_port:='/dev/ttyUSB1'
@@ -18,7 +19,12 @@
     "
   >
-  <material name="grey">
-    <color rgba="0.5 0.5 0.5 1"/>
-  </material>
+  <xacro:include filename="$(find clearpath_platform_description)/urdf/common.urdf.xacro" />
+  <xacro:include filename="$(find phoebe_description)/urdf/r100/r100.urdf.xacro" />
+  <xacro:r100
+      tf_prefix="${tf_prefix}"
+      use_fake_hardware="${use_fake_hardware}"
+      sim_ignition="${sim_ignition}"
+      ns="${ns}"
+  />
   <!-- Mounting rails for lifts -->
   <link name="${tf_prefix}lift_rails">
@@ -174,5 +180,5 @@
         <mesh filename="package://phoebe_description/meshes/visual/jaco01_meshes/ur_control_box.STL"/>
       </geometry>
-      <material name="grey" />
+      <material name="clearpath_aluminum" />
     </visual>
     <collision>
@@ -195,5 +201,5 @@
         <mesh filename="package://phoebe_description/meshes/visual/jaco01_meshes/ur_control_box.STL"/>
       </geometry>
-      <material name="grey" />
+      <material name="clearpath_aluminum" />
     </visual>
     <collision>
@@ -216,5 +222,5 @@
         <mesh filename="package://phoebe_description/meshes/visual/jaco01_meshes/scu.STL"/>
       </geometry>
-      <material name="grey" />
+      <material name="clearpath_aluminum" />
     </visual>
     <collision>
@@ -237,5 +243,5 @@
         <mesh filename="package://phoebe_description/meshes/visual/jaco01_meshes/scu.STL"/>
       </geometry>
-      <material name="grey" />
+      <material name="clearpath_aluminum" />
     </visual>
     <collision>
@@ -342,5 +348,5 @@
         <box size="0.2 0.2 0.015"/>
       </geometry>
-      <material name="grey"/>
+      <material name="clearpath_aluminum"/>
       <origin rpy="0 0 0" xyz="0 0 0.0075"/>
     </visual>
@@ -363,5 +369,5 @@
         <box size="0.2 0.2 0.015"/>
       </geometry>
-      <material name="grey"/>
+      <material name="clearpath_aluminum"/>
       <origin rpy="0 0 0" xyz="0 0 0.0075"/>
     </visual>

File: phoebe_description/urdf/r100/r100.urdf.xacro (robot description, xacro)
@@ -5,10 +5,11 @@
         params="wheel:='default'
                 tf_prefix
-                is_sim:=false
+                use_fake_hardware:=false
+                sim_ignition:=false
                 ns">
         <!-- Includes -->
         <xacro:include
-            filename="$(find phoebe_description)/urdf/wheels/wheel.urdf.xacro" ns="$(arg ns)" />
-        <xacro:include filename="$(find phoebe_description)/urdf/rocker.urdf.xacro" />
+            filename="$(find phoebe_description)/urdf/r100/wheels/wheel.urdf.xacro" ns="$(arg ns)" />
+        <xacro:include filename="$(find phoebe_description)/urdf/r100/rocker.urdf.xacro" />
         <xacro:arg name="gazebo_controllers"
             default="$(find phoebe_deploy)/config/${tf_prefix}control.yaml" />
@@ -269,37 +270,11 @@
         </joint>
         <!-- Gazebo Controller -->
-        <xacro:include filename="$(find phoebe_description)/urdf/gazebo.urdf.xacro"
-            ns="$(arg ns)" />
-        <!-- ROS2 controls -->
-        <ros2_control name="r100_hardware" type="system">
-            <hardware>
-                <xacro:if value="$(arg is_sim)">
-                    <plugin>ign_ros2_control/IgnitionSystem</plugin>
-                </xacro:if>
-                <xacro:unless value="$(arg is_sim)">
-                    <plugin>clearpath_platform/PumaHardware</plugin>
-                </xacro:unless>
-            </hardware>
-            <joint name="${tf_prefix}front_left_wheel_joint">
-                <command_interface name="velocity" />
-                <state_interface name="position" />
-                <state_interface name="velocity" />
-            </joint>
-            <joint name="${tf_prefix}front_right_wheel_joint">
-                <command_interface name="velocity" />
-                <state_interface name="position" />
-                <state_interface name="velocity" />
-            </joint>
-            <joint name="${tf_prefix}rear_left_wheel_joint">
-                <command_interface name="velocity" />
-                <state_interface name="position" />
-                <state_interface name="velocity" />
-            </joint>
-            <joint name="${tf_prefix}rear_right_wheel_joint">
-                <command_interface name="velocity" />
-                <state_interface name="position" />
-                <state_interface name="velocity" />
-            </joint>
-        </ros2_control>
+        <xacro:include filename="$(find phoebe_description)/urdf/r100/r100.ros2_control.xacro"/>
+        <xacro:r100_ros2_control
+          name="r100_ros2_control"
+          use_fake_hardware="${use_fake_hardware}"
+          sim_ignition="${sim_ignition}"
+          tf_prefix="${tf_prefix}"
+        />
     </xacro:macro>
 </robot>

File: phoebe_description/urdf/r100/rocker.urdf.xacro (robot description, xacro)
@@ -1,5 +1,5 @@
 <?xml version="1.0"?>
 <robot xmlns:xacro="http://ros.org/wiki/xacro" name="r100_rocker">
-  <xacro:include filename="$(find phoebe_description)/urdf/wheels/wheel.urdf.xacro" />
+  <xacro:include filename="$(find phoebe_description)/urdf/r100/wheels/wheel.urdf.xacro" />
   <xacro:macro name="r100_rocker" params="prefix joint_type location tf_prefix *joint_limits">
     <link name="${tf_prefix}${prefix}_rocker_link">

Commit message: adding lifkit calibration, and files for ur calibration

File: phoebe_description/urdf/phoebe.urdf.xacro (robot description, xacro)
@@ -13,4 +13,6 @@
     <xacro:arg name="left_ur_kinematics_file" default="$(find ur_description)/config/ur5e/default_kinematics.yaml" />
     <xacro:arg name="right_ur_kinematics_file" default="$(find ur_description)/config/ur5e/default_kinematics.yaml" />
+    <xacro:arg name="left_liftkit_calibration_file" default="$(find phoebe_description)/config/left_liftkit_calibration.yaml" />
+    <xacro:arg name="right_liftkit_calibration_file" default="$(find phoebe_description)/config/right_liftkit_calibration.yaml" />
     <!-- Includes -->
     <xacro:include filename="$(find phoebe_description)/urdf/phoebe_macro.xacro" />
@@ -28,4 +30,6 @@
         left_ur_kinematics_file="$(arg left_ur_kinematics_file)"
         right_ur_kinematics_file="$(arg right_ur_kinematics_file)"
+        left_liftkit_calibration_file="$(arg left_liftkit_calibration_file)"
+        right_liftkit_calibration_file="$(arg right_liftkit_calibration_file)"
     />
 </robot>

File: phoebe_description/urdf/phoebe_macro.xacro (robot description, xacro)
@@ -17,4 +17,6 @@
       left_ur_kinematics_file:='$(find ur_description)/config/ur5e/default_kinematics.yaml'
       right_ur_kinematics_file:='(find ur_description)/config/ur5e/default_kinematics.yaml'
+      left_liftkit_calibration_file:='$(find phoebe_description)/config/left_liftkit_calibration.yaml'
+      right_liftkit_calibration_file:='$(find phoebe_description)/config/right_liftkit_calibration.yaml'
     "
   >
@@ -388,4 +390,7 @@
   <xacro:include filename="$(find ewellix_liftkit_description)/urdf/ewellix_lift.xacro"/>
   <xacro:include filename="$(find ewellix_liftkit_description)/urdf/properties.xacro"/>
+  <!-- convert the arg into a property to be usable by the xacro -->
+  <xacro:property name="left_liftkit_calibration_file" value="$(arg left_liftkit_calibration_file)"/>
+  <xacro:property name="right_liftkit_calibration_file" value="$(arg right_liftkit_calibration_file)"/>
   <xacro:ewellix_lift
     name="${tf_prefix}left_ewellix"
@@ -398,4 +403,5 @@
     use_fake_hardware="${use_fake_hardware}"
     com_port="${left_ewellix_com_port}"
+    hw_calibration="${xacro.load_yaml(left_liftkit_calibration_file)}"
   >
     <origin xyz="0 0 ${0.0075+0.2457}" rpy="0 0 0"/>
@@ -411,4 +417,5 @@
     use_fake_hardware="${use_fake_hardware}"
     com_port="${right_ewellix_com_port}"
+    hw_calibration="${xacro.load_yaml(right_liftkit_calibration_file)}"
   >
     <origin xyz="0 0 ${0.0075+0.2457}" rpy="0 0 0"/>

Commit message: adding lifkit mount location calibration

File: phoebe_description/urdf/phoebe.urdf.xacro (robot description, xacro)
@@ -15,4 +15,5 @@
     <xacro:arg name="left_liftkit_calibration_file" default="$(find phoebe_description)/config/left_liftkit_calibration.yaml" />
     <xacro:arg name="right_liftkit_calibration_file" default="$(find phoebe_description)/config/right_liftkit_calibration.yaml" />
+    <xacro:arg name="liftkit_mount_calibration_file" default="$(find phoebe_description)/config/liftkit_mount_calibration.yaml" />
     <!-- Includes -->
     <xacro:include filename="$(find phoebe_description)/urdf/phoebe_macro.xacro" />
@@ -32,4 +33,5 @@
         left_liftkit_calibration_file="$(arg left_liftkit_calibration_file)"
         right_liftkit_calibration_file="$(arg right_liftkit_calibration_file)"
+        liftkit_mount_calibration_file="$(arg liftkit_mount_calibration_file)"
     />
 </robot>

File: phoebe_description/urdf/phoebe_macro.xacro (robot description, xacro)
@@ -19,4 +19,5 @@
       left_liftkit_calibration_file:='$(find phoebe_description)/config/left_liftkit_calibration.yaml'
       right_liftkit_calibration_file:='$(find phoebe_description)/config/right_liftkit_calibration.yaml'
+      liftkit_mount_calibration_file:='$(find phoebe_description)/config/liftkit_mount_calibration.yaml'
     "
   >
@@ -360,8 +361,14 @@
     </collision>
   </link>
+  <!-- load the liftkit mount calibration -->
+  <xacro:property name="liftkit_mount_calibration" value="${xacro.load_yaml(liftkit_mount_calibration_file)}"/>
+  <xacro:property name="left_edge_aligned_distance" value="${liftkit_mount_calibration['left_edge_aligned_distance']}"/>
+  <xacro:property name="right_edge_aligned_distance" value="${liftkit_mount_calibration['right_edge_aligned_distance']}"/>
+  <xacro:property name="left_liftkit_dist_from_edge" value="${liftkit_mount_calibration['left_liftkit_dist_from_edge']}"/>
+  <xacro:property name="right_liftkit_dist_from_edge" value="${liftkit_mount_calibration['right_liftkit_dist_from_edge']}"/>
   <joint name="${tf_prefix}left_ewellix_mount_flange_joint" type="fixed">
     <parent link="${tf_prefix}default_mount"/>
     <child link="${tf_prefix}left_ewellix_mount_flange_link"/>
-    <origin xyz="0 $(optenv LEFT_LIFT_Y 0.2) 0.04" rpy="0 0 0" />
+    <origin xyz="0 ${left_edge_aligned_distance-left_liftkit_dist_from_edge} 0.04" rpy="0 0 0" />
   </joint>
   <!-- Right Ewellix mounting flange -->
@@ -384,5 +391,5 @@
     <parent link="${tf_prefix}default_mount"/>
     <child link="${tf_prefix}right_ewellix_mount_flange_link"/>
-    <origin xyz="0 -$(optenv RIGHT_LIFT_Y 0.2) 0.04" rpy="0 0 0" />
+    <origin xyz="0 ${-right_edge_aligned_distance+right_liftkit_dist_from_edge} 0.04" rpy="0 0 0" />
   </joint>
 <!-- Ewellix lift column xacro -->

Commit message: ready to test calibration files

File: phoebe_description/urdf/phoebe.urdf.xacro (robot description, xacro)
@@ -5,4 +5,5 @@
     <xacro:arg name="use_fake_hardware" default="false" />
     <xacro:arg name="sim_ignition" default="false" />
+    <xacro:arg name="calibration_mode" default="false" />
     <xacro:arg name="left_ewellix_com_port" default="/dev/ewellix_left" />
     <xacro:arg name="right_ewellix_com_port" default="/dev/ewellix_right" />
@@ -23,4 +24,5 @@
         use_fake_hardware="$(arg use_fake_hardware)"
         sim_ignition="$(arg sim_ignition)"
+        calibration_mode="$(arg calibration_mode)"
         left_ewellix_com_port="$(arg left_ewellix_com_port)"
         right_ewellix_com_port="$(arg right_ewellix_com_port)"

File: phoebe_description/urdf/phoebe_macro.xacro (robot description, xacro)
@@ -9,4 +9,5 @@
       use_fake_hardware:='false'
       sim_ignition:='false'
+      calibration_mode:='false'
       left_ewellix_com_port:='/dev/ewellix_left'
       right_ewellix_com_port:='/dev/ewellix_right'
@@ -466,7 +467,21 @@
     <origin xyz="0 0 0" rpy="0 0 ${pi}" />
   </joint>
+  <!-- calibration links -->
+  <link name="${tf_prefix}left_arm_cal_link"> </link>
+  <joint name="${tf_prefix}left_arm_cal_joint" type="fixed">
+    <parent link="${tf_prefix}left_arm_mount_plate" />
+    <child link="${tf_prefix}left_arm_cal_link" />
+    <origin xyz="0 0 0" rpy="0 0 0"/>
+  </joint>
+  <link name="${tf_prefix}right_arm_cal_link"> </link>
+  <joint name="${tf_prefix}right_arm_cal_joint" type="fixed">
+    <parent link="${tf_prefix}right_arm_mount_plate" />
+    <child link="${tf_prefix}right_arm_cal_link" />
+    <origin xyz="0 0 0" rpy="0 0 0"/>
+  </joint>
+  <!-- end calibration links -->
   <link name="${tf_prefix}left_arm_mount_plate_2"> </link>
   <joint name="${tf_prefix}left_arm_mount_joint" type="fixed">
-    <parent link="${tf_prefix}left_arm_mount_plate" />
+    <parent link="${tf_prefix}left_arm_cal_link" />
     <child link="${tf_prefix}left_arm_mount_plate_2" />
     <origin xyz="0 0.01628 0.09117" rpy="-${pi/4} 0 0"/>
@@ -474,5 +489,5 @@
   <link name="${tf_prefix}right_arm_mount_plate_2"> </link>
   <joint name="${tf_prefix}right_arm_mount_joint" type="fixed">
-    <parent link="${tf_prefix}right_arm_mount_plate" />
+    <parent link="${tf_prefix}right_arm_cal_link" />
     <child link="${tf_prefix}right_arm_mount_plate_2" />
     <origin xyz="0 0.01628 0.09117" rpy="${pi/4} 0 ${pi}"/>
@@ -542,24 +557,66 @@
     <origin xyz="0 0 0.0" rpy="0 0 ${pi}"/>
   </xacro:ee_interface>
+  <!-- Calibration HW -->
+  <xacro:if value="${calibration_mode}">
+    <xacro:include filename="$(find phoebe_description)/urdf/calibration_interface.xacro"/>
+    <xacro:calibration_interface
+      tf_prefix="${tf_prefix}left_"
+      robot_parent="${tf_prefix}left_mtc_effector_side">
+      <origin xyz="0 0 0.024" rpy="0 0 ${pi}"/>
+    </xacro:calibration_interface>
+    <xacro:calibration_interface
+      tf_prefix="${tf_prefix}right_"
+      robot_parent="${tf_prefix}right_mtc_effector_side">
+      <origin xyz="0 0 0.024" rpy="0 0 ${pi}"/>
+    </xacro:calibration_interface>
+        <!-- calibration location-->
+    <link name="${tf_prefix}calibration_plate_target_side">
+      <visual>
+        <geometry>
+          <mesh filename="package://phoebe_description/meshes/visual/calibration/calibration_plate_target_side.stl" scale="0.0254 0.0254 0.0254"/>
+        </geometry>
+        <material name="clearpath_aluminum"/>
+      </visual>
+      <collision>
+        <geometry>
+          <mesh filename="package://phoebe_description/meshes/visual/calibration/calibration_plate_target_side.stl" scale="0.0254 0.0254 0.0254"/>
+        </geometry>
+      </collision>
+    </link>
+    <joint name="${tf_prefix}calibration_plate_target_joint_side" type="fixed">
+      <parent link="${tf_prefix}default_mount"/>
+      <child link="${tf_prefix}calibration_plate_target_side"/>
+      <origin xyz="0.4 0.0 0.22635" rpy="${pi} 0 ${-pi/2}" />
+    </joint>
+    <xacro:property name="cal_target_side_thickness" value="0.013335"/>
+    <joint name="${tf_prefix}calibration_face_target_side_joint" type="fixed">
+      <parent link="${tf_prefix}calibration_plate_target_side"/>
+      <child link="${tf_prefix}calibration_face_target_side"/>
+      <origin rpy="0 0 0" xyz="0 0 ${-1.0*cal_target_side_thickness}"/>
+    </joint>
+    <link name="${tf_prefix}calibration_face_target_side"/>
+  </xacro:if>
   <!-- Hand-E Grippers -->
-  <xacro:include filename="$(find dextivr_hande_description)/urdf/dextivr_hande.xacro"/>
-  <xacro:dextivr_hande
-    com_port="${right_hande_com_port}"
-    use_fake_hardware="${use_fake_hardware}"
-    name="${tf_prefix}right_dextivr_hande"
-    tf_prefix="${tf_prefix}right_"
-    parent="${tf_prefix}right_mtc_effector_side"
-    finger_xacro="fngr_original">
-    <origin xyz="0 0 0.024" rpy="0 0 ${pi}"/>
-  </xacro:dextivr_hande>
-  <xacro:dextivr_hande
-    com_port="${left_hande_com_port}"
-    use_fake_hardware="${use_fake_hardware}"
-    name="${tf_prefix}left_dextivr_hande"
-    tf_prefix="${tf_prefix}left_"
-    parent="${tf_prefix}left_mtc_effector_side"
-    finger_xacro="fngr_original">
-    <origin xyz="0 0 0.024" rpy="0 0 ${pi}"/>
-  </xacro:dextivr_hande>
+  <xacro:unless value="${calibration_mode}">
+    <xacro:include filename="$(find dextivr_hande_description)/urdf/dextivr_hande.xacro"/>
+    <xacro:dextivr_hande
+      com_port="${right_hande_com_port}"
+      use_fake_hardware="${use_fake_hardware}"
+      name="${tf_prefix}right_dextivr_hande"
+      tf_prefix="${tf_prefix}right_"
+      parent="${tf_prefix}right_mtc_effector_side"
+      finger_xacro="fngr_original">
+      <origin xyz="0 0 0.024" rpy="0 0 ${pi}"/>
+    </xacro:dextivr_hande>
+    <xacro:dextivr_hande
+      com_port="${left_hande_com_port}"
+      use_fake_hardware="${use_fake_hardware}"
+      name="${tf_prefix}left_dextivr_hande"
+      tf_prefix="${tf_prefix}left_"
+      parent="${tf_prefix}left_mtc_effector_side"
+      finger_xacro="fngr_original">
+      <origin xyz="0 0 0.024" rpy="0 0 ${pi}"/>
+    </xacro:dextivr_hande>
+  </xacro:unless>
   </xacro:macro>
 </robot>
