Commit message: almost working mujoco config

File: phoebe_description/urdf/phoebe.urdf.xacro (robot description, xacro)
@@ -17,4 +17,5 @@
     <xacro:arg name="right_liftkit_calibration_file" default="$(find phoebe_description)/config/right_liftkit_calibration.yaml" />
     <xacro:arg name="liftkit_mount_calibration_file" default="$(find phoebe_description)/config/liftkit_mount_calibration.yaml" />
+    <xacro:arg name="generate_ros2_control_tag" default="true" />
     <!-- Includes -->
     <xacro:include filename="$(find phoebe_description)/urdf/phoebe_macro.xacro" />
@@ -35,5 +36,5 @@
         left_liftkit_calibration_file="$(arg left_liftkit_calibration_file)"
         right_liftkit_calibration_file="$(arg right_liftkit_calibration_file)"
-        liftkit_mount_calibration_file="$(arg liftkit_mount_calibration_file)"
+        generate_ros2_control_tag="$(arg generate_ros2_control_tag)"
     />
 </robot>

File: phoebe_description/urdf/phoebe_macro.xacro (robot description, xacro)
@@ -17,8 +17,9 @@
       right_ur_ip_addr:='192.168.131.41'
       left_ur_kinematics_file:='$(find phoebe_description)/config/left_ur_calibration.yaml'
-      right_ur_kinematics_file:='(find phoebe_description)/config/right_ur_calibration.yaml'
+      right_ur_kinematics_file:='$(find phoebe_description)/config/right_ur_calibration.yaml'
       left_liftkit_calibration_file:='$(find phoebe_description)/config/left_liftkit_calibration.yaml'
       right_liftkit_calibration_file:='$(find phoebe_description)/config/right_liftkit_calibration.yaml'
       liftkit_mount_calibration_file:='$(find phoebe_description)/config/liftkit_mount_calibration.yaml'
+      generate_ros2_control_tag:='true'
     "
   >
@@ -30,4 +31,5 @@
       sim_ignition="${sim_ignition}"
       ns="${ns}"
+      generate_ros2_control_tag="${generate_ros2_control_tag}"
   />
   <!-- Mounting rails for lifts -->
@@ -179,5 +181,5 @@
   </joint>
   <!-- Rear UR Control Box -->
-  <link name="${tf_prefix}rear_ur_control_box">
+  <!-- <link name="${tf_prefix}rear_ur_control_box">
     <visual>
       <geometry>
@@ -190,5 +192,4 @@
       <geometry>
         <box size="0.199 0.502 0.195"/>
-        <!-- <mesh filename="package://phoebe_description/meshes/visual/jaco01_meshes/ur_control_box.STL"/> -->
       </geometry>
     </collision>
@@ -198,7 +199,7 @@
     <child link="${tf_prefix}rear_ur_control_box" />
     <origin xyz="-0.44274 0.13 0" rpy="0 0 0" />
-  </joint>
+  </joint> -->
   <!-- Front UR Control Box -->
-  <link name="${tf_prefix}front_ur_control_box">
+  <!-- <link name="${tf_prefix}front_ur_control_box">
     <visual>
       <geometry>
@@ -211,5 +212,4 @@
       <geometry>
         <box size="0.199 0.502 0.195"/>
-        <!-- <mesh filename="package://phoebe_description/meshes/visual/jaco01_meshes/ur_control_box.STL"/> -->
       </geometry>
     </collision>
@@ -219,5 +219,5 @@
     <child link="${tf_prefix}front_ur_control_box" />
     <origin xyz="0.44274 -0.13 0" rpy="0 0 ${pi}" />
-  </joint>
+  </joint> -->
   <!-- Rear Ewellix SCU -->
   <link name="${tf_prefix}rear_scu">
@@ -399,6 +399,6 @@
   <xacro:include filename="$(find ewellix_liftkit_description)/urdf/properties.xacro"/>
   <!-- convert the arg into a property to be usable by the xacro -->
-  <xacro:property name="left_liftkit_calibration_file" value="$(arg left_liftkit_calibration_file)"/>
-  <xacro:property name="right_liftkit_calibration_file" value="$(arg right_liftkit_calibration_file)"/>
+  <!-- <xacro:property name="left_liftkit_calibration_file" value="${left_liftkit_calibration_file}"/>
+  <xacro:property name="right_liftkit_calibration_file" value="${right_liftkit_calibration_file}"/> -->
   <xacro:ewellix_lift
     name="${tf_prefix}left_ewellix"
@@ -412,4 +412,5 @@
     com_port="${left_ewellix_com_port}"
     hw_calibration="${xacro.load_yaml(left_liftkit_calibration_file)}"
+    generate_ros2_control_tag="${generate_ros2_control_tag}"
   >
     <origin xyz="0 0 ${0.0075+0.2457}" rpy="0 0 0"/>
@@ -426,4 +427,5 @@
     com_port="${right_ewellix_com_port}"
     hw_calibration="${xacro.load_yaml(right_liftkit_calibration_file)}"
+    generate_ros2_control_tag="${generate_ros2_control_tag}"
   >
     <origin xyz="0 0 ${0.0075+0.2457}" rpy="0 0 0"/>
@@ -519,4 +521,5 @@
     input_recipe_filename="$(find ur_robot_driver)/resources/rtde_input_recipe.txt"
     output_recipe_filename="$(find ur_robot_driver)/resources/rtde_output_recipe.txt"
+    generate_ros2_control_tag="${generate_ros2_control_tag}"
     >
     <origin xyz="0 0 0" rpy="0 0 ${5*pi/4}" />
@@ -542,4 +545,5 @@
     input_recipe_filename="$(find ur_robot_driver)/resources/rtde_input_recipe.txt"
     output_recipe_filename="$(find ur_robot_driver)/resources/rtde_output_recipe.txt"
+    generate_ros2_control_tag="${generate_ros2_control_tag}"
     >
     <origin xyz="0 0 0" rpy="0 0 ${-pi/4}" /> <!-- TODO: need to integrate the OPTENV RIGEBACK_RIGHT_UR_XYZ stuff-->
@@ -606,5 +610,7 @@
       tf_prefix="${tf_prefix}right_"
       parent="${tf_prefix}right_ur_realsense_mount"
-      finger_xacro="fngr_original">
+      finger_xacro="fngr_original"
+      generate_ros2_control_tag="${generate_ros2_control_tag}"
+    >
       <origin xyz="0 0 0.008" rpy="0 0 ${pi}"/>
     </xacro:dextivr_hande>
@@ -615,5 +621,7 @@
       tf_prefix="${tf_prefix}left_"
       parent="${tf_prefix}left_ur_realsense_mount"
-      finger_xacro="fngr_original">
+      finger_xacro="fngr_original"
+      generate_ros2_control_tag="${generate_ros2_control_tag}"
+    >
       <origin xyz="0 0 0.008" rpy="0 0 ${pi}"/>
     </xacro:dextivr_hande>

File: phoebe_description/urdf/r100/r100_macro.xacro (robot description, xacro)
@@ -7,8 +7,9 @@
                 use_fake_hardware:=false
                 sim_ignition:=false
+                generate_ros2_control_tag:=true
                 ns">
         <!-- Includes -->
         <xacro:include
-            filename="$(find phoebe_description)/urdf/r100/wheels/wheel.urdf.xacro" ns="$(arg ns)" />
+            filename="$(find phoebe_description)/urdf/r100/wheels/wheel.urdf.xacro" ns="${ns}" />
         <xacro:include filename="$(find phoebe_description)/urdf/r100/rocker.urdf.xacro" />
         <xacro:arg name="gazebo_controllers"
@@ -270,11 +271,13 @@
         </joint>
         <!-- Gazebo Controller -->
-        <xacro:include filename="$(find phoebe_description)/urdf/r100/r100.ros2_control.xacro"/>
-        <xacro:r100_ros2_control
-          name="r100"
-          use_fake_hardware="${use_fake_hardware}"
-          sim_ignition="${sim_ignition}"
-          tf_prefix="${tf_prefix}"
-        />
+        <xacro:if value="${generate_ros2_control_tag}">
+            <xacro:include filename="$(find phoebe_description)/urdf/r100/r100.ros2_control.xacro"/>
+            <xacro:r100_ros2_control
+            name="r100"
+            use_fake_hardware="${use_fake_hardware}"
+            sim_ignition="${sim_ignition}"
+            tf_prefix="${tf_prefix}"
+            />
+        </xacro:if>
     </xacro:macro>
 </robot>

Commit message: Added launch and xacro argument for replacing the left Ewellix liftkit with the static pedestal. Modified urdf and xacro files accordingly.

File: phoebe_description/urdf/phoebe.urdf.xacro (robot description, xacro)
@@ -19,4 +19,5 @@
     <xacro:arg name="liftkit_mount_calibration_file" default="$(find phoebe_description)/config/liftkit_mount_calibration.yaml" />
     <xacro:arg name="generate_ros2_control_tag" default="true" />
+    <xacro:arg name="use_left_static_pedestal" default="false" />
     <!-- Includes -->
     <xacro:include filename="$(find phoebe_description)/urdf/phoebe_macro.xacro" />
@@ -39,4 +40,5 @@
         right_liftkit_calibration_file="$(arg right_liftkit_calibration_file)"
         generate_ros2_control_tag="$(arg generate_ros2_control_tag)"
+        use_left_static_pedestal="$(arg use_left_static_pedestal)"
     />
 </robot>

File: phoebe_description/urdf/phoebe_macro.xacro (robot description, xacro)
@@ -25,4 +25,5 @@
       add_grasp_push_frames:='true'
       use_camera_mesh:='true'
+      use_left_static_pedestal:='false'
     "
   >
@@ -392,30 +393,52 @@
   </joint>
   <!-- Left Ewellix mounting flange -->
-  <link name="${tf_prefix}left_ewellix_mount_flange_link">
-    <visual>
-      <geometry>
-        <box size="0.2 0.2 0.015"/>
-      </geometry>
-      <material name="clearpath_aluminum"/>
-      <origin rpy="0 0 0" xyz="0 0 0.0075"/>
-    </visual>
-    <collision>
-      <geometry>
-        <box size="0.2 0.2 0.015"/>
-      </geometry>
-      <origin rpy="0 0 0" xyz="0 0 0.0075"/>
-    </collision>
-  </link>
   <!-- load the liftkit mount calibration -->
-  <xacro:property name="liftkit_mount_calibration" value="${xacro.load_yaml(liftkit_mount_calibration_file)}"/>
-  <xacro:property name="left_edge_aligned_distance" value="${liftkit_mount_calibration['left_edge_aligned_distance']}"/>
-  <xacro:property name="right_edge_aligned_distance" value="${liftkit_mount_calibration['right_edge_aligned_distance']}"/>
-  <xacro:property name="left_liftkit_dist_from_edge" value="${liftkit_mount_calibration['left_liftkit_dist_from_edge']}"/>
-  <xacro:property name="right_liftkit_dist_from_edge" value="${liftkit_mount_calibration['right_liftkit_dist_from_edge']}"/>
-  <joint name="${tf_prefix}left_ewellix_mount_flange_joint" type="fixed">
-    <parent link="${tf_prefix}default_mount"/>
-    <child link="${tf_prefix}left_ewellix_mount_flange_link"/>
-    <origin xyz="0 ${left_edge_aligned_distance-left_liftkit_dist_from_edge} 0.04" rpy="0 0 0" />
-  </joint>
+    <xacro:property name="liftkit_mount_calibration" value="${xacro.load_yaml(liftkit_mount_calibration_file)}"/>
+    <xacro:property name="left_edge_aligned_distance" value="${liftkit_mount_calibration['left_edge_aligned_distance']}"/>
+    <xacro:property name="right_edge_aligned_distance" value="${liftkit_mount_calibration['right_edge_aligned_distance']}"/>
+    <xacro:property name="left_liftkit_dist_from_edge" value="${liftkit_mount_calibration['left_liftkit_dist_from_edge']}"/>
+    <xacro:property name="right_liftkit_dist_from_edge" value="${liftkit_mount_calibration['right_liftkit_dist_from_edge']}"/>
+  <xacro:unless value="${use_left_static_pedestal}">
+    <link name="${tf_prefix}left_ewellix_mount_flange_link">
+      <visual>
+        <geometry>
+          <box size="0.2 0.2 0.015"/>
+        </geometry>
+        <material name="clearpath_aluminum"/>
+        <origin rpy="0 0 0" xyz="0 0 0.0075"/>
+      </visual>
+      <collision>
+        <geometry>
+          <box size="0.2 0.2 0.015"/>
+        </geometry>
+        <origin rpy="0 0 0" xyz="0 0 0.0075"/>
+      </collision>
+    </link>
+    <joint name="${tf_prefix}left_ewellix_mount_flange_joint" type="fixed">
+      <parent link="${tf_prefix}default_mount"/>
+      <child link="${tf_prefix}left_ewellix_mount_flange_link"/>
+      <origin xyz="0 ${left_edge_aligned_distance-left_liftkit_dist_from_edge} 0.04" rpy="0 0 0" />
+    </joint>
+  </xacro:unless>
+  <xacro:if value="${use_left_static_pedestal}">
+    <link name="${tf_prefix}left_static_pedestal_link">
+      <visual>
+        <geometry>
+          <mesh filename="package://phoebe_description/meshes/visual/static_pedestal.stl" scale="0.0254 0.0254 0.0254"/>
+        </geometry>
+        <material name="clearpath_aluminum"/>
+      </visual>
+      <collision>
+        <geometry>
+          <mesh filename="package://phoebe_description/meshes/visual/static_pedestal.stl" scale="0.0254 0.0254 0.0254"/>
+        </geometry>
+      </collision>
+    </link>
+    <joint name="${tf_prefix}left_ewellix_pedestal_link_joint" type="fixed">
+      <parent link="${tf_prefix}default_mount"/>
+      <child link="${tf_prefix}left_static_pedestal_link"/>
+      <origin xyz="0 ${left_edge_aligned_distance-left_liftkit_dist_from_edge} 0.04" rpy="0 0 0" />
+    </joint>
+  </xacro:if>
   <!-- Right Ewellix mounting flange -->
   <link name="${tf_prefix}right_ewellix_mount_flange_link">
@@ -446,53 +469,83 @@
   <!-- <xacro:property name="left_liftkit_calibration_file" value="${left_liftkit_calibration_file}"/>
   <xacro:property name="right_liftkit_calibration_file" value="${right_liftkit_calibration_file}"/> -->
+  <xacro:unless value="${use_left_static_pedestal}">
+    <xacro:ewellix_lift
+      name="${tf_prefix}left_ewellix"
+      is_700="false"
+      is_500="true"
+      tf_prefix="${tf_prefix}left_"
+      parent="${tf_prefix}left_ewellix_mount_flange_link"
+      height_limit="0.5"
+      initial_value="0.26644069061695785"
+      omit_plates="true"
+      use_fake_hardware="${use_fake_hardware}"
+      com_port="${left_ewellix_com_port}"
+      generate_ros2_control_tag="${generate_ros2_control_tag}"
+    >
+      <origin xyz="0 0 ${0.0075+0.2457}" rpy="0 0 0"/>
+    </xacro:ewellix_lift>
+    <!-- Left arm mount plate -->
+    <link name="${tf_prefix}left_arm_mount_plate">
+      <visual>
+        <geometry>
+          <mesh filename="package://phoebe_description/meshes/visual/jaco01_meshes/arm_mount.STL"/>
+        </geometry>
+        <material name="clearpath_black" />
+      </visual>
+      <collision>
+        <geometry>
+          <mesh filename="package://phoebe_description/meshes/visual/jaco01_meshes/arm_mount_collision.STL"/>
+        </geometry>
+      </collision>
+    </link>
+    <joint name="${tf_prefix}left_arm_mount_plate_joint" type="fixed">
+      <parent link="${tf_prefix}left_ewellix_lift_tip_link" />
+      <child link="${tf_prefix}left_arm_mount_plate" />
+      <origin xyz="0 0 0" rpy="0 0 0" />
+    </joint>
+  </xacro:unless>
+  <xacro:if value="${use_left_static_pedestal}">
+     <link name="${tf_prefix}left_ewellix_lift_tip_link">
+     </link>
+     <joint name="${tf_prefix}ewellix_lift_tip_joint" type="fixed">
+      <parent link="${tf_prefix}left_static_pedestal_link"/>
+      <child link="${tf_prefix}left_ewellix_lift_tip_link"/>
+      <origin xyz="0 0 0.6096" rpy="0 0 0"/>
+    </joint>
+    <!-- Left arm mount plate -->
+    <link name="${tf_prefix}left_arm_mount_plate">
+      <visual>
+        <geometry>
+          <mesh filename="package://phoebe_description/meshes/visual/jaco01_meshes/arm_mount.STL"/>
+        </geometry>
+        <material name="clearpath_black" />
+      </visual>
+      <collision>
+        <geometry>
+          <mesh filename="package://phoebe_description/meshes/visual/jaco01_meshes/arm_mount_collision.STL"/>
+        </geometry>
+      </collision>
+    </link>
+    <joint name="${tf_prefix}left_arm_mount_plate_joint" type="fixed">
+      <parent link="${tf_prefix}left_ewellix_lift_tip_link" />
+      <child link="${tf_prefix}left_arm_mount_plate" />
+      <origin xyz="0 0 0" rpy="0 0 0" />
+    </joint>
+  </xacro:if>
   <xacro:ewellix_lift
-    name="${tf_prefix}left_ewellix"
-    is_700="false"
-    is_500="true"
-    tf_prefix="${tf_prefix}left_"
-    parent="${tf_prefix}left_ewellix_mount_flange_link"
-    height_limit="0.5"
-    initial_value="0.26644069061695785"
-    omit_plates="true"
-    use_fake_hardware="${use_fake_hardware}"
-    com_port="${left_ewellix_com_port}"
-    generate_ros2_control_tag="${generate_ros2_control_tag}"
-  >
-    <origin xyz="0 0 ${0.0075+0.2457}" rpy="0 0 0"/>
+      name="${tf_prefix}right_ewellix"
+      is_700="false"
+      is_500="true"
+      tf_prefix="${tf_prefix}right_"
+      parent="${tf_prefix}right_ewellix_mount_flange_link"
+      height_limit="0.5"
+      initial_value="0.259764889515653"
+      omit_plates="true"
+      use_fake_hardware="${use_fake_hardware}"
+      com_port="${right_ewellix_com_port}"
+      generate_ros2_control_tag="${generate_ros2_control_tag}"
+    >
+      <origin xyz="0 0 ${0.0075+0.2457}" rpy="0 0 0"/>
   </xacro:ewellix_lift>
-  <xacro:ewellix_lift
-    name="${tf_prefix}right_ewellix"
-    is_700="false"
-    is_500="true"
-    tf_prefix="${tf_prefix}right_"
-    parent="${tf_prefix}right_ewellix_mount_flange_link"
-    height_limit="0.5"
-    initial_value="0.259764889515653"
-    omit_plates="true"
-    use_fake_hardware="${use_fake_hardware}"
-    com_port="${right_ewellix_com_port}"
-    generate_ros2_control_tag="${generate_ros2_control_tag}"
-  >
-    <origin xyz="0 0 ${0.0075+0.2457}" rpy="0 0 0"/>
-  </xacro:ewellix_lift>
-  <!-- Left arm mount plate -->
-  <link name="${tf_prefix}left_arm_mount_plate">
-    <visual>
-      <geometry>
-        <mesh filename="package://phoebe_description/meshes/visual/jaco01_meshes/arm_mount.STL"/>
-      </geometry>
-      <material name="clearpath_black" />
-    </visual>
-    <collision>
-      <geometry>
-        <mesh filename="package://phoebe_description/meshes/visual/jaco01_meshes/arm_mount_collision.STL"/>
-      </geometry>
-    </collision>
-  </link>
-  <joint name="${tf_prefix}left_arm_mount_plate_joint" type="fixed">
-    <parent link="${tf_prefix}left_ewellix_lift_tip_link" />
-    <child link="${tf_prefix}left_arm_mount_plate" />
-    <origin xyz="0 0 0" rpy="0 0 0" />
-  </joint>
   <!-- Right arm mount plate -->
   <link name="${tf_prefix}right_arm_mount_plate">

Commit message: update urdf and options

File: phoebe_description/urdf/phoebe.urdf.xacro (robot description, xacro)
@@ -9,4 +9,6 @@
     <xacro:arg name="left_ewellix_com_port" default="/dev/ewellix_left" />
     <xacro:arg name="right_ewellix_com_port" default="/dev/ewellix_right" />
+    <xacro:arg name="left_hand_type" default="hande" />
+    <xacro:arg name="right_hand_type" default="hande" />
     <xacro:arg name="left_hande_com_port" default="/tmp/hande_left" />
     <xacro:arg name="right_hande_com_port" default="/tmp/hande_right" />
@@ -31,4 +33,6 @@
         left_ewellix_com_port="$(arg left_ewellix_com_port)"
         right_ewellix_com_port="$(arg right_ewellix_com_port)"
+        left_hand_type="$(arg left_hand_type)"
+        right_hand_type="$(arg right_hand_type)"
         left_hande_com_port="$(arg left_hande_com_port)"
         right_hande_com_port="$(arg right_hande_com_port)"

File: phoebe_description/urdf/phoebe_macro.xacro (robot description, xacro)
@@ -14,4 +14,6 @@
       left_ewellix_com_port:='/dev/ewellix_left'
       right_ewellix_com_port:='/dev/ewellix_right'
+      left_hand_type:='hande'
+      right_hand_type:='hande'
       left_hande_com_port:='/tmp/hande_left'
       right_hande_com_port:='/tmp/hande_right'
@@ -712,29 +714,58 @@
       <origin xyz="-6.4777232475001029e-02 1.1461581058038600e-04 1.2884814853441564e-02" rpy="-9.9487205554735336e-02 -1.4520756449714673e+00 1.0569277772629829e-01"/>
     </xacro:sensor_d435>
-    <!-- right gripper - 2F-85 -->
     <xacro:include filename="$(find phoebe_description)/urdf/robotiq_2f_85_macro.xacro"/>
-    <xacro:robotiq_2f_85
-      com_port="${right_hande_com_port}"
-      use_fake_hardware="${use_fake_hardware}"
-      name="${tf_prefix}right_dextivr_hande"
-      tf_prefix="${tf_prefix}right_"
-      parent="${tf_prefix}right_ur_realsense_mount"
-      generate_ros2_control_tag="${generate_ros2_control_tag}"
-      add_grasp_push_frames="${add_grasp_push_frames}">
-      <origin xyz="0 0 0.003" rpy="0 0 ${pi/2}"/>
-    </xacro:robotiq_2f_85>
-    <!-- Left gripper - Hand-E -->
     <xacro:include filename="$(find dextivr_hande_description)/urdf/dextivr_hande.xacro"/>
-    <xacro:dextivr_hande
-      com_port="${left_hande_com_port}"
-      use_fake_hardware="${use_fake_hardware}"
-      name="${tf_prefix}left_dextivr_hande"
-      tf_prefix="${tf_prefix}left_"
-      parent="${tf_prefix}left_ur_realsense_mount"
-      generate_ros2_control_tag="${generate_ros2_control_tag}"
-      add_grasp_push_frames="${add_grasp_push_frames}"
-      finger_xacro="fngr_original">
-      <origin xyz="0 0 0.003" rpy="0 0 ${pi/2}"/>
-    </xacro:dextivr_hande>
+    <!-- right hand - can be either hande or 2f85 -->
+    <xacro:if value="${right_hand_type == 'hande'}">
+        <xacro:dextivr_hande
+        com_port="${right_hande_com_port}"
+        use_fake_hardware="${use_fake_hardware}"
+        name="${tf_prefix}right_dextivr_hande"
+        tf_prefix="${tf_prefix}right_"
+        parent="${tf_prefix}right_ur_realsense_mount"
+        generate_ros2_control_tag="${generate_ros2_control_tag}"
+        add_grasp_push_frames="${add_grasp_push_frames}"
+        finger_xacro="fngr_original">
+        <origin xyz="0 0 0.003" rpy="0 0 ${pi/2}"/>
+      </xacro:dextivr_hande>
+    </xacro:if>
+    <xacro:if value="${right_hand_type == '2f85'}">
+      <xacro:robotiq_2f_85
+        com_port="${right_hande_com_port}"
+        use_fake_hardware="${use_fake_hardware}"
+        name="${tf_prefix}right_dextivr_hande"
+        tf_prefix="${tf_prefix}right_"
+        parent="${tf_prefix}right_ur_realsense_mount"
+        generate_ros2_control_tag="${generate_ros2_control_tag}"
+        add_grasp_push_frames="${add_grasp_push_frames}">
+        <origin xyz="0 0 0.003" rpy="0 0 ${pi/2}"/>
+      </xacro:robotiq_2f_85>
+    </xacro:if>
+    <!-- left hand - can be either hande or 2f85 -->
+    <xacro:if value="${left_hand_type == 'hande'}">
+      <xacro:dextivr_hande
+        com_port="${left_hande_com_port}"
+        use_fake_hardware="${use_fake_hardware}"
+        name="${tf_prefix}left_dextivr_hande"
+        tf_prefix="${tf_prefix}left_"
+        parent="${tf_prefix}left_ur_realsense_mount"
+        generate_ros2_control_tag="${generate_ros2_control_tag}"
+        add_grasp_push_frames="${add_grasp_push_frames}"
+        finger_xacro="fngr_original">
+        <origin xyz="0 0 0.003" rpy="0 0 ${pi/2}"/>
+      </xacro:dextivr_hande>
+    </xacro:if>
+    <xacro:if value="${left_hand_type == '2f85'}">
+      <xacro:robotiq_2f_85
+        com_port="${left_hande_com_port}"
+        use_fake_hardware="${use_fake_hardware}"
+        name="${tf_prefix}left_dextivr_hande"
+        tf_prefix="${tf_prefix}left_"
+        parent="${tf_prefix}left_ur_realsense_mount"
+        generate_ros2_control_tag="${generate_ros2_control_tag}"
+        add_grasp_push_frames="${add_grasp_push_frames}">
+        <origin xyz="0 0 0.003" rpy="0 0 ${pi/2}"/>
+      </xacro:robotiq_2f_85>
+    </xacro:if>
   </xacro:unless>
   <!-- Calibration HW -->
