Commit message: Fixes for launching Phoebe + WilbUR together

File: phoebe_description/urdf/calibration_interface.xacro (robot description, xacro)
@@ -17,5 +17,5 @@
           <mesh filename="package://phoebe_description/meshes/visual/calibration/calibration_plate_robot_side.stl" scale="0.0254 0.0254 0.0254"/>
         </geometry>
-        <material name="clearpath_aluminum"/>
+        <material name="phoebe_aluminum"/>
       </visual>
       <!-- collision -->

File: phoebe_description/urdf/phoebe_macro.xacro (robot description, xacro)
@@ -102,5 +102,5 @@
         <mesh filename="package://phoebe_description/meshes/visual/jaco01_meshes/lift_rails.STL"/>
       </geometry>
-      <material name="clearpath_black" />
+      <material name="phoebe_black" />
     </visual>
     <collision>
@@ -123,5 +123,5 @@
         <mesh filename="package://phoebe_description/meshes/visual/jaco01_meshes/shelf.STL"/>
       </geometry>
-      <material name="clearpath_black" />
+      <material name="phoebe_black" />
     </visual>
     <collision>
@@ -144,5 +144,5 @@
         <mesh filename="package://phoebe_description/meshes/visual/jaco01_meshes/shelf.STL"/>
       </geometry>
-      <material name="clearpath_black" />
+      <material name="phoebe_black" />
     </visual>
     <collision>
@@ -165,5 +165,5 @@
         <mesh filename="package://phoebe_description/meshes/visual/jaco01_meshes/monitor_hinge_base.STL"/>
       </geometry>
-      <material name="clearpath_black" />
+      <material name="phoebe_black" />
     </visual>
     <collision>
@@ -186,5 +186,5 @@
         <mesh filename="package://phoebe_description/meshes/visual/jaco01_meshes/monitor_hinge_top.STL"/>
       </geometry>
-      <material name="clearpath_black" />
+      <material name="phoebe_black" />
     </visual>
     <collision>
@@ -207,5 +207,5 @@
         <mesh filename="package://phoebe_description/meshes/visual/jaco01_meshes/monitor.STL"/>
       </geometry>
-      <material name="clearpath_black" />
+      <material name="phoebe_black" />
     </visual>
     <collision>
@@ -228,5 +228,5 @@
         <mesh filename="package://phoebe_description/meshes/visual/jaco01_meshes/monitor.STL"/>
       </geometry>
-      <material name="clearpath_black" />
+      <material name="phoebe_black" />
     </visual>
     <collision>
@@ -249,5 +249,5 @@
         <mesh filename="package://phoebe_description/meshes/visual/jaco01_meshes/ur_control_box.STL"/>
       </geometry>
-      <material name="clearpath_aluminum" />
+      <material name="phoebe_aluminum" />
     </visual>
     <collision>
@@ -269,5 +269,5 @@
         <mesh filename="package://phoebe_description/meshes/visual/jaco01_meshes/ur_control_box.STL"/>
       </geometry>
-      <material name="clearpath_aluminum" />
+      <material name="phoebe_aluminum" />
     </visual>
     <collision>
@@ -289,5 +289,5 @@
         <mesh filename="package://phoebe_description/meshes/visual/jaco01_meshes/scu.STL"/>
       </geometry>
-      <material name="clearpath_aluminum" />
+      <material name="phoebe_aluminum" />
     </visual>
     <collision>
@@ -310,5 +310,5 @@
         <mesh filename="package://phoebe_description/meshes/visual/jaco01_meshes/scu.STL"/>
       </geometry>
-      <material name="clearpath_aluminum" />
+      <material name="phoebe_aluminum" />
     </visual>
     <collision>
@@ -331,5 +331,5 @@
         <mesh filename="package://phoebe_description/meshes/visual/jaco01_meshes/autec_receiver.STL"/>
       </geometry>
-      <material name="clearpath_yellow" />
+      <material name="phoebe_yellow" />
     </visual>
     <collision>
@@ -352,5 +352,5 @@
         <mesh filename="package://phoebe_description/meshes/visual/jaco01_meshes/wifi_antenna.STL"/>
       </geometry>
-      <material name="clearpath_black" />
+      <material name="phoebe_black" />
     </visual>
     <collision>
@@ -373,5 +373,5 @@
         <mesh filename="package://phoebe_description/meshes/visual/jaco01_meshes/wifi_antenna.STL"/>
       </geometry>
-      <material name="clearpath_black" />
+      <material name="phoebe_black" />
     </visual>
     <collision>
@@ -394,5 +394,5 @@
         <mesh filename="package://phoebe_description/meshes/visual/jaco01_meshes/autec_antenna.STL"/>
       </geometry>
-      <material name="clearpath_black" />
+      <material name="phoebe_black" />
     </visual>
     <collision>
@@ -421,5 +421,5 @@
           <box size="0.2 0.2 0.015"/>
         </geometry>
-        <material name="clearpath_aluminum"/>
+        <material name="phoebe_aluminum"/>
         <origin rpy="0 0 0" xyz="0 0 0.0075"/>
       </visual>
@@ -443,5 +443,5 @@
           <mesh filename="package://phoebe_description/meshes/visual/static_pedestal_with_mount.stl" scale="0.0254 0.0254 0.0254"/>
         </geometry>
-        <material name="clearpath_aluminum"/>
+        <material name="phoebe_aluminum"/>
       </visual>
       <collision>
@@ -463,5 +463,5 @@
         <box size="0.2 0.2 0.015"/>
       </geometry>
-      <material name="clearpath_aluminum"/>
+      <material name="phoebe_aluminum"/>
       <origin rpy="0 0 0" xyz="0 0 0.0075"/>
     </visual>
@@ -507,5 +507,5 @@
           <mesh filename="package://phoebe_description/meshes/visual/jaco01_meshes/arm_mount.STL"/>
         </geometry>
-        <material name="clearpath_black" />
+        <material name="phoebe_black" />
       </visual>
       <collision>
@@ -535,5 +535,5 @@
           <mesh filename="package://phoebe_description/meshes/visual/jaco01_meshes/arm_mount_swivellink_new.stl" scale="0.0254 0.0254 0.0254"/>
         </geometry>
-        <material name="clearpath_black" />
+        <material name="phoebe_black" />
       </visual>
       <collision>
@@ -570,5 +570,5 @@
         <mesh filename="package://phoebe_description/meshes/visual/jaco01_meshes/arm_mount.STL"/>
       </geometry>
-      <material name="clearpath_black" />
+      <material name="phoebe_black" />
     </visual>
     <collision>
@@ -752,5 +752,6 @@
         parent="${tf_prefix}right_ur_realsense_mount"
         generate_ros2_control_tag="${generate_ros2_control_tag}"
-        add_grasp_push_frames="${add_grasp_push_frames}">
+        add_grasp_push_frames="${add_grasp_push_frames}"
+        sim_ignition="${sim_ignition}">
         <origin xyz="0 0 0.003" rpy="0 0 ${pi/2}"/>
       </xacro:robotiq_2f_85>
@@ -778,5 +779,6 @@
         parent="${tf_prefix}left_ur_realsense_mount"
         generate_ros2_control_tag="${generate_ros2_control_tag}"
-        add_grasp_push_frames="${add_grasp_push_frames}">
+        add_grasp_push_frames="${add_grasp_push_frames}"
+        sim_ignition="${sim_ignition}">
         <origin xyz="0 0 0.003" rpy="0 0 ${pi/2}"/>
       </xacro:robotiq_2f_85>
@@ -802,5 +804,5 @@
           <mesh filename="package://phoebe_description/meshes/visual/calibration/calibration_plate_target_side.stl" scale="0.0254 0.0254 0.0254"/>
         </geometry>
-        <material name="clearpath_aluminum"/>
+        <material name="phoebe_aluminum"/>
       </visual>
       <collision>

File: phoebe_description/urdf/r100/r100_macro.xacro (robot description, xacro)
@@ -58,5 +58,5 @@
                     <mesh filename="package://phoebe_description/meshes/visual/body.stl" />
                 </geometry>
-                <material name="clearpath_black" />
+                <material name="phoebe_black" />
             </visual>
             <collision>
@@ -92,5 +92,5 @@
                     <mesh filename="package://phoebe_description/meshes/visual/side-cover.stl" />
                 </geometry>
-                <material name="clearpath_yellow" />
+                <material name="phoebe_yellow" />
             </visual>
         </link>
@@ -101,5 +101,5 @@
                     <mesh filename="package://phoebe_description/meshes/visual/side-cover.stl" />
                 </geometry>
-                <material name="clearpath_yellow" />
+                <material name="phoebe_yellow" />
             </visual>
         </link>
@@ -115,5 +115,5 @@
                     <mesh filename="package://phoebe_description/meshes/visual/end-cover.stl" />
                 </geometry>
-                <material name="clearpath_black" />
+                <material name="phoebe_black" />
             </visual>
         </link>
@@ -129,5 +129,5 @@
                     <mesh filename="package://phoebe_description/meshes/visual/end-cover.stl" />
                 </geometry>
-                <material name="clearpath_black" />
+                <material name="phoebe_black" />
             </visual>
         </link>
@@ -149,5 +149,5 @@
                     <mesh filename="package://phoebe_description/meshes/visual/lights.stl" />
                 </geometry>
-                <material name="clearpath_white" />
+                <material name="phoebe_white" />
             </visual>
         </link>
@@ -158,5 +158,5 @@
                     <mesh filename="package://phoebe_description/meshes/visual/lights.stl" />
                 </geometry>
-                <material name="clearpath_black" />
+                <material name="phoebe_black" />
             </visual>
         </link>
@@ -173,5 +173,5 @@
                     <mesh filename="package://phoebe_description/meshes/visual/axle.stl" />
                 </geometry>
-                <material name="clearpath_black" />
+                <material name="phoebe_black" />
             </visual>
         </link>
@@ -188,5 +188,5 @@
                     <box size="0.493 0.493 ${riser_height}" />
                 </geometry>
-                <material name="clearpath_light_grey" />
+                <material name="phoebe_light_grey" />
             </visual>
             <collision>
@@ -209,5 +209,5 @@
                     <mesh filename="package://phoebe_description/meshes/visual/top.stl" />
                 </geometry>
-                <material name="clearpath_black" />
+                <material name="phoebe_black" />
             </visual>
             <collision>

File: phoebe_description/urdf/r100/rocker.urdf.xacro (robot description, xacro)
@@ -9,5 +9,5 @@
           <mesh filename="package://phoebe_description/meshes/visual/rocker.stl" />
         </geometry>
-        <material name="clearpath_black" />
+        <material name="phoebe_black" />
       </visual>
       <inertial>

File: phoebe_description/urdf/r100/wheels/wheel.urdf.xacro (robot description, xacro)
@@ -9,5 +9,5 @@
           <mesh filename="package://phoebe_description/meshes/visual/wheel.stl" />
         </geometry>
-        <material name="clearpath_black" />
+        <material name="phoebe_black" />
       </visual>
       <collision>

File: phoebe_description/urdf/robotiq_2f_85_macro.xacro (robot description, xacro)
@@ -11,5 +11,6 @@
     com_port:=/dev/ttyUSB1
     add_grasp_push_frames:=true
-    generate_ros2_control_tag:=true">
+    generate_ros2_control_tag:=true
+    sim_ignition:=false">
     <material name="${tf_prefix}black">
       <color rgba="0 0 0 1"/>

File: phoebe_mujoco_config/urdf/phoebe_mujoco_processed_inputs.xacro (robot description, xacro)
@@ -33,19 +33,19 @@
       <!-- elbow params, at least for the shoulder + elbow. The wrist joints are guess. -->
       <xacro:unless value="${use_left_static_pedestal}">
-        <modify_element type="joint" name="${tf_prefix}left_ewellix_lift_lower_to_higher" class="size5"/>
+        <modify_element type="joint" name="${tf_prefix}left_ewellix_lift_lower_to_higher" class="phoebe_size5"/>
       </xacro:unless>
-      <modify_element type="joint" name="${tf_prefix}left_ur_arm_shoulder_pan_joint" class="size3" damping="10.6" frictionloss="4.67" armature="1.44"/>
-      <modify_element type="joint" name="${tf_prefix}left_ur_arm_shoulder_lift_joint" class="size3" damping="10.6" frictionloss="4.67" armature="1.44"/>
-      <modify_element type="joint" name="${tf_prefix}left_ur_arm_elbow_joint" class="size3_limited" damping="10.6" frictionloss="4.67" armature="1.44"/>
-      <modify_element type="joint" name="${tf_prefix}left_ur_arm_wrist_1_joint" class="size1" damping="2.75" frictionloss="1.9" armature="0.21"/>
-      <modify_element type="joint" name="${tf_prefix}left_ur_arm_wrist_2_joint" class="size1" damping="2.1" frictionloss="1.85" armature="0.19"/>
-      <modify_element type="joint" name="${tf_prefix}left_ur_arm_wrist_3_joint" class="size1" damping="2.1" frictionloss="2.0" armature="0.17"/>
-      <modify_element type="joint" name="${tf_prefix}right_ewellix_lift_lower_to_higher" class="size5"/>
-      <modify_element type="joint" name="${tf_prefix}right_ur_arm_shoulder_pan_joint" class="size3" damping="10.6" frictionloss="4.67" armature="1.44"/>
-      <modify_element type="joint" name="${tf_prefix}right_ur_arm_shoulder_lift_joint" class="size3" damping="10.6" frictionloss="4.67" armature="1.44"/>
-      <modify_element type="joint" name="${tf_prefix}right_ur_arm_elbow_joint" class="size3_limited" damping="10.6" frictionloss="4.67" armature="1.44"/>
-      <modify_element type="joint" name="${tf_prefix}right_ur_arm_wrist_1_joint" class="size1" damping="2.75" frictionloss="1.9" armature="0.21"/>
-      <modify_element type="joint" name="${tf_prefix}right_ur_arm_wrist_2_joint" class="size1" damping="2.1" frictionloss="1.85" armature="0.19"/>
-      <modify_element type="joint" name="${tf_prefix}right_ur_arm_wrist_3_joint" class="size1" damping="2.1" frictionloss="2.0" armature="0.17"/>
+      <modify_element type="joint" name="${tf_prefix}left_ur_arm_shoulder_pan_joint" class="phoebe_size3" damping="10.6" frictionloss="4.67" armature="1.44"/>
+      <modify_element type="joint" name="${tf_prefix}left_ur_arm_shoulder_lift_joint" class="phoebe_size3" damping="10.6" frictionloss="4.67" armature="1.44"/>
+      <modify_element type="joint" name="${tf_prefix}left_ur_arm_elbow_joint" class="phoebe_size3_limited" damping="10.6" frictionloss="4.67" armature="1.44"/>
+      <modify_element type="joint" name="${tf_prefix}left_ur_arm_wrist_1_joint" class="phoebe_size1" damping="2.75" frictionloss="1.9" armature="0.21"/>
+      <modify_element type="joint" name="${tf_prefix}left_ur_arm_wrist_2_joint" class="phoebe_size1" damping="2.1" frictionloss="1.85" armature="0.19"/>
+      <modify_element type="joint" name="${tf_prefix}left_ur_arm_wrist_3_joint" class="phoebe_size1" damping="2.1" frictionloss="2.0" armature="0.17"/>
+      <modify_element type="joint" name="${tf_prefix}right_ewellix_lift_lower_to_higher" class="phoebe_size5"/>
+      <modify_element type="joint" name="${tf_prefix}right_ur_arm_shoulder_pan_joint" class="phoebe_size3" damping="10.6" frictionloss="4.67" armature="1.44"/>
+      <modify_element type="joint" name="${tf_prefix}right_ur_arm_shoulder_lift_joint" class="phoebe_size3" damping="10.6" frictionloss="4.67" armature="1.44"/>
+      <modify_element type="joint" name="${tf_prefix}right_ur_arm_elbow_joint" class="phoebe_size3_limited" damping="10.6" frictionloss="4.67" armature="1.44"/>
+      <modify_element type="joint" name="${tf_prefix}right_ur_arm_wrist_1_joint" class="phoebe_size1" damping="2.75" frictionloss="1.9" armature="0.21"/>
+      <modify_element type="joint" name="${tf_prefix}right_ur_arm_wrist_2_joint" class="phoebe_size1" damping="2.1" frictionloss="1.85" armature="0.19"/>
+      <modify_element type="joint" name="${tf_prefix}right_ur_arm_wrist_3_joint" class="phoebe_size1" damping="2.1" frictionloss="2.0" armature="0.17"/>
       <xacro:if value="${left_hand_type == 'hande'}">
         <modify_element type="joint" name="${tf_prefix}left_finger_1_joint" armature="0.5" frictionloss="5.0" />

File: phoebe_mujoco_config/urdf/phoebe_mujoco_raw_inputs.xacro (robot description, xacro)
@@ -16,24 +16,24 @@
             <material specular="0.5" shininess="0.25"/>
             <joint armature="0.1" actuatorgravcomp="true"/>
-            <default class="size5">
+            <default class="phoebe_size5">
                 <joint actuatorfrclimited="true" actuatorfrcrange="-1000 1000"/>
                 <position ctrlrange="0.0 0.7" kp="75000" dampratio="1.0" forcerange="-1000 1000"/>
             </default>
-            <default class="size4">
+            <default class="phoebe_size4">
                 <joint damping="10"/>
                 <general forcerange="-330 330" ctrlrange="-330 330"/>
             </default>
-            <default class="size3">
+            <default class="phoebe_size3">
                 <joint damping="5"/>
                 <general forcerange="-150 150" ctrlrange="-150 150"/>
-                <default class="size3_limited">
+                <default class="phoebe_size3_limited">
                     <joint range="-3.1415 3.1415"/>
                 </default>
             </default>
-            <default class="size2">
+            <default class="phoebe_size2">
                 <joint damping="2" />
                 <general forcerange="-56 56" ctrlrange="-56 56"/>
             </default>
-            <default class="size1">
+            <default class="phoebe_size1">
                 <joint damping="1" />
                 <general forcerange="-28 28" ctrlrange="-28 28"/>
@@ -73,19 +73,19 @@
         </xacro:if>
         <xacro:unless value="${use_left_static_pedestal}">
-            <position class="size5" name="${tf_prefix}left_ewellix_lift_lower_to_higher" joint="${tf_prefix}left_ewellix_lift_lower_to_higher"/>
+            <position class="phoebe_size5" name="${tf_prefix}left_ewellix_lift_lower_to_higher" joint="${tf_prefix}left_ewellix_lift_lower_to_higher"/>
         </xacro:unless>
-        <motor class="size3" name="${tf_prefix}left_ur_arm_shoulder_pan_joint" joint="${tf_prefix}left_ur_arm_shoulder_pan_joint"/>
-        <motor class="size3" name="${tf_prefix}left_ur_arm_shoulder_lift_joint" joint="${tf_prefix}left_ur_arm_shoulder_lift_joint"/>
-        <motor class="size3_limited" name="${tf_prefix}left_ur_arm_elbow_joint" joint="${tf_prefix}left_ur_arm_elbow_joint"/>
-        <motor class="size1" name="${tf_prefix}left_ur_arm_wrist_1_joint" joint="${tf_prefix}left_ur_arm_wrist_1_joint"/>
-        <motor class="size1" name="${tf_prefix}left_ur_arm_wrist_2_joint" joint="${tf_prefix}left_ur_arm_wrist_2_joint"/>
-        <motor class="size1" name="${tf_prefix}left_ur_arm_wrist_3_joint" joint="${tf_prefix}left_ur_arm_wrist_3_joint"/>
-        <position class="size5" name="${tf_prefix}right_ewellix_lift_lower_to_higher" joint="${tf_prefix}right_ewellix_lift_lower_to_higher"/>
-        <motor class="size3" name="${tf_prefix}right_ur_arm_shoulder_pan_joint" joint="${tf_prefix}right_ur_arm_shoulder_pan_joint"/>
-        <motor class="size3" name="${tf_prefix}right_ur_arm_shoulder_lift_joint" joint="${tf_prefix}right_ur_arm_shoulder_lift_joint"/>
-        <motor class="size3_limited" name="${tf_prefix}right_ur_arm_elbow_joint" joint="${tf_prefix}right_ur_arm_elbow_joint"/>
-        <motor class="size1" name="${tf_prefix}right_ur_arm_wrist_1_joint" joint="${tf_prefix}right_ur_arm_wrist_1_joint"/>
-        <motor class="size1" name="${tf_prefix}right_ur_arm_wrist_2_joint" joint="${tf_prefix}right_ur_arm_wrist_2_joint"/>
-        <motor class="size1" name="${tf_prefix}right_ur_arm_wrist_3_joint" joint="${tf_prefix}right_ur_arm_wrist_3_joint"/>
+        <motor class="phoebe_size3" name="${tf_prefix}left_ur_arm_shoulder_pan_joint" joint="${tf_prefix}left_ur_arm_shoulder_pan_joint"/>
+        <motor class="phoebe_size3" name="${tf_prefix}left_ur_arm_shoulder_lift_joint" joint="${tf_prefix}left_ur_arm_shoulder_lift_joint"/>
+        <motor class="phoebe_size3_limited" name="${tf_prefix}left_ur_arm_elbow_joint" joint="${tf_prefix}left_ur_arm_elbow_joint"/>
+        <motor class="phoebe_size1" name="${tf_prefix}left_ur_arm_wrist_1_joint" joint="${tf_prefix}left_ur_arm_wrist_1_joint"/>
+        <motor class="phoebe_size1" name="${tf_prefix}left_ur_arm_wrist_2_joint" joint="${tf_prefix}left_ur_arm_wrist_2_joint"/>
+        <motor class="phoebe_size1" name="${tf_prefix}left_ur_arm_wrist_3_joint" joint="${tf_prefix}left_ur_arm_wrist_3_joint"/>
+        <position class="phoebe_size5" name="${tf_prefix}right_ewellix_lift_lower_to_higher" joint="${tf_prefix}right_ewellix_lift_lower_to_higher"/>
+        <motor class="phoebe_size3" name="${tf_prefix}right_ur_arm_shoulder_pan_joint" joint="${tf_prefix}right_ur_arm_shoulder_pan_joint"/>
+        <motor class="phoebe_size3" name="${tf_prefix}right_ur_arm_shoulder_lift_joint" joint="${tf_prefix}right_ur_arm_shoulder_lift_joint"/>
+        <motor class="phoebe_size3_limited" name="${tf_prefix}right_ur_arm_elbow_joint" joint="${tf_prefix}right_ur_arm_elbow_joint"/>
+        <motor class="phoebe_size1" name="${tf_prefix}right_ur_arm_wrist_1_joint" joint="${tf_prefix}right_ur_arm_wrist_1_joint"/>
+        <motor class="phoebe_size1" name="${tf_prefix}right_ur_arm_wrist_2_joint" joint="${tf_prefix}right_ur_arm_wrist_2_joint"/>
+        <motor class="phoebe_size1" name="${tf_prefix}right_ur_arm_wrist_3_joint" joint="${tf_prefix}right_ur_arm_wrist_3_joint"/>
         <!-- Nominally include the wheels -->
         <xacro:unless value="${include_world_joints}">
