Commit message: initial working nav2, uses phobes odom smoother

File: phoebe_description/urdf/r100/r100_macro.xacro (robot description, xacro)
@@ -30,4 +30,7 @@
         <xacro:property name="imu_offset_y" value="-0.2902" />
         <xacro:property name="imu_offset_z" value="0.1681" />
+        <xacro:property name="lidar_offset_x" value="0.3" />
+        <xacro:property name="lidar_offset_y" value="0.0" />
+        <xacro:property name="lidar_offset_z" value="0.05" />
         <xacro:property name="dummy_inertia" value="1e-09" />
         <!-- Chassis -->
@@ -253,4 +256,17 @@
             <child link="${tf_prefix}imu_0_link" />
             <origin xyz="${imu_offset_x} ${imu_offset_y} ${imu_offset_z}" rpy="0 0 0" />
+        </joint>
+        <link name="${tf_prefix}lidar2d_0_laser">
+            <inertial>
+                <mass value="0.001" />
+                <origin xyz="0 0 0" rpy="0 0 0" />
+                <inertia ixx="${dummy_inertia}" ixy="0.0" ixz="0.0" iyy="${dummy_inertia}" iyz="0.0"
+                    izz="${dummy_inertia}" />
+            </inertial>
+        </link>
+        <joint name="${tf_prefix}lidar_2d_0_joint" type="fixed">
+            <parent link="${tf_prefix}default_mount" />
+            <child link="${tf_prefix}lidar2d_0_laser" />
+            <origin xyz="${lidar_offset_x} ${lidar_offset_y} ${lidar_offset_z}" rpy="0 0 0" />
         </joint>
         <gazebo reference="${tf_prefix}imu_0_link">

Commit message: fixing lidar location to be reasonable

File: phoebe_description/urdf/r100/r100_macro.xacro (robot description, xacro)
@@ -30,7 +30,8 @@
         <xacro:property name="imu_offset_y" value="-0.2902" />
         <xacro:property name="imu_offset_z" value="0.1681" />
-        <xacro:property name="lidar_offset_x" value="0.3" />
+        <!-- these values are not actually correct, but they are close enough to be useful -->
+        <xacro:property name="lidar_offset_x" value="0.4" />
         <xacro:property name="lidar_offset_y" value="0.0" />
-        <xacro:property name="lidar_offset_z" value="0.05" />
+        <xacro:property name="lidar_offset_z" value="-0.03" />
         <xacro:property name="dummy_inertia" value="1e-09" />
         <!-- Chassis -->

Commit message: fixing inertial properties on base link

File: phoebe_description/urdf/r100/r100_macro.xacro (robot description, xacro)
@@ -36,6 +36,15 @@
         <xacro:property name="lidar_offset_z" value="-0.03" />
         <xacro:property name="dummy_inertia" value="1e-09" />
-        <!-- Chassis -->
-        <link name="${tf_prefix}base_link"></link>
+        <!-- Chassis w dummy mass/inertia so mujoco converter processes properly -->
+        <link name="${tf_prefix}base_link">
+            <inertial>
+                <origin xyz="0 0 0" rpy="0 0 0" />
+                <mass value="0.01" />
+                <inertia
+                    ixx="1e-3" ixy="0.0" ixz="0.0"
+                    iyy="1e-3" iyz="0.0"
+                    izz="1e-3" />
+            </inertial>
+        </link>
         <joint name="${tf_prefix}base_link_joint" type="fixed">
             <origin xyz="0 0 0" rpy="0 0 0" />
