Commit message: Restructuring files. Renamed to imetro_mobile_environment. Rescaled cylinder mockup model files.

File: phoebe_description/urdf/imetro_mobile_environment/imetro_mobile_environment_colors.xacro (robot description, xacro)
@@ -2,14 +2,14 @@
 <robot xmlns:xacro="http://wiki.ros.org/xacro" name="phoebe_colors">
   <!-- ===================== MATERIALS/COLORS ===================== -->
-  <material name="phoebe_environment_black">
+  <material name="imetro_mobile_environment_black">
     <color rgba="0.1 0.1 0.1 1"/>
   </material>
-  <material name="phoebe_environment_blue">
+  <material name="imetro_mobile_environment_blue">
     <color rgba="0.1 0.1 0.3 1"/>
   </material>
-  <material name="phoebe_environment_brown">
+  <material name="imetro_mobile_environment_brown">
     <color rgba="0.42 0.22 0.16 1"/>
   </material>
-  <material name="phoebe_environment_gray">
+  <material name="imetro_mobile_environment_gray">
     <color rgba="0.7 0.7 0.7 1"/>
   </material>

File: phoebe_description/urdf/imetro_mobile_environment/imetro_mobile_environment_macro.xacro (robot description, xacro)
@@ -1,7 +1,7 @@
 <?xml version="1.0"?>
-<robot xmlns:xacro="http://wiki.ros.org/xacro" name="phoebe_environment">
-  <xacro:macro name="phoebe_environment" params="parent">
+<robot xmlns:xacro="http://wiki.ros.org/xacro" name="imetro_mobile_environment">
+  <xacro:macro name="imetro_mobile_environment" params="parent">
     <!-- Include color xacro -->
-    <xacro:include filename="$(find phoebe_description)/urdf/phoebe_environment_colors.xacro"/>
+    <xacro:include filename="$(find phoebe_description)/urdf/imetro_mobile_environment/imetro_mobile_environment_colors.xacro"/>
     <!-- ===================== BOOKSHELVES (CABINETS) ===================== -->
     <link name="bookshelves">
@@ -12,5 +12,5 @@
           <box size="3.0 0.5 1.5"/>
         </geometry>
-        <material name="phoebe_environment_black"/>
+        <material name="imetro_mobile_environment_black"/>
       </visual>
       <collision>
@@ -26,5 +26,5 @@
           <box size="3.0 0.5 1.5"/>
         </geometry>
-        <material name="phoebe_environment_black"/>
+        <material name="imetro_mobile_environment_black"/>
       </visual>
       <collision>
@@ -47,5 +47,5 @@
           <box size="0.666 1.332 0.666"/>
         </geometry>
-        <material name="phoebe_environment_blue"/>
+        <material name="imetro_mobile_environment_blue"/>
       </visual>
       <collision>
@@ -61,5 +61,5 @@
           <box size="0.666 0.666 0.666"/>
         </geometry>
-        <material name="phoebe_environment_blue"/>
+        <material name="imetro_mobile_environment_blue"/>
       </visual>
       <collision>
@@ -82,5 +82,5 @@
           <box size="0.666 1.332 0.666"/>
         </geometry>
-        <material name="phoebe_environment_brown"/>
+        <material name="imetro_mobile_environment_brown"/>
       </visual>
       <collision>
@@ -96,5 +96,5 @@
           <box size="0.666 1.332 0.666"/>
         </geometry>
-        <material name="phoebe_environment_brown"/>
+        <material name="imetro_mobile_environment_brown"/>
       </visual>
       <collision>
@@ -110,5 +110,5 @@
           <box size="0.666 2.5 0.666"/>
         </geometry>
-        <material name="phoebe_environment_brown"/>
+        <material name="imetro_mobile_environment_brown"/>
       </visual>
       <collision>
@@ -135,5 +135,5 @@
           <origin xyz="2.75 -0.666 0.665"/>
           <geometry>
-              <mesh filename="package://phoebe_description/meshes/visual/cylinder/cylinder_mockup_full_length.stl" scale="0.001 0.001 0.001"/>
+              <mesh filename="package://phoebe_description/meshes/visual/cylinder/cylinder_mockup_full_length_m.stl"/>
           </geometry>
        </collision>
@@ -146,9 +146,9 @@
     <link name="cylinder_jig">
       <visual>
-        <origin xyz="-2.1 -0.666 0.667" rpy="3.14 3.14 0"/>
+        <origin xyz="-2.1 -0.666 0.667" rpy="3.14 3.14 -1.57"/>
         <geometry>
-          <mesh filename="package://phoebe_description/meshes/visual/cylinder/cylinder_jig/cylinder_jig.stl" scale="0.001 0.001 0.001"/>
+          <mesh filename="package://phoebe_description/meshes/visual/cylinder/cylinder_jig/cylinder_jig_m.stl"/>
         </geometry>
-        <material name="phoebe_environment_black"/>
+        <material name="imetro_mobile_environment_black"/>
       </visual>
     </link>
