Commit message: Added origins.

File: phoebe_description/urdf/imetro_mobile_environment/imetro_mobile_environment.urdf.xacro (robot description, xacro)
@@ -4,4 +4,6 @@
   <xacro:include filename="$(find phoebe_description)/urdf/imetro_mobile_environment/imetro_mobile_environment_macro.xacro"/>
   <link name="world"/>
-  <xacro:imetro_mobile_environment parent="world"/>
+  <xacro:imetro_mobile_environment parent="world">
+    <origin xyz="0 0 0" rpy="0 0 0" />
+  </xacro:imetro_mobile_environment>
 </robot>

File: phoebe_description/urdf/imetro_mobile_environment/imetro_mobile_environment_macro.xacro (robot description, xacro)
@@ -1,5 +1,11 @@
 <?xml version="1.0"?>
 <robot xmlns:xacro="http://wiki.ros.org/xacro" name="imetro_mobile_environment">
-  <xacro:macro name="imetro_mobile_environment" params="parent">
+  <xacro:macro name="imetro_mobile_environment" params="parent *origin">
+  <link name="mobile_environment_base"/>
+  <joint name="mobile_environment_base_joint" type="fixed">
+    <parent link="${parent}"/>
+    <child link="mobile_environment_base"/>
+    <xacro:insert_block name="origin" />
+  </joint>
     <!-- Include color xacro -->
     <xacro:include filename="$(find phoebe_description)/urdf/imetro_mobile_environment/imetro_mobile_environment_colors.xacro"/>
@@ -8,5 +14,5 @@
       <!-- right shelf -->
       <visual>
-        <origin xyz="1.55 -2.25 0.75"/>
+        <origin xyz="1.55 0 0.75"/>
         <geometry>
           <box size="3.0 0.5 1.5"/>
@@ -15,5 +21,5 @@
       </visual>
       <collision>
-        <origin xyz="1.55 -2.25 0.75"/>
+        <origin xyz="1.55 0 0.75"/>
         <geometry>
           <box size="3.0 0.5 1.5"/>
@@ -22,5 +28,5 @@
       <!-- left shelf -->
       <visual>
-        <origin xyz="-1.55 -2.25 0.75"/>
+        <origin xyz="-1.55 0 0.75"/>
         <geometry>
           <box size="3.0 0.5 1.5"/>
@@ -29,5 +35,5 @@
       </visual>
       <collision>
-        <origin xyz="-1.55 -2.25 0.75"/>
+        <origin xyz="-1.55 0 0.75"/>
         <geometry>
           <box size="3.0 0.5 1.5"/>
@@ -36,12 +42,13 @@
     </link>
     <joint name="bookshelves_joint" type="fixed">
-      <parent link="${parent}"/>
-      <child link="bookshelves"/>
+      <parent link="mobile_environment_base"/>
+      <child link="bookshelves"/>
+      <origin xyz="0 -2.25 0"/>
     </joint>
     <!-- ===================== TABLES ===================== -->
-    <link name="tables">
-      <!-- pick table -->
+    <!-- pick table -->
+    <link name="pick_table">
       <visual>
-        <origin xyz="3.0 -0.666 0.333"/>
+        <origin xyz="0 0 0.333"/>
         <geometry>
           <box size="0.666 1.332 0.666"/>
@@ -50,12 +57,19 @@
       </visual>
       <collision>
-        <origin xyz="3.0 -0.666 0.333"/>
+        <origin xyz="0 0 0.333"/>
         <geometry>
           <box size="0.666 1.332 0.666"/>
         </geometry>
       </collision>
+    </link>
+    <joint name="pick_table_joint" type="fixed">
+      <parent link="mobile_environment_base"/>
+      <child link="pick_table"/>
+      <origin xyz="3.0 -0.666 0" rpy="0 0 0"/>
+    </joint>
       <!-- place table -->
+    <link name="place_table">
       <visual>
-        <origin xyz="-2.25 -0.666 0.333"/>
+        <origin xyz="0 0 0.333"/>
         <geometry>
           <box size="0.666 0.666 0.666"/>
@@ -64,5 +78,5 @@
       </visual>
       <collision>
-        <origin xyz="-2.25 -0.666 0.333"/>
+        <origin xyz="0 0 0.333"/>
         <geometry>
           <box size="0.666 0.666 0.666"/>
@@ -70,7 +84,8 @@
       </collision>
     </link>
-    <joint name="tables_joint" type="fixed">
-      <parent link="${parent}"/>
-      <child link="tables"/>
+    <joint name="place_table_joint" type="fixed">
+      <parent link="mobile_environment_base"/>
+      <child link="place_table"/>
+      <origin xyz="-2.25 -0.666 0" rpy="0 0 0"/>
     </joint>
     <!-- ===================== DESKS ===================== -->
@@ -78,5 +93,5 @@
       <!-- desk 1 -->
       <visual>
-        <origin xyz="3.0 1.0 0.333" rpy="0 0 0.523599"/>
+        <origin xyz="1.15 -1.0 0.333" rpy="0 0 0.523599"/>
         <geometry>
           <box size="0.666 1.332 0.666"/>
@@ -85,5 +100,5 @@
       </visual>
       <collision>
-        <origin xyz="3.0 1.0 0.333" rpy="0 0 0.523599"/>
+        <origin xyz="1.15 -1.0 0.333" rpy="0 0 0.523599"/>
         <geometry>
           <box size="0.666 1.332 0.666"/>
@@ -92,5 +107,5 @@
       <!-- desk 2 -->
       <visual>
-        <origin xyz="1.85 2.0 0.333" rpy="0 0 1.2"/>
+        <origin xyz="0 0 0.333" rpy="0 0 1.2"/>
         <geometry>
           <box size="0.666 1.332 0.666"/>
@@ -99,5 +114,5 @@
       </visual>
       <collision>
-        <origin xyz="1.85 2.0 0.333" rpy="0 0 1.2"/>
+        <origin xyz="0 0 0.333" rpy="0 0 1.2"/>
         <geometry>
           <box size="0.666 1.332 0.666"/>
@@ -106,5 +121,5 @@
       <!-- desk 3 -->
       <visual>
-        <origin xyz="-0.25 2.25 0.333" rpy="0 0 1.57"/>
+        <origin xyz="-2.1 0.25 0.333" rpy="0 0 1.57"/>
         <geometry>
           <box size="0.666 2.5 0.666"/>
@@ -113,5 +128,5 @@
       </visual>
       <collision>
-        <origin xyz="-0.25 2.25 0.333" rpy="0 0 1.57"/>
+        <origin xyz="-2.1 0.25 0.333" rpy="0 0 1.57"/>
         <geometry>
           <box size="0.666 2.5 0.666"/>
@@ -120,6 +135,7 @@
     </link>
     <joint name="desks_joint" type="fixed">
-      <parent link="${parent}"/>
-      <child link="desks"/>
+     <parent link="mobile_environment_base"/>
+      <child link="desks"/>
+      <origin xyz="1.85 2.0 0" rpy="0 0 0"/>
     </joint>
     <!-- ===================== CYLINDER ===================== -->
@@ -140,5 +156,5 @@
     </link>
     <joint name="cylinder_joint" type="fixed">
-      <parent link="${parent}"/>
+      <parent link="mobile_environment_base"/>
       <child link="cylinder"/>
     </joint>
@@ -154,5 +170,5 @@
     </link>
     <joint name="cylinder_jig_joint" type="fixed">
-      <parent link="${parent}"/>
+      <parent link="mobile_environment_base"/>
       <child link="cylinder_jig"/>
     </joint>
