Commit message: fixing space/tabs and fixing small cylinder issues

File: phoebe_description/urdf/imetro_mobile_environment/imetro_mobile_environment.urdf.xacro (robot description, xacro)
@@ -5,5 +5,5 @@
   <link name="world"/>
   <xacro:imetro_mobile_environment parent="world">
-    <origin xyz="0 0 0" rpy="0 0 0" />
+    <origin xyz="0 0 0" rpy="0 0 0" />
   </xacro:imetro_mobile_environment>
 </robot>

File: phoebe_description/urdf/imetro_mobile_environment/imetro_mobile_environment_macro.xacro (robot description, xacro)
@@ -3,9 +3,9 @@
   <xacro:macro name="imetro_mobile_environment" params="parent *origin">
   <link name="mobile_environment_base"/>
-  <joint name="mobile_environment_base_joint" type="fixed">
-    <parent link="${parent}"/>
-    <child link="mobile_environment_base"/>
-    <xacro:insert_block name="origin" />
-  </joint>
+  <joint name="mobile_environment_base_joint" type="fixed">
+    <parent link="${parent}"/>
+    <child link="mobile_environment_base"/>
+    <xacro:insert_block name="origin" />
+  </joint>
     <!-- Include color xacro -->
     <xacro:include filename="$(find phoebe_description)/urdf/imetro_mobile_environment/imetro_mobile_environment_colors.xacro"/>
@@ -43,6 +43,6 @@
     <joint name="bookshelves_joint" type="fixed">
       <parent link="mobile_environment_base"/>
-      <child link="bookshelves"/>
-      <origin xyz="0 -2.25 0"/>
+      <child link="bookshelves"/>
+      <origin xyz="0 -2.25 0"/>
     </joint>
     <!-- ===================== TABLES ===================== -->
@@ -136,6 +136,6 @@
     <joint name="desks_joint" type="fixed">
      <parent link="mobile_environment_base"/>
-      <child link="desks"/>
-      <origin xyz="1.85 2.0 0" rpy="0 0 0"/>
+      <child link="desks"/>
+      <origin xyz="1.85 2.0 0" rpy="0 0 0"/>
     </joint>
     <!-- ===================== CYLINDER ===================== -->
@@ -149,5 +149,5 @@
        </visual>
        <collision>
-          <origin xyz="2.75 -0.666 0.665"/>
+          <origin xyz="0 0 0"/>
           <geometry>
               <mesh filename="package://phoebe_description/meshes/visual/cylinder/cylinder_mockup_full_length_m.stl"/>
@@ -155,5 +155,5 @@
        </collision>
     </link>
-    <joint name="cylinder_joint" type="fixed">
+    <joint name="cylinder_joint" type="floating">
       <parent link="mobile_environment_base"/>
       <child link="cylinder"/>
@@ -183,8 +183,8 @@
   <link name="apriltag_0">
     <visual>
-      <geometry>
+      <geometry>
         <mesh filename="package://phoebe_description/meshes/visual/april_tags/AprilTag_0000.dae"/>
-      </geometry>
-      <material name="tag36h11-0">
+      </geometry>
+      <material name="tag36h11-0">
         <texture filename="package://phoebe_description/meshes/visual/april_tags/tag36_11_00000.png"/>
      </material>
@@ -198,8 +198,8 @@
   <link name="apriltag_4">
     <visual>
-      <geometry>
+      <geometry>
         <mesh filename="package://phoebe_description/meshes/visual/april_tags/AprilTag_0004.dae"/>
-      </geometry>
-      <material name="tag36h11-4">
+      </geometry>
+      <material name="tag36h11-4">
         <texture filename="package://phoebe_description/meshes/visual/april_tags/tag36_11_00004.png"/>
       </material>
