Commit message: Making joint names for the environment objects static.

File: phoebe_description/urdf/imetro_mobile_environment/imetro_mobile_environment_macro.xacro (robot description, xacro)
@@ -35,5 +35,5 @@
       </collision>
     </link>
-    <joint name="${parent}_to_bookshelves" type="fixed">
+    <joint name="bookshelves_joint" type="fixed">
       <parent link="${parent}"/>
       <child link="bookshelves"/>
@@ -70,5 +70,5 @@
       </collision>
     </link>
-    <joint name="${parent}_to_tables" type="fixed">
+    <joint name="tables_joint" type="fixed">
       <parent link="${parent}"/>
       <child link="tables"/>
@@ -119,5 +119,5 @@
       </collision>
     </link>
-    <joint name="${parent}_to_desks" type="fixed">
+    <joint name="desks_joint" type="fixed">
       <parent link="${parent}"/>
       <child link="desks"/>
@@ -139,5 +139,5 @@
        </collision>
     </link>
-    <joint name="${parent}_to_cylinder" type="fixed">
+    <joint name="cylinder_joint" type="fixed">
       <parent link="${parent}"/>
       <child link="cylinder"/>
@@ -153,5 +153,5 @@
       </visual>
     </link>
-    <joint name="${parent}_to_cylinder_jig" type="fixed">
+    <joint name="cylinder_jig_joint" type="fixed">
       <parent link="${parent}"/>
       <child link="cylinder_jig"/>

Commit message: Added april tags into environment URDF. Cleaned up URDF. Took out world bodies that are in the enviroment urdf out of the Mujoco scene urdf.

File: phoebe_description/urdf/imetro_mobile_environment/imetro_mobile_environment_macro.xacro (robot description, xacro)
@@ -142,7 +142,7 @@
     <link name="cylinder">
        <visual>
-          <origin xyz="2.75 -0.666 0.665"/>
+          <origin xyz="0 0 0"/>
           <geometry>
-              <mesh filename="package://phoebe_description/meshes/visual/cylinder/cylinder_mockup_full_length.stl" scale="0.001 0.001 0.001"/>
+              <mesh filename="package://phoebe_description/meshes/visual/cylinder/cylinder_mockup_full_length_m.stl"/>
           </geometry>
           <material name="cylinder_bottle_blue"/>
@@ -158,9 +158,10 @@
       <parent link="mobile_environment_base"/>
       <child link="cylinder"/>
-    </joint>
-    <!-- ===================== CYLINDER JIG ===================== -->
+      <origin xyz="2.75 -0.666 0.665" rpy="0 0 0"/>
+    </joint>
+    <!-- ===================== CYLINDER JIG + APRIL TAGS ===================== -->
     <link name="cylinder_jig">
       <visual>
-        <origin xyz="-2.1 -0.666 0.667" rpy="3.14 3.14 -1.57"/>
+        <origin xyz="0 0 0" rpy="0 0 0"/>
         <geometry>
           <mesh filename="package://phoebe_description/meshes/visual/cylinder/cylinder_jig/cylinder_jig_m.stl"/>
@@ -168,9 +169,61 @@
         <material name="imetro_mobile_environment_black"/>
       </visual>
+      <collision>
+        <origin xyz="0 0 0" rpy="0 0 0"/>
+        <geometry>
+          <mesh filename="package://phoebe_description/meshes/visual/cylinder/cylinder_jig/cylinder_jig_m.stl"/>
+        </geometry>
+      </collision>
     </link>
     <joint name="cylinder_jig_joint" type="fixed">
       <parent link="mobile_environment_base"/>
       <child link="cylinder_jig"/>
-    </joint>
+      <origin xyz="-2.1 -0.666 0.667" rpy="3.14 3.14 -1.57"/>
+    </joint>
+  <link name="apriltag_0">
+    <visual>
+      <origin xyz="-0.089 0 0.066" rpy="${1.57+0.53} ${0} ${1.57}"/>
+      <geometry>
+      <box size="0.073 0.073 0.002"/>
+      </geometry>
+    <material name="tag36h11-0">
+     <texture filename="package://phoebe_description/meshes/visual/april_tags/tag36_11_00000.png"/>
+    </material>
+   </visual>
+ </link>
+   <joint name="apriltag_0_joint" type="fixed">
+     <parent link="cylinder_jig"/>
+     <child link="apriltag_0"/>
+   </joint>
+  <link name="apriltag_4">
+    <visual>
+      <origin xyz="0 -0.089 0.066" rpy="${-0.523599+1.57} 0 0"/>
+      <geometry>
+      <box size="0.073 0.073 0.002"/>
+      </geometry>
+    <material name="tag36h11-4">
+     <texture filename="package://phoebe_description/meshes/visual/april_tags/tag36_11_00004.png"/>
+    </material>
+   </visual>
+ </link>
+   <joint name="apriltag_4_joint" type="fixed">
+     <parent link="cylinder_jig"/>
+     <child link="apriltag_4"/>
+   </joint>
+  <link name="apriltag_1">
+    <visual>
+      <origin xyz="0.134059 -1.788736 2.822666" rpy="-0.785 0 3.14159"/>
+      <geometry>
+        <box size="0.214 0.214 0.002"/>
+      </geometry>
+      <material name="tag36h11-1">
+        <texture filename="package://phoebe_description/meshes/visual/april_tags/tag36_11_00001.png"/>
+      </material>
+    </visual>
+  </link>
+   <joint name="apriltag_1_joint" type="fixed">
+    <parent link="mobile_environment_base"/>
+    <child link="apriltag_1"/>
+   </joint>
   </xacro:macro>
 </robot>

File: phoebe_mujoco_config/urdf/phoebe_mujoco_scene.xacro (robot description, xacro)
@@ -13,142 +13,16 @@
             <global azimuth="-120" elevation="-30" offwidth="1280" offheight="720"/>
         </visual>
-        <!-- this stuff will go away once Zarrin gets the environment urdf-ified -->
+        <!-- [In progress] this stuff will go away once Zarrin gets the environment urdf-ified -->
         <compiler angle="radian"/><!-- assetdir="assets" /> -->
-        <!-- <default>
-            <default class="cylinder_jig">
-            <geom group="3" type="mesh" condim="3" friction="0.01 0.005 0.0001" solimp="0.0 0.99 0.01 0.1 6" priority="2"/>
-            </default>
-        </default> -->
         <asset>
-            <!-- <texture type="2d" name="tag36_11_00000" file="tag36_11_00000.png"/>
-            <texture type="2d" name="tag36_11_00001" file="tag36_11_00001.png"/>
-            <texture type="2d" name="tag36_11_00004" file="tag36_11_00004.png"/>
-            <texture type="2d" name="tag36_11_00006" file="tag36_11_00006.png"/>
-            <material name="tag36h11-0" texture="tag36_11_00000" specular="0.5" shininess="0.25"/>
-            <material name="tag36h11-1" texture="tag36_11_00001" specular="0.5" shininess="0.25" texrepeat="-1 1"/>
-            <material name="tag36h11-4" texture="tag36_11_00004" specular="0.5" shininess="0.25"/>
-            <material name="tag36h11-6" texture="tag36_11_00006" specular="0.5" shininess="0.25"/> -->
             <texture type="skybox" builtin="gradient" rgb1="0.3 0.5 0.7" rgb2="0 0 0" width="512" height="3072"/>
-            <material name="cabinet_black" reflectance="0.2" rgba="0.1 0.1 0.1 1.0"/>
-            <material name="table_blue" reflectance="0.2" rgba="0.1 0.1 0.3 1.0"/>
-            <material name="desk_brown" reflectance="0.2" rgba="0.42 0.22 0.16 1.0"/>
             <texture type="2d" name="groundplane" builtin="checker" mark="edge" rgb1="0.8 0.8 0.8" rgb2="0.8 0.8 0.8"
             markrgb="0.5 0.5 0.5" width="300" height="300"/>
             <material name="groundplane" texture="groundplane" texuniform="true" texrepeat="3.0 3.0" reflectance="0.0"/>
-            <!-- <mesh name="cylinder" file="cylinder_mockup_full_length.stl" scale="0.001 0.001 0.001"/> -->
-            <!-- cylinder jig - decomposed bc convexity doesn't work well for it -->
-            <!-- <mesh file="cylinder_jig/cylinder_jig.obj" scale="0.001 0.001 0.001"/>
-            <mesh file="cylinder_jig/cylinder_jig_collision_0.obj" scale="0.001 0.001 0.001"/>
-            <mesh file="cylinder_jig/cylinder_jig_collision_1.obj" scale="0.001 0.001 0.001"/>
-            <mesh file="cylinder_jig/cylinder_jig_collision_2.obj" scale="0.001 0.001 0.001"/>
-            <mesh file="cylinder_jig/cylinder_jig_collision_3.obj" scale="0.001 0.001 0.001"/>
-            <mesh file="cylinder_jig/cylinder_jig_collision_4.obj" scale="0.001 0.001 0.001"/>
-            <mesh file="cylinder_jig/cylinder_jig_collision_5.obj" scale="0.001 0.001 0.001"/>
-            <mesh file="cylinder_jig/cylinder_jig_collision_6.obj" scale="0.001 0.001 0.001"/>
-            <mesh file="cylinder_jig/cylinder_jig_collision_7.obj" scale="0.001 0.001 0.001"/>
-            <mesh file="cylinder_jig/cylinder_jig_collision_8.obj" scale="0.001 0.001 0.001"/>
-            <mesh file="cylinder_jig/cylinder_jig_collision_9.obj" scale="0.001 0.001 0.001"/>
-            <mesh file="cylinder_jig/cylinder_jig_collision_10.obj" scale="0.001 0.001 0.001"/>
-            <mesh file="cylinder_jig/cylinder_jig_collision_11.obj" scale="0.001 0.001 0.001"/>
-            <mesh file="cylinder_jig/cylinder_jig_collision_12.obj" scale="0.001 0.001 0.001"/>
-            <mesh file="cylinder_jig/cylinder_jig_collision_13.obj" scale="0.001 0.001 0.001"/>
-            <mesh file="cylinder_jig/cylinder_jig_collision_14.obj" scale="0.001 0.001 0.001"/>
-            <mesh file="cylinder_jig/cylinder_jig_collision_15.obj" scale="0.001 0.001 0.001"/>
-            <mesh file="cylinder_jig/cylinder_jig_collision_16.obj" scale="0.001 0.001 0.001"/>
-            <mesh file="cylinder_jig/cylinder_jig_collision_17.obj" scale="0.001 0.001 0.001"/>
-            <mesh file="cylinder_jig/cylinder_jig_collision_18.obj" scale="0.001 0.001 0.001"/>
-            <mesh file="cylinder_jig/cylinder_jig_collision_19.obj" scale="0.001 0.001 0.001"/>
-            <mesh file="cylinder_jig/cylinder_jig_collision_20.obj" scale="0.001 0.001 0.001"/>
-            <mesh file="cylinder_jig/cylinder_jig_collision_21.obj" scale="0.001 0.001 0.001"/>
-            <mesh file="cylinder_jig/cylinder_jig_collision_22.obj" scale="0.001 0.001 0.001"/> -->
         </asset>
         <worldbody>
             <light pos="0 0 3" dir="0 0 -1" directional="true" castshadow="false"/>
+            <!-- Keeping the floor because the floor isn't defined in the URDF -->
             <geom name="floor" size="0 0 0.05" type="plane" material="groundplane"/>
-            <!-- left bookshelf -->
-            <geom size="1.5 0.25 0.75" pos="1.55 -2.25 0.75" quat="1 0 0 0" type="box" material="cabinet_black" class="visual"/>
-            <geom size="1.5 0.25 0.75" pos="1.55 -2.25 0.75" quat="1 0 0 0" type="box" class="collision"/>
-            <!-- right bookshelf -->
-            <geom size="1.5 0.25 0.75" pos="-1.55 -2.25 0.75" quat="1 0 0 0" type="box" material="cabinet_black" class="visual"/>
-            <geom size="1.5 0.25 0.75" pos="-1.55 -2.25 0.75" quat="1 0 0 0" type="box" class="collision"/>
-            <!-- pick table -->
-            <geom size="0.333 0.666 0.333" pos="3.0 -0.666 0.333" quat="1 0 0 0" type="box" material="table_blue" class="visual"/>
-            <geom size="0.333 0.666 0.333" pos="3.0 -0.666 0.333" quat="1 0 0 0" type="box" class="collision"/>
-            <!-- place table -->
-            <geom size="0.333 0.333 0.333" pos="-2.25 -0.666 0.333" quat="1 0 0 0" type="box" material="table_blue" class="visual"/>
-            <geom size="0.333 0.333 0.333" pos="-2.25 -0.666 0.333" quat="1 0 0 0" type="box" class="collision"/>
-            <!-- left operator desk -->
-            <geom size="0.333 0.666 0.333" pos="3.0 1.0 0.333" euler="0 0 0.523599" type="box" material="desk_brown" class="visual"/>
-            <geom size="0.333 0.666 0.333" pos="3.0 1.0 0.333" euler="0 0 0.523599" type="box" class="collision"/>
-            <!-- right operator desk -->
-            <geom size="0.333 0.666 0.333" pos="1.85 2.0 0.333" euler="0 0 1.2" type="box" material="desk_brown" class="visual"/>
-            <geom size="0.333 0.666 0.333" pos="1.85 2.0 0.333" euler="0 0 1.2" type="box" class="collision"/>
-            <!-- extra operator desks -->
-            <geom size="0.333 1.25 0.333" pos="-0.25 2.25 0.333" euler="0 0 1.57" type="box" material="desk_brown" class="visual"/>
-            <geom size="0.333 1.25 0.333" pos="-0.25 2.25 0.333" euler="0 0 1.57" type="box" class="collision"/>
-            <!-- <body name="cylinder" pos="2.75 -0.666 0.665">
-            <inertial pos="0 0 0.19" quat="1 0 0 0" mass="0.750" diaginertia="0.0005 0.0005 3e-5"/>
-            <joint name="free_joint" type="free"/>
-            <geom name="cylinder_vis" type="mesh" mesh="cylinder" rgba="1.0 0.1 0.1 1" class="visual"/>
-            <geom name="cylinder_col" type="mesh" mesh="cylinder" class="rubber"/>
-            </body> -->
-            <!-- <body name="cylinder_jig2" pos="0.8 2.2 1.1" euler="2.793 0 0">
-            <geom mesh="cylinder_jig" class="visual" rgba="0.1 0.1 0.1 1"/>
-            <geom mesh="cylinder_jig_collision_0" rgba="0.8900706191757303 0.9713592020957457 0.5780404029665048 1" class="cylinder_jig"/>
-            <geom mesh="cylinder_jig_collision_1" rgba="0.5545276775470052 0.47601813929328296 0.35862291685158143 1" class="cylinder_jig"/>
-            <geom mesh="cylinder_jig_collision_2" rgba="0.13197806700948966 0.6471947445059179 0.7095739691734154 1" class="cylinder_jig"/>
-            <geom mesh="cylinder_jig_collision_3" rgba="0.7327672247839327 0.06423444375100495 0.8043783305091261 1" class="cylinder_jig"/>
-            <geom mesh="cylinder_jig_collision_4" rgba="0.2021803460953837 0.8744426278588913 0.3386706933649809 1" class="cylinder_jig"/>
-            <geom mesh="cylinder_jig_collision_5" rgba="0.37872295514623133 0.6631442663595145 0.15468060498609038 1" class="cylinder_jig"/>
-            <geom mesh="cylinder_jig_collision_6" rgba="0.6679580209979851 0.3060642452647271 0.20193549290426838 1" class="cylinder_jig"/>
-            <geom mesh="cylinder_jig_collision_7" rgba="0.47177191206702973 0.6540724362279718 0.8740551402007518 1" class="cylinder_jig"/>
-            <geom mesh="cylinder_jig_collision_8" rgba="0.5899446431026785 0.6311655960711683 0.027869920889558975 1" class="cylinder_jig"/>
-            <geom mesh="cylinder_jig_collision_9" rgba="0.2591704408287576 0.6300630983154788 0.25980279876281087 1" class="cylinder_jig"/>
-            <geom  mesh="cylinder_jig_collision_10" rgba="0.6408079987631246 0.4613069677941516 0.8155322240665396 1" class="cylinder_jig"/>
-            <geom  mesh="cylinder_jig_collision_11" rgba="0.3962835623849993 0.19715408034338555 0.5191951688125966 1" class="cylinder_jig"/>
-            <geom  mesh="cylinder_jig_collision_12" rgba="0.13721703394572005 0.26619449837891695 0.7535914591211844 1" class="cylinder_jig"/>
-            <geom  mesh="cylinder_jig_collision_13" rgba="0.8013209941740281 0.623267868073114 0.5249186188051098 1" class="cylinder_jig"/>
-            <geom  mesh="cylinder_jig_collision_14" rgba="0.12000656712564839 0.24490833975705906 0.6437845642161399 1" class="cylinder_jig"/>
-            <geom  mesh="cylinder_jig_collision_15" rgba="0.6989912314637909 0.8834574961444431 0.2365143868062637 1" class="cylinder_jig"/>
-            <geom  mesh="cylinder_jig_collision_16" rgba="0.18990052529297574 0.5675369407151897 0.7895952869553159 1" class="cylinder_jig"/>
-            <geom  mesh="cylinder_jig_collision_17" rgba="0.40779119532224406 0.7556777891725958 0.49631518694962695 1" class="cylinder_jig"/>
-            <geom  mesh="cylinder_jig_collision_18" rgba="0.1863716966990977 0.5551044180319202 0.6785043125909683 1" class="cylinder_jig"/>
-            <geom  mesh="cylinder_jig_collision_19" rgba="0.048451371073279015 0.6758287766400523 0.4051556228153562 1" class="cylinder_jig"/>
-            <geom  mesh="cylinder_jig_collision_20" rgba="0.018782822474950556 0.15708435070778426 0.515621244371689 1" class="cylinder_jig"/>
-            <geom  mesh="cylinder_jig_collision_21" rgba="0.6460655150070409 0.42822465655561837 0.18481563322749284 1" class="cylinder_jig"/>
-            <geom  mesh="cylinder_jig_collision_22" rgba="0.7648716961996037 0.8822818672407353 0.1549012556710525 1" class="cylinder_jig"/>
-            <geom material="tag36h11-6" size="0.0365 0.0365 0.001" pos="0 0.175 0.12" euler="-1.57 0 0" type="box" class="visual"/>
-            <geom material="tag36h11-0" size="0.0365 0.0365 0.001" pos="-0.088 0.068 0" euler="-1.5707963 -1.0471975 -1.5707963" type="box" class="visual"/>
-            </body> -->
-            <!-- <body name="cylinder_jig" pos="-2.1 -0.666 0.667" euler="1.57 1.57 0">
-            <geom mesh="cylinder_jig" class="visual" rgba="0.1 0.1 0.1 1"/>
-            <geom mesh="cylinder_jig_collision_0" rgba="0.8900706191757303 0.9713592020957457 0.5780404029665048 1" class="cylinder_jig"/>
-            <geom mesh="cylinder_jig_collision_1" rgba="0.5545276775470052 0.47601813929328296 0.35862291685158143 1" class="cylinder_jig"/>
-            <geom mesh="cylinder_jig_collision_2" rgba="0.13197806700948966 0.6471947445059179 0.7095739691734154 1" class="cylinder_jig"/>
-            <geom mesh="cylinder_jig_collision_3" rgba="0.7327672247839327 0.06423444375100495 0.8043783305091261 1" class="cylinder_jig"/>
-            <geom mesh="cylinder_jig_collision_4" rgba="0.2021803460953837 0.8744426278588913 0.3386706933649809 1" class="cylinder_jig"/>
-            <geom mesh="cylinder_jig_collision_5" rgba="0.37872295514623133 0.6631442663595145 0.15468060498609038 1" class="cylinder_jig"/>
-            <geom mesh="cylinder_jig_collision_6" rgba="0.6679580209979851 0.3060642452647271 0.20193549290426838 1" class="cylinder_jig"/>
-            <geom mesh="cylinder_jig_collision_7" rgba="0.47177191206702973 0.6540724362279718 0.8740551402007518 1" class="cylinder_jig"/>
-            <geom mesh="cylinder_jig_collision_8" rgba="0.5899446431026785 0.6311655960711683 0.027869920889558975 1" class="cylinder_jig"/>
-            <geom mesh="cylinder_jig_collision_9" rgba="0.2591704408287576 0.6300630983154788 0.25980279876281087 1" class="cylinder_jig"/>
-            <geom  mesh="cylinder_jig_collision_10" rgba="0.6408079987631246 0.4613069677941516 0.8155322240665396 1" class="cylinder_jig"/>
-            <geom  mesh="cylinder_jig_collision_11" rgba="0.3962835623849993 0.19715408034338555 0.5191951688125966 1" class="cylinder_jig"/>
-            <geom  mesh="cylinder_jig_collision_12" rgba="0.13721703394572005 0.26619449837891695 0.7535914591211844 1" class="cylinder_jig"/>
-            <geom  mesh="cylinder_jig_collision_13" rgba="0.8013209941740281 0.623267868073114 0.5249186188051098 1" class="cylinder_jig"/>
-            <geom  mesh="cylinder_jig_collision_14" rgba="0.12000656712564839 0.24490833975705906 0.6437845642161399 1" class="cylinder_jig"/>
-            <geom  mesh="cylinder_jig_collision_15" rgba="0.6989912314637909 0.8834574961444431 0.2365143868062637 1" class="cylinder_jig"/>
-            <geom  mesh="cylinder_jig_collision_16" rgba="0.18990052529297574 0.5675369407151897 0.7895952869553159 1" class="cylinder_jig"/>
-            <geom  mesh="cylinder_jig_collision_17" rgba="0.40779119532224406 0.7556777891725958 0.49631518694962695 1" class="cylinder_jig"/>
-            <geom  mesh="cylinder_jig_collision_18" rgba="0.1863716966990977 0.5551044180319202 0.6785043125909683 1" class="cylinder_jig"/>
-            <geom  mesh="cylinder_jig_collision_19" rgba="0.048451371073279015 0.6758287766400523 0.4051556228153562 1" class="cylinder_jig"/>
-            <geom  mesh="cylinder_jig_collision_20" rgba="0.018782822474950556 0.15708435070778426 0.515621244371689 1" class="cylinder_jig"/>
-            <geom  mesh="cylinder_jig_collision_21" rgba="0.6460655150070409 0.42822465655561837 0.18481563322749284 1" class="cylinder_jig"/>
-            <geom  mesh="cylinder_jig_collision_22" rgba="0.7648716961996037 0.8822818672407353 0.1549012556710525 1" class="cylinder_jig"/>
-            <geom material="tag36h11-4" size="0.0365 0.0365 0.001" pos="0 0.068 0.088" euler="-0.523599 0 0" type="box" class="visual"/>
-            <geom material="tag36h11-0" size="0.0365 0.0365 0.001" pos="-0.088 0.068 0" euler="-1.5707963 -1.0471975 -1.5707963" type="box" class="visual"/>
-            </body> -->
-            <!-- april tag -->
-            <!-- <geom material="tag36h11-1" size="0.107 0.107 0.001" pos="0.134059 -1.788736 2.822666" euler="0.785 0 3.14159" type="box" class="visual"/> -->
         </worldbody>
     </scene>

Commit message: Preliminary edits to get Mujoco urdf conversion working for the environment.

File: phoebe_description/urdf/imetro_mobile_environment/imetro_mobile_environment_macro.xacro (robot description, xacro)
@@ -183,4 +183,5 @@
   <link name="apriltag_0">
     <visual>
+     <!-- pos="-0.088 0.068 0" euler="-1.5707963 -1.0471975 -1.5707963"  -->
       <origin xyz="-0.089 0 0.066" rpy="${1.57+0.53} ${0} ${1.57}"/>
       <geometry>
@@ -211,7 +212,7 @@
      <child link="apriltag_4"/>
    </joint>
+   <!-- ===================== WORLD APRIL TAG ===================== -->
   <link name="apriltag_1">
     <visual>
-      <origin xyz="0.134059 -1.788736 2.822666" rpy="-0.785 0 3.14159"/>
       <geometry>
         <box size="0.214 0.214 0.002"/>
@@ -225,4 +226,5 @@
     <parent link="mobile_environment_base"/>
     <child link="apriltag_1"/>
+    <origin xyz="0.134059 -1.788736 2.822666" rpy="-0.785 0 3.14159"/>
    </joint>
   </xacro:macro>

File: phoebe_description/urdf/phoebe_macro.xacro (robot description, xacro)
@@ -9,4 +9,5 @@
       use_fake_hardware:='false'
       sim_ignition:='false'
+      parent:='world'
       include_world_joints:='false'
       calibration_mode:='false'

File: phoebe_mujoco_config/urdf/phoebe_mujoco_xacro.urdf (robot description, URDF)
Before this commit: robot phoebe, 1 links, 0 joints
Joints:
- added joint floating_base_joint: type floating, parent world, child base_link

Commit message: Added .dae files for the april tags so they translate to Mujoco. Implementation needs work.

File: phoebe_description/urdf/imetro_mobile_environment/imetro_mobile_environment_macro.xacro (robot description, xacro)
@@ -187,4 +187,5 @@
       <geometry>
       <box size="0.073 0.073 0.002"/>
+          <!-- <mesh filename="package://phoebe_description/meshes/visual/april_tags/AprilTag_000.dae"/> -->
       </geometry>
     <material name="tag36h11-0">
@@ -202,4 +203,5 @@
       <geometry>
       <box size="0.073 0.073 0.002"/>
+        <!-- <mesh filename="package://phoebe_description/meshes/visual/april_tags/AprilTag_004.dae"/> -->
       </geometry>
     <material name="tag36h11-4">
@@ -217,4 +219,5 @@
       <geometry>
         <box size="0.214 0.214 0.002"/>
+        <!-- <mesh filename="package://phoebe_description/meshes/visual/april_tags/AprilTag_001.dae"/> -->
       </geometry>
       <material name="tag36h11-1">
