Commit message: Brought in .dae mesh files for the april tags and adjusted orientation of them in the urdf. Now the april tags translate to Mujoco.

File: phoebe_description/urdf/imetro_mobile_environment/imetro_mobile_environment_macro.xacro (robot description, xacro)
@@ -184,8 +184,8 @@
     <visual>
      <!-- pos="-0.088 0.068 0" euler="-1.5707963 -1.0471975 -1.5707963"  -->
-      <origin xyz="-0.089 0 0.066" rpy="${1.57+0.53} ${0} ${1.57}"/>
+      <origin xyz="-0.089 0 0.066" rpy="0 0.52360 0"/>
       <geometry>
-      <box size="0.073 0.073 0.002"/>
-          <!-- <mesh filename="package://phoebe_description/meshes/visual/april_tags/AprilTag_000.dae"/> -->
+ <!--      <box size="0.073 0.073 0.002"/> -->
+          <mesh filename="package://phoebe_description/meshes/visual/april_tags/AprilTag_0000.dae"/>
       </geometry>
     <material name="tag36h11-0">
@@ -200,8 +200,8 @@
   <link name="apriltag_4">
     <visual>
-      <origin xyz="0 -0.089 0.066" rpy="${-0.523599+1.57} 0 0"/>
+      <origin xyz="0 -0.089 0.066" rpy="0 0.52360 1.57"/>
       <geometry>
-      <box size="0.073 0.073 0.002"/>
-        <!-- <mesh filename="package://phoebe_description/meshes/visual/april_tags/AprilTag_004.dae"/> -->
+ <!--      <box size="0.073 0.073 0.002"/> -->
+        <mesh filename="package://phoebe_description/meshes/visual/april_tags/AprilTag_0004.dae"/>
       </geometry>
     <material name="tag36h11-4">
@@ -218,6 +218,6 @@
     <visual>
       <geometry>
-        <box size="0.214 0.214 0.002"/>
-        <!-- <mesh filename="package://phoebe_description/meshes/visual/april_tags/AprilTag_001.dae"/> -->
+        <!-- <box size="0.214 0.214 0.002"/> -->
+        <mesh filename="package://phoebe_description/meshes/visual/april_tags/AprilTag_0001.dae"/>
       </geometry>
       <material name="tag36h11-1">
@@ -229,5 +229,5 @@
     <parent link="mobile_environment_base"/>
     <child link="apriltag_1"/>
-    <origin xyz="0.134059 -1.788736 2.822666" rpy="-0.785 0 3.14159"/>
+    <origin xyz="0.134059 -1.788736 2.822666" rpy="-3.14159 0.52360 1.57"/>
    </joint>
   </xacro:macro>

Commit message: General clean up and pre commit fixed.

File: phoebe_description/urdf/imetro_mobile_environment/imetro_mobile_environment_macro.xacro (robot description, xacro)
@@ -184,7 +184,6 @@
     <visual>
      <!-- pos="-0.088 0.068 0" euler="-1.5707963 -1.0471975 -1.5707963"  -->
-      <origin xyz="-0.089 0 0.066" rpy="0 0.52360 0"/>
       <geometry>
- <!--      <box size="0.073 0.073 0.002"/> -->
+          <!--<box size="0.073 0.073 0.002"/> -->
           <mesh filename="package://phoebe_description/meshes/visual/april_tags/AprilTag_0000.dae"/>
       </geometry>
@@ -197,10 +196,10 @@
      <parent link="cylinder_jig"/>
      <child link="apriltag_0"/>
+     <origin xyz="-0.089 0 0.066" rpy="0 0.52360 0"/>
    </joint>
   <link name="apriltag_4">
     <visual>
-      <origin xyz="0 -0.089 0.066" rpy="0 0.52360 1.57"/>
       <geometry>
- <!--      <box size="0.073 0.073 0.002"/> -->
+        <!--<box size="0.073 0.073 0.002"/> -->
         <mesh filename="package://phoebe_description/meshes/visual/april_tags/AprilTag_0004.dae"/>
       </geometry>
@@ -213,4 +212,5 @@
      <parent link="cylinder_jig"/>
      <child link="apriltag_4"/>
+     <origin xyz="0 -0.089 0.066" rpy="0 0.52360 1.57"/>
    </joint>
    <!-- ===================== WORLD APRIL TAG ===================== -->

Commit message: Formatting + cleaned up obselete comments.

File: phoebe_description/urdf/imetro_mobile_environment/imetro_mobile_environment_macro.xacro (robot description, xacro)
@@ -183,13 +183,11 @@
   <link name="apriltag_0">
     <visual>
-     <!-- pos="-0.088 0.068 0" euler="-1.5707963 -1.0471975 -1.5707963"  -->
       <geometry>
-          <!--<box size="0.073 0.073 0.002"/> -->
-          <mesh filename="package://phoebe_description/meshes/visual/april_tags/AprilTag_0000.dae"/>
+        <mesh filename="package://phoebe_description/meshes/visual/april_tags/AprilTag_0000.dae"/>
       </geometry>
-    <material name="tag36h11-0">
-     <texture filename="package://phoebe_description/meshes/visual/april_tags/tag36_11_00000.png"/>
-    </material>
-   </visual>
+      <material name="tag36h11-0">
+        <texture filename="package://phoebe_description/meshes/visual/april_tags/tag36_11_00000.png"/>
+     </material>
+    </visual>
  </link>
    <joint name="apriltag_0_joint" type="fixed">
@@ -201,11 +199,10 @@
     <visual>
       <geometry>
-        <!--<box size="0.073 0.073 0.002"/> -->
         <mesh filename="package://phoebe_description/meshes/visual/april_tags/AprilTag_0004.dae"/>
       </geometry>
-    <material name="tag36h11-4">
-     <texture filename="package://phoebe_description/meshes/visual/april_tags/tag36_11_00004.png"/>
-    </material>
-   </visual>
+      <material name="tag36h11-4">
+        <texture filename="package://phoebe_description/meshes/visual/april_tags/tag36_11_00004.png"/>
+      </material>
+    </visual>
  </link>
    <joint name="apriltag_4_joint" type="fixed">
@@ -218,5 +215,4 @@
     <visual>
       <geometry>
-        <!-- <box size="0.214 0.214 0.002"/> -->
         <mesh filename="package://phoebe_description/meshes/visual/april_tags/AprilTag_0001.dae"/>
       </geometry>

Commit message: Making cylinder floating, and adjusting world tag tilt angle.

File: phoebe_description/urdf/imetro_mobile_environment/imetro_mobile_environment_macro.xacro (robot description, xacro)
@@ -141,4 +141,8 @@
     <!-- ===================== CYLINDER ===================== -->
     <link name="cylinder">
+       <inertial>
+          <mass value="0.750"/>
+          <inertia ixx="0.0005" ixy="0" ixz="0" iyy="0.0005" iyz="0" izz="3e-5"/>
+        </inertial>
        <visual>
           <origin xyz="0 0 0"/>
@@ -155,5 +159,5 @@
        </collision>
     </link>
-    <joint name="cylinder_joint" type="fixed">
+    <joint name="cylinder_joint" type="floating">
       <parent link="mobile_environment_base"/>
       <child link="cylinder"/>
@@ -225,5 +229,5 @@
     <parent link="mobile_environment_base"/>
     <child link="apriltag_1"/>
-    <origin xyz="0.134059 -1.788736 2.822666" rpy="-3.14159 0.52360 1.57"/>
+    <origin xyz="0.134059 -1.788736 2.822666" rpy="-3.14159 0.785 1.57"/>
    </joint>
   </xacro:macro>

Commit message: fixing inertia of cylinder

File: phoebe_description/urdf/imetro_mobile_environment/imetro_mobile_environment_macro.xacro (robot description, xacro)
@@ -143,5 +143,6 @@
        <inertial>
           <mass value="0.750"/>
-          <inertia ixx="0.0005" ixy="0" ixz="0" iyy="0.0005" iyz="0" izz="3e-5"/>
+          <inertia ixx="0.007" ixy="0" ixz="0" iyy="0.007" iyz="0" izz="0.0003"/>
+          <origin xyz="0 0 0.16"/>
         </inertial>
        <visual>
