Commit message: adding rough inertial values for cylinder so mujoco is happy

File: phoebe_description/urdf/imetro_mobile_environment/imetro_mobile_environment_macro.xacro (robot description, xacro)
@@ -141,4 +141,10 @@
     <!-- ===================== CYLINDER ===================== -->
     <link name="cylinder">
+      <!-- placeholder values for now so mujoco is happy enough -->
+      <inertial>
+        <mass value="0.75"/>
+        <origin xyz="0 0 0"/>
+        <inertia ixx="1e-4" ixy="0" ixz="0" iyy="1e-4" iyz="0" izz="1e-4"/>
+      </inertial>
        <visual>
           <origin xyz="0 0 0"/>

Commit message: Tweak cylinder masses

File: phoebe_description/urdf/imetro_mobile_environment/imetro_mobile_environment_macro.xacro (robot description, xacro)
@@ -141,9 +141,9 @@
     <!-- ===================== CYLINDER ===================== -->
     <link name="cylinder">
-      <!-- placeholder values for now so mujoco is happy enough -->
+      <!-- Placeholder mass params for the 3d printed cylinder, likely needs updates -->
       <inertial>
-        <mass value="0.75"/>
-        <origin xyz="0 0 0"/>
-        <inertia ixx="1e-4" ixy="0" ixz="0" iyy="1e-4" iyz="0" izz="1e-4"/>
+          <mass value="0.5" />
+          <origin xyz="0 0 0.182975" rpy="0 0 0" />
+          <inertia ixx="0.005691726" ixy="0.0" ixz="0.0" iyy="0.005691726" iyz="0.0" izz="0.000223503" />
       </inertial>
        <visual>
