Commit message: remove ignition block in wheels urdf

File: phoebe_description/urdf/r100/wheels/wheel.urdf.xacro (robot description, xacro)
@@ -27,17 +27,4 @@
       </inertial>
     </link>
-    <gazebo reference="${tf_prefix}${prefix}_wheel_link">
-      <collision>
-        <surface>
-          <friction>
-            <ode>
-              <mu>1.0</mu>
-              <mu2>0.0</mu2>
-              <fdir1 ignition:expressed_in="${tf_prefix}base_link">1 ${side} 0</fdir1>
-            </ode>
-          </friction>
-        </surface>
-      </collision>
-    </gazebo>
     <joint name="${tf_prefix}${prefix}_wheel_joint" type="continuous">
       <parent link="${parent}" />
