Commit message: Add tf prefixes

File: phoebe_mujoco_config/urdf/phoebe_mujoco_ros2_control_macros.xacro (robot description, xacro)
@@ -1,19 +1,21 @@
 <?xml version="1.0"?>
 <robot name="phoebe_mujoco_ros2_control_macros" xmlns:xacro="http://ros.org/wiki/xacro">
-  <xacro:macro name="phoebe_mujoco_ros2_control_sensors">
-    <sensor name="left_wrist_mounted_camera">
-      <param name="frame_name">left_wrist_mounted_camera_color_optical_frame</param>
-      <param name="info_topic">/left_wrist_mounted_camera_/color/camera_info</param>
-      <param name="image_topic">/left_wrist_mounted_camera_/color/image_raw</param>
-      <param name="depth_topic">/left_wrist_mounted_camera_/aligned_depth_to_color/image_raw</param>
-    </sensor>
-    <sensor name="right_wrist_mounted_camera">
-      <param name="frame_name">right_wrist_mounted_camera_color_optical_frame</param>
-      <param name="info_topic">/right_wrist_mounted_camera_/color/camera_info</param>
-      <param name="image_topic">/right_wrist_mounted_camera_/color/image_raw</param>
-      <param name="depth_topic">/right_wrist_mounted_camera_/aligned_depth_to_color/image_raw</param>
-    </sensor>
-    <sensor name="lidar2d_0">
-      <param name="frame_name">lidar2d_0_laser</param>
+  <xacro:macro name="phoebe_mujoco_ros2_control_sensors" params="
+    tf_prefix:=''
+  ">
+    <sensor name="${tf_prefix}left_wrist_mounted_camera">
+      <param name="frame_name">${tf_prefix}left_wrist_mounted_camera_color_optical_frame</param>
+      <param name="info_topic">/${tf_prefix}left_wrist_mounted_camera_/color/camera_info</param>
+      <param name="image_topic">/${tf_prefix}left_wrist_mounted_camera_/color/image_raw</param>
+      <param name="depth_topic">/${tf_prefix}left_wrist_mounted_camera_/aligned_depth_to_color/image_raw</param>
+    </sensor>
+    <sensor name="${tf_prefix}right_wrist_mounted_camera">
+      <param name="frame_name">${tf_prefix}right_wrist_mounted_camera_color_optical_frame</param>
+      <param name="info_topic">/${tf_prefix}right_wrist_mounted_camera_/color/camera_info</param>
+      <param name="image_topic">/${tf_prefix}right_wrist_mounted_camera_/color/image_raw</param>
+      <param name="depth_topic">/${tf_prefix}right_wrist_mounted_camera_/aligned_depth_to_color/image_raw</param>
+    </sensor>
+    <sensor name="${tf_prefix}lidar2d_0">
+      <param name="frame_name">${tf_prefix}lidar2d_0_laser</param>
       <param name="angle_increment">0.1</param>
       <param name="min_angle">-2.3</param>
@@ -21,10 +23,9 @@
       <param name="range_min">0.05</param>
       <param name="range_max">10</param>
-      <param name="laserscan_topic">lidar2d_0_laser/scan</param>
-    </sensor>
-    <sensor name="imu_sensor">
+      <param name="laserscan_topic">${tf_prefix}lidar2d_0_laser/scan</param>
+    </sensor>
+    <sensor name="${tf_prefix}imu_sensor">
       <param name="mujoco_type">imu</param>
-      <!-- There is no requirement for the mujoco_sensor_name to match the ros2_control sensor name -->
-      <param name="mujoco_sensor_name">imu_sensor</param>
+      <param name="mujoco_sensor_name">${tf_prefix}imu_sensor</param>
       <state_interface name="orientation.x"/>
       <state_interface name="orientation.y"/>
@@ -38,7 +39,7 @@
       <state_interface name="linear_acceleration.z"/>
     </sensor>
-    <sensor name="right_ur_arm_tcp_fts_sensor">
+    <sensor name="${tf_prefix}right_ur_arm_tcp_fts_sensor">
       <param name="mujoco_type">fts</param>
-      <param name="mujoco_sensor_name">right_ur_arm_tcp_fts_sensor</param>
+      <param name="mujoco_sensor_name">${tf_prefix}right_ur_arm_tcp_fts_sensor</param>
       <state_interface name="force.x"/>
       <state_interface name="force.y"/>
@@ -48,7 +49,7 @@
       <state_interface name="torque.z"/>
     </sensor>
-    <sensor name="left_ur_arm_tcp_fts_sensor">
+    <sensor name="${tf_prefix}left_ur_arm_tcp_fts_sensor">
       <param name="mujoco_type">fts</param>
-      <param name="mujoco_sensor_name">left_ur_arm_tcp_fts_sensor</param>
+      <param name="mujoco_sensor_name">${tf_prefix}left_ur_arm_tcp_fts_sensor</param>
       <state_interface name="force.x"/>
       <state_interface name="force.y"/>
@@ -60,8 +61,9 @@
   </xacro:macro>
   <xacro:macro name="phoebe_mujoco_ros2_control_joints" params="
+    tf_prefix:=''
     use_left_static_pedestal:=false
   ">
     <xacro:unless value="${use_left_static_pedestal}">
-      <joint name="left_ewellix_lift_lower_to_higher">
+      <joint name="${tf_prefix}left_ewellix_lift_lower_to_higher">
         <command_interface name="position"/>
         <state_interface name="position">
@@ -72,5 +74,5 @@
       </joint>
     </xacro:unless>
-    <joint name="right_ewellix_lift_lower_to_higher">
+    <joint name="${tf_prefix}right_ewellix_lift_lower_to_higher">
       <command_interface name="position"/>
       <state_interface name="position">
@@ -80,5 +82,5 @@
       <state_interface name="effort"/>
     </joint>
-    <joint name="left_finger_1_joint">
+<joint name="${tf_prefix}left_finger_1_joint">
       <command_interface name="position"/>
       <state_interface name="position">
@@ -88,19 +90,19 @@
       <state_interface name="effort"/>
     </joint>
-    <joint name="right_robotiq_85_left_knuckle_joint">
-      <command_interface name="position"/>
-      <state_interface name="position">
-        <param name="initial_value">0.0</param>
-      </state_interface>
-      <state_interface name="velocity"/>
-      <state_interface name="effort"/>
-    </joint>
-    <joint name="left_ur_arm_shoulder_pan_joint">
-      <command_interface name="position"/>
-      <state_interface name="position">
-        <xacro:if value="${use_left_static_pedestal}">
+    <joint name="${tf_prefix}right_robotiq_85_left_knuckle_joint">
+      <command_interface name="position"/>
+      <state_interface name="position">
+        <param name="initial_value">0.0</param>
+      </state_interface>
+      <state_interface name="velocity"/>
+      <state_interface name="effort"/>
+    </joint>
+    <joint name="${tf_prefix}left_ur_arm_shoulder_pan_joint">
+      <command_interface name="position"/>
+      <state_interface name="position">
+        <xacro:if value="$(arg use_left_static_pedestal)">
           <param name="initial_value">${radians(8)}</param>
         </xacro:if>
-        <xacro:unless value="${use_left_static_pedestal}">
+        <xacro:unless value="$(arg use_left_static_pedestal)">
           <param name="initial_value">${radians(-33)}</param>
         </xacro:unless>
@@ -109,5 +111,5 @@
       <state_interface name="effort"/>
     </joint>
-    <joint name="left_ur_arm_shoulder_lift_joint">
+    <joint name="${tf_prefix}left_ur_arm_shoulder_lift_joint">
       <command_interface name="position"/>
       <state_interface name="position">
@@ -117,5 +119,5 @@
       <state_interface name="effort"/>
     </joint>
-    <joint name="left_ur_arm_elbow_joint">
+    <joint name="${tf_prefix}left_ur_arm_elbow_joint">
       <command_interface name="position"/>
       <state_interface name="position">
@@ -125,5 +127,5 @@
       <state_interface name="effort"/>
     </joint>
-    <joint name="left_ur_arm_wrist_1_joint">
+    <joint name="${tf_prefix}left_ur_arm_wrist_1_joint">
       <command_interface name="position"/>
       <state_interface name="position">
@@ -133,5 +135,5 @@
       <state_interface name="effort"/>
     </joint>
-    <joint name="left_ur_arm_wrist_2_joint">
+    <joint name="${tf_prefix}left_ur_arm_wrist_2_joint">
       <command_interface name="position"/>
       <state_interface name="position">
@@ -141,5 +143,5 @@
       <state_interface name="effort"/>
     </joint>
-    <joint name="left_ur_arm_wrist_3_joint">
+    <joint name="${tf_prefix}left_ur_arm_wrist_3_joint">
       <command_interface name="position"/>
       <state_interface name="position">
@@ -149,5 +151,5 @@
       <state_interface name="effort"/>
     </joint>
-    <joint name="right_ur_arm_shoulder_pan_joint">
+    <joint name="${tf_prefix}right_ur_arm_shoulder_pan_joint">
       <command_interface name="position"/>
       <state_interface name="position">
@@ -157,5 +159,5 @@
       <state_interface name="effort"/>
     </joint>
-    <joint name="right_ur_arm_shoulder_lift_joint">
+    <joint name="${tf_prefix}right_ur_arm_shoulder_lift_joint">
       <command_interface name="position"/>
       <state_interface name="position">
@@ -165,5 +167,5 @@
       <state_interface name="effort"/>
     </joint>
-    <joint name="right_ur_arm_elbow_joint">
+    <joint name="${tf_prefix}right_ur_arm_elbow_joint">
       <command_interface name="position"/>
       <state_interface name="position">
@@ -173,5 +175,5 @@
       <state_interface name="effort"/>
     </joint>
-    <joint name="right_ur_arm_wrist_1_joint">
+    <joint name="${tf_prefix}right_ur_arm_wrist_1_joint">
       <command_interface name="position"/>
       <state_interface name="position">
@@ -181,5 +183,5 @@
       <state_interface name="effort"/>
     </joint>
-    <joint name="right_ur_arm_wrist_2_joint">
+    <joint name="${tf_prefix}right_ur_arm_wrist_2_joint">
       <command_interface name="position"/>
       <state_interface name="position">
@@ -189,5 +191,5 @@
       <state_interface name="effort"/>
     </joint>
-    <joint name="right_ur_arm_wrist_3_joint">
+    <joint name="${tf_prefix}right_ur_arm_wrist_3_joint">
       <command_interface name="position"/>
       <state_interface name="position">
@@ -197,35 +199,35 @@
       <state_interface name="effort"/>
     </joint>
-    <joint name="front_left_wheel_joint">
-      <command_interface name="velocity" />
-      <state_interface name="position" >
-        <param name="initial_value">0.0</param>
-      </state_interface>
-      <state_interface name="velocity" />
-      <state_interface name="effort" />
-    </joint>
-    <joint name="front_right_wheel_joint">
-      <command_interface name="velocity" />
-      <state_interface name="position" >
-        <param name="initial_value">0.0</param>
-      </state_interface>
-      <state_interface name="velocity" />
-      <state_interface name="effort" />
-    </joint>
-    <joint name="rear_left_wheel_joint">
-      <command_interface name="velocity" />
-      <state_interface name="position" >
-        <param name="initial_value">0.0</param>
-      </state_interface>
-      <state_interface name="velocity" />
-      <state_interface name="effort" />
-    </joint>
-    <joint name="rear_right_wheel_joint">
-      <command_interface name="velocity" />
-      <state_interface name="position" >
-        <param name="initial_value">0.0</param>
-      </state_interface>
-      <state_interface name="velocity" />
-      <state_interface name="effort" />
+    <joint name="${tf_prefix}front_left_wheel_joint">
+      <command_interface name="velocity"/>
+      <state_interface name="position">
+        <param name="initial_value">0.0</param>
+      </state_interface>
+      <state_interface name="velocity"/>
+      <state_interface name="effort"/>
+    </joint>
+    <joint name="${tf_prefix}front_right_wheel_joint">
+      <command_interface name="velocity"/>
+      <state_interface name="position">
+        <param name="initial_value">0.0</param>
+      </state_interface>
+      <state_interface name="velocity"/>
+      <state_interface name="effort"/>
+    </joint>
+    <joint name="${tf_prefix}rear_left_wheel_joint">
+      <command_interface name="velocity"/>
+      <state_interface name="position">
+        <param name="initial_value">0.0</param>
+      </state_interface>
+      <state_interface name="velocity"/>
+      <state_interface name="effort"/>
+    </joint>
+    <joint name="${tf_prefix}rear_right_wheel_joint">
+      <command_interface name="velocity"/>
+      <state_interface name="position">
+        <param name="initial_value">0.0</param>
+      </state_interface>
+      <state_interface name="velocity"/>
+      <state_interface name="effort"/>
     </joint>
   </xacro:macro>
