Commit message: Parameterize mujoco inputs for PB

File: phoebe_mujoco_config/urdf/phoebe_mujoco_raw_inputs.xacro (robot description, xacro)
@@ -1,205 +1,221 @@
 <?xml version="1.0"?>
 <robot xmlns:xacro="http://wiki.ros.org/xacro">
-  <xacro:macro name="phoebe_mujoco_raw_inputs" params="
+  <xacro:macro name="phoebe_mujoco_raw_inputs_content" params="
     use_left_static_pedestal:=false
   ">
-    <raw_inputs>
-        <option integrator="implicitfast" impratio="20" cone="elliptic" noslip_iterations="5">
-            <flag multiccd="enable"/>
-        </option>
-        <default>
-            <default class="phoebe">
-                <material specular="0.5" shininess="0.25"/>
-                <joint axis="0 1 0" range="-6.28319 6.28319" armature="0.1"/>
-                <position ctrlrange="-6.2831 6.2831"/>
-                <general biastype="affine" ctrlrange="-6.2831 6.2831"/>
-                <default class="size4">
-                    <joint damping="10"/>
-                    <general forcerange="-330 330" gainprm="100000" biasprm="0 -100000 -10000"/>
+    <option integrator="implicitfast" impratio="20" cone="elliptic" noslip_iterations="5">
+        <flag multiccd="enable"/>
+    </option>
+    <default>
+        <default class="phoebe">
+            <material specular="0.5" shininess="0.25"/>
+            <joint axis="0 1 0" range="-6.28319 6.28319" armature="0.1"/>
+            <position ctrlrange="-6.2831 6.2831"/>
+            <general biastype="affine" ctrlrange="-6.2831 6.2831"/>
+            <default class="size4">
+                <joint damping="10"/>
+                <general forcerange="-330 330" gainprm="100000" biasprm="0 -100000 -10000"/>
+            </default>
+            <default class="size3">
+                <joint damping="5"/>
+                <general forcerange="-150 150" gainprm="100000" biasprm="0 -100000 -5000"/>
+                <default class="size3_limited">
+                    <joint range="-3.1415 3.1415"/>
+                    <general ctrlrange="-3.1415 3.1415"/>
                 </default>
-                <default class="size3">
-                    <joint damping="5"/>
-                    <general forcerange="-150 150" gainprm="100000" biasprm="0 -100000 -5000"/>
-                    <default class="size3_limited">
-                        <joint range="-3.1415 3.1415"/>
-                        <general ctrlrange="-3.1415 3.1415"/>
-                    </default>
+            </default>
+            <default class="size2">
+                <joint damping="2"/>
+                <general forcerange="-56 56" gainprm="100000" biasprm="0 -100000 -1000"/>
+            </default>
+            <default class="visual">
+                <geom group="2" type="mesh" contype="0" conaffinity="0"/>
+            </default>
+            <default class="collision">
+                <geom group="3" type="mesh"/>
+                <default class="wheels">
+                    <geom condim="3" friction="0.5 0.005 0.0001" solimp="0.95 0.99 0.001 0.1 6"/>
                 </default>
-                <default class="size2">
-                    <joint damping="2"/>
-                    <general forcerange="-56 56" gainprm="100000" biasprm="0 -100000 -1000"/>
+                <default class="rubber">
+                    <geom condim="4" friction="5 1.0 1.0" priority="1" solimp="0.9 0.95 0.001" solref="0.002 1" conaffinity="1"/>
                 </default>
-                <default class="visual">
-                    <geom group="2" type="mesh" contype="0" conaffinity="0"/>
-                </default>
-                <default class="collision">
-                    <geom group="3" type="mesh"/>
-                    <default class="wheels">
-                        <geom condim="3" friction="0.5 0.005 0.0001" solimp="0.95 0.99 0.001 0.1 6"/>
-                    </default>
-                    <default class="rubber">
-                        <geom condim="4" friction="5 1.0 1.0" priority="1" solimp="0.9 0.95 0.001" solref="0.002 1" conaffinity="1"/>
-                    </default>
-                </default>
-                <default class="right_spring_link">
-                    <joint range="-0.9 0.29670597283" armature="0.001" stiffness="0.05" springref="-2.62" damping="0.00125"/>
-                </default>
-                <default class="left_spring_link">
-                    <joint range="-0.29670597283 0.9" armature="0.001" stiffness="0.05" springref="2.62" damping="0.00125"/>
-                </default>
+            </default>
+            <default class="right_spring_link">
+                <joint range="-0.9 0.29670597283" armature="0.001" stiffness="0.05" springref="-2.62" damping="0.00125"/>
+            </default>
+            <default class="left_spring_link">
+                <joint range="-0.29670597283 0.9" armature="0.001" stiffness="0.05" springref="2.62" damping="0.00125"/>
             </default>
         </default>
-        <actuator>
-            <xacro:unless value="${use_left_static_pedestal}">
-                <position joint="left_ewellix_lift_lower_to_higher" name="left_ewellix_lift_lower_to_higher" kp="75000" dampratio="1.0" ctrlrange="0.0 0.7" />
-            </xacro:unless>
-            <position joint="right_ewellix_lift_lower_to_higher" name="right_ewellix_lift_lower_to_higher" kp="75000" dampratio="1.0" ctrlrange="0.0 0.7" />
-            <position tendon="right_split" name="right_robotiq_85_left_knuckle_joint" kp="100000" dampratio="10.0" ctrlrange="0.0 0.8" forcerange="-20 20"/>
-            <position tendon="left_split" name="left_finger_1_joint" kp="10000" dampratio="10.0" ctrlrange="0.0 0.025" forcerange="-130 130"/>
-            <general class="size4" name="left_ur_arm_shoulder_pan_joint" joint="left_ur_arm_shoulder_pan_joint"/>
-            <general class="size4" name="left_ur_arm_shoulder_lift_joint" joint="left_ur_arm_shoulder_lift_joint"/>
-            <general class="size3_limited" name="left_ur_arm_elbow_joint" joint="left_ur_arm_elbow_joint"/>
-            <general class="size2" name="left_ur_arm_wrist_1_joint" joint="left_ur_arm_wrist_1_joint"/>
-            <general class="size2" name="left_ur_arm_wrist_2_joint" joint="left_ur_arm_wrist_2_joint"/>
-            <general class="size2" name="left_ur_arm_wrist_3_joint" joint="left_ur_arm_wrist_3_joint"/>
-            <general class="size4" name="right_ur_arm_shoulder_pan_joint" joint="right_ur_arm_shoulder_pan_joint"/>
-            <general class="size4" name="right_ur_arm_shoulder_lift_joint" joint="right_ur_arm_shoulder_lift_joint"/>
-            <general class="size3_limited" name="right_ur_arm_elbow_joint" joint="right_ur_arm_elbow_joint"/>
-            <general class="size2" name="right_ur_arm_wrist_1_joint" joint="right_ur_arm_wrist_1_joint"/>
-            <general class="size2" name="right_ur_arm_wrist_2_joint" joint="right_ur_arm_wrist_2_joint"/>
-            <general class="size2" name="right_ur_arm_wrist_3_joint" joint="right_ur_arm_wrist_3_joint"/>
-            <velocity name="front_right_wheel_joint" joint="front_right_wheel_joint" ctrlrange="-15 15" kv="50"/>
-            <velocity name="front_left_wheel_joint" joint="front_left_wheel_joint" ctrlrange="-15 15" kv="50"/>
-            <velocity name="rear_right_wheel_joint" joint="rear_right_wheel_joint" ctrlrange="-15 15" kv="50"/>
-            <velocity name="rear_left_wheel_joint" joint="rear_left_wheel_joint" ctrlrange="-15 15" kv="50"/>
-        </actuator>
-        <contact>
-            <xacro:unless value="${use_left_static_pedestal}">
-                <exclude body1="base_link" body2="left_ewellix_lift_higher_link"/>
-                <exclude body1="base_link" body2="left_ewellix_lift_middle_link"/>
-            </xacro:unless>
-            <exclude body1="base_link" body2="right_ewellix_lift_higher_link"/>
-            <exclude body1="base_link" body2="right_ewellix_lift_middle_link"/>
-            <exclude body1="base_link" body2="rear_left_wheel_link"/>
-            <exclude body1="base_link" body2="rear_left_wheel_roller_0_link"/>
-            <exclude body1="base_link" body2="rear_left_wheel_roller_1_link"/>
-            <exclude body1="base_link" body2="rear_left_wheel_roller_2_link"/>
-            <exclude body1="base_link" body2="rear_left_wheel_roller_3_link"/>
-            <exclude body1="base_link" body2="rear_left_wheel_roller_4_link"/>
-            <exclude body1="base_link" body2="rear_left_wheel_roller_5_link"/>
-            <exclude body1="base_link" body2="rear_left_wheel_roller_6_link"/>
-            <exclude body1="base_link" body2="rear_left_wheel_roller_7_link"/>
-            <exclude body1="base_link" body2="rear_right_wheel_link"/>
-            <exclude body1="base_link" body2="rear_right_wheel_roller_0_link"/>
-            <exclude body1="base_link" body2="rear_right_wheel_roller_1_link"/>
-            <exclude body1="base_link" body2="rear_right_wheel_roller_2_link"/>
-            <exclude body1="base_link" body2="rear_right_wheel_roller_3_link"/>
-            <exclude body1="base_link" body2="rear_right_wheel_roller_4_link"/>
-            <exclude body1="base_link" body2="rear_right_wheel_roller_5_link"/>
-            <exclude body1="base_link" body2="rear_right_wheel_roller_6_link"/>
-            <exclude body1="base_link" body2="rear_right_wheel_roller_7_link"/>
-            <exclude body1="base_link" body2="front_left_wheel_link"/>
-            <exclude body1="base_link" body2="front_left_wheel_roller_0_link"/>
-            <exclude body1="base_link" body2="front_left_wheel_roller_1_link"/>
-            <exclude body1="base_link" body2="front_left_wheel_roller_2_link"/>
-            <exclude body1="base_link" body2="front_left_wheel_roller_3_link"/>
-            <exclude body1="base_link" body2="front_left_wheel_roller_4_link"/>
-            <exclude body1="base_link" body2="front_left_wheel_roller_5_link"/>
-            <exclude body1="base_link" body2="front_left_wheel_roller_6_link"/>
-            <exclude body1="base_link" body2="front_left_wheel_roller_7_link"/>
-            <exclude body1="base_link" body2="front_right_wheel_link"/>
-            <exclude body1="base_link" body2="front_right_wheel_roller_0_link"/>
-            <exclude body1="base_link" body2="front_right_wheel_roller_1_link"/>
-            <exclude body1="base_link" body2="front_right_wheel_roller_2_link"/>
-            <exclude body1="base_link" body2="front_right_wheel_roller_3_link"/>
-            <exclude body1="base_link" body2="front_right_wheel_roller_4_link"/>
-            <exclude body1="base_link" body2="front_right_wheel_roller_5_link"/>
-            <exclude body1="base_link" body2="front_right_wheel_roller_6_link"/>
-            <exclude body1="base_link" body2="front_right_wheel_roller_7_link"/>
-        </contact>
-        <!-- let hand - hande -->
+    </default>
+    <actuator>
+        <xacro:unless value="${use_left_static_pedestal}">
+            <position joint="left_ewellix_lift_lower_to_higher" name="left_ewellix_lift_lower_to_higher" kp="75000" dampratio="1.0" ctrlrange="0.0 0.7" />
+        </xacro:unless>
+        <position joint="right_ewellix_lift_lower_to_higher" name="right_ewellix_lift_lower_to_higher" kp="75000" dampratio="1.0" ctrlrange="0.0 0.7" />
+        <position tendon="right_split" name="right_robotiq_85_left_knuckle_joint" kp="100000" dampratio="10.0" ctrlrange="0.0 0.8" forcerange="-20 20"/>
+        <position tendon="left_split" name="left_finger_1_joint" kp="10000" dampratio="10.0" ctrlrange="0.0 0.025" forcerange="-130 130"/>
+        <general class="size4" name="left_ur_arm_shoulder_pan_joint" joint="left_ur_arm_shoulder_pan_joint"/>
+        <general class="size4" name="left_ur_arm_shoulder_lift_joint" joint="left_ur_arm_shoulder_lift_joint"/>
+        <general class="size3_limited" name="left_ur_arm_elbow_joint" joint="left_ur_arm_elbow_joint"/>
+        <general class="size2" name="left_ur_arm_wrist_1_joint" joint="left_ur_arm_wrist_1_joint"/>
+        <general class="size2" name="left_ur_arm_wrist_2_joint" joint="left_ur_arm_wrist_2_joint"/>
+        <general class="size2" name="left_ur_arm_wrist_3_joint" joint="left_ur_arm_wrist_3_joint"/>
+        <general class="size4" name="right_ur_arm_shoulder_pan_joint" joint="right_ur_arm_shoulder_pan_joint"/>
+        <general class="size4" name="right_ur_arm_shoulder_lift_joint" joint="right_ur_arm_shoulder_lift_joint"/>
+        <general class="size3_limited" name="right_ur_arm_elbow_joint" joint="right_ur_arm_elbow_joint"/>
+        <general class="size2" name="right_ur_arm_wrist_1_joint" joint="right_ur_arm_wrist_1_joint"/>
+        <general class="size2" name="right_ur_arm_wrist_2_joint" joint="right_ur_arm_wrist_2_joint"/>
+        <general class="size2" name="right_ur_arm_wrist_3_joint" joint="right_ur_arm_wrist_3_joint"/>
+        <velocity name="front_right_wheel_joint" joint="front_right_wheel_joint" ctrlrange="-15 15" kv="50"/>
+        <velocity name="front_left_wheel_joint" joint="front_left_wheel_joint" ctrlrange="-15 15" kv="50"/>
+        <velocity name="rear_right_wheel_joint" joint="rear_right_wheel_joint" ctrlrange="-15 15" kv="50"/>
+        <velocity name="rear_left_wheel_joint" joint="rear_left_wheel_joint" ctrlrange="-15 15" kv="50"/>
+    </actuator>
+    <contact>
+        <xacro:unless value="${use_left_static_pedestal}">
+            <exclude body1="base_link" body2="left_ewellix_lift_higher_link"/>
+            <exclude body1="base_link" body2="left_ewellix_lift_middle_link"/>
+        </xacro:unless>
+        <exclude body1="base_link" body2="right_ewellix_lift_higher_link"/>
+        <exclude body1="base_link" body2="right_ewellix_lift_middle_link"/>
+        <exclude body1="base_link" body2="rear_left_wheel_link"/>
+        <exclude body1="base_link" body2="rear_left_wheel_roller_0_link"/>
+        <exclude body1="base_link" body2="rear_left_wheel_roller_1_link"/>
+        <exclude body1="base_link" body2="rear_left_wheel_roller_2_link"/>
+        <exclude body1="base_link" body2="rear_left_wheel_roller_3_link"/>
+        <exclude body1="base_link" body2="rear_left_wheel_roller_4_link"/>
+        <exclude body1="base_link" body2="rear_left_wheel_roller_5_link"/>
+        <exclude body1="base_link" body2="rear_left_wheel_roller_6_link"/>
+        <exclude body1="base_link" body2="rear_left_wheel_roller_7_link"/>
+        <exclude body1="base_link" body2="rear_right_wheel_link"/>
+        <exclude body1="base_link" body2="rear_right_wheel_roller_0_link"/>
+        <exclude body1="base_link" body2="rear_right_wheel_roller_1_link"/>
+        <exclude body1="base_link" body2="rear_right_wheel_roller_2_link"/>
+        <exclude body1="base_link" body2="rear_right_wheel_roller_3_link"/>
+        <exclude body1="base_link" body2="rear_right_wheel_roller_4_link"/>
+        <exclude body1="base_link" body2="rear_right_wheel_roller_5_link"/>
+        <exclude body1="base_link" body2="rear_right_wheel_roller_6_link"/>
+        <exclude body1="base_link" body2="rear_right_wheel_roller_7_link"/>
+        <exclude body1="base_link" body2="front_left_wheel_link"/>
+        <exclude body1="base_link" body2="front_left_wheel_roller_0_link"/>
+        <exclude body1="base_link" body2="front_left_wheel_roller_1_link"/>
+        <exclude body1="base_link" body2="front_left_wheel_roller_2_link"/>
+        <exclude body1="base_link" body2="front_left_wheel_roller_3_link"/>
+        <exclude body1="base_link" body2="front_left_wheel_roller_4_link"/>
+        <exclude body1="base_link" body2="front_left_wheel_roller_5_link"/>
+        <exclude body1="base_link" body2="front_left_wheel_roller_6_link"/>
+        <exclude body1="base_link" body2="front_left_wheel_roller_7_link"/>
+        <exclude body1="base_link" body2="front_right_wheel_link"/>
+        <exclude body1="base_link" body2="front_right_wheel_roller_0_link"/>
+        <exclude body1="base_link" body2="front_right_wheel_roller_1_link"/>
+        <exclude body1="base_link" body2="front_right_wheel_roller_2_link"/>
+        <exclude body1="base_link" body2="front_right_wheel_roller_3_link"/>
+        <exclude body1="base_link" body2="front_right_wheel_roller_4_link"/>
+        <exclude body1="base_link" body2="front_right_wheel_roller_5_link"/>
+        <exclude body1="base_link" body2="front_right_wheel_roller_6_link"/>
+        <exclude body1="base_link" body2="front_right_wheel_roller_7_link"/>
+    </contact>
+    <!-- let hand - hande -->
+    <tendon>
+        <fixed name="left_split">
+        <joint joint="left_finger_1_joint" coef="0.5"/>
+        <joint joint="left_finger_2_joint" coef="0.5"/>
+        </fixed>
+    </tendon>
+    <equality>
+        <joint joint1="left_finger_1_joint" joint2="left_finger_2_joint" polycoef="0 1 0 0 0" solimp="0.95 0.99 0.001" solref="0.005 1"/>
+    </equality>
+    <!-- right hand - 2f-85 -->
+    <tendon>
+        <fixed name="right_split">
+        <joint joint="right_robotiq_85_left_knuckle_joint" coef="0.485"/>
+        <joint joint="right_robotiq_85_right_knuckle_joint" coef="-0.485"/>
+        </fixed>
+    </tendon>
+    <equality>
+        <connect anchor="-0.0371575 0.0 0.043422" body1="right_robotiq_85_right_inner_knuckle_link" body2="right_robotiq_85_right_finger_tip_link" solimp="0.95 0.99 0.001" solref="0.005 1"/>
+        <connect anchor="0.0371575 0.0 0.043422" body1="right_robotiq_85_left_inner_knuckle_link" body2="right_robotiq_85_left_finger_tip_link" solimp="0.95 0.99 0.001" solref="0.005 1"/>
+        <joint joint1="right_robotiq_85_left_knuckle_joint" joint2="right_robotiq_85_right_knuckle_joint" polycoef="0 -1 0 0 0" solimp="0.95 0.99 0.001"
+        solref="0.005 1"/>
+    </equality>
+    <contact>
+        <exclude body1="right_ur_arm_wrist_3_link" body2="right_robotiq_85_right_inner_knuckle_link"/>
+        <exclude body1="right_ur_arm_wrist_3_link" body2="right_robotiq_85_left_inner_knuckle_link"/>
+        <exclude body1="right_ur_arm_wrist_3_link" body2="right_robotiq_85_right_knuckle_link"/>
+        <exclude body1="right_ur_arm_wrist_3_link" body2="right_robotiq_85_left_knuckle_link"/>
+        <exclude body1="right_ur_arm_wrist_3_link" body2="right_robotiq_85_right_finger_tip_link"/>
+        <exclude body1="right_ur_arm_wrist_3_link" body2="right_robotiq_85_left_finger_tip_link"/>
+        <exclude body1="right_robotiq_85_right_finger_tip_link" body2="right_robotiq_85_right_knuckle_link"/>
+        <exclude body1="right_robotiq_85_left_finger_tip_link" body2="right_robotiq_85_left_knuckle_link"/>
+        <exclude body1="right_robotiq_85_right_finger_tip_link" body2="right_robotiq_85_right_finger_coupler_link"/>
+        <exclude body1="right_robotiq_85_left_finger_tip_link" body2="right_robotiq_85_left_finger_coupler_link"/>
+        <exclude body1="right_robotiq_85_right_knuckle_link" body2="right_robotiq_85_right_finger_coupler_link"/>
+        <exclude body1="right_robotiq_85_left_knuckle_link" body2="right_robotiq_85_left_finger_coupler_link"/>
+        <exclude body1="right_robotiq_85_right_inner_knuckle_link" body2="right_robotiq_85_right_finger_tip_link"/>
+        <exclude body1="right_robotiq_85_left_inner_knuckle_link" body2="right_robotiq_85_left_finger_tip_link"/>
+        <exclude body1="right_robotiq_85_right_inner_knuckle_link" body2="right_robotiq_85_right_finger_coupler_link"/>
+        <exclude body1="right_robotiq_85_left_inner_knuckle_link" body2="right_robotiq_85_left_finger_coupler_link"/>
+        <exclude body1="right_robotiq_85_right_inner_knuckle_link" body2="right_robotiq_85_right_knuckle_link"/>
+        <exclude body1="right_robotiq_85_left_inner_knuckle_link" body2="right_robotiq_85_left_knuckle_link"/>
+    </contact>
+    <!-- Same logic as above... but for liftkits -->
+    <xacro:unless value="${use_left_static_pedestal}">
         <tendon>
-            <fixed name="left_split">
-            <joint joint="left_finger_1_joint" coef="0.5"/>
-            <joint joint="left_finger_2_joint" coef="0.5"/>
+            <fixed name="left_lift_middle_mimic_higher">
+            <joint joint="left_ewellix_lift_lower_to_higher" coef="0.5"/>
+            <joint joint="left_middle_mimic_higher" coef="0.5"/>
             </fixed>
         </tendon>
+    </xacro:unless>
+    <tendon>
+        <fixed name="right_lift_middle_mimic_higher">
+        <joint joint="right_ewellix_lift_lower_to_higher" coef="0.5"/>
+        <joint joint="right_middle_mimic_higher" coef="0.5"/>
+        </fixed>
+    </tendon>
+    <!-- The mimic joint is scaled by 50% in the URDF -->
+    <xacro:unless value="${use_left_static_pedestal}">
         <equality>
-            <joint joint1="left_finger_1_joint" joint2="left_finger_2_joint" polycoef="0 1 0 0 0" solimp="0.95 0.99 0.001" solref="0.005 1"/>
+            <joint name="left_upper_mimic_lower" joint1="left_ewellix_lift_lower_to_higher" joint2="left_middle_mimic_higher" polycoef="0 2 0 0 0"/>
         </equality>
-        <!-- right hand - 2f-85 -->
-        <tendon>
-            <fixed name="right_split">
-            <joint joint="right_robotiq_85_left_knuckle_joint" coef="0.485"/>
-            <joint joint="right_robotiq_85_right_knuckle_joint" coef="-0.485"/>
-            </fixed>
-        </tendon>
-        <equality>
-            <connect anchor="-0.0371575 0.0 0.043422" body1="right_robotiq_85_right_inner_knuckle_link" body2="right_robotiq_85_right_finger_tip_link" solimp="0.95 0.99 0.001" solref="0.005 1"/>
-            <connect anchor="0.0371575 0.0 0.043422" body1="right_robotiq_85_left_inner_knuckle_link" body2="right_robotiq_85_left_finger_tip_link" solimp="0.95 0.99 0.001" solref="0.005 1"/>
-            <joint joint1="right_robotiq_85_left_knuckle_joint" joint2="right_robotiq_85_right_knuckle_joint" polycoef="0 -1 0 0 0" solimp="0.95 0.99 0.001"
-            solref="0.005 1"/>
-        </equality>
-        <contact>
-            <exclude body1="right_ur_arm_wrist_3_link" body2="right_robotiq_85_right_inner_knuckle_link"/>
-            <exclude body1="right_ur_arm_wrist_3_link" body2="right_robotiq_85_left_inner_knuckle_link"/>
-            <exclude body1="right_ur_arm_wrist_3_link" body2="right_robotiq_85_right_knuckle_link"/>
-            <exclude body1="right_ur_arm_wrist_3_link" body2="right_robotiq_85_left_knuckle_link"/>
-            <exclude body1="right_ur_arm_wrist_3_link" body2="right_robotiq_85_right_finger_tip_link"/>
-            <exclude body1="right_ur_arm_wrist_3_link" body2="right_robotiq_85_left_finger_tip_link"/>
-            <exclude body1="right_robotiq_85_right_finger_tip_link" body2="right_robotiq_85_right_knuckle_link"/>
-            <exclude body1="right_robotiq_85_left_finger_tip_link" body2="right_robotiq_85_left_knuckle_link"/>
-            <exclude body1="right_robotiq_85_right_finger_tip_link" body2="right_robotiq_85_right_finger_coupler_link"/>
-            <exclude body1="right_robotiq_85_left_finger_tip_link" body2="right_robotiq_85_left_finger_coupler_link"/>
-            <exclude body1="right_robotiq_85_right_knuckle_link" body2="right_robotiq_85_right_finger_coupler_link"/>
-            <exclude body1="right_robotiq_85_left_knuckle_link" body2="right_robotiq_85_left_finger_coupler_link"/>
-            <exclude body1="right_robotiq_85_right_inner_knuckle_link" body2="right_robotiq_85_right_finger_tip_link"/>
-            <exclude body1="right_robotiq_85_left_inner_knuckle_link" body2="right_robotiq_85_left_finger_tip_link"/>
-            <exclude body1="right_robotiq_85_right_inner_knuckle_link" body2="right_robotiq_85_right_finger_coupler_link"/>
-            <exclude body1="right_robotiq_85_left_inner_knuckle_link" body2="right_robotiq_85_left_finger_coupler_link"/>
-            <exclude body1="right_robotiq_85_right_inner_knuckle_link" body2="right_robotiq_85_right_knuckle_link"/>
-            <exclude body1="right_robotiq_85_left_inner_knuckle_link" body2="right_robotiq_85_left_knuckle_link"/>
-        </contact>
-        <!-- Same logic as above... but for liftkits -->
-        <xacro:unless value="${use_left_static_pedestal}">
-            <tendon>
-                <fixed name="left_lift_middle_mimic_higher">
-                <joint joint="left_ewellix_lift_lower_to_higher" coef="0.5"/>
-                <joint joint="left_middle_mimic_higher" coef="0.5"/>
-                </fixed>
-            </tendon>
-        </xacro:unless>
-        <tendon>
-            <fixed name="right_lift_middle_mimic_higher">
-            <joint joint="right_ewellix_lift_lower_to_higher" coef="0.5"/>
-            <joint joint="right_middle_mimic_higher" coef="0.5"/>
-            </fixed>
-        </tendon>
-        <!-- The mimic joint is scaled by 50% in the URDF -->
-        <xacro:unless value="${use_left_static_pedestal}">
-            <equality>
-                <joint name="left_upper_mimic_lower" joint1="left_ewellix_lift_lower_to_higher" joint2="left_middle_mimic_higher" polycoef="0 2 0 0 0"/>
-            </equality>
-        </xacro:unless>
-        <equality>
-            <joint name="right_upper_mimic_lower" joint1="right_ewellix_lift_lower_to_higher" joint2="right_middle_mimic_higher" polycoef="0 2 0 0 0"/>
-        </equality>
-        <sensor>
-            <force name="left_ur_arm_tcp_fts_sensor_force" site="left_ur_arm_ft_frame"/>
-            <torque name="left_ur_arm_tcp_fts_sensor_torque" site="left_ur_arm_ft_frame"/>
-        </sensor>
-        <sensor>
-            <force name="right_ur_arm_tcp_fts_sensor_force" site="right_ur_arm_ft_frame"/>
-            <torque name="right_ur_arm_tcp_fts_sensor_torque" site="right_ur_arm_ft_frame"/>
-        </sensor>
-        <sensor>
-            <framequat name="imu_sensor_quat" objtype="site" objname="imu_0_link" />
-            <gyro name="imu_sensor_gyro" site="imu_0_link" />
-            <accelerometer name="imu_sensor_accel" site="imu_0_link" />
-        </sensor>
-        <sensor>
-            <rangefinder name="lidar2d_0" site="lidar2d_0"/>
-        </sensor>
-    </raw_inputs>
+    </xacro:unless>
+    <equality>
+        <joint name="right_upper_mimic_lower" joint1="right_ewellix_lift_lower_to_higher" joint2="right_middle_mimic_higher" polycoef="0 2 0 0 0"/>
+    </equality>
+    <sensor>
+        <force name="left_ur_arm_tcp_fts_sensor_force" site="left_ur_arm_ft_frame"/>
+        <torque name="left_ur_arm_tcp_fts_sensor_torque" site="left_ur_arm_ft_frame"/>
+    </sensor>
+    <sensor>
+        <force name="right_ur_arm_tcp_fts_sensor_force" site="right_ur_arm_ft_frame"/>
+        <torque name="right_ur_arm_tcp_fts_sensor_torque" site="right_ur_arm_ft_frame"/>
+    </sensor>
+    <sensor>
+        <framequat name="imu_sensor_quat" objtype="site" objname="imu_0_link" />
+        <gyro name="imu_sensor_gyro" site="imu_0_link" />
+        <accelerometer name="imu_sensor_accel" site="imu_0_link" />
+    </sensor>
+    <sensor>
+        <rangefinder name="lidar2d_0" site="lidar2d_0"/>
+    </sensor>
   </xacro:macro>
+    <!-- Can use `skip_tags` to include the macro in other files without duplicating inputs -->
+    <xacro:macro name="phoebe_mujoco_raw_inputs" params="
+      use_left_static_pedestal:=false
+      skip_tags:=false
+    ">
+      <xacro:unless value="${skip_tags}">
+        <raw_inputs>
+          <xacro:phoebe_mujoco_raw_inputs_content
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