Commit message: mujoco launches with dual handes

File: phoebe_mujoco_config/urdf/phoebe_mujoco_processed_inputs.xacro (robot description, xacro)
@@ -3,4 +3,6 @@
   <xacro:macro name="phoebe_mujoco_processed_inputs" params="
     tf_prefix:=''
+    left_hand_type:='hande'
+    right_hand_type:='hande'
   ">
     <!-- Process arguments for the URDF -->
@@ -10,9 +12,4 @@
       <camera site="${tf_prefix}right_wrist_mounted_camera_color_optical_frame" name="${tf_prefix}right_wrist_mounted_camera" fovy="58" mode="fixed" resolution="1280 720"/>
       <lidar ref_site="${tf_prefix}lidar2d_0_laser" sensor_name="${tf_prefix}lidar2d_0" min_angle="-2.3" max_angle="2.3" angle_increment="0.1" />    <!-- <decompose_mesh mesh_name="finger_v6" threshold="0.05"/> -->
-      <!-- Add frictionloss and armature to fingers to help with backdriving -->
-      <modify_element type="joint" name="${tf_prefix}left_finger_1_joint" armature="0.5" frictionloss="5.0" />
-      <modify_element type="joint" name="${tf_prefix}left_finger_2_joint" armature="0.5" frictionloss="5.0" />
-      <modify_element type="joint" name="${tf_prefix}right_finger_1_joint" armature="0.5" frictionloss="5.0" />
-      <modify_element type="joint" name="${tf_prefix}right_finger_2_joint" armature="0.5" frictionloss="5.0" />.
       <!-- Add gravcomp so that control will make the joints move about the desired position-->
       <modify_element type="body" name="${tf_prefix}left_ewellix_lift_higher_link" gravcomp="1.0"/>
@@ -24,4 +21,16 @@
       <modify_element type="body" name="${tf_prefix}left_ur_arm_wrist_2_link" gravcomp="1.0"/>
       <modify_element type="body" name="${tf_prefix}left_ur_arm_wrist_3_link" gravcomp="1.0"/>
+      <xacro:if value="${left_hand_type == 'hande'}">
+        <modify_element type="joint" name="${tf_prefix}left_finger_1_joint" armature="0.5" frictionloss="5.0" />
+        <modify_element type="joint" name="${tf_prefix}left_finger_2_joint" armature="0.5" frictionloss="5.0" />
+        <modify_element type="body" name="${tf_prefix}left_finger_1_link" gravcomp="1.0"/>
+        <modify_element type="body" name="${tf_prefix}left_finger_2_link" gravcomp="1.0"/>
+      </xacro:if>
+      <xacro:if value="${right_hand_type == 'hande'}">
+        <modify_element type="joint" name="${tf_prefix}right_finger_1_joint" armature="0.5" frictionloss="5.0" />
+        <modify_element type="joint" name="${tf_prefix}right_finger_2_joint" armature="0.5" frictionloss="5.0" />
+        <modify_element type="body" name="${tf_prefix}right_finger_1_link" gravcomp="1.0"/>
+        <modify_element type="body" name="${tf_prefix}right_finger_2_link" gravcomp="1.0"/>
+      </xacro:if>
       <modify_element type="body" name="${tf_prefix}left_finger_1_link" gravcomp="1.0"/>
       <modify_element type="body" name="${tf_prefix}left_finger_2_link" gravcomp="1.0"/>

File: phoebe_mujoco_config/urdf/phoebe_mujoco_raw_inputs.xacro (robot description, xacro)
@@ -4,4 +4,6 @@
     use_left_static_pedestal:=false
     tf_prefix:=''
+    left_hand_type:='hande'
+    right_hand_type:='hande'
     defaults_prefix:=''
   ">
@@ -56,6 +58,16 @@
         </xacro:unless>
         <position joint="${tf_prefix}right_ewellix_lift_lower_to_higher" name="${tf_prefix}right_ewellix_lift_lower_to_higher" kp="75000" dampratio="1.0" ctrlrange="0.0 0.7" />
-        <position tendon="${tf_prefix}right_split" name="${tf_prefix}right_robotiq_85_left_knuckle_joint" kp="100000" dampratio="10.0" ctrlrange="0.0 0.8" forcerange="-20 20"/>
-        <position tendon="${tf_prefix}left_split" name="${tf_prefix}left_finger_1_joint" kp="10000" dampratio="10.0" ctrlrange="0.0 0.025" forcerange="-130 130"/>
+        <xacro:if value="${right_hand_type == 'hande'}">
+            <position tendon="${tf_prefix}right_split" name="${tf_prefix}right_finger_1_joint" kp="10000" dampratio="10.0" ctrlrange="0.0 0.025" forcerange="-130 130"/>
+        </xacro:if>
+        <xacro:if value="${right_hand_type == '2f85'}">
+            <position tendon="${tf_prefix}right_split" name="${tf_prefix}right_robotiq_85_left_knuckle_joint" kp="100000" dampratio="10.0" ctrlrange="0.0 0.8" forcerange="-20 20"/>
+        </xacro:if>
+        <xacro:if value="${left_hand_type == 'hande'}">
+            <position tendon="${tf_prefix}left_split" name="${tf_prefix}left_finger_1_joint" kp="10000" dampratio="10.0" ctrlrange="0.0 0.025" forcerange="-130 130"/>
+        </xacro:if>
+        <xacro:if value="${left_hand_type == '2f85'}">
+            <position tendon="${tf_prefix}left_split" name="${tf_prefix}left_robotiq_85_left_knuckle_joint" kp="100000" dampratio="10.0" ctrlrange="0.0 0.8" forcerange="-20 20"/>
+        </xacro:if>
         <general class="size4" name="${tf_prefix}left_ur_arm_shoulder_pan_joint" joint="${tf_prefix}left_ur_arm_shoulder_pan_joint"/>
         <general class="size4" name="${tf_prefix}left_ur_arm_shoulder_lift_joint" joint="${tf_prefix}left_ur_arm_shoulder_lift_joint"/>
@@ -119,47 +131,96 @@
         <exclude body1="${tf_prefix}base_link" body2="${tf_prefix}front_right_wheel_roller_7_link"/>
     </contact>
-    <!-- let hand - hande -->
-    <tendon>
-        <fixed name="${tf_prefix}left_split">
-        <joint joint="${tf_prefix}left_finger_1_joint" coef="0.5"/>
-        <joint joint="${tf_prefix}left_finger_2_joint" coef="0.5"/>
-        </fixed>
-    </tendon>
-    <equality>
-        <joint joint1="${tf_prefix}left_finger_1_joint" joint2="${tf_prefix}left_finger_2_joint" polycoef="0 1 0 0 0" solimp="0.95 0.99 0.001" solref="0.005 1"/>
-    </equality>
-    <!-- right hand - 2f-85 -->
-    <tendon>
-        <fixed name="${tf_prefix}right_split">
-        <joint joint="${tf_prefix}right_robotiq_85_left_knuckle_joint" coef="0.485"/>
-        <joint joint="${tf_prefix}right_robotiq_85_right_knuckle_joint" coef="-0.485"/>
-        </fixed>
-    </tendon>
-    <equality>
-        <connect anchor="-0.0371575 0.0 0.043422" body1="${tf_prefix}right_robotiq_85_right_inner_knuckle_link" body2="${tf_prefix}right_robotiq_85_right_finger_tip_link" solimp="0.95 0.99 0.001" solref="0.005 1"/>
-        <connect anchor="0.0371575 0.0 0.043422" body1="${tf_prefix}right_robotiq_85_left_inner_knuckle_link" body2="${tf_prefix}right_robotiq_85_left_finger_tip_link" solimp="0.95 0.99 0.001" solref="0.005 1"/>
-        <joint joint1="${tf_prefix}right_robotiq_85_left_knuckle_joint" joint2="${tf_prefix}right_robotiq_85_right_knuckle_joint" polycoef="0 -1 0 0 0" solimp="0.95 0.99 0.001"
-        solref="0.005 1"/>
-    </equality>
-    <contact>
-        <exclude body1="${tf_prefix}right_ur_arm_wrist_3_link" body2="${tf_prefix}right_robotiq_85_right_inner_knuckle_link"/>
-        <exclude body1="${tf_prefix}right_ur_arm_wrist_3_link" body2="${tf_prefix}right_robotiq_85_left_inner_knuckle_link"/>
-        <exclude body1="${tf_prefix}right_ur_arm_wrist_3_link" body2="${tf_prefix}right_robotiq_85_right_knuckle_link"/>
-        <exclude body1="${tf_prefix}right_ur_arm_wrist_3_link" body2="${tf_prefix}right_robotiq_85_left_knuckle_link"/>
-        <exclude body1="${tf_prefix}right_ur_arm_wrist_3_link" body2="${tf_prefix}right_robotiq_85_right_finger_tip_link"/>
-        <exclude body1="${tf_prefix}right_ur_arm_wrist_3_link" body2="${tf_prefix}right_robotiq_85_left_finger_tip_link"/>
-        <exclude body1="${tf_prefix}right_robotiq_85_right_finger_tip_link" body2="${tf_prefix}right_robotiq_85_right_knuckle_link"/>
-        <exclude body1="${tf_prefix}right_robotiq_85_left_finger_tip_link" body2="${tf_prefix}right_robotiq_85_left_knuckle_link"/>
-        <exclude body1="${tf_prefix}right_robotiq_85_right_finger_tip_link" body2="${tf_prefix}right_robotiq_85_right_finger_coupler_link"/>
-        <exclude body1="${tf_prefix}right_robotiq_85_left_finger_tip_link" body2="${tf_prefix}right_robotiq_85_left_finger_coupler_link"/>
-        <exclude body1="${tf_prefix}right_robotiq_85_right_knuckle_link" body2="${tf_prefix}right_robotiq_85_right_finger_coupler_link"/>
-        <exclude body1="${tf_prefix}right_robotiq_85_left_knuckle_link" body2="${tf_prefix}right_robotiq_85_left_finger_coupler_link"/>
-        <exclude body1="${tf_prefix}right_robotiq_85_right_inner_knuckle_link" body2="${tf_prefix}right_robotiq_85_right_finger_tip_link"/>
-        <exclude body1="${tf_prefix}right_robotiq_85_left_inner_knuckle_link" body2="${tf_prefix}right_robotiq_85_left_finger_tip_link"/>
-        <exclude body1="${tf_prefix}right_robotiq_85_right_inner_knuckle_link" body2="${tf_prefix}right_robotiq_85_right_finger_coupler_link"/>
-        <exclude body1="${tf_prefix}right_robotiq_85_left_inner_knuckle_link" body2="${tf_prefix}right_robotiq_85_left_finger_coupler_link"/>
-        <exclude body1="${tf_prefix}right_robotiq_85_right_inner_knuckle_link" body2="${tf_prefix}right_robotiq_85_right_knuckle_link"/>
-        <exclude body1="${tf_prefix}right_robotiq_85_left_inner_knuckle_link" body2="${tf_prefix}right_robotiq_85_left_knuckle_link"/>
-    </contact>
+    <!-- left hand - hande or 2f85 -->
+    <xacro:if value="${left_hand_type == 'hande'}">
+        <tendon>
+            <fixed name="${tf_prefix}left_split">
+            <joint joint="${tf_prefix}left_finger_1_joint" coef="0.5"/>
+            <joint joint="${tf_prefix}left_finger_2_joint" coef="0.5"/>
+            </fixed>
+        </tendon>
+        <equality>
+            <joint joint1="${tf_prefix}left_finger_1_joint" joint2="${tf_prefix}left_finger_2_joint" polycoef="0 1 0 0 0" solimp="0.95 0.99 0.001" solref="0.005 1"/>
+        </equality>
+    </xacro:if>
+    <xacro:if value="${left_hand_type == '2f85'}">
+        <tendon>
+            <fixed name="${tf_prefix}left_split">
+            <joint joint="${tf_prefix}left_robotiq_85_left_knuckle_joint" coef="0.485"/>
+            <joint joint="${tf_prefix}left_robotiq_85_right_knuckle_joint" coef="-0.485"/>
+            </fixed>
+        </tendon>
+        <equality>
+            <connect anchor="-0.0371575 0.0 0.043422" body1="${tf_prefix}left_robotiq_85_right_inner_knuckle_link" body2="${tf_prefix}left_robotiq_85_right_finger_tip_link" solimp="0.95 0.99 0.001" solref="0.005 1"/>
+            <connect anchor="0.0371575 0.0 0.043422" body1="${tf_prefix}left_robotiq_85_left_inner_knuckle_link" body2="${tf_prefix}left_robotiq_85_left_finger_tip_link" solimp="0.95 0.99 0.001" solref="0.005 1"/>
+            <joint joint1="${tf_prefix}left_robotiq_85_left_knuckle_joint" joint2="${tf_prefix}left_robotiq_85_right_knuckle_joint" polycoef="0 -1 0 0 0" solimp="0.95 0.99 0.001"
+            solref="0.005 1"/>
+        </equality>
+        <contact>
+            <exclude body1="${tf_prefix}left_ur_arm_wrist_3_link" body2="${tf_prefix}left_robotiq_85_right_inner_knuckle_link"/>
+            <exclude body1="${tf_prefix}left_ur_arm_wrist_3_link" body2="${tf_prefix}left_robotiq_85_left_inner_knuckle_link"/>
+            <exclude body1="${tf_prefix}left_ur_arm_wrist_3_link" body2="${tf_prefix}left_robotiq_85_right_knuckle_link"/>
+            <exclude body1="${tf_prefix}left_ur_arm_wrist_3_link" body2="${tf_prefix}left_robotiq_85_left_knuckle_link"/>
+            <exclude body1="${tf_prefix}left_ur_arm_wrist_3_link" body2="${tf_prefix}left_robotiq_85_right_finger_tip_link"/>
+            <exclude body1="${tf_prefix}left_ur_arm_wrist_3_link" body2="${tf_prefix}left_robotiq_85_left_finger_tip_link"/>
+            <exclude body1="${tf_prefix}left_robotiq_85_right_finger_tip_link" body2="${tf_prefix}left_robotiq_85_right_knuckle_link"/>
+            <exclude body1="${tf_prefix}left_robotiq_85_left_finger_tip_link" body2="${tf_prefix}left_robotiq_85_left_knuckle_link"/>
+            <exclude body1="${tf_prefix}left_robotiq_85_right_finger_tip_link" body2="${tf_prefix}left_robotiq_85_right_finger_coupler_link"/>
+            <exclude body1="${tf_prefix}left_robotiq_85_left_finger_tip_link" body2="${tf_prefix}left_robotiq_85_left_finger_coupler_link"/>
+            <exclude body1="${tf_prefix}left_robotiq_85_right_knuckle_link" body2="${tf_prefix}left_robotiq_85_right_finger_coupler_link"/>
+            <exclude body1="${tf_prefix}left_robotiq_85_left_knuckle_link" body2="${tf_prefix}left_robotiq_85_left_finger_coupler_link"/>
+            <exclude body1="${tf_prefix}left_robotiq_85_right_inner_knuckle_link" body2="${tf_prefix}left_robotiq_85_right_finger_tip_link"/>
+            <exclude body1="${tf_prefix}left_robotiq_85_left_inner_knuckle_link" body2="${tf_prefix}left_robotiq_85_left_finger_tip_link"/>
+            <exclude body1="${tf_prefix}left_robotiq_85_right_inner_knuckle_link" body2="${tf_prefix}left_robotiq_85_right_finger_coupler_link"/>
+            <exclude body1="${tf_prefix}left_robotiq_85_left_inner_knuckle_link" body2="${tf_prefix}left_robotiq_85_left_finger_coupler_link"/>
+            <exclude body1="${tf_prefix}left_robotiq_85_right_inner_knuckle_link" body2="${tf_prefix}left_robotiq_85_right_knuckle_link"/>
+            <exclude body1="${tf_prefix}left_robotiq_85_left_inner_knuckle_link" body2="${tf_prefix}left_robotiq_85_left_knuckle_link"/>
+        </contact>
+    </xacro:if>
+    <!-- right hand - hande or 2f85 -->
+    <xacro:if value="${right_hand_type == 'hande'}">
+        <tendon>
+            <fixed name="${tf_prefix}right_split">
+            <joint joint="${tf_prefix}right_finger_1_joint" coef="0.5"/>
+            <joint joint="${tf_prefix}right_finger_2_joint" coef="0.5"/>
+            </fixed>
+        </tendon>
+        <equality>
+            <joint joint1="${tf_prefix}right_finger_1_joint" joint2="${tf_prefix}right_finger_2_joint" polycoef="0 1 0 0 0" solimp="0.95 0.99 0.001" solref="0.005 1"/>
+        </equality>
+    </xacro:if>
+    <xacro:if value="${right_hand_type == '2f85'}">
+        <tendon>
+            <fixed name="${tf_prefix}right_split">
+            <joint joint="${tf_prefix}right_robotiq_85_left_knuckle_joint" coef="0.485"/>
+            <joint joint="${tf_prefix}right_robotiq_85_right_knuckle_joint" coef="-0.485"/>
+            </fixed>
+        </tendon>
+        <equality>
+            <connect anchor="-0.0371575 0.0 0.043422" body1="${tf_prefix}right_robotiq_85_right_inner_knuckle_link" body2="${tf_prefix}right_robotiq_85_right_finger_tip_link" solimp="0.95 0.99 0.001" solref="0.005 1"/>
+            <connect anchor="0.0371575 0.0 0.043422" body1="${tf_prefix}right_robotiq_85_left_inner_knuckle_link" body2="${tf_prefix}right_robotiq_85_left_finger_tip_link" solimp="0.95 0.99 0.001" solref="0.005 1"/>
+            <joint joint1="${tf_prefix}right_robotiq_85_left_knuckle_joint" joint2="${tf_prefix}right_robotiq_85_right_knuckle_joint" polycoef="0 -1 0 0 0" solimp="0.95 0.99 0.001"
+            solref="0.005 1"/>
+        </equality>
+        <contact>
+            <exclude body1="${tf_prefix}right_ur_arm_wrist_3_link" body2="${tf_prefix}right_robotiq_85_right_inner_knuckle_link"/>
+            <exclude body1="${tf_prefix}right_ur_arm_wrist_3_link" body2="${tf_prefix}right_robotiq_85_left_inner_knuckle_link"/>
+            <exclude body1="${tf_prefix}right_ur_arm_wrist_3_link" body2="${tf_prefix}right_robotiq_85_right_knuckle_link"/>
+            <exclude body1="${tf_prefix}right_ur_arm_wrist_3_link" body2="${tf_prefix}right_robotiq_85_left_knuckle_link"/>
+            <exclude body1="${tf_prefix}right_ur_arm_wrist_3_link" body2="${tf_prefix}right_robotiq_85_right_finger_tip_link"/>
+            <exclude body1="${tf_prefix}right_ur_arm_wrist_3_link" body2="${tf_prefix}right_robotiq_85_left_finger_tip_link"/>
+            <exclude body1="${tf_prefix}right_robotiq_85_right_finger_tip_link" body2="${tf_prefix}right_robotiq_85_right_knuckle_link"/>
+            <exclude body1="${tf_prefix}right_robotiq_85_left_finger_tip_link" body2="${tf_prefix}right_robotiq_85_left_knuckle_link"/>
+            <exclude body1="${tf_prefix}right_robotiq_85_right_finger_tip_link" body2="${tf_prefix}right_robotiq_85_right_finger_coupler_link"/>
+            <exclude body1="${tf_prefix}right_robotiq_85_left_finger_tip_link" body2="${tf_prefix}right_robotiq_85_left_finger_coupler_link"/>
+            <exclude body1="${tf_prefix}right_robotiq_85_right_knuckle_link" body2="${tf_prefix}right_robotiq_85_right_finger_coupler_link"/>
+            <exclude body1="${tf_prefix}right_robotiq_85_left_knuckle_link" body2="${tf_prefix}right_robotiq_85_left_finger_coupler_link"/>
+            <exclude body1="${tf_prefix}right_robotiq_85_right_inner_knuckle_link" body2="${tf_prefix}right_robotiq_85_right_finger_tip_link"/>
+            <exclude body1="${tf_prefix}right_robotiq_85_left_inner_knuckle_link" body2="${tf_prefix}right_robotiq_85_left_finger_tip_link"/>
+            <exclude body1="${tf_prefix}right_robotiq_85_right_inner_knuckle_link" body2="${tf_prefix}right_robotiq_85_right_finger_coupler_link"/>
+            <exclude body1="${tf_prefix}right_robotiq_85_left_inner_knuckle_link" body2="${tf_prefix}right_robotiq_85_left_finger_coupler_link"/>
+            <exclude body1="${tf_prefix}right_robotiq_85_right_inner_knuckle_link" body2="${tf_prefix}right_robotiq_85_right_knuckle_link"/>
+            <exclude body1="${tf_prefix}right_robotiq_85_left_inner_knuckle_link" body2="${tf_prefix}right_robotiq_85_left_knuckle_link"/>
+        </contact>
+    </xacro:if>
     <!-- Same logic as above... but for liftkits -->
     <xacro:unless value="${use_left_static_pedestal}">

File: phoebe_mujoco_config/urdf/phoebe_mujoco_ros2_control_macros.xacro (robot description, xacro)
@@ -62,4 +62,6 @@
   <xacro:macro name="phoebe_mujoco_ros2_control_joints" params="
     tf_prefix:=''
+    left_hand_type:='hande'
+    right_hand_type:='hande'
     use_left_static_pedestal:=false
   ">
@@ -82,20 +84,44 @@
       <state_interface name="effort"/>
     </joint>
-<joint name="${tf_prefix}left_finger_1_joint">
-      <command_interface name="position"/>
-      <state_interface name="position">
-        <param name="initial_value">0.02</param>
-      </state_interface>
-      <state_interface name="velocity"/>
-      <state_interface name="effort"/>
-    </joint>
-    <joint name="${tf_prefix}right_robotiq_85_left_knuckle_joint">
-      <command_interface name="position"/>
-      <state_interface name="position">
-        <param name="initial_value">0.0</param>
-      </state_interface>
-      <state_interface name="velocity"/>
-      <state_interface name="effort"/>
-    </joint>
+    <xacro:if value="${left_hand_type == 'hande'}">
+      <joint name="${tf_prefix}left_finger_1_joint">
+        <command_interface name="position"/>
+        <state_interface name="position">
+          <param name="initial_value">0.02</param>
+        </state_interface>
+        <state_interface name="velocity"/>
+        <state_interface name="effort"/>
+      </joint>
+    </xacro:if>
+    <xacro:if value="${left_hand_type == '2f85'}">
+      <joint name="${tf_prefix}left_robotiq_85_left_knuckle_joint">
+        <command_interface name="position"/>
+        <state_interface name="position">
+          <param name="initial_value">0.0</param>
+        </state_interface>
+        <state_interface name="velocity"/>
+        <state_interface name="effort"/>
+      </joint>
+    </xacro:if>
+    <xacro:if value="${right_hand_type == 'hande'}">
+      <joint name="${tf_prefix}right_finger_1_joint">
+        <command_interface name="position"/>
+        <state_interface name="position">
+          <param name="initial_value">0.02</param>
+        </state_interface>
+        <state_interface name="velocity"/>
+        <state_interface name="effort"/>
+      </joint>
+    </xacro:if>
+    <xacro:if value="${right_hand_type == '2f85'}">
+      <joint name="${tf_prefix}right_robotiq_85_left_knuckle_joint">
+        <command_interface name="position"/>
+        <state_interface name="position">
+          <param name="initial_value">0.0</param>
+        </state_interface>
+        <state_interface name="velocity"/>
+        <state_interface name="effort"/>
+      </joint>
+    </xacro:if>
     <joint name="${tf_prefix}left_ur_arm_shoulder_pan_joint">
       <command_interface name="position"/>
