Commit message: Replace body gravity compensation with actuator variant

File: phoebe_mujoco_config/urdf/phoebe_mujoco_processed_inputs.xacro (robot description, xacro)
@@ -26,42 +26,27 @@
       <camera site="${tf_prefix}left_wrist_mounted_camera_color_optical_frame" name="${tf_prefix}left_wrist_mounted_camera" fovy="58" mode="fixed" resolution="1280 720"/>
       <camera site="${tf_prefix}right_wrist_mounted_camera_color_optical_frame" name="${tf_prefix}right_wrist_mounted_camera" fovy="58" mode="fixed" resolution="1280 720"/>
-      <!-- Apply default classes to Phoebe joints -->
-      <modify_element type="joint" name="${tf_prefix}shoulder_pan_joint" class="size4"/>
-      <modify_element type="joint" name="${tf_prefix}shoulder_lift_joint" class="size4"/>
-      <modify_element type="joint" name="${tf_prefix}elbow_joint" class="size3_limited"/>
-      <modify_element type="joint" name="${tf_prefix}wrist_1_joint" class="size2"/>
-      <modify_element type="joint" name="${tf_prefix}wrist_2_joint" class="size2"/>
-      <modify_element type="joint" name="${tf_prefix}wrist_3_joint" class="size2"/>
-      <!-- Add gravcomp so that control will make the joints move about the desired position-->
-      <modify_element type="body" name="${tf_prefix}left_ewellix_lift_higher_link" gravcomp="1.0"/>
-      <modify_element type="body" name="${tf_prefix}left_ewellix_lift_middle_link" gravcomp="1.0"/>
-      <modify_element type="body" name="${tf_prefix}left_ur_arm_shoulder_link" gravcomp="1.0"/>
-      <modify_element type="body" name="${tf_prefix}left_ur_arm_upper_arm_link" gravcomp="1.0"/>
-      <modify_element type="body" name="${tf_prefix}left_ur_arm_forearm_link" gravcomp="1.0"/>
-      <modify_element type="body" name="${tf_prefix}left_ur_arm_wrist_1_link" gravcomp="1.0"/>
-      <modify_element type="body" name="${tf_prefix}left_ur_arm_wrist_2_link" gravcomp="1.0"/>
-      <modify_element type="body" name="${tf_prefix}left_ur_arm_wrist_3_link" gravcomp="1.0"/>
+      <!-- Apply default classes to Phoebe joints. -->
+      <modify_element type="joint" name="${tf_prefix}left_ewellix_lift_lower_to_higher" class="size5"/>
+      <modify_element type="joint" name="${tf_prefix}left_ur_arm_shoulder_pan_joint" class="size4"/>
+      <modify_element type="joint" name="${tf_prefix}left_ur_arm_shoulder_lift_joint" class="size4"/>
+      <modify_element type="joint" name="${tf_prefix}left_ur_arm_elbow_joint" class="size3_limited"/>
+      <modify_element type="joint" name="${tf_prefix}left_ur_arm_wrist_1_joint" class="size2"/>
+      <modify_element type="joint" name="${tf_prefix}left_ur_arm_wrist_2_joint" class="size2"/>
+      <modify_element type="joint" name="${tf_prefix}left_ur_arm_wrist_3_joint" class="size2"/>
+      <modify_element type="joint" name="${tf_prefix}right_ewellix_lift_lower_to_higher" class="size5"/>
+      <modify_element type="joint" name="${tf_prefix}right_ur_arm_shoulder_pan_joint" class="size4"/>
+      <modify_element type="joint" name="${tf_prefix}right_ur_arm_shoulder_lift_joint" class="size4"/>
+      <modify_element type="joint" name="${tf_prefix}right_ur_arm_elbow_joint" class="size3_limited"/>
+      <modify_element type="joint" name="${tf_prefix}right_ur_arm_wrist_1_joint" class="size2"/>
+      <modify_element type="joint" name="${tf_prefix}right_ur_arm_wrist_2_joint" class="size2"/>
+      <modify_element type="joint" name="${tf_prefix}right_ur_arm_wrist_3_joint" class="size2"/>
       <xacro:if value="${left_hand_type == 'hande'}">
         <modify_element type="joint" name="${tf_prefix}left_finger_1_joint" armature="0.5" frictionloss="5.0" />
         <modify_element type="joint" name="${tf_prefix}left_finger_2_joint" armature="0.5" frictionloss="5.0" />
-        <modify_element type="body" name="${tf_prefix}left_finger_1_link" gravcomp="1.0"/>
-        <modify_element type="body" name="${tf_prefix}left_finger_2_link" gravcomp="1.0"/>
       </xacro:if>
       <xacro:if value="${right_hand_type == 'hande'}">
         <modify_element type="joint" name="${tf_prefix}right_finger_1_joint" armature="0.5" frictionloss="5.0" />
         <modify_element type="joint" name="${tf_prefix}right_finger_2_joint" armature="0.5" frictionloss="5.0" />
-        <modify_element type="body" name="${tf_prefix}right_finger_1_link" gravcomp="1.0"/>
-        <modify_element type="body" name="${tf_prefix}right_finger_2_link" gravcomp="1.0"/>
       </xacro:if>
-      <modify_element type="body" name="${tf_prefix}left_finger_1_link" gravcomp="1.0"/>
-      <modify_element type="body" name="${tf_prefix}left_finger_2_link" gravcomp="1.0"/>
-      <modify_element type="body" name="${tf_prefix}right_ewellix_lift_higher_link" gravcomp="1.0"/>
-      <modify_element type="body" name="${tf_prefix}right_ewellix_lift_middle_link" gravcomp="1.0"/>
-      <modify_element type="body" name="${tf_prefix}right_ur_arm_shoulder_link" gravcomp="1.0"/>
-      <modify_element type="body" name="${tf_prefix}right_ur_arm_upper_arm_link" gravcomp="1.0"/>
-      <modify_element type="body" name="${tf_prefix}right_ur_arm_forearm_link" gravcomp="1.0"/>
-      <modify_element type="body" name="${tf_prefix}right_ur_arm_wrist_1_link" gravcomp="1.0"/>
-      <modify_element type="body" name="${tf_prefix}right_ur_arm_wrist_2_link" gravcomp="1.0"/>
-      <modify_element type="body" name="${tf_prefix}right_ur_arm_wrist_3_link" gravcomp="1.0"/>
   </xacro:macro>
 </robot>

File: phoebe_mujoco_config/urdf/phoebe_mujoco_raw_inputs.xacro (robot description, xacro)
@@ -17,10 +17,14 @@
             <position ctrlrange="-6.2831 6.2831"/>
             <general biastype="affine" ctrlrange="-6.2831 6.2831"/>
+            <default class="size5">
+                <joint actuatorfrclimited="true" actuatorfrcrange="-1000 1000"/>
+                <position ctrlrange="0.0 0.7" kp="75000" dampratio="1.0" forcerange="-1000 1000"/>
+            </default>
             <default class="size4">
-                <joint damping="10"/>
+                <joint damping="10" actuatorgravcomp="true"/>
                 <general forcerange="-330 330" gainprm="100000" biasprm="0 -100000 -10000"/>
             </default>
             <default class="size3">
-                <joint damping="5"/>
+                <joint damping="5" actuatorgravcomp="true"/>
                 <general forcerange="-150 150" gainprm="100000" biasprm="0 -100000 -5000"/>
                 <default class="size3_limited">
@@ -30,5 +34,5 @@
             </default>
             <default class="size2">
-                <joint damping="2"/>
+                <joint damping="2" actuatorgravcomp="true" />
                 <general forcerange="-56 56" gainprm="10000" biasprm="0 -10000 -1000"/>
             </default>
@@ -54,8 +58,4 @@
     </default>
     <actuator>
-        <xacro:unless value="${use_left_static_pedestal}">
-            <position joint="${tf_prefix}left_ewellix_lift_lower_to_higher" name="${tf_prefix}left_ewellix_lift_lower_to_higher" kp="75000" dampratio="1.0" ctrlrange="0.0 0.7" />
-        </xacro:unless>
-        <position joint="${tf_prefix}right_ewellix_lift_lower_to_higher" name="${tf_prefix}right_ewellix_lift_lower_to_higher" kp="75000" dampratio="1.0" ctrlrange="0.0 0.7" />
         <xacro:if value="${right_hand_type == 'hande'}">
             <position tendon="${tf_prefix}right_split" name="${tf_prefix}right_finger_1_joint" kp="10000" dampratio="10.0" ctrlrange="0.0 0.025" forcerange="-130 130"/>
@@ -70,4 +70,5 @@
             <general biastype="affine" name="${tf_prefix}left_robotiq_85_left_knuckle_joint" tendon="${tf_prefix}left_split" forcerange="-10 10" ctrlrange="0 0.8" gainprm="100 0 0" biasprm="0 -100 -25"/>
         </xacro:if>
+        <position class="size5" name="${tf_prefix}left_ewellix_lift_lower_to_higher" joint="${tf_prefix}left_ewellix_lift_lower_to_higher"/>
         <general class="size4" name="${tf_prefix}left_ur_arm_shoulder_pan_joint" joint="${tf_prefix}left_ur_arm_shoulder_pan_joint"/>
         <general class="size4" name="${tf_prefix}left_ur_arm_shoulder_lift_joint" joint="${tf_prefix}left_ur_arm_shoulder_lift_joint"/>
@@ -76,4 +77,5 @@
         <general class="size2" name="${tf_prefix}left_ur_arm_wrist_2_joint" joint="${tf_prefix}left_ur_arm_wrist_2_joint"/>
         <general class="size2" name="${tf_prefix}left_ur_arm_wrist_3_joint" joint="${tf_prefix}left_ur_arm_wrist_3_joint"/>
+        <position class="size5" name="${tf_prefix}right_ewellix_lift_lower_to_higher" joint="${tf_prefix}right_ewellix_lift_lower_to_higher"/>
         <general class="size4" name="${tf_prefix}right_ur_arm_shoulder_pan_joint" joint="${tf_prefix}right_ur_arm_shoulder_pan_joint"/>
         <general class="size4" name="${tf_prefix}right_ur_arm_shoulder_lift_joint" joint="${tf_prefix}right_ur_arm_shoulder_lift_joint"/>

Commit message: fixing gravcomp and joint classifications

File: phoebe_mujoco_config/urdf/phoebe_mujoco_processed_inputs.xacro (robot description, xacro)
@@ -31,17 +31,17 @@
         <modify_element type="joint" name="${tf_prefix}left_ewellix_lift_lower_to_higher" class="size5"/>
       </xacro:unless>
-      <modify_element type="joint" name="${tf_prefix}left_ur_arm_shoulder_pan_joint" class="size4"/>
-      <modify_element type="joint" name="${tf_prefix}left_ur_arm_shoulder_lift_joint" class="size4"/>
+      <modify_element type="joint" name="${tf_prefix}left_ur_arm_shoulder_pan_joint" class="size3"/>
+      <modify_element type="joint" name="${tf_prefix}left_ur_arm_shoulder_lift_joint" class="size3"/>
       <modify_element type="joint" name="${tf_prefix}left_ur_arm_elbow_joint" class="size3_limited"/>
-      <modify_element type="joint" name="${tf_prefix}left_ur_arm_wrist_1_joint" class="size2"/>
-      <modify_element type="joint" name="${tf_prefix}left_ur_arm_wrist_2_joint" class="size2"/>
-      <modify_element type="joint" name="${tf_prefix}left_ur_arm_wrist_3_joint" class="size2"/>
+      <modify_element type="joint" name="${tf_prefix}left_ur_arm_wrist_1_joint" class="size1"/>
+      <modify_element type="joint" name="${tf_prefix}left_ur_arm_wrist_2_joint" class="size1"/>
+      <modify_element type="joint" name="${tf_prefix}left_ur_arm_wrist_3_joint" class="size1"/>
       <modify_element type="joint" name="${tf_prefix}right_ewellix_lift_lower_to_higher" class="size5"/>
-      <modify_element type="joint" name="${tf_prefix}right_ur_arm_shoulder_pan_joint" class="size4"/>
-      <modify_element type="joint" name="${tf_prefix}right_ur_arm_shoulder_lift_joint" class="size4"/>
+      <modify_element type="joint" name="${tf_prefix}right_ur_arm_shoulder_pan_joint" class="size3"/>
+      <modify_element type="joint" name="${tf_prefix}right_ur_arm_shoulder_lift_joint" class="size3"/>
       <modify_element type="joint" name="${tf_prefix}right_ur_arm_elbow_joint" class="size3_limited"/>
-      <modify_element type="joint" name="${tf_prefix}right_ur_arm_wrist_1_joint" class="size2"/>
-      <modify_element type="joint" name="${tf_prefix}right_ur_arm_wrist_2_joint" class="size2"/>
-      <modify_element type="joint" name="${tf_prefix}right_ur_arm_wrist_3_joint" class="size2"/>
+      <modify_element type="joint" name="${tf_prefix}right_ur_arm_wrist_1_joint" class="size1"/>
+      <modify_element type="joint" name="${tf_prefix}right_ur_arm_wrist_2_joint" class="size1"/>
+      <modify_element type="joint" name="${tf_prefix}right_ur_arm_wrist_3_joint" class="size1"/>
       <xacro:if value="${left_hand_type == 'hande'}">
         <modify_element type="joint" name="${tf_prefix}left_finger_1_joint" armature="0.5" frictionloss="5.0" />
@@ -52,4 +52,29 @@
         <modify_element type="joint" name="${tf_prefix}right_finger_2_joint" armature="0.5" frictionloss="5.0" />
       </xacro:if>
+      <!-- Add gravcomp so that control will make the joints move about the desired position-->
+      <modify_element type="body" name="${tf_prefix}left_ewellix_lift_higher_link" gravcomp="1.0"/>
+      <modify_element type="body" name="${tf_prefix}left_ewellix_lift_middle_link" gravcomp="1.0"/>
+      <modify_element type="body" name="${tf_prefix}left_ur_arm_shoulder_link" gravcomp="1.0"/>
+      <modify_element type="body" name="${tf_prefix}left_ur_arm_upper_arm_link" gravcomp="1.0"/>
+      <modify_element type="body" name="${tf_prefix}left_ur_arm_forearm_link" gravcomp="1.0"/>
+      <modify_element type="body" name="${tf_prefix}left_ur_arm_wrist_1_link" gravcomp="1.0"/>
+      <modify_element type="body" name="${tf_prefix}left_ur_arm_wrist_2_link" gravcomp="1.0"/>
+      <modify_element type="body" name="${tf_prefix}left_ur_arm_wrist_3_link" gravcomp="1.0"/>
+      <xacro:if value="${left_hand_type == 'hande'}">
+        <modify_element type="body" name="${tf_prefix}left_finger_1_link" gravcomp="1.0"/>
+        <modify_element type="body" name="${tf_prefix}left_finger_2_link" gravcomp="1.0"/>
+      </xacro:if>
+      <modify_element type="body" name="${tf_prefix}right_ewellix_lift_higher_link" gravcomp="1.0"/>
+      <modify_element type="body" name="${tf_prefix}right_ewellix_lift_middle_link" gravcomp="1.0"/>
+      <modify_element type="body" name="${tf_prefix}right_ur_arm_shoulder_link" gravcomp="1.0"/>
+      <modify_element type="body" name="${tf_prefix}right_ur_arm_upper_arm_link" gravcomp="1.0"/>
+      <modify_element type="body" name="${tf_prefix}right_ur_arm_forearm_link" gravcomp="1.0"/>
+      <modify_element type="body" name="${tf_prefix}right_ur_arm_wrist_1_link" gravcomp="1.0"/>
+      <modify_element type="body" name="${tf_prefix}right_ur_arm_wrist_2_link" gravcomp="1.0"/>
+      <modify_element type="body" name="${tf_prefix}right_ur_arm_wrist_3_link" gravcomp="1.0"/>
+      <xacro:if value="${left_hand_type == 'hande'}">
+        <modify_element type="body" name="${tf_prefix}right_finger_1_link" gravcomp="1.0"/>
+        <modify_element type="body" name="${tf_prefix}right_finger_2_link" gravcomp="1.0"/>
+      </xacro:if>
   </xacro:macro>
 </robot>

File: phoebe_mujoco_config/urdf/phoebe_mujoco_raw_inputs.xacro (robot description, xacro)
@@ -15,5 +15,5 @@
         <default class="phoebe">
             <material specular="0.5" shininess="0.25"/>
-            <joint axis="0 1 0" range="-6.28319 6.28319" armature="0.1"/>
+            <joint axis="0 1 0" range="-6.28319 6.28319" armature="0.1" actuatorgravcomp="true"/>
             <general ctrlrange="-6.2831 6.2831"/>
             <default class="size5">
@@ -22,9 +22,9 @@
             </default>
             <default class="size4">
-                <joint damping="10" actuatorgravcomp="true"/>
+                <joint damping="10"/>
                 <general forcerange="-330 330" ctrlrange="-330 330"/>
             </default>
             <default class="size3">
-                <joint damping="5" actuatorgravcomp="true"/>
+                <joint damping="5"/>
                 <general forcerange="-150 150" ctrlrange="-150 150"/>
                 <default class="size3_limited">
@@ -33,9 +33,9 @@
             </default>
             <default class="size2">
-                <joint damping="2" actuatorgravcomp="true" />
+                <joint damping="2" />
                 <general forcerange="-56 56" ctrlrange="-56 56"/>
             </default>
             <default class="size1">
-                <joint damping="1" actuatorgravcomp="true" />
+                <joint damping="1" />
                 <general forcerange="-28 28" ctrlrange="-28 28"/>
             </default>

Commit message: adding mujoco collision objects for objects of interest

File: phoebe_mujoco_config/urdf/phoebe_mujoco_processed_inputs.xacro (robot description, xacro)
@@ -89,4 +89,49 @@
         <modify_element type="body" name="${tf_prefix}right_finger_2_link" gravcomp="1.0"/>
       </xacro:if>
+      <replace_collision link="${tf_prefix}rear_shelf" stage="urdf">
+        <collision>
+          <geometry>
+            <mesh filename="package://phoebe_description/meshes/visual/jaco01_meshes/shelf.STL"/>
+          </geometry>
+        </collision>
+      </replace_collision>
+      <replace_collision link="${tf_prefix}front_shelf" stage="urdf">
+        <collision>
+          <geometry>
+            <mesh filename="package://phoebe_description/meshes/visual/jaco01_meshes/shelf.STL"/>
+          </geometry>
+        </collision>
+      </replace_collision>
+      <replace_collision link="${tf_prefix}right_wifi_antenna" stage="urdf">
+        <collision>
+          <geometry>
+            <mesh filename="package://phoebe_description/meshes/visual/jaco01_meshes/wifi_antenna.STL"/>
+          </geometry>
+        </collision>
+      </replace_collision>
+      <replace_collision link="${tf_prefix}left_wifi_antenna" stage="urdf">
+        <collision>
+          <geometry>
+            <mesh filename="package://phoebe_description/meshes/visual/jaco01_meshes/wifi_antenna.STL"/>
+          </geometry>
+        </collision>
+      </replace_collision>
+      <replace_collision link="${tf_prefix}right_monitor" stage="urdf">
+        <collision>
+          <geometry>
+            <mesh filename="package://phoebe_description/meshes/visual/jaco01_meshes/monitor.STL"/>
+          </geometry>
+        </collision>
+      </replace_collision>
+      <replace_collision link="${tf_prefix}left_monitor" stage="urdf">
+        <collision>
+          <geometry>
+            <mesh filename="package://phoebe_description/meshes/visual/jaco01_meshes/monitor.STL"/>
+          </geometry>
+        </collision>
+      </replace_collision>
+      <xacro:include filename="$(find dextivr_hande_description)/urdf/dextivr_hande.xacro"/>
+      <xacro:hande_gripper_base_link_mujoco_collision_mesh tf_prefix="${tf_prefix}left_"/>
+      <xacro:hande_gripper_base_link_mujoco_collision_mesh tf_prefix="${tf_prefix}right_"/>
   </xacro:macro>
 </robot>
