Commit message: parameterizing mujoco things for static pedestal

File: phoebe_mujoco_config/urdf/phoebe_mujoco_raw_inputs.xacro (robot description, xacro)
@@ -1,5 +1,7 @@
 <?xml version="1.0"?>
 <robot xmlns:xacro="http://wiki.ros.org/xacro">
-  <xacro:macro name="phoebe_mujoco_raw_inputs">
+  <xacro:macro name="phoebe_mujoco_raw_inputs" params="
+    use_left_static_pedestal:=false
+  ">
     <raw_inputs>
         <option integrator="implicitfast" impratio="20" cone="elliptic" noslip_iterations="5">
@@ -46,5 +48,7 @@
         </default>
         <actuator>
-            <position joint="left_ewellix_lift_lower_to_higher" name="left_ewellix_lift_lower_to_higher" kp="75000" dampratio="1.0" ctrlrange="0.0 0.7" />
+            <xacro:unless value="${use_left_static_pedestal}">
+                <position joint="left_ewellix_lift_lower_to_higher" name="left_ewellix_lift_lower_to_higher" kp="75000" dampratio="1.0" ctrlrange="0.0 0.7" />
+            </xacro:unless>
             <position joint="right_ewellix_lift_lower_to_higher" name="right_ewellix_lift_lower_to_higher" kp="75000" dampratio="1.0" ctrlrange="0.0 0.7" />
             <position tendon="right_split" name="right_robotiq_85_left_knuckle_joint" kp="100000" dampratio="10.0" ctrlrange="0.0 0.8" forcerange="-20 20"/>
@@ -68,6 +72,8 @@
         </actuator>
         <contact>
-            <exclude body1="base_link" body2="left_ewellix_lift_higher_link"/>
-            <exclude body1="base_link" body2="left_ewellix_lift_middle_link"/>
+            <xacro:unless value="${use_left_static_pedestal}">
+                <exclude body1="base_link" body2="left_ewellix_lift_higher_link"/>
+                <exclude body1="base_link" body2="left_ewellix_lift_middle_link"/>\
+            </xacro:unless>
             <exclude body1="base_link" body2="right_ewellix_lift_higher_link"/>
             <exclude body1="base_link" body2="right_ewellix_lift_middle_link"/>
@@ -153,10 +159,12 @@
         </contact>
         <!-- Same logic as above... but for liftkits -->
-        <tendon>
-            <fixed name="left_lift_middle_mimic_higher">
-            <joint joint="left_ewellix_lift_lower_to_higher" coef="0.5"/>
-            <joint joint="left_middle_mimic_higher" coef="0.5"/>
-            </fixed>
-        </tendon>
+        <xacro:unless value="${use_left_static_pedestal}">
+            <tendon>
+                <fixed name="left_lift_middle_mimic_higher">
+                <joint joint="left_ewellix_lift_lower_to_higher" coef="0.5"/>
+                <joint joint="left_middle_mimic_higher" coef="0.5"/>
+                </fixed>
+            </tendon>
+        </xacro:unless>
         <tendon>
             <fixed name="right_lift_middle_mimic_higher">
@@ -166,7 +174,9 @@
         </tendon>
         <!-- The mimic joint is scaled by 50% in the URDF -->
-        <equality>
-            <joint name="left_upper_mimic_lower" joint1="left_ewellix_lift_lower_to_higher" joint2="left_middle_mimic_higher" polycoef="0 2 0 0 0"/>
-        </equality>
+        <xacro:unless value="${use_left_static_pedestal}">
+            <equality>
+                <joint name="left_upper_mimic_lower" joint1="left_ewellix_lift_lower_to_higher" joint2="left_middle_mimic_higher" polycoef="0 2 0 0 0"/>
+            </equality>
+        </xacro:unless>
         <equality>
             <joint name="right_upper_mimic_lower" joint1="right_ewellix_lift_lower_to_higher" joint2="right_middle_mimic_higher" polycoef="0 2 0 0 0"/>

Commit message: re-adding wheel contact params bc apparently they got lost at some point

File: phoebe_mujoco_config/urdf/phoebe_mujoco_raw_inputs.xacro (robot description, xacro)
@@ -15,33 +15,36 @@
                 <general biastype="affine" ctrlrange="-6.2831 6.2831"/>
                 <default class="size4">
-                <joint damping="10"/>
-                <general forcerange="-330 330" gainprm="100000" biasprm="0 -100000 -10000"/>
+                    <joint damping="10"/>
+                    <general forcerange="-330 330" gainprm="100000" biasprm="0 -100000 -10000"/>
                 </default>
                 <default class="size3">
-                <joint damping="5"/>
-                <general forcerange="-150 150" gainprm="100000" biasprm="0 -100000 -5000"/>
-                <default class="size3_limited">
-                    <joint range="-3.1415 3.1415"/>
-                    <general ctrlrange="-3.1415 3.1415"/>
-                </default>
+                    <joint damping="5"/>
+                    <general forcerange="-150 150" gainprm="100000" biasprm="0 -100000 -5000"/>
+                    <default class="size3_limited">
+                        <joint range="-3.1415 3.1415"/>
+                        <general ctrlrange="-3.1415 3.1415"/>
+                    </default>
                 </default>
                 <default class="size2">
-                <joint damping="2"/>
-                <general forcerange="-56 56" gainprm="100000" biasprm="0 -100000 -1000"/>
+                    <joint damping="2"/>
+                    <general forcerange="-56 56" gainprm="100000" biasprm="0 -100000 -1000"/>
                 </default>
                 <default class="visual">
-                <geom group="2" type="mesh" contype="0" conaffinity="0"/>
+                    <geom group="2" type="mesh" contype="0" conaffinity="0"/>
                 </default>
                 <default class="collision">
-                <geom group="3" type="mesh"/>
-                <default class="rubber">
-                    <geom condim="4" friction="5 1.0 1.0" priority="1" solimp="0.9 0.95 0.001" solref="0.002 1" conaffinity="1"/>
-                </default>
+                    <geom group="3" type="mesh"/>
+                    <default class="wheels">
+                        <geom condim="3" friction="0.5 0.005 0.0001" solimp="0.95 0.99 0.001 0.1 6"/>
+                    </default>
+                    <default class="rubber">
+                        <geom condim="4" friction="5 1.0 1.0" priority="1" solimp="0.9 0.95 0.001" solref="0.002 1" conaffinity="1"/>
+                    </default>
                 </default>
                 <default class="right_spring_link">
-                <joint range="-0.9 0.29670597283" armature="0.001" stiffness="0.05" springref="-2.62" damping="0.00125"/>
+                    <joint range="-0.9 0.29670597283" armature="0.001" stiffness="0.05" springref="-2.62" damping="0.00125"/>
                 </default>
                 <default class="left_spring_link">
-                <joint range="-0.29670597283 0.9" armature="0.001" stiffness="0.05" springref="2.62" damping="0.00125"/>
+                    <joint range="-0.29670597283 0.9" armature="0.001" stiffness="0.05" springref="2.62" damping="0.00125"/>
                 </default>
             </default>
@@ -74,5 +77,5 @@
             <xacro:unless value="${use_left_static_pedestal}">
                 <exclude body1="base_link" body2="left_ewellix_lift_higher_link"/>
-                <exclude body1="base_link" body2="left_ewellix_lift_middle_link"/>\
+                <exclude body1="base_link" body2="left_ewellix_lift_middle_link"/>
             </xacro:unless>
             <exclude body1="base_link" body2="right_ewellix_lift_higher_link"/>

Commit message: More prefixes

File: phoebe_mujoco_config/urdf/phoebe_mujoco_raw_inputs.xacro (robot description, xacro)
@@ -127,5 +127,5 @@
     </tendon>
     <equality>
-        <joint joint1="left_finger_1_joint" joint2="left_finger_2_joint" polycoef="0 1 0 0 0" solimp="0.95 0.99 0.001" solref="0.005 1"/>
+        <joint joint1="${tf_prefix}left_finger_1_joint" joint2="${tf_prefix}left_finger_2_joint" polycoef="0 1 0 0 0" solimp="0.95 0.99 0.001" solref="0.005 1"/>
     </equality>
     <!-- right hand - 2f-85 -->
@@ -139,5 +139,5 @@
         <connect anchor="-0.0371575 0.0 0.043422" body1="${tf_prefix}right_robotiq_85_right_inner_knuckle_link" body2="${tf_prefix}right_robotiq_85_right_finger_tip_link" solimp="0.95 0.99 0.001" solref="0.005 1"/>
         <connect anchor="0.0371575 0.0 0.043422" body1="${tf_prefix}right_robotiq_85_left_inner_knuckle_link" body2="${tf_prefix}right_robotiq_85_left_finger_tip_link" solimp="0.95 0.99 0.001" solref="0.005 1"/>
-        <joint joint1="right_robotiq_85_left_knuckle_joint" joint2="right_robotiq_85_right_knuckle_joint" polycoef="0 -1 0 0 0" solimp="0.95 0.99 0.001"
+        <joint joint1="${tf_prefix}right_robotiq_85_left_knuckle_joint" joint2="${tf_prefix}right_robotiq_85_right_knuckle_joint" polycoef="0 -1 0 0 0" solimp="0.95 0.99 0.001"
         solref="0.005 1"/>
     </equality>
@@ -184,21 +184,21 @@
     </xacro:unless>
     <equality>
-        <joint name="${tf_prefix}right_upper_mimic_lower" joint1="right_ewellix_lift_lower_to_higher" joint2="right_middle_mimic_higher" polycoef="0 2 0 0 0"/>
+        <joint name="${tf_prefix}right_upper_mimic_lower" joint1="${tf_prefix}right_ewellix_lift_lower_to_higher" joint2="${tf_prefix}right_middle_mimic_higher" polycoef="0 2 0 0 0"/>
     </equality>
     <sensor>
-        <force name="${tf_prefix}left_ur_arm_tcp_fts_sensor_force" site="left_ur_arm_ft_frame"/>
-        <torque name="${tf_prefix}left_ur_arm_tcp_fts_sensor_torque" site="left_ur_arm_ft_frame"/>
-    </sensor>
-    <sensor>
-        <force name="${tf_prefix}right_ur_arm_tcp_fts_sensor_force" site="right_ur_arm_ft_frame"/>
-        <torque name="${tf_prefix}right_ur_arm_tcp_fts_sensor_torque" site="right_ur_arm_ft_frame"/>
-    </sensor>
-    <sensor>
-        <framequat name="${tf_prefix}imu_sensor_quat" objtype="site" objname="imu_0_link" />
-        <gyro name="${tf_prefix}imu_sensor_gyro" site="imu_0_link" />
-        <accelerometer name="${tf_prefix}imu_sensor_accel" site="imu_0_link" />
-    </sensor>
-    <sensor>
-        <rangefinder name="${tf_prefix}lidar2d_0" site="lidar2d_0"/>
+        <force name="${tf_prefix}left_ur_arm_tcp_fts_sensor_force" site="${tf_prefix}left_ur_arm_ft_frame"/>
+        <torque name="${tf_prefix}left_ur_arm_tcp_fts_sensor_torque" site="${tf_prefix}left_ur_arm_ft_frame"/>
+    </sensor>
+    <sensor>
+        <force name="${tf_prefix}right_ur_arm_tcp_fts_sensor_force" site="${tf_prefix}right_ur_arm_ft_frame"/>
+        <torque name="${tf_prefix}right_ur_arm_tcp_fts_sensor_torque" site="${tf_prefix}right_ur_arm_ft_frame"/>
+    </sensor>
+    <sensor>
+        <framequat name="${tf_prefix}imu_sensor_quat" objtype="site" objname="${tf_prefix}imu_0_link" />
+        <gyro name="${tf_prefix}imu_sensor_gyro" site="${tf_prefix}imu_0_link" />
+        <accelerometer name="${tf_prefix}imu_sensor_accel" site="${tf_prefix}imu_0_link" />
+    </sensor>
+    <sensor>
+        <rangefinder name="${tf_prefix}lidar2d_0" site="${tf_prefix}lidar2d_0"/>
     </sensor>
   </xacro:macro>

Commit message: Missing prefix

File: phoebe_mujoco_config/urdf/phoebe_mujoco_raw_inputs.xacro (robot description, xacro)
@@ -241,5 +241,5 @@
     <xacro:unless value="${use_left_static_pedestal}">
         <equality>
-            <joint name="${tf_prefix}left_upper_mimic_lower" joint1="left_ewellix_lift_lower_to_higher" joint2="left_middle_mimic_higher" polycoef="0 2 0 0 0"/>
+            <joint name="${tf_prefix}left_upper_mimic_lower" joint1="${tf_prefix}left_ewellix_lift_lower_to_higher" joint2="${tf_prefix}left_middle_mimic_higher" polycoef="0 2 0 0 0"/>
         </equality>
     </xacro:unless>
