Commit message: support pid controllers and fix actuator configs

File: phoebe_mujoco_config/urdf/phoebe_mujoco_raw_inputs.xacro (robot description, xacro)
@@ -16,6 +16,5 @@
             <material specular="0.5" shininess="0.25"/>
             <joint axis="0 1 0" range="-6.28319 6.28319" armature="0.1"/>
-            <position ctrlrange="-6.2831 6.2831"/>
-            <general biastype="affine" ctrlrange="-6.2831 6.2831"/>
+            <general ctrlrange="-6.2831 6.2831"/>
             <default class="size5">
                 <joint actuatorfrclimited="true" actuatorfrcrange="-1000 1000"/>
@@ -24,17 +23,20 @@
             <default class="size4">
                 <joint damping="10" actuatorgravcomp="true"/>
-                <general forcerange="-330 330" gainprm="100000" biasprm="0 -100000 -10000"/>
+                <general forcerange="-330 330" ctrlrange="-330 330"/>
             </default>
             <default class="size3">
                 <joint damping="5" actuatorgravcomp="true"/>
-                <general forcerange="-150 150" gainprm="100000" biasprm="0 -100000 -5000"/>
+                <general forcerange="-150 150" ctrlrange="-150 150"/>
                 <default class="size3_limited">
                     <joint range="-3.1415 3.1415"/>
-                    <general ctrlrange="-3.1415 3.1415"/>
                 </default>
             </default>
             <default class="size2">
                 <joint damping="2" actuatorgravcomp="true" />
-                <general forcerange="-56 56" gainprm="10000" biasprm="0 -10000 -1000"/>
+                <general forcerange="-56 56" ctrlrange="-56 56"/>
+            </default>
+            <default class="size1">
+                <joint damping="1" actuatorgravcomp="true" />
+                <general forcerange="-28 28" ctrlrange="-28 28"/>
             </default>
             <default class="${defaults_prefix}visual">
@@ -74,17 +76,17 @@
             <position class="size5" name="${tf_prefix}left_ewellix_lift_lower_to_higher" joint="${tf_prefix}left_ewellix_lift_lower_to_higher"/>
         </xacro:unless>
-        <general class="size4" name="${tf_prefix}left_ur_arm_shoulder_pan_joint" joint="${tf_prefix}left_ur_arm_shoulder_pan_joint"/>
-        <general class="size4" name="${tf_prefix}left_ur_arm_shoulder_lift_joint" joint="${tf_prefix}left_ur_arm_shoulder_lift_joint"/>
-        <general class="size3_limited" name="${tf_prefix}left_ur_arm_elbow_joint" joint="${tf_prefix}left_ur_arm_elbow_joint"/>
-        <general class="size2" name="${tf_prefix}left_ur_arm_wrist_1_joint" joint="${tf_prefix}left_ur_arm_wrist_1_joint"/>
-        <general class="size2" name="${tf_prefix}left_ur_arm_wrist_2_joint" joint="${tf_prefix}left_ur_arm_wrist_2_joint"/>
-        <general class="size2" name="${tf_prefix}left_ur_arm_wrist_3_joint" joint="${tf_prefix}left_ur_arm_wrist_3_joint"/>
+        <motor class="size3" name="${tf_prefix}left_ur_arm_shoulder_pan_joint" joint="${tf_prefix}left_ur_arm_shoulder_pan_joint"/>
+        <motor class="size3" name="${tf_prefix}left_ur_arm_shoulder_lift_joint" joint="${tf_prefix}left_ur_arm_shoulder_lift_joint"/>
+        <motor class="size3_limited" name="${tf_prefix}left_ur_arm_elbow_joint" joint="${tf_prefix}left_ur_arm_elbow_joint"/>
+        <motor class="size1" name="${tf_prefix}left_ur_arm_wrist_1_joint" joint="${tf_prefix}left_ur_arm_wrist_1_joint"/>
+        <motor class="size1" name="${tf_prefix}left_ur_arm_wrist_2_joint" joint="${tf_prefix}left_ur_arm_wrist_2_joint"/>
+        <motor class="size1" name="${tf_prefix}left_ur_arm_wrist_3_joint" joint="${tf_prefix}left_ur_arm_wrist_3_joint"/>
         <position class="size5" name="${tf_prefix}right_ewellix_lift_lower_to_higher" joint="${tf_prefix}right_ewellix_lift_lower_to_higher"/>
-        <general class="size4" name="${tf_prefix}right_ur_arm_shoulder_pan_joint" joint="${tf_prefix}right_ur_arm_shoulder_pan_joint"/>
-        <general class="size4" name="${tf_prefix}right_ur_arm_shoulder_lift_joint" joint="${tf_prefix}right_ur_arm_shoulder_lift_joint"/>
-        <general class="size3_limited" name="${tf_prefix}right_ur_arm_elbow_joint" joint="${tf_prefix}right_ur_arm_elbow_joint"/>
-        <general class="size2" name="${tf_prefix}right_ur_arm_wrist_1_joint" joint="${tf_prefix}right_ur_arm_wrist_1_joint"/>
-        <general class="size2" name="${tf_prefix}right_ur_arm_wrist_2_joint" joint="${tf_prefix}right_ur_arm_wrist_2_joint"/>
-        <general class="size2" name="${tf_prefix}right_ur_arm_wrist_3_joint" joint="${tf_prefix}right_ur_arm_wrist_3_joint"/>
+        <motor class="size3" name="${tf_prefix}right_ur_arm_shoulder_pan_joint" joint="${tf_prefix}right_ur_arm_shoulder_pan_joint"/>
+        <motor class="size3" name="${tf_prefix}right_ur_arm_shoulder_lift_joint" joint="${tf_prefix}right_ur_arm_shoulder_lift_joint"/>
+        <motor class="size3_limited" name="${tf_prefix}right_ur_arm_elbow_joint" joint="${tf_prefix}right_ur_arm_elbow_joint"/>
+        <motor class="size1" name="${tf_prefix}right_ur_arm_wrist_1_joint" joint="${tf_prefix}right_ur_arm_wrist_1_joint"/>
+        <motor class="size1" name="${tf_prefix}right_ur_arm_wrist_2_joint" joint="${tf_prefix}right_ur_arm_wrist_2_joint"/>
+        <motor class="size1" name="${tf_prefix}right_ur_arm_wrist_3_joint" joint="${tf_prefix}right_ur_arm_wrist_3_joint"/>
         <!-- Nominally include the wheels -->
         <xacro:unless value="${include_world_joints}">

Commit message: Fix wheel joint limits in MuJoCo

File: phoebe_mujoco_config/urdf/phoebe_mujoco_raw_inputs.xacro (robot description, xacro)
@@ -15,6 +15,5 @@
         <default class="phoebe">
             <material specular="0.5" shininess="0.25"/>
-            <joint axis="0 1 0" range="-6.28319 6.28319" armature="0.1" actuatorgravcomp="true"/>
-            <general ctrlrange="-6.2831 6.2831"/>
+            <joint axis="0 1 0" armature="0.1" actuatorgravcomp="true"/>
             <default class="size5">
                 <joint actuatorfrclimited="true" actuatorfrcrange="-1000 1000"/>

Commit message: Remove the joint axis arg

File: phoebe_mujoco_config/urdf/phoebe_mujoco_raw_inputs.xacro (robot description, xacro)
@@ -15,5 +15,5 @@
         <default class="phoebe">
             <material specular="0.5" shininess="0.25"/>
-            <joint axis="0 1 0" armature="0.1" actuatorgravcomp="true"/>
+            <joint armature="0.1" actuatorgravcomp="true"/>
             <default class="size5">
                 <joint actuatorfrclimited="true" actuatorfrcrange="-1000 1000"/>
