Commit message: remove duplicate tf_prefix

File: phoebe_moveit_config/config/phoebe_macro.srdf.xacro (robot description, xacro)
@@ -16,8 +16,8 @@
       <!--SUBGROUPS: Groups can also be formed by referencing to already defined group names-->
       <xacro:if value="$(arg calibration_mode)">
-          <xacro:property name="tip_link_name" value="${tf_prefix}calibration_plate_robot_side"/>
+          <xacro:property name="tip_link_name" value="calibration_plate_robot_side"/>
       </xacro:if>
       <xacro:unless value="$(arg calibration_mode)">
-          <xacro:property name="tip_link_name" value="${tf_prefix}grasp_frame"/>
+          <xacro:property name="tip_link_name" value="grasp_frame"/>
       </xacro:unless>
       <group name="left_push1">

Commit message: parameterizing moveit config. handes seem to work but 2f85 mujoco is borked somehow

File: phoebe_moveit_config/config/phoebe_macro.srdf.xacro (robot description, xacro)
@@ -9,4 +9,6 @@
     calibration_mode=false
     use_left_static_pedestal=false
+    left_hand_type='hande'
+    right_hand_type='hande'
     ">
       <!--GROUPS: Representation of a set of joints and links. This can be useful for specifying DOF to plan for, defining arms, end effectors, etc-->
@@ -49,10 +51,26 @@
       </group>
       <xacro:unless value="$(arg calibration_mode)">
+        <!-- left hand -->
+        <xacro:if value="${left_hand_type == 'hande'}">
           <group name="left_hande">
-              <joint name="${tf_prefix}left_finger_1_joint"/>
+            <joint name="${tf_prefix}left_finger_1_joint"/>
           </group>
+        </xacro:if>
+        <xacro:if value="${left_hand_type == '2f85'}">
+          <group name="left_hande">
+            <joint name="${tf_prefix}left_robotiq_85_left_knuckle_joint"/>
+          </group>
+        </xacro:if>
+        <!-- right hand -->
+        <xacro:if value="${right_hand_type == 'hande'}">
           <group name="right_hande">
-              <joint name="${tf_prefix}right_robotiq_85_left_knuckle_joint"/>
+            <joint name="${tf_prefix}right_finger_1_joint"/>
           </group>
+        </xacro:if>
+        <xacro:if value="${right_hand_type == '2f85'}">
+          <group name="right_hande">
+            <joint name="${tf_prefix}right_robotiq_85_left_knuckle_joint"/>
+          </group>
+        </xacro:if>
       </xacro:unless>
       <group name="right_lift_ur">
@@ -69,12 +87,34 @@
       </group>
       <group name="left_gripper">
-        <link name="${tf_prefix}left_gripper_base_link"/>
-        <link name="${tf_prefix}left_finger_1_link"/>
-        <link name="${tf_prefix}left_finger_2_link"/>
-        <link name="${tf_prefix}left_grasp_frame" />
-        <joint name="${tf_prefix}left_finger_1_joint"/>
-        <passive_joint name="${tf_prefix}left_finger_2_joint"/>
+        <xacro:if value="${left_hand_type == 'hande'}">
+          <link name="${tf_prefix}left_gripper_base_link"/>
+          <link name="${tf_prefix}left_finger_1_link"/>
+          <link name="${tf_prefix}left_finger_2_link"/>
+          <link name="${tf_prefix}left_grasp_frame" />
+          <joint name="${tf_prefix}left_finger_1_joint"/>
+          <passive_joint name="${tf_prefix}left_finger_2_joint"/>
+        </xacro:if>
+        <xacro:if value="${left_hand_type == '2f85'}">
+          <joint name="${tf_prefix}left_robotiq_85_left_finger_tip_joint"/>
+          <joint name="${tf_prefix}left_robotiq_85_left_finger_joint"/>
+          <joint name="${tf_prefix}left_robotiq_85_left_inner_knuckle_joint"/>
+          <joint name="${tf_prefix}left_robotiq_85_left_knuckle_joint"/>
+          <joint name="${tf_prefix}left_robotiq_85_right_finger_tip_joint"/>
+          <joint name="${tf_prefix}left_robotiq_85_right_finger_joint"/>
+          <joint name="${tf_prefix}left_robotiq_85_right_inner_knuckle_joint"/>
+          <joint name="${tf_prefix}left_robotiq_85_right_knuckle_joint"/>
+          <link name="${tf_prefix}left_grasp_frame"/>
+        </xacro:if>
       </group>
       <group name="right_gripper">
+        <xacro:if value="${right_hand_type == 'hande'}">
+          <link name="${tf_prefix}right_gripper_base_link"/>
+          <link name="${tf_prefix}right_finger_1_link"/>
+          <link name="${tf_prefix}right_finger_2_link"/>
+          <link name="${tf_prefix}right_grasp_frame" />
+          <joint name="${tf_prefix}right_finger_1_joint"/>
+          <passive_joint name="${tf_prefix}right_finger_2_joint"/>
+        </xacro:if>
+        <xacro:if value="${right_hand_type == '2f85'}">
           <joint name="${tf_prefix}right_robotiq_85_left_finger_tip_joint"/>
           <joint name="${tf_prefix}right_robotiq_85_left_finger_joint"/>
@@ -86,4 +126,5 @@
           <joint name="${tf_prefix}right_robotiq_85_right_knuckle_joint"/>
           <link name="${tf_prefix}right_grasp_frame"/>
+        </xacro:if>
       </group>
       <end_effector group="left_gripper" name="left_gripper" parent_link="${tf_prefix}left_ur_arm_tool0"/>
@@ -133,16 +174,38 @@
       <!-- Grippers -->
       <xacro:unless value="$(arg calibration_mode)">
+        <!-- left hand -->
+        <xacro:if value="${left_hand_type == 'hande'}">
           <group_state group="left_hande" name="open">
-              <joint name="${tf_prefix}left_finger_1_joint" value="0.025"/>
+            <joint name="${tf_prefix}left_finger_1_joint" value="0.025"/>
           </group_state>
-          <group_state group="left_hande" name="close">
-              <joint name="${tf_prefix}left_finger_1_joint" value="0"/>
+         <group_state group="left_hande" name="close">
+            <joint name="${tf_prefix}left_finger_1_joint" value="0"/>
           </group_state>
+        </xacro:if>
+        <xacro:if value="${left_hand_type == '2f85'}">
+          <group_state group="left_hande" name="open">
+            <joint name="${tf_prefix}left_robotiq_85_left_knuckle_joint" value="0"/>
+          </group_state>
+         <group_state group="left_hande" name="close">
+            <joint name="${tf_prefix}left_robotiq_85_left_knuckle_joint" value="${radians(45)}"/>
+          </group_state>
+        </xacro:if>
+        <!-- right hand -->
+        <xacro:if value="${right_hand_type == 'hande'}">
           <group_state group="right_hande" name="open">
-              <joint name="${tf_prefix}right_robotiq_85_left_knuckle_joint" value="0"/>
+            <joint name="${tf_prefix}right_finger_1_joint" value="0.025"/>
           </group_state>
-          <group_state group="right_hande" name="close">
-              <joint name="${tf_prefix}right_robotiq_85_left_knuckle_joint" value="${radians(45)}"/>
+         <group_state group="right_hande" name="close">
+            <joint name="${tf_prefix}right_finger_1_joint" value="0"/>
           </group_state>
+        </xacro:if>
+        <xacro:if value="${right_hand_type == '2f85'}">
+          <group_state group="right_hande" name="open">
+            <joint name="${tf_prefix}right_robotiq_85_left_knuckle_joint" value="0"/>
+          </group_state>
+         <group_state group="right_hande" name="close">
+            <joint name="${tf_prefix}right_robotiq_85_left_knuckle_joint" value="${radians(45)}"/>
+          </group_state>
+        </xacro:if>
       </xacro:unless>
       <!-- Lifts -->
@@ -925,4 +988,33 @@
       <disable_collisions link1="${tf_prefix}right_robotiq_85_left_inner_knuckle_link" link2="${tf_prefix}right_robotiq_85_right_knuckle_link" reason="Adjacent"/>
       <disable_collisions link1="${tf_prefix}right_robotiq_85_right_inner_knuckle_link" link2="${tf_prefix}right_robotiq_85_right_knuckle_link" reason="Adjacent"/>
+      <disable_collisions link1="${tf_prefix}left_robotiq_85_base_link" link2="${tf_prefix}left_robotiq_85_left_inner_knuckle_link" reason="Adjacent"/>
+      <disable_collisions link1="${tf_prefix}left_robotiq_85_base_link" link2="${tf_prefix}left_robotiq_85_left_knuckle_link" reason="Adjacent"/>
+      <disable_collisions link1="${tf_prefix}left_robotiq_85_base_link" link2="${tf_prefix}left_robotiq_85_right_inner_knuckle_link" reason="Adjacent"/>
+      <disable_collisions link1="${tf_prefix}left_robotiq_85_base_link" link2="${tf_prefix}left_robotiq_85_right_knuckle_link" reason="Adjacent"/>
+      <disable_collisions link1="${tf_prefix}left_robotiq_85_base_link" link2="${tf_prefix}left_robotiq_hande_cb_adapter" reason="Adjacent"/>
+      <disable_collisions link1="${tf_prefix}left_robotiq_85_base_link" link2="${tf_prefix}left_robotiq_85_right_finger_link" reason="Never"/>
+      <disable_collisions link1="${tf_prefix}left_robotiq_85_base_link" link2="${tf_prefix}left_robotiq_85_left_finger_tip_link" reason="Never"/>
+      <disable_collisions link1="${tf_prefix}left_robotiq_85_base_link" link2="${tf_prefix}left_robotiq_85_base_link" reason="Never"/>
+      <disable_collisions link1="${tf_prefix}left_robotiq_85_base_link" link2="${tf_prefix}left_robotiq_85_right_finger_tip_link" reason="Never"/>
+      <disable_collisions link1="${tf_prefix}left_robotiq_85_base_link" link2="${tf_prefix}left_robotiq_85_left_finger_link" reason="Never"/>
+      <disable_collisions link1="${tf_prefix}left_robotiq_85_base_link" link2="${tf_prefix}left_ur_realsense_mount" reason="Never"/>
+      <disable_collisions link1="${tf_prefix}left_robotiq_85_left_finger_link" link2="${tf_prefix}left_robotiq_85_left_finger_tip_link" reason="Adjacent"/>
+      <disable_collisions link1="${tf_prefix}left_robotiq_85_left_finger_link" link2="${tf_prefix}left_robotiq_85_left_knuckle_link" reason="Adjacent"/>
+      <disable_collisions link1="${tf_prefix}left_robotiq_85_left_finger_tip_link" link2="${tf_prefix}left_robotiq_85_left_inner_knuckle_link" reason="Adjacent"/>
+      <disable_collisions link1="${tf_prefix}left_robotiq_85_left_finger_tip_link" link2="${tf_prefix}left_robotiq_85_right_inner_knuckle_link" reason="Adjacent"/>
+      <disable_collisions link1="${tf_prefix}left_robotiq_85_left_finger_tip_link" link2="${tf_prefix}left_robotiq_85_right_finger_tip_link" reason="Adjacent"/>
+      <disable_collisions link1="${tf_prefix}left_robotiq_85_right_finger_link" link2="${tf_prefix}left_robotiq_85_right_finger_tip_link" reason="Adjacent"/>
+      <disable_collisions link1="${tf_prefix}left_robotiq_85_right_finger_link" link2="${tf_prefix}left_robotiq_85_right_knuckle_link" reason="Adjacent"/>
+      <disable_collisions link1="${tf_prefix}left_robotiq_85_right_finger_tip_link" link2="${tf_prefix}left_robotiq_85_right_inner_knuckle_link" reason="Adjacent"/>
+      <disable_collisions link1="${tf_prefix}left_robotiq_85_left_finger_link" link2="${tf_prefix}left_robotiq_85_left_inner_knuckle_link" reason="Adjacent"/>
+      <disable_collisions link1="${tf_prefix}left_robotiq_85_right_finger_link" link2="${tf_prefix}left_robotiq_85_right_inner_knuckle_link" reason="Adjacent"/>
+      <disable_collisions link1="${tf_prefix}left_robotiq_85_left_inner_knuckle_link" link2="${tf_prefix}left_robotiq_85_left_knuckle_link" reason="Adjacent"/>
+      <disable_collisions link1="${tf_prefix}left_robotiq_85_left_inner_knuckle_link" link2="${tf_prefix}left_robotiq_85_right_inner_knuckle_link" reason="Adjacent"/>
+      <disable_collisions link1="${tf_prefix}left_robotiq_85_left_inner_knuckle_link" link2="${tf_prefix}left_robotiq_85_right_finger_tip_link" reason="Adjacent"/>
+      <disable_collisions link1="${tf_prefix}left_robotiq_85_left_inner_knuckle_link" link2="${tf_prefix}left_robotiq_85_right_knuckle_link" reason="Adjacent"/>
+      <disable_collisions link1="${tf_prefix}left_robotiq_85_right_inner_knuckle_link" link2="${tf_prefix}left_robotiq_85_right_knuckle_link" reason="Adjacent"/>
+      <disable_collisions link1="${tf_prefix}right_finger_1_link" link2="${tf_prefix}right_gripper_base_link"/>
+      <disable_collisions link1="${tf_prefix}right_finger_2_link" link2="${tf_prefix}right_gripper_base_link"/>
+      <disable_collisions link1="${tf_prefix}right_gripper_base_link" link2="${tf_prefix}right_robotiq_hande_cb_adapter"/>
       <xacro:if value="$(arg calibration_mode)">
           <disable_collisions link1="${tf_prefix}front_shelf" link2="${tf_prefix}calibration_plate_target_side" reason="Adjacent"/>
